Commit message: removing WAM from urdf path name

File: models/arm.urdf.xacro (robot description, xacro)
@@ -36,8 +36,8 @@
     <xacro:ForceTorque prefix="${prefix}"/>
     <xacro:LowerWristFTPalm prefix="${prefix}"/>
-    <link name="${prefix}/WAM/PalmLink" />
-    <joint name="${prefix}/WAM/PalmJoint" type="fixed">
-      <parent link="${prefix}/WAM/LowerWristFTPalmLink"/>
-      <child link="${prefix}/WAM/PalmLink"/>
+    <link name="${prefix}/PalmLink" />
+    <joint name="${prefix}/PalmJoint" type="fixed">
+      <parent link="${prefix}/LowerWristFTPalmLink"/>
+      <child link="${prefix}/PalmLink"/>
       <!--             <origin xyz="0 0 0.1293166" rpy="0 0 0"/> -->
       <origin xyz="0 0 0.0793166" rpy="0 0 ${PI/2}"/>

File: models/common.urdf.xacro (robot description, xacro)
@@ -30,7 +30,14 @@
   xmlns:geom="http://playerstage.sourceforge.net/gazebo/xmlschema/#geom"
   xmlns:xacro="http://ros.org/wiki/xacro">
+  <!-- Directories -->
   <xacro:property name="homeDirectory" value="package://bard_urdf" />
   <xacro:property name="highResModelDirectory" value="${homeDirectory}/models/componentSTL/splitModels" />
+  <!-- Constants -->
   <xacro:property name="PI" value="3.1415926535897931" />
+  <!-- Materials -->
+  <material name="WAMGrey">
+    <color rgba="0.9 0.9 0.9 1.0"/>
+  </material>
+  <!-- Gazebo macros -->
   <xacro:macro name="gazeboReference" params="name material">
     <gazebo reference="${name}">
@@ -56,4 +63,5 @@
     </gazebo>
   </xacro:macro>
+  <!-- Controller macros -->
   <xacro:macro name="control" params="name topicName linkName jointName">
     <transmission type="pr2_mechanism_model/SimpleTransmission" name="${name}_trans">

File: models/components.urdf.xacro (robot description, xacro)
@@ -33,5 +33,5 @@
   <include filename="$(find bard_urdf)/models/common.urdf.xacro"/>
   <xacro:macro name="Shoulder" params="prefix parentLink xyz rpy">
-    <link name="${prefix}/WAM/ShoulderLink" >
+    <link name="${prefix}/ShoulderLink" >
       <inertial>
         <origin xyz="-.00443422 0.1289039 -.00066489" />
@@ -56,9 +56,9 @@
       </collision>
     </link>
-    <xacro:gazeboReferenceDAE name="${prefix}/WAM/ShoulderLink"/>
-    <xacro:control topicName="${prefix}/WAM/ShoulderYaw" name="DarmSim_${prefix}Arm_WAM_ShoulderYaw" linkName="${prefix}/WAM/ShoulderLink" jointName="${prefix}/WAM/YawJoint" />
-    <joint name="${prefix}/WAM/YawJoint" type="revolute">
+    <xacro:gazeboReferenceDAE name="${prefix}/ShoulderLink"/>
+    <xacro:control topicName="${prefix}/ShoulderYaw" name="DarmSim_${prefix}Arm_WAM_ShoulderYaw" linkName="${prefix}/ShoulderLink" jointName="${prefix}/YawJoint" />
+    <joint name="${prefix}/YawJoint" type="revolute">
       <parent link="${parentLink}"/>
-      <child link="${prefix}/WAM/ShoulderLink"/>
+      <child link="${prefix}/ShoulderLink"/>
       <origin xyz="${xyz}" rpy="${rpy}"/>
       <axis xyz="0 -1 0"/>
@@ -69,5 +69,5 @@
   </xacro:macro>
   <xacro:macro name="UpperArmInShoulder" params="prefix">
-    <link name="${prefix}/WAM/UpperArmInShoulderLink" >
+    <link name="${prefix}/UpperArmInShoulderLink" >
       <visual>
         <material name="WAMGrey" />
@@ -91,9 +91,9 @@
       </collision>
     </link>
-    <xacro:gazeboReferenceDAE name="${prefix}/WAM/UpperArmInShoulderLink"/>
-    <xacro:control topicName="${prefix}/WAM/ShoulderPitch" name="DarmSim_${prefix}Arm_WAM_ShoulderPitch" linkName="${prefix}/WAM/UpperArmInShoulderLink" jointName="${prefix}/WAM/ShoulderPitchJoint" />
-    <joint name="${prefix}/WAM/ShoulderPitchJoint" type="revolute">
-      <parent link="${prefix}/WAM/ShoulderLink"/>
-      <child link="${prefix}/WAM/UpperArmInShoulderLink"/>
+    <xacro:gazeboReferenceDAE name="${prefix}/UpperArmInShoulderLink"/>
+    <xacro:control topicName="${prefix}/ShoulderPitch" name="DarmSim_${prefix}Arm_WAM_ShoulderPitch" linkName="${prefix}/UpperArmInShoulderLink" jointName="${prefix}/ShoulderPitchJoint" />
+    <joint name="${prefix}/ShoulderPitchJoint" type="revolute">
+      <parent link="${prefix}/ShoulderLink"/>
+      <child link="${prefix}/UpperArmInShoulderLink"/>
       <origin xyz="0 0 0" rpy="${0.5 * PI} 0 0"/>
       <axis xyz="0 1 0"/>
@@ -104,5 +104,5 @@
   </xacro:macro>
   <xacro:macro name="UpperArm" params="prefix">
-    <link name="${prefix}/WAM/UpperArmLink" >
+    <link name="${prefix}/UpperArmLink" >
       <inertial>
         <origin xyz="-.03826 .20751 .00003" />
@@ -126,9 +126,9 @@
       </collision>
     </link>
-    <xacro:gazeboReferenceDAE name="${prefix}/WAM/UpperArmLink" />
-    <xacro:control topicName="${prefix}/WAM/UpperArmYaw" name="DarmSim_${prefix}Arm_WAM_UpperArmYaw" linkName="${prefix}/WAM/UpperArmLink" jointName="${prefix}/WAM/ShoulderYawJoint" />
-    <joint name="${prefix}/WAM/ShoulderYawJoint" type="revolute">
-      <parent link="${prefix}/WAM/UpperArmInShoulderLink"/>
-      <child link="${prefix}/WAM/UpperArmLink"/>
+    <xacro:gazeboReferenceDAE name="${prefix}/UpperArmLink" />
+    <xacro:control topicName="${prefix}/UpperArmYaw" name="DarmSim_${prefix}Arm_WAM_UpperArmYaw" linkName="${prefix}/UpperArmLink" jointName="${prefix}/ShoulderYawJoint" />
+    <joint name="${prefix}/ShoulderYawJoint" type="revolute">
+      <parent link="${prefix}/UpperArmInShoulderLink"/>
+      <child link="${prefix}/UpperArmLink"/>
       <origin xyz="0 0 0" rpy="-${0.5 * PI} 0 0"/>
       <axis xyz="0 -1 0"/>
@@ -139,5 +139,5 @@
   </xacro:macro>
   <xacro:macro name="ForeArm" params="prefix">
-    <link name="${prefix}/WAM/ForeArmLink" >
+    <link name="${prefix}/ForeArmLink" >
       <inertial>
         <origin xyz="0 0 0" />
@@ -162,9 +162,9 @@
       </collision>
     </link>
-    <xacro:gazeboReferenceDAE name="${prefix}/WAM/ForeArmLink" />
-    <xacro:control topicName="${prefix}/WAM/ElbowPitch" name="DarmSim_${prefix}Arm_WAM_ElbowPitch" linkName="${prefix}/WAM/ForeArmLink" jointName="${prefix}/WAM/ElbowJoint" />
-    <joint name="${prefix}/WAM/ElbowJoint" type="revolute">
-      <parent link="${prefix}/WAM/UpperArmLink"/>
-      <child link="${prefix}/WAM/ForeArmLink"/>
+    <xacro:gazeboReferenceDAE name="${prefix}/ForeArmLink" />
+    <xacro:control topicName="${prefix}/ElbowPitch" name="DarmSim_${prefix}Arm_WAM_ElbowPitch" linkName="${prefix}/ForeArmLink" jointName="${prefix}/ElbowJoint" />
+    <joint name="${prefix}/ElbowJoint" type="revolute">
+      <parent link="${prefix}/UpperArmLink"/>
+      <child link="${prefix}/ForeArmLink"/>
       <origin xyz="0.045 -0.55 0" rpy="${0.5 * PI} 0 0"/>
       <axis xyz="0 1 0"/>
@@ -175,5 +175,5 @@
   </xacro:macro>
   <xacro:macro name="UpperWristYaw" params="prefix">
-    <link name="${prefix}/WAM/UpperWristYawLink" >
+    <link name="${prefix}/UpperWristYawLink" >
       <inertial>
         <origin xyz="0.00008921 0.00511217 0.00435824" />
@@ -197,9 +197,9 @@
       </collision>
     </link>
-    <xacro:gazeboReferenceDAE name="${prefix}/WAM/UpperWristYawLink" />
-    <xacro:control topicName="${prefix}/WAM/UpperWristYaw" name="DarmSim_${prefix}Arm_WAM_UpperWristYaw" linkName="${prefix}/WAM/UpperWristYawLink" jointName="${prefix}/WAM/UpperWristYawJoint" />
-    <joint name="${prefix}/WAM/UpperWristYawJoint" type="revolute">
-      <parent link="${prefix}/WAM/ForeArmLink"/>
-      <child link="${prefix}/WAM/UpperWristYawLink"/>
+    <xacro:gazeboReferenceDAE name="${prefix}/UpperWristYawLink" />
+    <xacro:control topicName="${prefix}/UpperWristYaw" name="DarmSim_${prefix}Arm_WAM_UpperWristYaw" linkName="${prefix}/UpperWristYawLink" jointName="${prefix}/UpperWristYawJoint" />
+    <joint name="${prefix}/UpperWristYawJoint" type="revolute">
+      <parent link="${prefix}/ForeArmLink"/>
+      <child link="${prefix}/UpperWristYawLink"/>
       <origin xyz="-0.045 0 .3" rpy="-${0.5 * PI} 0 ${0.5 * PI}"/>
       <axis xyz="0 -1 0"/>
@@ -210,5 +210,5 @@
   </xacro:macro>
   <xacro:macro name="UpperWristPitch" params="prefix">
-    <link name="${prefix}/WAM/UpperWristPitchLink" >
+    <link name="${prefix}/UpperWristPitchLink" >
       <inertial>
         <origin xyz="-0.00012262 -0.01703194 0.02468336" rpy="0 0 0" />
@@ -232,9 +232,9 @@
       </collision>
     </link>
-    <xacro:gazeboReferenceDAE name="${prefix}/WAM/UpperWristPitchLink" />
-    <xacro:control topicName="${prefix}/WAM/UpperWristPitch" name="DarmSim_${prefix}Arm_WAM_UpperWristPitch" linkName="${prefix}/WAM/UpperWristPitchLink" jointName="${prefix}/WAM/UpperWristPitchJoint" />
-    <joint name="${prefix}/WAM/UpperWristPitchJoint" type="revolute">
-      <parent link="${prefix}/WAM/UpperWristYawLink"/>
-      <child link="${prefix}/WAM/UpperWristPitchLink"/>
+    <xacro:gazeboReferenceDAE name="${prefix}/UpperWristPitchLink" />
+    <xacro:control topicName="${prefix}/UpperWristPitch" name="DarmSim_${prefix}Arm_WAM_UpperWristPitch" linkName="${prefix}/UpperWristPitchLink" jointName="${prefix}/UpperWristPitchJoint" />
+    <joint name="${prefix}/UpperWristPitchJoint" type="revolute">
+      <parent link="${prefix}/UpperWristYawLink"/>
+      <child link="${prefix}/UpperWristPitchLink"/>
       <origin xyz="0 0 0" rpy="${0.5 * PI} ${0.5 * PI} 0"/>
       <axis xyz="0 1 0"/>
@@ -245,5 +245,5 @@
   </xacro:macro>
   <xacro:macro name="ForceTorque" params="prefix">
-    <link name="${prefix}/WAM/ForceTorqueLink" >
+    <link name="${prefix}/ForceTorqueLink" >
       <inertial>
         <origin xyz="-0.00000134 -0.00228167 -0.00000141" rpy="0 0 0" />
@@ -267,9 +267,9 @@
       </collision>
     </link>
-    <xacro:gazeboReferenceDAE name="${prefix}/WAM/ForceTorqueLink"/>
-    <xacro:control topicName="${prefix}/WAM/LowerWristYaw" name="DarmSim_${prefix}Arm_WAM_LowerWristYaw" linkName="${prefix}/WAM/ForceTorqueLink" jointName="${prefix}/WAM/LowerWristYawJoint" />
-    <joint name="${prefix}/WAM/LowerWristYawJoint" type="revolute">
-      <parent link="${prefix}/WAM/UpperWristPitchLink"/>
-      <child link="${prefix}/WAM/ForceTorqueLink"/>
+    <xacro:gazeboReferenceDAE name="${prefix}/ForceTorqueLink"/>
+    <xacro:control topicName="${prefix}/LowerWristYaw" name="DarmSim_${prefix}Arm_WAM_LowerWristYaw" linkName="${prefix}/ForceTorqueLink" jointName="${prefix}/LowerWristYawJoint" />
+    <joint name="${prefix}/LowerWristYawJoint" type="revolute">
+      <parent link="${prefix}/UpperWristPitchLink"/>
+      <child link="${prefix}/ForceTorqueLink"/>
       <origin xyz="0 0 0.06713340" rpy="0 0 0"/>
       <axis xyz="0 0 1"/>
@@ -280,5 +280,5 @@
   </xacro:macro>
   <xacro:macro name="LowerWristFTPalm" params="prefix">
-    <link name="${prefix}/WAM/LowerWristFTPalmLink" >
+    <link name="${prefix}/LowerWristFTPalmLink" >
       <inertial>
         <origin xyz="0.00035500 -0.00499005 0.04864979" />
@@ -302,12 +302,12 @@
       </collision>
     </link>
-    <xacro:gazeboReferenceDAE name="${prefix}/WAM/LowerWristFTPalmLink"/>
-    <joint name="${prefix}/WAM/FTPalmJoint" type="fixed">
-      <parent link="${prefix}/WAM/ForceTorqueLink"/>
-      <child link="${prefix}/WAM/LowerWristFTPalmLink"/>
+    <xacro:gazeboReferenceDAE name="${prefix}/LowerWristFTPalmLink"/>
+    <joint name="${prefix}/FTPalmJoint" type="fixed">
+      <parent link="${prefix}/ForceTorqueLink"/>
+      <child link="${prefix}/LowerWristFTPalmLink"/>
       <origin xyz="0 0 0.0048" rpy="0 0 -${0.5 * PI}"/>
       <provideFeedback value="true"/>
     </joint>
-    <gazebo reference="${prefix}/WAM/FTPalmJoint">
+    <gazebo reference="${prefix}/FTPalmJoint">
       <provideFeedback value="true"/>
     </gazebo>
@@ -316,19 +316,19 @@
         <alwaysOn>true</alwaysOn>
         <updateRate>100.0</updateRate>
-        <jointName>${prefix}/WAM/FTPalmJoint</jointName>
+        <jointName>${prefix}/FTPalmJoint</jointName>
         <topicName>${prefix}/BHand/ForceTorqueSensor</topicName>
         <bodyRelation>child</bodyRelation>
-        <frameName>${prefix}/WAM/LowerWristFTPalmLink</frameName>
+        <frameName>${prefix}/LowerWristFTPalmLink</frameName>
         <interface:position name="${prefix}_JointFTsensor_force_iface" />
       </controller:gazebo_ros_jointFeedback>
     </gazebo>
-    <gazebo reference="${prefix}/WAM/LowerWristFTPalmLink">
+    <gazebo reference="${prefix}/LowerWristFTPalmLink">
       <sensor:contact name="${prefix}Palm_contact_sensor">
-        <geom>${prefix}/WAM/LowerWristFTPalmLink_geom</geom>
+        <geom>${prefix}/LowerWristFTPalmLink_geom</geom>
         <updateRate>100.0</updateRate>
-        <controller:gazebo_ros_bumper name="${prefix}/WAM/LowerWristFTPalmLink/bumperController" plugin="libgazebo_ros_bumper.so">
+        <controller:gazebo_ros_bumper name="${prefix}/LowerWristFTPalmLink/bumperController" plugin="libgazebo_ros_bumper.so">
           <alwaysOn>true</alwaysOn>
           <updateRate>100.0</updateRate>
-          <frameName>${prefix}/WAM/LowerWristFTPalmLink</frameName>
+          <frameName>${prefix}/LowerWristFTPalmLink</frameName>
           <bumperTopicName>${prefix}/BHand/Palm/bumper</bumperTopicName>
           <interface:bumper name="DarmSim${prefix}ArmWAMLowerWristFTPalmLink_bumper_iface" />
@@ -367,5 +367,5 @@
     <xacro:control topicName="${prefix}/BHand/Finger${number}/KnuckleOne" name="DarmSim_${prefix}Arm_BHand_Finger${number}KnuckleOne" linkName="${prefix}/BHand/Finger${number}/KnuckleOneLink" jointName="${prefix}/BHand/Finger${number}/KnuckleOneJoint" />
     <joint name="${prefix}/BHand/Finger${number}/KnuckleOneJoint" type="revolute">
-      <parent link="${prefix}/WAM/LowerWristFTPalmLink"/>
+      <parent link="${prefix}/LowerWristFTPalmLink"/>
       <child link="${prefix}/BHand/Finger${number}/KnuckleOneLink"/>
       <origin xyz="${xyz}" rpy="${rpy}"/>

File: models/hand.urdf.xacro (robot description, xacro)
@@ -47,5 +47,5 @@
   </xacro:macro>
   <xacro:macro name="darpa_hand" params="prefix">
-    <xacro:fingers prefix="${prefix}" parent="${prefix}/WAM/LowerWristFTPalmLink" number="Three" xyz="0 -0.05 0.0801966" rpy="-${0.5 * PI} -0.0429350996 -${0.5 * PI}"/>
+    <xacro:fingers prefix="${prefix}" parent="${prefix}/LowerWristFTPalmLink" number="Three" xyz="0 -0.05 0.0801966" rpy="-${0.5 * PI} -0.0429350996 -${0.5 * PI}"/>
     <xacro:KnuckleOne prefix="${prefix}" number="One" xyz=".02497 0 0.0587966" rpy="0 0 ${0.5 * PI}" axis="0 0 -1"/>
     <xacro:fingers prefix="${prefix}" parent="${prefix}/BHand/FingerOne/KnuckleOneLink" number="One" xyz=".05 0 0.02140" rpy="-${0.5 * PI} -0.0429350996 0"/>

File: models/root.urdf.xacro (robot description, xacro)
@@ -23,17 +23,10 @@
  * of or in connection with the use or performance of this software.
 -->
-<robot name="darpa_arm_robot"
+<robot name="dual_wam_robot"
   xmlns:xacro="http://www.ros.org/wiki/xacro"
   xmlns:controller="http://playerstage.sourceforge.net/gazebo/xmlschema/#controller">
   <include filename="$(find bard_urdf)/models/common.urdf.xacro"/>
   <include filename="$(find bard_urdf)/models/arm.urdf.xacro"/>
-  <include filename="$(find bard_urdf)/models/headAssembly.urdf.xacro"/>
   <include filename="$(find bard_urdf)/models/components.urdf.xacro"/>
-  <material name="WAMGrey">
-    <color rgba="0.9 0.9 0.9 1.0"/>
-  </material>
-  <material name="DarpaBlue">
-    <color rgba="0.0 0.5 0.5 1.0"/>
-  </material>
   <link name = "world"/>
   <xacro:base xyz="0 0 0.813372" rpy="0 0 0" parent="world"/>
@@ -59,6 +52,6 @@
   </link>
   <xacro:gazeboReferenceDAE name="cylinderLink" />
-  <link name = "DarmSim/RightArm/WAM/FixedLink" />
-  <link name = "DarmSim/LeftArm/WAM/FixedLink" />
+  <link name = "LeftWAM/FixedLink" />
+  <link name = "RightWAM/FixedLink" />
   <joint name="cylinderJoint" type="fixed">
     <parent link="baseLink"/>
@@ -68,10 +61,10 @@
   <joint name="rightFixedJoint" type="fixed">
     <parent link="baseLink"/>
-    <child link="DarmSim/RightArm/WAM/FixedLink"/>
+    <child link="RightWAM/FixedLink"/>
     <origin xyz="-0.350177361 -0.350177361 .37836125" rpy="0 ${-0.5*PI} ${0.25*PI}"/>
   </joint>
   <joint name="leftFixedJoint" type="fixed">
     <parent link="baseLink"/>
-    <child link="DarmSim/LeftArm/WAM/FixedLink"/>
+    <child link="LeftWAM/FixedLink"/>
     <origin xyz="0.350177361 -0.350177361 .37836125" rpy="0 ${-0.5*PI} ${0.75*PI}"/>
   </joint>
@@ -82,6 +75,6 @@
     </controller:gazebo_ros_controller_manager>
   </gazebo>
-  <xacro:darpa_arm prefix="Right" parentLink="baseLink" xyz="-0.350177361 -0.350177361 .37836125" rpy="-${0.5 * PI} -${0.5 * PI} ${0.25*PI}" />
-  <xacro:darpa_arm prefix="Left" parentLink="baseLink" xyz="0.350177361 -0.350177361 .37836125" rpy="-${0.5 * PI} -${0.5 * PI} ${0.75*PI}" />
+  <xacro:darpa_arm prefix="RightWAM" parentLink="baseLink" xyz="-0.350177361 -0.350177361 .37836125" rpy="-${0.5 * PI} -${0.5 * PI} ${0.25*PI}" />
+  <xacro:darpa_arm prefix="LeftWAM" parentLink="baseLink" xyz="0.350177361 -0.350177361 .37836125" rpy="-${0.5 * PI} -${0.5 * PI} ${0.75*PI}" />
   <xacro:darpa_head_assembly parent="baseLink" xyz="0 -.1292225 .52971" rpy="${0.5 * PI} 0 0"/>
 </robot>

Commit message: renaming darpa_arm to wam_arm

File: models/arm.urdf.xacro (robot description, xacro)
@@ -27,5 +27,5 @@
   <include filename="$(find bard_urdf)/models/common.urdf.xacro"/>
   <include filename="$(find bard_urdf)/models/components.urdf.xacro"/>
-  <xacro:macro name="darpa_arm" params="prefix parentLink xyz rpy">
+  <xacro:macro name="wam_arm" params="prefix parentLink xyz rpy">
     <xacro:Shoulder prefix="${prefix}" parentLink="${parentLink}" xyz="${xyz}" rpy="${rpy}"/>
     <xacro:UpperArmInShoulder prefix="${prefix}"/>

File: models/root.urdf.xacro (robot description, xacro)
@@ -83,5 +83,5 @@
   </gazebo>
   <!-- Construct the actual arms -->
-  <xacro:darpa_arm prefix="RightWAM" parentLink="RightWAM/FixedLink" xyz="0 0 0 " rpy="0 0 0" />
-  <xacro:darpa_arm prefix="LeftWAM" parentLink="LeftWAM/FixedLink" xyz="0 0 0" rpy="0 0 0" />
+  <xacro:wam_arm prefix="RightWAM" parentLink="RightWAM/FixedLink" xyz="0 0 0 " rpy="0 0 0" />
+  <xacro:wam_arm prefix="LeftWAM" parentLink="LeftWAM/FixedLink" xyz="0 0 0" rpy="0 0 0" />
 </robot>

Commit message: renaming root to example, and separating the wam arm with and without a hand

File: models/arm.urdf.xacro (robot description, xacro)
@@ -27,4 +27,5 @@
   <include filename="$(find bard_urdf)/models/common.urdf.xacro"/>
   <include filename="$(find bard_urdf)/models/components.urdf.xacro"/>
+  <!-- Define a macro to construct the arm -->
   <xacro:macro name="wam_arm" params="prefix parentLink xyz rpy">
     <xacro:Shoulder prefix="${prefix}" parentLink="${parentLink}" xyz="${xyz}" rpy="${rpy}"/>
@@ -34,4 +35,8 @@
     <xacro:UpperWristYaw prefix="${prefix}"/>
     <xacro:UpperWristPitch prefix="${prefix}"/>
+  </xacro:macro>
+  <!-- Define a macro to construct the arm with a Barrett BHand on the end of it -->
+  <xacro:macro name="wam_arm_and_hand" params="prefix parentLink xyz rpy">
+    <xacro:wam_arm prefix="${prefix}" parentLink="${parentLink}" xyz="${xyz}" rpy="${rpy}"/>
     <xacro:ForceTorque prefix="${prefix}"/>
     <xacro:LowerWristFTPalm prefix="${prefix}"/>
@@ -43,5 +48,5 @@
       <origin xyz="0 0 0.0793166" rpy="0 0 ${PI/2}"/>
     </joint>
-    <xacro:darpa_hand prefix="${prefix}" />
+    <xacro:barrett_hand prefix="${prefix}" />
   </xacro:macro>
 </robot>

File: models/hand.urdf.xacro (robot description, xacro)
@@ -46,5 +46,5 @@
     </gazebo>
   </xacro:macro>
-  <xacro:macro name="darpa_hand" params="prefix">
+  <xacro:macro name="barrett_hand" params="prefix">
     <xacro:fingers prefix="${prefix}" parent="${prefix}/LowerWristFTPalmLink" number="Three" xyz="0 -0.05 0.0801966" rpy="-${0.5 * PI} -0.0429350996 -${0.5 * PI}"/>
     <xacro:KnuckleOne prefix="${prefix}" number="One" xyz=".02497 0 0.0587966" rpy="0 0 ${0.5 * PI}" axis="0 0 -1"/>

File: models/two_arms_example.urdf.xacro (robot description, xacro)
@@ -52,5 +52,5 @@
         <origin xyz="0 0 0" rpy="0 0 0" />
         <geometry>
-          <mesh filename="package://bard_urdf/models/componentSTL/baseLinkTwoArms.stl"/>
+          <mesh filename="package://bard_urdf/models/componentSTL/bench_lattice.stl"/>
         </geometry>
       </collision>
@@ -83,5 +83,5 @@
   </gazebo>
   <!-- Construct the actual arms -->
-  <xacro:wam_arm prefix="RightWAM" parentLink="RightWAM/FixedLink" xyz="0 0 0 " rpy="0 0 0" />
-  <xacro:wam_arm prefix="LeftWAM" parentLink="LeftWAM/FixedLink" xyz="0 0 0" rpy="0 0 0" />
+  <xacro:wam_arm_and_hand prefix="RightWAM" parentLink="RightWAM/FixedLink" xyz="0 0 0 " rpy="0 0 0" />
+  <xacro:wam_arm_and_hand prefix="LeftWAM" parentLink="LeftWAM/FixedLink" xyz="0 0 0" rpy="0 0 0" />
 </robot>
