Commit message: adding non-ft barrett wrist

File: models/arm.urdf.xacro (robot description, xacro)
@@ -36,7 +36,16 @@
     <xacro:UpperWristPitch prefix="${prefix}"/>
   </xacro:macro>
+  <xacro:macro name="barret_palm" params="prefix">
+    <xacro:LowerWrist prefix="${prefix}"/>
+    <link name="${prefix}/PalmLink" />
+    <joint name="${prefix}/PalmJoint" type="fixed">
+      <parent link="${prefix}/LowerWristLink"/>
+      <child link="${prefix}/PalmLink"/>
+      <!--             <origin xyz="0 0 0.1293166" rpy="0 0 0"/> -->
+      <origin xyz="0 0 0.0793166" rpy="0 0 ${PI/2}"/>
+    </joint>
+  </xacro:macro>
   <!-- Define a macro to construct the arm with a Barrett BHand on the end of it -->
-  <xacro:macro name="wam_arm_and_hand" params="prefix parentLink xyz rpy">
-    <xacro:wam_arm prefix="${prefix}" parentLink="${parentLink}" xyz="${xyz}" rpy="${rpy}"/>
+  <xacro:macro name="barrett_ft_palm" params="prefix">
     <xacro:ForceTorque prefix="${prefix}"/>
     <xacro:LowerWristFTPalm prefix="${prefix}"/>

File: models/components.urdf.xacro (robot description, xacro)
@@ -244,4 +244,47 @@
     </joint>
   </xacro:macro>
+  <xacro:macro name="LowerWrist" params="prefix">
+    <link name="${prefix}/LowerWristLink" >
+      <inertial>
+        <origin xyz="0.00035500 -0.00499005 0.04864979" />
+        <mass value="0.63352875" />
+        <inertia  ixx="0.00102103" ixy="0.00000775"  ixz="-0.00001230"
+          iyy="0.00080944"  iyz="-0.00014417"
+          izz="0.00068788" />
+      </inertial>
+      <visual>
+        <material name="WAMGrey" />
+        <origin xyz="0 0 0" rpy="0 0 0" />
+        <geometry>
+          <mesh filename="${homeDirectory}/models/componentSTL/palm.DAE"/>
+        </geometry>
+      </visual>
+      <collision>
+        <origin xyz="0 0 0" rpy="0 0 0" />
+        <geometry>
+          <mesh filename="${homeDirectory}/models/componentSTL/palm.stl"/>
+        </geometry>
+      </collision>
+    </link>
+    <xacro:gazeboReferenceDAE name="${prefix}/LowerWristLink"/>
+    <joint name="${prefix}/LowerWristYawJoint" type="revolute">
+      <parent link="${prefix}/UpperWristPitchLink"/>
+      <child link="${prefix}/PalmLink"/>
+      <origin xyz="0 0 0.06713340" rpy="0 0 0"/>
+      <axis xyz="0 0 1"/>
+      <limit effort="5" lower="-2.95" upper="2.95" velocity="3.27"/><!-- 2.95 is a limit taken in from 3 due to saftey and differences between arms. -->
+      <!-- <safety_controller k_position="100" k_velocity="3" soft_lower_limit="-100.0" soft_upper_limit="100.0" /> -->
+      <dynamics damping="1.0" friction="100.0"/>
+    </joint>
+    <joint name="${prefix}/PalmJoint" type="fixed">
+      <parent link="${prefix}/ForceTorqueLink"/>
+      <child link="${prefix}/LowerWristFTPalmLink"/>
+      <origin xyz="0 0 0.0048" rpy="0 0 -${0.5 * PI}"/>
+      <provideFeedback value="true"/>
+    </joint>
+    <gazebo reference="${prefix}/PalmJoint">
+      <provideFeedback value="true"/>
+    </gazebo>
+  </xacro:macro>
   <xacro:macro name="ForceTorque" params="prefix">
     <link name="${prefix}/ForceTorqueLink" >

Commit message: updating bard urdf to have non-ft stuff

File: models/arm.urdf.xacro (robot description, xacro)
@@ -38,19 +38,21 @@
   <xacro:macro name="barret_palm" params="prefix">
     <xacro:LowerWrist prefix="${prefix}"/>
+    <xacro:LowerWristPalm prefix="${prefix}"/>
     <link name="${prefix}/PalmLink" />
     <joint name="${prefix}/PalmJoint" type="fixed">
-      <parent link="${prefix}/LowerWristLink"/>
+      <parent link="${prefix}/LowerWristPalmLink"/>
       <child link="${prefix}/PalmLink"/>
       <!--             <origin xyz="0 0 0.1293166" rpy="0 0 0"/> -->
       <origin xyz="0 0 0.0793166" rpy="0 0 ${PI/2}"/>
     </joint>
+    <xacro:barrett_hand prefix="${prefix}" />
   </xacro:macro>
   <!-- Define a macro to construct the arm with a Barrett BHand on the end of it -->
   <xacro:macro name="barrett_ft_palm" params="prefix">
-    <xacro:ForceTorque prefix="${prefix}"/>
-    <xacro:LowerWristFTPalm prefix="${prefix}"/>
+    <xacro:LowerWristFT prefix="${prefix}"/>
+    <xacro:LowerWristPalmFT prefix="${prefix}"/>
     <link name="${prefix}/PalmLink" />
     <joint name="${prefix}/PalmJoint" type="fixed">
-      <parent link="${prefix}/LowerWristFTPalmLink"/>
+      <parent link="${prefix}/LowerWristPalmLink"/>
       <child link="${prefix}/PalmLink"/>
       <!--             <origin xyz="0 0 0.1293166" rpy="0 0 0"/> -->

File: models/components.urdf.xacro (robot description, xacro)
@@ -245,7 +245,6 @@
   </xacro:macro>
   <!-- Palm without force-torque sensor -->
-  <!-- ForceTorque macros -->
-  <xacro:macro name="ForceTorque" params="prefix">
-    <link name="${prefix}/ForceTorqueLink" >
+  <xacro:macro name="LowerWrist" params="prefix">
+    <link name="${prefix}/LowerWristYawLink" >
       <inertial>
         <origin xyz="-0.00000134 -0.00228167 -0.00000141" rpy="0 0 0" />
@@ -269,10 +268,10 @@
       </collision>
     </link>
-    <xacro:gazeboReferenceDAE name="${prefix}/ForceTorqueLink"/>
-    <xacro:control topicName="${prefix}/LowerWristYaw" name="DarmSim_${prefix}Arm_WAM_LowerWristYaw" linkName="${prefix}/ForceTorqueLink" jointName="${prefix}/LowerWristYawJoint" />
+    <xacro:gazeboReferenceDAE name="${prefix}/LowerWristYawLink"/>
+    <xacro:control topicName="${prefix}/LowerWristYaw" name="DarmSim_${prefix}Arm_WAM_LowerWristYaw" linkName="${prefix}/LowerWristYawLink" jointName="${prefix}/LowerWristYawJoint" />
     <joint name="${prefix}/LowerWristYawJoint" type="revolute">
       <parent link="${prefix}/UpperWristPitchLink"/>
-      <child link="${prefix}/ForceTorqueLink"/>
-      <origin xyz="0 0 0.06713340" rpy="0 0 0"/>
+      <child link="${prefix}/LowerWristYawLink"/>
+      <origin xyz="0 0 0.060" rpy="0 0 0"/>
       <axis xyz="0 0 1"/>
       <limit effort="5" lower="-2.95" upper="2.95" velocity="3.27"/><!-- 2.95 is a limit taken in from 3 due to saftey and differences between arms. -->
@@ -281,6 +280,6 @@
     </joint>
   </xacro:macro>
-  <xacro:macro name="LowerWristFTPalm" params="prefix">
-    <link name="${prefix}/LowerWristFTPalmLink" >
+  <xacro:macro name="LowerWristPalm" params="prefix">
+    <link name="${prefix}/LowerWristPalmLink" >
       <inertial>
         <origin xyz="0.00035500 -0.00499005 0.04864979" />
@@ -304,12 +303,12 @@
       </collision>
     </link>
-    <xacro:gazeboReferenceDAE name="${prefix}/LowerWristFTPalmLink"/>
-    <joint name="${prefix}/FTPalmJoint" type="fixed">
-      <parent link="${prefix}/ForceTorqueLink"/>
-      <child link="${prefix}/LowerWristFTPalmLink"/>
-      <origin xyz="0 0 0.0048" rpy="0 0 -${0.5 * PI}"/>
+    <xacro:gazeboReferenceDAE name="${prefix}/LowerWristPalmLink"/>
+    <joint name="${prefix}/LowerWristPalmJoint" type="fixed">
+      <parent link="${prefix}/LowerWristYawLink"/>
+      <child link="${prefix}/LowerWristPalmLink"/>
+      <origin xyz="0 0 0" rpy="0 0 -${0.5 * PI}"/>
       <provideFeedback value="true"/>
     </joint>
-    <gazebo reference="${prefix}/FTPalmJoint">
+    <gazebo reference="${prefix}/LowerWristPalmJoint">
       <provideFeedback value="true"/>
     </gazebo>
@@ -318,21 +317,115 @@
         <alwaysOn>true</alwaysOn>
         <updateRate>100.0</updateRate>
-        <jointName>${prefix}/FTPalmJoint</jointName>
+        <jointName>${prefix}/LowerWristPalmJoint</jointName>
         <topicName>${prefix}/BHand/ForceTorqueSensor</topicName>
         <bodyRelation>child</bodyRelation>
-        <frameName>${prefix}/LowerWristFTPalmLink</frameName>
+        <frameName>${prefix}/LowerWristPalmLink</frameName>
         <interface:position name="${prefix}_JointFTsensor_force_iface" />
       </controller:gazebo_ros_jointFeedback>
     </gazebo>
-    <gazebo reference="${prefix}/LowerWristFTPalmLink">
+    <gazebo reference="${prefix}/LowerWristPalmLink">
       <sensor:contact name="${prefix}Palm_contact_sensor">
-        <geom>${prefix}/LowerWristFTPalmLink_geom</geom>
+        <geom>${prefix}/LowerWristPalmLink_geom</geom>
         <updateRate>100.0</updateRate>
-        <controller:gazebo_ros_bumper name="${prefix}/LowerWristFTPalmLink/bumperController" plugin="libgazebo_ros_bumper.so">
+        <controller:gazebo_ros_bumper name="${prefix}/LowerWristPalmLink/bumperController" plugin="libgazebo_ros_bumper.so">
           <alwaysOn>true</alwaysOn>
           <updateRate>100.0</updateRate>
-          <frameName>${prefix}/LowerWristFTPalmLink</frameName>
+          <frameName>${prefix}/LowerWristPalmLink</frameName>
           <bumperTopicName>${prefix}/BHand/Palm/bumper</bumperTopicName>
-          <interface:bumper name="DarmSim${prefix}ArmWAMLowerWristFTPalmLink_bumper_iface" />
+          <interface:bumper name="DarmSim${prefix}ArmWAMLowerWristPalmLink_bumper_iface" />
+        </controller:gazebo_ros_bumper>
+      </sensor:contact>
+    </gazebo>
+  </xacro:macro>
+  <!-- Palm with ForceTorque macros -->
+  <xacro:macro name="LowerWristFT" params="prefix">
+    <link name="${prefix}/LowerWristYawLink" >
+      <inertial>
+        <origin xyz="-0.00000134 -0.00228167 -0.00000141" rpy="0 0 0" />
+        <mass value="0.17286134" />
+        <inertia  ixx="0.00010859" ixy="0.00000000"  ixz="-0.00000000"
+          iyy="0.00020683"  iyz="-0.0000000"
+          izz="0.00010851" />
+      </inertial>
+      <visual>
+        <material name="WAMGrey" />
+        <origin xyz="0 0 0" rpy="0 0 0" />
+        <geometry>
+          <mesh filename="${homeDirectory}/models/componentSTL/forceTorqueSensor.DAE"/>
+        </geometry>
+      </visual>
+      <collision>
+        <origin xyz="0 0 0" rpy="0 0 0" />
+        <geometry>
+          <mesh filename="${homeDirectory}/models/componentSTL/forceTorqueSensor.stl"/>
+        </geometry>
+      </collision>
+    </link>
+    <xacro:gazeboReferenceDAE name="${prefix}/LowerWristYawLink"/>
+    <xacro:control topicName="${prefix}/LowerWristYaw" name="DarmSim_${prefix}Arm_WAM_LowerWristYaw" linkName="${prefix}/LowerWristYawLink" jointName="${prefix}/LowerWristYawJoint" />
+    <joint name="${prefix}/LowerWristYawJoint" type="revolute">
+      <parent link="${prefix}/UpperWristPitchLink"/>
+      <child link="${prefix}/LowerWristYawLink"/>
+      <origin xyz="0 0 0.06713340" rpy="0 0 0"/>
+      <axis xyz="0 0 1"/>
+      <limit effort="5" lower="-2.95" upper="2.95" velocity="3.27"/><!-- 2.95 is a limit taken in from 3 due to saftey and differences between arms. -->
+      <!-- <safety_controller k_position="100" k_velocity="3" soft_lower_limit="-100.0" soft_upper_limit="100.0" /> -->
+      <dynamics damping="1.0" friction="100.0"/>
+    </joint>
+  </xacro:macro>
+  <xacro:macro name="LowerWristPalmFT" params="prefix">
+    <link name="${prefix}/LowerWristPalmLink" >
+      <inertial>
+        <origin xyz="0.00035500 -0.00499005 0.04864979" />
+        <mass value="0.63352875" />
+        <inertia  ixx="0.00102103" ixy="0.00000775"  ixz="-0.00001230"
+          iyy="0.00080944"  iyz="-0.00014417"
+          izz="0.00068788" />
+      </inertial>
+      <visual>
+        <material name="WAMGrey" />
+        <origin xyz="0 0 0" rpy="0 0 0" />
+        <geometry>
+          <mesh filename="${homeDirectory}/models/componentSTL/palm.DAE"/>
+        </geometry>
+      </visual>
+      <collision>
+        <origin xyz="0 0 0" rpy="0 0 0" />
+        <geometry>
+          <mesh filename="${homeDirectory}/models/componentSTL/palm.stl"/>
+        </geometry>
+      </collision>
+    </link>
+    <xacro:gazeboReferenceDAE name="${prefix}/LowerWristPalmLink"/>
+    <joint name="${prefix}/LowerWristPalmJoint" type="fixed">
+      <parent link="${prefix}/LowerWristYawLink"/>
+      <child link="${prefix}/LowerWristPalmLink"/>
+      <origin xyz="0 0 0.0048" rpy="0 0 -${0.5 * PI}"/>
+      <provideFeedback value="true"/>
+    </joint>
+    <gazebo reference="${prefix}/LowerWristPalmJoint">
+      <provideFeedback value="true"/>
+    </gazebo>
+    <gazebo>
+      <controller:gazebo_ros_jointFeedback name="${prefix}_JointFTsensor" plugin="libgazebo_ros_jointFeedback.so">
+        <alwaysOn>true</alwaysOn>
+        <updateRate>100.0</updateRate>
+        <jointName>${prefix}/LowerWristPalmJoint</jointName>
+        <topicName>${prefix}/BHand/ForceTorqueSensor</topicName>
+        <bodyRelation>child</bodyRelation>
+        <frameName>${prefix}/LowerWristPalmLink</frameName>
+        <interface:position name="${prefix}_JointFTsensor_force_iface" />
+      </controller:gazebo_ros_jointFeedback>
+    </gazebo>
+    <gazebo reference="${prefix}/LowerWristPalmLink">
+      <sensor:contact name="${prefix}Palm_contact_sensor">
+        <geom>${prefix}/LowerWristPalmLink_geom</geom>
+        <updateRate>100.0</updateRate>
+        <controller:gazebo_ros_bumper name="${prefix}/LowerWristPalmLink/bumperController" plugin="libgazebo_ros_bumper.so">
+          <alwaysOn>true</alwaysOn>
+          <updateRate>100.0</updateRate>
+          <frameName>${prefix}/LowerWristPalmLink</frameName>
+          <bumperTopicName>${prefix}/BHand/Palm/bumper</bumperTopicName>
+          <interface:bumper name="DarmSim${prefix}ArmWAMLowerWristPalmLink_bumper_iface" />
         </controller:gazebo_ros_bumper>
       </sensor:contact>
@@ -370,5 +463,5 @@
     <xacro:control topicName="${prefix}/BHand/Finger${number}/KnuckleOne" name="DarmSim_${prefix}Arm_BHand_Finger${number}KnuckleOne" linkName="${prefix}/BHand/Finger${number}/KnuckleOneLink" jointName="${prefix}/BHand/Finger${number}/KnuckleOneJoint" />
     <joint name="${prefix}/BHand/Finger${number}/KnuckleOneJoint" type="revolute">
-      <parent link="${prefix}/LowerWristFTPalmLink"/>
+      <parent link="${prefix}/LowerWristPalmLink"/>
       <child link="${prefix}/BHand/Finger${number}/KnuckleOneLink"/>
       <origin xyz="${xyz}" rpy="${rpy}"/>

File: models/hand.urdf.xacro (robot description, xacro)
@@ -47,5 +47,5 @@
   </xacro:macro>
   <xacro:macro name="barrett_hand" params="prefix">
-    <xacro:fingers prefix="${prefix}" parent="${prefix}/LowerWristFTPalmLink" number="Three" xyz="0 -0.05 0.0801966" rpy="-${0.5 * PI} -0.0429350996 -${0.5 * PI}"/>
+    <xacro:fingers prefix="${prefix}" parent="${prefix}/LowerWristPalmLink" number="Three" xyz="0 -0.05 0.0801966" rpy="-${0.5 * PI} -0.0429350996 -${0.5 * PI}"/>
     <xacro:KnuckleOne prefix="${prefix}" number="One" xyz=".02497 0 0.0587966" rpy="0 0 ${0.5 * PI}" axis="0 0 -1"/>
     <xacro:fingers prefix="${prefix}" parent="${prefix}/BHand/FingerOne/KnuckleOneLink" number="One" xyz=".05 0 0.02140" rpy="-${0.5 * PI} -0.0429350996 0"/>

Commit message: kdl chain solver takes link names and not joint names as arguments

File: models/arm.urdf.xacro (robot description, xacro)
@@ -36,5 +36,5 @@
     <xacro:UpperWristPitch prefix="${prefix}"/>
   </xacro:macro>
-  <xacro:macro name="barret_palm" params="prefix">
+  <xacro:macro name="barrett_palm" params="prefix">
     <xacro:LowerWrist prefix="${prefix}"/>
     <xacro:LowerWristPalm prefix="${prefix}"/>

Commit message: functioning grav comp

File: models/arm.urdf.xacro (robot description, xacro)
@@ -46,5 +46,4 @@
       <origin xyz="0 0 0.0793166" rpy="0 0 ${PI/2}"/>
     </joint>
-    <xacro:barrett_hand prefix="${prefix}" />
   </xacro:macro>
   <!-- Define a macro to construct the arm with a Barrett BHand on the end of it -->
@@ -59,5 +58,4 @@
       <origin xyz="0 0 0.0793166" rpy="0 0 ${PI/2}"/>
     </joint>
-    <xacro:barrett_hand prefix="${prefix}" />
   </xacro:macro>
 </robot>

File: models/components.urdf.xacro (robot description, xacro)
@@ -142,5 +142,5 @@
       <inertial>
         <origin xyz="0 0 0" />
-        <mass value="3.40016804" />
+        <mass value="3.20016804" />
         <origin xyz="-0.04001488 -.00022942 .13271662" rpy="0 0 0" />
         <inertia  ixx="0.01491672" ixy="0.00001741"   ixz="-0.00150604"
