Commit message: lots of updates

File: models/arm.urdf.xacro (robot description, xacro)
@@ -27,9 +27,28 @@
   <include filename="$(find bard_urdf)/models/common.urdf.xacro"/>
   <include filename="$(find bard_urdf)/models/components.urdf.xacro"/>
+  <!-- different types of arms -->
+  <xacro:macro name="wam_4dof" params="prefix parentLink xyz rpy">
+    <xacro:wam_upper_arm prefix="${prefix}" parentLink="${parentLink}" xyz="${xyz}" rpy="${rpy}"/>
+    <xacro:hollow_forearm prefix="${prefix}"/>
+  </xacro:macro>
+  <xacro:macro name="wam_7dof" params="prefix parentLink xyz rpy">
+    <xacro:wam_upper_arm prefix="${prefix}" parentLink="${parentLink}" xyz="${xyz}" rpy="${rpy}"/>
+    <xacro:actuated_forearm prefix="${prefix}"/>
+  </xacro:macro>
+  <xacro:macro name="wam_4dof_hand" params="prefix parentLink xyz rpy">
+  </xacro:macro>
+  <xacro:macro name="wam_7dof_hand" params="prefix parentLink xyz rpy">
+  </xacro:macro>
   <!-- Define a macro to construct the arm -->
-  <xacro:macro name="wam_arm" params="prefix parentLink xyz rpy">
+  <xacro:macro name="wam_upper_arm" params="prefix parentLink xyz rpy">
     <xacro:Shoulder prefix="${prefix}" parentLink="${parentLink}" xyz="${xyz}" rpy="${rpy}"/>
     <xacro:UpperArmInShoulder prefix="${prefix}"/>
     <xacro:UpperArm prefix="${prefix}"/>
+  </xacro:macro>
+  <xacro macro name="hollow_forearm" params="prefix"/>
+    <xacro:HollowForeArm prefix="${prefix}"/>
+    <xacro:HollowWrist prefix="${prefix}"/>
+  </xacro:macro>
+  <xacro macro name="actuated_forearm" params="prefix"/>
     <xacro:ForeArm prefix="${prefix}"/>
     <xacro:UpperWristYaw prefix="${prefix}"/>

File: models/components.urdf.xacro (robot description, xacro)
@@ -32,30 +32,6 @@
   <include filename="$(find bard_urdf)/models/hand.urdf.xacro"/>
   <include filename="$(find bard_urdf)/models/common.urdf.xacro"/>
+  <!-- Upper arm macros -->
   <xacro:macro name="Shoulder" params="prefix parentLink xyz rpy">
-    <link name="${prefix}/ShoulderLink" >
-      <inertial>
-        <origin xyz="-.00443422 0.1289039 -.00066489" />
-        <mass value="10.7677" />
-        <inertia  ixx=".13488033" ixy="-.00213041"   ixz="-.00012485"
-          iyy=".11328369"  iyz=".00068555"
-          izz=".09046330" />
-      </inertial>
-      <visual>
-        <material name="WAMGrey" />
-        <!--  this orgin is not centered because the origin in our model is not at the same spot as the origin barret uses for inertia-->
-        <origin xyz="0 .189 0" rpy="${PI} 0 0" />
-        <geometry>
-          <mesh filename="${homeDirectory}/models/componentSTL/wamShoulderLink1.DAE"/>
-        </geometry>
-      </visual>
-      <collision>
-        <origin xyz="0 .189 0" rpy="${PI} 0 0" />
-        <geometry>
-          <mesh filename="${homeDirectory}/models/componentSTL/wamShoulderLink1.stl"/>
-        </geometry>
-      </collision>
-    </link>
-    <xacro:gazeboReferenceDAE name="${prefix}/ShoulderLink"/>
-    <xacro:control topicName="${prefix}/ShoulderYaw" name="DarmSim_${prefix}Arm_WAM_ShoulderYaw" linkName="${prefix}/ShoulderLink" jointName="${prefix}/YawJoint" />
     <joint name="${prefix}/YawJoint" type="revolute">
       <parent link="${parentLink}"/>
@@ -67,30 +43,31 @@
       <dynamics damping="1.0" friction="100.0"/>
     </joint>
+    <link name="${prefix}/ShoulderLink" >
+      <inertial>
+        <origin xyz="-.00443422 0.1289039 -.00066489" />
+        <mass value="10.7677" />
+        <inertia  ixx=".13488033" ixy="-.00213041"   ixz="-.00012485"
+          iyy=".11328369"  iyz=".00068555"
+          izz=".09046330" />
+      </inertial>
+      <visual>
+        <material name="WAMGrey" />
+        <!--  this orgin is not centered because the origin in our model is not at the same spot as the origin barret uses for inertia-->
+        <origin xyz="0 .189 0" rpy="${PI} 0 0" />
+        <geometry>
+          <mesh filename="${homeDirectory}/models/componentSTL/wamShoulderLink1.DAE"/>
+        </geometry>
+      </visual>
+      <collision>
+        <origin xyz="0 .189 0" rpy="${PI} 0 0" />
+        <geometry>
+          <mesh filename="${homeDirectory}/models/componentSTL/wamShoulderLink1.stl"/>
+        </geometry>
+      </collision>
+    </link>
+    <xacro:gazeboReferenceDAE name="${prefix}/ShoulderLink"/>
+    <xacro:control topicName="${prefix}/ShoulderYaw" name="DarmSim_${prefix}Arm_WAM_ShoulderYaw" linkName="${prefix}/ShoulderLink" jointName="${prefix}/YawJoint" />
   </xacro:macro>
   <xacro:macro name="UpperArmInShoulder" params="prefix">
-    <link name="${prefix}/UpperArmInShoulderLink" >
-      <visual>
-        <material name="WAMGrey" />
-        <origin xyz="0 0 0" rpy="${PI} 0 0" />
-        <geometry>
-          <mesh filename="${homeDirectory}/models/componentSTL/wamUpperArmInShoulderLink.DAE"/>
-        </geometry>
-      </visual>
-      <inertial>
-        <origin xyz="-.00236981 .03105614 .01542114" />
-        <mass value="3.87493756" />
-        <inertia  ixx=".02140958" ixy=".00027172"  ixz=".00002461"
-          iyy=".01377875"  iyz="-.00181920"
-          izz=".01558906" />
-      </inertial>
-      <collision>
-        <origin xyz="0 0 0" rpy="${PI} 0 0" />
-        <geometry>
-          <mesh filename="${homeDirectory}/models/componentSTL/wamUpperArmInShoulderLink2.stl"/>
-        </geometry>
-      </collision>
-    </link>
-    <xacro:gazeboReferenceDAE name="${prefix}/UpperArmInShoulderLink"/>
-    <xacro:control topicName="${prefix}/ShoulderPitch" name="DarmSim_${prefix}Arm_WAM_ShoulderPitch" linkName="${prefix}/UpperArmInShoulderLink" jointName="${prefix}/ShoulderPitchJoint" />
     <joint name="${prefix}/ShoulderPitchJoint" type="revolute">
       <parent link="${prefix}/ShoulderLink"/>
@@ -102,30 +79,30 @@
       <dynamics damping="1.0" friction="100.0"/>
     </joint>
+    <link name="${prefix}/UpperArmInShoulderLink" >
+      <visual>
+        <material name="WAMGrey" />
+        <origin xyz="0 0 0" rpy="${PI} 0 0" />
+        <geometry>
+          <mesh filename="${homeDirectory}/models/componentSTL/wamUpperArmInShoulderLink.DAE"/>
+        </geometry>
+      </visual>
+      <inertial>
+        <origin xyz="-.00236981 .03105614 .01542114" />
+        <mass value="3.87493756" />
+        <inertia  ixx=".02140958" ixy=".00027172"  ixz=".00002461"
+          iyy=".01377875"  iyz="-.00181920"
+          izz=".01558906" />
+      </inertial>
+      <collision>
+        <origin xyz="0 0 0" rpy="${PI} 0 0" />
+        <geometry>
+          <mesh filename="${homeDirectory}/models/componentSTL/wamUpperArmInShoulderLink2.stl"/>
+        </geometry>
+      </collision>
+    </link>
+    <xacro:gazeboReferenceDAE name="${prefix}/UpperArmInShoulderLink"/>
+    <xacro:control topicName="${prefix}/ShoulderPitch" name="DarmSim_${prefix}Arm_WAM_ShoulderPitch" linkName="${prefix}/UpperArmInShoulderLink" jointName="${prefix}/ShoulderPitchJoint" />
   </xacro:macro>
   <xacro:macro name="UpperArm" params="prefix">
-    <link name="${prefix}/UpperArmLink" >
-      <inertial>
-        <origin xyz="-.03826 .20751 .00003" />
-        <mass value="1.80228141" />
-        <inertia  ixx=".05911077" ixy="-.00249612"  ixz=".00000738"
-          iyy=".00324550"   iyz="-.00001767"
-          izz=".05927043" />
-      </inertial>
-      <visual>
-        <material name="WAMGrey" />
-        <origin xyz="0 0 0" rpy="0 0 0" />
-        <geometry>
-          <mesh filename="${homeDirectory}/models/componentSTL/wamUpperArmLink3.DAE"/>
-        </geometry>
-      </visual>
-      <collision>
-        <origin xyz="0 0 0" rpy="0 0 0" />
-        <geometry>
-          <mesh filename="${homeDirectory}/models/componentSTL/wamUpperArmLink3.stl"/>
-        </geometry>
-      </collision>
-    </link>
-    <xacro:gazeboReferenceDAE name="${prefix}/UpperArmLink" />
-    <xacro:control topicName="${prefix}/UpperArmYaw" name="DarmSim_${prefix}Arm_WAM_UpperArmYaw" linkName="${prefix}/UpperArmLink" jointName="${prefix}/ShoulderYawJoint" />
     <joint name="${prefix}/ShoulderYawJoint" type="revolute">
       <parent link="${prefix}/UpperArmInShoulderLink"/>
@@ -137,6 +114,40 @@
       <dynamics damping="1.0" friction="100.0"/>
     </joint>
-  </xacro:macro>
-  <xacro:macro name="ForeArm" params="prefix">
+    <link name="${prefix}/UpperArmLink" >
+      <inertial>
+        <origin xyz="-.03826 .20751 .00003" />
+        <mass value="1.80228141" />
+        <inertia  ixx=".05911077" ixy="-.00249612"  ixz=".00000738"
+          iyy=".00324550"   iyz="-.00001767"
+          izz=".05927043" />
+      </inertial>
+      <visual>
+        <material name="WAMGrey" />
+        <origin xyz="0 0 0" rpy="0 0 0" />
+        <geometry>
+          <mesh filename="${homeDirectory}/models/componentSTL/wamUpperArmLink3.DAE"/>
+        </geometry>
+      </visual>
+      <collision>
+        <origin xyz="0 0 0" rpy="0 0 0" />
+        <geometry>
+          <mesh filename="${homeDirectory}/models/componentSTL/wamUpperArmLink3.stl"/>
+        </geometry>
+      </collision>
+    </link>
+    <xacro:gazeboReferenceDAE name="${prefix}/UpperArmLink" />
+    <xacro:control topicName="${prefix}/UpperArmYaw" name="DarmSim_${prefix}Arm_WAM_UpperArmYaw" linkName="${prefix}/UpperArmLink" jointName="${prefix}/ShoulderYawJoint" />
+  </xacro:macro>
+  <!-- Hollow forearm macros -->
+  <xacro macro name="HollowForeArm" params="prefix">
+    <joint name="${prefix}/ElbowJoint" type="revolute">
+      <parent link="${prefix}/UpperArmLink"/>
+      <child link="${prefix}/ForeArmLink"/>
+      <origin xyz="0.045 -0.55 0" rpy="${0.5 * PI} 0 0"/>
+      <axis xyz="0 1 0"/>
+      <limit effort="15" lower="-0.9" upper="${PI}" velocity="3.27"/>
+      <!-- <safety_controller k_position="100" k_velocity="3" soft_lower_limit="-100.0" soft_upper_limit="100.0" /> -->
+      <dynamics damping="1.0" friction="100.0"/>
+    </joint>
     <link name="${prefix}/ForeArmLink" >
       <inertial>
@@ -164,4 +175,42 @@
     <xacro:gazeboReferenceDAE name="${prefix}/ForeArmLink" />
     <xacro:control topicName="${prefix}/ElbowPitch" name="DarmSim_${prefix}Arm_WAM_ElbowPitch" linkName="${prefix}/ForeArmLink" jointName="${prefix}/ElbowJoint" />
+  </xacro:macro>
+  <xacro:macro name="HollowWrist" params="prefix">
+    <joint name="${prefix}/UpperWristJoint" type="fixed">
+      <parent link="${prefix}/ForeArmLink"/>
+      <child link="${prefix}/LowerWristPalmLink"/>
+      <origin xyz="-0.045 0 .35" rpy="-${0.5 * PI} 0 ${0.5 * PI}"/>
+      <axis xyz="0 -1 0"/>
+      <limit effort="5" lower="-4.8" upper="1.3" velocity="3.27"/>
+      <!-- <safety_controller k_position="100" k_velocity="3" soft_lower_limit="-100.0" soft_upper_limit="100.0" /> -->
+      <dynamics damping="1.0" friction="100.0"/>
+    </joint>
+    <link name="${prefix}/LowerWristPalmLink" >
+      <inertial>
+        <origin xyz="0.00008921 0.00511217 0.00435824" />
+        <mass value="1.12376019" />
+        <inertia  ixx="0.00005029" ixy="0.00000020"  ixz="0.00007582"
+          iyy="0.00007582"  iyz="-0.00000359"
+          izz="0.00006270" />
+      </inertial>
+      <visual>
+        <material name="WAMGrey" />
+        <origin xyz="0 0.02711 0" rpy="${PI} 0 0" />
+        <geometry>
+          <mesh filename="${homeDirectory}/models/componentSTL/wamUpperWristYawLink.DAE"/>
+        </geometry>
+      </visual>
+      <collision>
+        <origin xyz="0 0.02711 0" rpy="${PI} 0 0" />
+        <geometry>
+          <mesh filename="${homeDirectory}/models/componentSTL/wamUpperWristYawLink5.stl"/>
+        </geometry>
+      </collision>
+    </link>
+    <xacro:gazeboReferenceDAE name="${prefix}/UpperWristYawLink" />
+    <xacro:control topicName="${prefix}/UpperWristYaw" name="DarmSim_${prefix}Arm_WAM_UpperWristYaw" linkName="${prefix}/UpperWristYawLink" jointName="${prefix}/UpperWristYawJoint" />
+  </xacro:macro>
+  <!-- Forearm macros -->
+  <xacro:macro name="ForeArm" params="prefix">
     <joint name="${prefix}/ElbowJoint" type="revolute">
       <parent link="${prefix}/UpperArmLink"/>
@@ -173,30 +222,31 @@
       <dynamics damping="1.0" friction="100.0"/>
     </joint>
+    <link name="${prefix}/ForeArmLink" >
+      <inertial>
+        <origin xyz="0 0 0" />
+        <mass value="3.20016804" />
+        <origin xyz="-0.04001488 -.00022942 .13271662" rpy="0 0 0" />
+        <inertia  ixx="0.01491672" ixy="0.00001741"   ixz="-0.00150604"
+          iyy="0.01482988"   iyz="-0.00002109"
+          izz="0.00294463" />
+      </inertial>
+      <visual>
+        <material name="WAMGrey" />
+        <origin xyz="0 0 0" rpy="-${PI} 0 0" />
+        <geometry>
+          <mesh filename="${homeDirectory}/models/componentSTL/wamForeArmLink4.DAE"/>
+        </geometry>
+      </visual>
+      <collision>
+        <origin xyz="0 0 0" rpy="-${PI} 0 0" />
+        <geometry>
+          <mesh filename="${homeDirectory}/models/componentSTL/wamForeArmLink4.stl"/>
+        </geometry>
+      </collision>
+    </link>
+    <xacro:gazeboReferenceDAE name="${prefix}/ForeArmLink" />
+    <xacro:control topicName="${prefix}/ElbowPitch" name="DarmSim_${prefix}Arm_WAM_ElbowPitch" linkName="${prefix}/ForeArmLink" jointName="${prefix}/ElbowJoint" />
   </xacro:macro>
   <xacro:macro name="UpperWristYaw" params="prefix">
-    <link name="${prefix}/UpperWristYawLink" >
-      <inertial>
-        <origin xyz="0.00008921 0.00511217 0.00435824" />
-        <mass value="1.12376019" />
-        <inertia  ixx="0.00005029" ixy="0.00000020"  ixz="0.00007582"
-          iyy="0.00007582"  iyz="-0.00000359"
-          izz="0.00006270" />
-      </inertial>
-      <visual>
-        <material name="WAMGrey" />
-        <origin xyz="0 0.02711 0" rpy="${PI} 0 0" />
-        <geometry>
-          <mesh filename="${homeDirectory}/models/componentSTL/wamUpperWristYawLink.DAE"/>
-        </geometry>
-      </visual>
-      <collision>
-        <origin xyz="0 0.02711 0" rpy="${PI} 0 0" />
-        <geometry>
-          <mesh filename="${homeDirectory}/models/componentSTL/wamUpperWristYawLink5.stl"/>
-        </geometry>
-      </collision>
-    </link>
-    <xacro:gazeboReferenceDAE name="${prefix}/UpperWristYawLink" />
-    <xacro:control topicName="${prefix}/UpperWristYaw" name="DarmSim_${prefix}Arm_WAM_UpperWristYaw" linkName="${prefix}/UpperWristYawLink" jointName="${prefix}/UpperWristYawJoint" />
     <joint name="${prefix}/UpperWristYawJoint" type="revolute">
       <parent link="${prefix}/ForeArmLink"/>
@@ -208,30 +258,30 @@
       <dynamics damping="1.0" friction="100.0"/>
     </joint>
+    <link name="${prefix}/UpperWristYawLink" >
+      <inertial>
+        <origin xyz="0.00008921 0.00511217 0.00435824" />
+        <mass value="1.12376019" />
+        <inertia  ixx="0.00005029" ixy="0.00000020"  ixz="0.00007582"
+          iyy="0.00007582"  iyz="-0.00000359"
+          izz="0.00006270" />
+      </inertial>
+      <visual>
+        <material name="WAMGrey" />
+        <origin xyz="0 0.02711 0" rpy="${PI} 0 0" />
+        <geometry>
+          <mesh filename="${homeDirectory}/models/componentSTL/wamUpperWristYawLink.DAE"/>
+        </geometry>
+      </visual>
+      <collision>
+        <origin xyz="0 0.02711 0" rpy="${PI} 0 0" />
+        <geometry>
+          <mesh filename="${homeDirectory}/models/componentSTL/wamUpperWristYawLink5.stl"/>
+        </geometry>
+      </collision>
+    </link>
+    <xacro:gazeboReferenceDAE name="${prefix}/UpperWristYawLink" />
+    <xacro:control topicName="${prefix}/UpperWristYaw" name="DarmSim_${prefix}Arm_WAM_UpperWristYaw" linkName="${prefix}/UpperWristYawLink" jointName="${prefix}/UpperWristYawJoint" />
   </xacro:macro>
   <xacro:macro name="UpperWristPitch" params="prefix">
-    <link name="${prefix}/UpperWristPitchLink" >
-      <inertial>
-        <origin xyz="-0.00012262 -0.01703194 0.02468336" rpy="0 0 0" />
-        <mass value="0.41797364" />
-        <inertia  ixx="0.00055516" ixy="0.00000061"  ixz="-0.00000074"
-          iyy="0.00024367"  iyz="-0.00004590"
-          izz="0.00045358" />
-      </inertial>
-      <visual>
-        <material name="WAMGrey" />
-        <origin xyz="0 0 0" rpy="${0.5 * PI} 0 ${0.5 * PI}" />
-        <geometry>
-          <mesh filename="${homeDirectory}/models/componentSTL/wamUpperWristPitchLink6.DAE"/>
-        </geometry>
-      </visual>
-      <collision>
-        <origin xyz="0 0 0" rpy="${0.5 * PI} 0 ${0.5 * PI}" />
-        <geometry>
-          <mesh filename="${homeDirectory}/models/componentSTL/wamUpperWristPitchLink6.stl"/>
-        </geometry>
-      </collision>
-    </link>
-    <xacro:gazeboReferenceDAE name="${prefix}/UpperWristPitchLink" />
-    <xacro:control topicName="${prefix}/UpperWristPitch" name="DarmSim_${prefix}Arm_WAM_UpperWristPitch" linkName="${prefix}/UpperWristPitchLink" jointName="${prefix}/UpperWristPitchJoint" />
     <joint name="${prefix}/UpperWristPitchJoint" type="revolute">
       <parent link="${prefix}/UpperWristYawLink"/>
@@ -243,31 +293,31 @@
       <dynamics damping="1.0" friction="100.0"/>
     </joint>
+    <link name="${prefix}/UpperWristPitchLink" >
+      <inertial>
+        <origin xyz="-0.00012262 -0.01703194 0.02468336" rpy="0 0 0" />
+        <mass value="0.41797364" />
+        <inertia  ixx="0.00055516" ixy="0.00000061"  ixz="-0.00000074"
+          iyy="0.00024367"  iyz="-0.00004590"
+          izz="0.00045358" />
+      </inertial>
+      <visual>
+        <material name="WAMGrey" />
+        <origin xyz="0 0 0" rpy="${0.5 * PI} 0 ${0.5 * PI}" />
+        <geometry>
+          <mesh filename="${homeDirectory}/models/componentSTL/wamUpperWristPitchLink6.DAE"/>
+        </geometry>
+      </visual>
+      <collision>
+        <origin xyz="0 0 0" rpy="${0.5 * PI} 0 ${0.5 * PI}" />
+        <geometry>
+          <mesh filename="${homeDirectory}/models/componentSTL/wamUpperWristPitchLink6.stl"/>
+        </geometry>
+      </collision>
+    </link>
+    <xacro:gazeboReferenceDAE name="${prefix}/UpperWristPitchLink" />
+    <xacro:control topicName="${prefix}/UpperWristPitch" name="DarmSim_${prefix}Arm_WAM_UpperWristPitch" linkName="${prefix}/UpperWristPitchLink" jointName="${prefix}/UpperWristPitchJoint" />
   </xacro:macro>
   <!-- Palm without force-torque sensor -->
   <xacro:macro name="LowerWrist" params="prefix">
-    <link name="${prefix}/LowerWristYawLink" >
-      <inertial>
-        <origin xyz="-0.00000134 -0.00228167 -0.00000141" rpy="0 0 0" />
-        <mass value="0.17286134" />
-        <inertia  ixx="0.00010859" ixy="0.00000000"  ixz="-0.00000000"
-          iyy="0.00020683"  iyz="-0.0000000"
-          izz="0.00010851" />
-      </inertial>
-      <visual>
-        <material name="WAMGrey" />
-        <origin xyz="0 0 0" rpy="0 0 0" />
-        <geometry>
-          <mesh filename="${homeDirectory}/models/componentSTL/forceTorqueSensor.DAE"/>
-        </geometry>
-      </visual>
-      <collision>
-        <origin xyz="0 0 0" rpy="0 0 0" />
-        <geometry>
-          <mesh filename="${homeDirectory}/models/componentSTL/forceTorqueSensor.stl"/>
-        </geometry>
-      </collision>
-    </link>
-    <xacro:gazeboReferenceDAE name="${prefix}/LowerWristYawLink"/>
-    <xacro:control topicName="${prefix}/LowerWristYaw" name="DarmSim_${prefix}Arm_WAM_LowerWristYaw" linkName="${prefix}/LowerWristYawLink" jointName="${prefix}/LowerWristYawJoint" />
     <joint name="${prefix}/LowerWristYawJoint" type="revolute">
       <parent link="${prefix}/UpperWristPitchLink"/>
@@ -279,6 +329,36 @@
       <dynamics damping="1.0" friction="100.0"/>
     </joint>
+    <link name="${prefix}/LowerWristYawLink" >
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
Commit message: updating launchfile and fixing urdf

File: models/arm.urdf.xacro (robot description, xacro)
@@ -31,12 +31,10 @@
     <xacro:wam_upper_arm prefix="${prefix}" parentLink="${parentLink}" xyz="${xyz}" rpy="${rpy}"/>
     <xacro:hollow_forearm prefix="${prefix}"/>
+    <xacro:barrett_palm prefix="${prefix}"/>
   </xacro:macro>
   <xacro:macro name="wam_7dof" params="prefix parentLink xyz rpy">
     <xacro:wam_upper_arm prefix="${prefix}" parentLink="${parentLink}" xyz="${xyz}" rpy="${rpy}"/>
     <xacro:actuated_forearm prefix="${prefix}"/>
-  </xacro:macro>
-  <xacro:macro name="wam_4dof_hand" params="prefix parentLink xyz rpy">
-  </xacro:macro>
-  <xacro:macro name="wam_7dof_hand" params="prefix parentLink xyz rpy">
+    <xacro:barrett_palm prefix="${prefix}"/>
   </xacro:macro>
   <!-- Define a macro to construct the arm -->
@@ -46,9 +44,9 @@
     <xacro:UpperArm prefix="${prefix}"/>
   </xacro:macro>
-  <xacro macro name="hollow_forearm" params="prefix"/>
+  <xacro:macro name="hollow_forearm" params="prefix">
     <xacro:HollowForeArm prefix="${prefix}"/>
     <xacro:HollowWrist prefix="${prefix}"/>
   </xacro:macro>
-  <xacro macro name="actuated_forearm" params="prefix"/>
+  <xacro:macro name="actuated_forearm" params="prefix">
     <xacro:ForeArm prefix="${prefix}"/>
     <xacro:UpperWristYaw prefix="${prefix}"/>

File: models/components.urdf.xacro (robot description, xacro)
@@ -140,5 +140,5 @@
   </xacro:macro>
   <!-- Hollow forearm macros -->
-  <xacro macro name="HollowForeArm" params="prefix">
+  <xacro:macro name="HollowForeArm" params="prefix">
     <joint name="${prefix}/ElbowJoint" type="revolute">
       <parent link="${prefix}/UpperArmLink"/>
