Commit message: fixing urdf

File: models/arm.urdf.xacro (robot description, xacro)
@@ -31,12 +31,14 @@
     <xacro:wam_upper_arm prefix="${prefix}" parentLink="${parentLink}" xyz="${xyz}" rpy="${rpy}"/>
     <xacro:hollow_forearm prefix="${prefix}"/>
-    <xacro:barrett_palm prefix="${prefix}"/>
   </xacro:macro>
   <xacro:macro name="wam_7dof" params="prefix parentLink xyz rpy">
     <xacro:wam_upper_arm prefix="${prefix}" parentLink="${parentLink}" xyz="${xyz}" rpy="${rpy}"/>
     <xacro:actuated_forearm prefix="${prefix}"/>
-    <xacro:barrett_palm prefix="${prefix}"/>
   </xacro:macro>
-  <!-- Define a macro to construct the arm -->
+  <xacro:macro name="wam_7dof_ft" params="prefix parentLink xyz rpy">
+    <xacro:wam_upper_arm prefix="${prefix}" parentLink="${parentLink}" xyz="${xyz}" rpy="${rpy}"/>
+    <xacro:actuated_forearm_ft prefix="${prefix}"/>
+  </xacro:macro>
+  <!-- upper arm only -->
   <xacro:macro name="wam_upper_arm" params="prefix parentLink xyz rpy">
     <xacro:Shoulder prefix="${prefix}" parentLink="${parentLink}" xyz="${xyz}" rpy="${rpy}"/>
@@ -44,35 +46,27 @@
     <xacro:UpperArm prefix="${prefix}"/>
   </xacro:macro>
+  <!-- forearm with no actuation "wrist" -->
   <xacro:macro name="hollow_forearm" params="prefix">
     <xacro:HollowForeArm prefix="${prefix}"/>
     <xacro:HollowWrist prefix="${prefix}"/>
+    <xacro:Palm prefix="${prefix}"/>
   </xacro:macro>
+  <!-- forearm with actuation "wrist" -->
   <xacro:macro name="actuated_forearm" params="prefix">
     <xacro:ForeArm prefix="${prefix}"/>
     <xacro:UpperWristYaw prefix="${prefix}"/>
     <xacro:UpperWristPitch prefix="${prefix}"/>
-  </xacro:macro>
-  <xacro:macro name="barrett_palm" params="prefix">
     <xacro:LowerWrist prefix="${prefix}"/>
     <xacro:LowerWristPalm prefix="${prefix}"/>
-    <link name="${prefix}/PalmLink" />
-    <joint name="${prefix}/PalmJoint" type="fixed">
-      <parent link="${prefix}/LowerWristPalmLink"/>
-      <child link="${prefix}/PalmLink"/>
-      <!--             <origin xyz="0 0 0.1293166" rpy="0 0 0"/> -->
-      <origin xyz="0 0 0.0793166" rpy="0 0 ${PI/2}"/>
-    </joint>
+    <xacro:Palm prefix="${prefix}"/>
   </xacro:macro>
   <!-- Define a macro to construct the arm with a Barrett BHand on the end of it -->
-  <xacro:macro name="barrett_ft_palm" params="prefix">
+  <xacro:macro name="actuated_forearm_ft" params="prefix">
+    <xacro:ForeArm prefix="${prefix}"/>
+    <xacro:UpperWristYaw prefix="${prefix}"/>
+    <xacro:UpperWristPitch prefix="${prefix}"/>
     <xacro:LowerWristFT prefix="${prefix}"/>
     <xacro:LowerWristPalmFT prefix="${prefix}"/>
-    <link name="${prefix}/PalmLink" />
-    <joint name="${prefix}/PalmJoint" type="fixed">
-      <parent link="${prefix}/LowerWristPalmLink"/>
-      <child link="${prefix}/PalmLink"/>
-      <!--             <origin xyz="0 0 0.1293166" rpy="0 0 0"/> -->
-      <origin xyz="0 0 0.0793166" rpy="0 0 ${PI/2}"/>
-    </joint>
+    <xacro:Palm prefix="${prefix}"/>
   </xacro:macro>
 </robot>

File: models/components.urdf.xacro (robot description, xacro)
@@ -506,4 +506,14 @@
     </gazebo>
   </xacro:macro>
+  <!-- Palm -->
+  <xacro:macro name="Palm" params="prefix">
+    <link name="${prefix}/PalmLink" />
+    <joint name="${prefix}/PalmJoint" type="fixed">
+      <parent link="${prefix}/LowerWristPalmLink"/>
+      <child link="${prefix}/PalmLink"/>
+      <!--             <origin xyz="0 0 0.1293166" rpy="0 0 0"/> -->
+      <origin xyz="0 0 0.0793166" rpy="0 0 ${PI/2}"/>
+    </joint>
+  </xacro:macro>
   <!-- Hand macros -->
   <xacro:macro name="KnuckleOne" params="prefix number xyz rpy axis">

File: models/left_arm.urdf.xacro (robot description, xacro)
@@ -48,5 +48,4 @@
   </joint>
   <xacro:wam_7dof prefix="LeftWAM" parentLink="LeftWAM/FixedLink" xyz="0 0 0" rpy="0 0 0" />
-  <xacro:barrett_palm prefix="LeftWAM"/>
   <!--xacro:barrett_hand prefix="LeftWAM" /-->
   <!-- Simulation stuff -->

Commit message: working ik pose controller

File: models/arm.urdf.xacro (robot description, xacro)
@@ -50,5 +50,4 @@
     <xacro:HollowForeArm prefix="${prefix}"/>
     <xacro:HollowWrist prefix="${prefix}"/>
-    <xacro:Palm prefix="${prefix}"/>
   </xacro:macro>
   <!-- forearm with actuation "wrist" -->
@@ -58,6 +57,4 @@
     <xacro:UpperWristPitch prefix="${prefix}"/>
     <xacro:LowerWrist prefix="${prefix}"/>
-    <xacro:LowerWristPalm prefix="${prefix}"/>
-    <xacro:Palm prefix="${prefix}"/>
   </xacro:macro>
   <!-- Define a macro to construct the arm with a Barrett BHand on the end of it -->
@@ -67,6 +64,4 @@
     <xacro:UpperWristPitch prefix="${prefix}"/>
     <xacro:LowerWristFT prefix="${prefix}"/>
-    <xacro:LowerWristPalmFT prefix="${prefix}"/>
-    <xacro:Palm prefix="${prefix}"/>
   </xacro:macro>
 </robot>

File: models/components.urdf.xacro (robot description, xacro)
@@ -287,5 +287,5 @@
       <parent link="${prefix}/UpperWristYawLink"/>
       <child link="${prefix}/UpperWristPitchLink"/>
-      <origin xyz="0 0 0" rpy="${0.5 * PI} ${0.5 * PI} 0"/>
+      <origin xyz="0 0 0" rpy="${0.5 * PI} ${PI} 0"/>
       <axis xyz="0 1 0"/>
       <limit effort="5" lower="-1.45" upper="1.45" velocity="3.27"/><!-- 1.45 is a limit taken in from 1.5 due to saftey and differences between arms. -->
@@ -296,5 +296,5 @@
       <inertial>
         <origin xyz="-0.00012262 -0.01703194 0.02468336" rpy="0 0 0" />
-        <mass value="0.41797364" />
+        <mass value="0.51797364" />
         <inertia  ixx="0.00055516" ixy="0.00000061"  ixz="-0.00000074"
           iyy="0.00024367"  iyz="-0.00004590"
@@ -332,5 +332,5 @@
       <inertial>
         <origin xyz="-0.00000134 -0.00228167 -0.00000141" rpy="0 0 0" />
-        <mass value="0.17286134" />
+        <mass value="0.08286134" />
         <inertia  ixx="0.00010859" ixy="0.00000000"  ixz="-0.00000000"
           iyy="0.00020683"  iyz="-0.0000000"
@@ -353,62 +353,4 @@
     <xacro:gazeboReferenceDAE name="${prefix}/LowerWristYawLink"/>
     <xacro:control topicName="${prefix}/LowerWristYaw" name="DarmSim_${prefix}Arm_WAM_LowerWristYaw" linkName="${prefix}/LowerWristYawLink" jointName="${prefix}/LowerWristYawJoint" />
-  </xacro:macro>
-  <xacro:macro name="LowerWristPalm" params="prefix">
-    <joint name="${prefix}/LowerWristPalmJoint" type="fixed">
-      <parent link="${prefix}/LowerWristYawLink"/>
-      <child link="${prefix}/LowerWristPalmLink"/>
-      <origin xyz="0 0 0" rpy="0 0 -${0.5 * PI}"/>
-      <provideFeedback value="true"/>
-    </joint>
-    <link name="${prefix}/LowerWristPalmLink" >
-      <inertial>
-        <origin xyz="0.00035500 -0.00499005 0.04864979" />
-        <mass value="0.63352875" />
-        <inertia  ixx="0.00102103" ixy="0.00000775"  ixz="-0.00001230"
-          iyy="0.00080944"  iyz="-0.00014417"
-          izz="0.00068788" />
-      </inertial>
-      <visual>
-        <material name="WAMGrey" />
-        <origin xyz="0 0 0" rpy="0 0 0" />
-        <geometry>
-          <mesh filename="${homeDirectory}/models/componentSTL/palm.DAE"/>
-        </geometry>
-      </visual>
-      <collision>
-        <origin xyz="0 0 0" rpy="0 0 0" />
-        <geometry>
-          <mesh filename="${homeDirectory}/models/componentSTL/palm.stl"/>
-        </geometry>
-      </collision>
-    </link>
-    <xacro:gazeboReferenceDAE name="${prefix}/LowerWristPalmLink"/>
-    <gazebo reference="${prefix}/LowerWristPalmJoint">
-      <provideFeedback value="true"/>
-    </gazebo>
-    <gazebo>
-      <controller:gazebo_ros_jointFeedback name="${prefix}_JointFTsensor" plugin="libgazebo_ros_jointFeedback.so">
-        <alwaysOn>true</alwaysOn>
-        <updateRate>100.0</updateRate>
-        <jointName>${prefix}/LowerWristPalmJoint</jointName>
-        <topicName>${prefix}/BHand/ForceTorqueSensor</topicName>
-        <bodyRelation>child</bodyRelation>
-        <frameName>${prefix}/LowerWristPalmLink</frameName>
-        <interface:position name="${prefix}_JointFTsensor_force_iface" />
-      </controller:gazebo_ros_jointFeedback>
-    </gazebo>
-    <gazebo reference="${prefix}/LowerWristPalmLink">
-      <sensor:contact name="${prefix}Palm_contact_sensor">
-        <geom>${prefix}/LowerWristPalmLink_geom</geom>
-        <updateRate>100.0</updateRate>
-        <controller:gazebo_ros_bumper name="${prefix}/LowerWristPalmLink/bumperController" plugin="libgazebo_ros_bumper.so">
-          <alwaysOn>true</alwaysOn>
-          <updateRate>100.0</updateRate>
-          <frameName>${prefix}/LowerWristPalmLink</frameName>
-          <bumperTopicName>${prefix}/BHand/Palm/bumper</bumperTopicName>
-          <interface:bumper name="DarmSim${prefix}ArmWAMLowerWristPalmLink_bumper_iface" />
-        </controller:gazebo_ros_bumper>
-      </sensor:contact>
-    </gazebo>
   </xacro:macro>
   <!-- Palm with ForceTorque macros -->
@@ -447,72 +389,4 @@
     <xacro:gazeboReferenceDAE name="${prefix}/LowerWristYawLink"/>
     <xacro:control topicName="${prefix}/LowerWristYaw" name="DarmSim_${prefix}Arm_WAM_LowerWristYaw" linkName="${prefix}/LowerWristYawLink" jointName="${prefix}/LowerWristYawJoint" />
-  </xacro:macro>
-  <xacro:macro name="LowerWristPalmFT" params="prefix">
-    <joint name="${prefix}/LowerWristPalmJoint" type="fixed">
-      <parent link="${prefix}/LowerWristYawLink"/>
-      <child link="${prefix}/LowerWristPalmLink"/>
-      <origin xyz="0 0 0.0048" rpy="0 0 -${0.5 * PI}"/>
-      <provideFeedback value="true"/>
-    </joint>
-    <link name="${prefix}/LowerWristPalmLink" >
-      <inertial>
-        <origin xyz="0.00035500 -0.00499005 0.04864979" />
-        <mass value="0.63352875" />
-        <inertia  ixx="0.00102103" ixy="0.00000775"  ixz="-0.00001230"
-          iyy="0.00080944"  iyz="-0.00014417"
-          izz="0.00068788" />
-      </inertial>
-      <visual>
-        <material name="WAMGrey" />
-        <origin xyz="0 0 0" rpy="0 0 0" />
-        <geometry>
-          <mesh filename="${homeDirectory}/models/componentSTL/palm.DAE"/>
-        </geometry>
-      </visual>
-      <collision>
-        <origin xyz="0 0 0" rpy="0 0 0" />
-        <geometry>
-          <mesh filename="${homeDirectory}/models/componentSTL/palm.stl"/>
-        </geometry>
-      </collision>
-    </link>
-    <xacro:gazeboReferenceDAE name="${prefix}/LowerWristPalmLink"/>
-    <gazebo reference="${prefix}/LowerWristPalmJoint">
-      <provideFeedback value="true"/>
-    </gazebo>
-    <gazebo>
-      <controller:gazebo_ros_jointFeedback name="${prefix}_JointFTsensor" plugin="libgazebo_ros_jointFeedback.so">
-        <alwaysOn>true</alwaysOn>
-        <updateRate>100.0</updateRate>
-        <jointName>${prefix}/LowerWristPalmJoint</jointName>
-        <topicName>${prefix}/BHand/ForceTorqueSensor</topicName>
-        <bodyRelation>child</bodyRelation>
-        <frameName>${prefix}/LowerWristPalmLink</frameName>
-        <interface:position name="${prefix}_JointFTsensor_force_iface" />
-      </controller:gazebo_ros_jointFeedback>
-    </gazebo>
-    <gazebo reference="${prefix}/LowerWristPalmLink">
-      <sensor:contact name="${prefix}Palm_contact_sensor">
-        <geom>${prefix}/LowerWristPalmLink_geom</geom>
-        <updateRate>100.0</updateRate>
-        <controller:gazebo_ros_bumper name="${prefix}/LowerWristPalmLink/bumperController" plugin="libgazebo_ros_bumper.so">
-          <alwaysOn>true</alwaysOn>
-          <updateRate>100.0</updateRate>
-          <frameName>${prefix}/LowerWristPalmLink</frameName>
-          <bumperTopicName>${prefix}/BHand/Palm/bumper</bumperTopicName>
-          <interface:bumper name="DarmSim${prefix}ArmWAMLowerWristPalmLink_bumper_iface" />
-        </controller:gazebo_ros_bumper>
-      </sensor:contact>
-    </gazebo>
-  </xacro:macro>
-  <!-- Palm -->
-  <xacro:macro name="Palm" params="prefix">
-    <link name="${prefix}/PalmLink" />
-    <joint name="${prefix}/PalmJoint" type="fixed">
-      <parent link="${prefix}/LowerWristPalmLink"/>
-      <child link="${prefix}/PalmLink"/>
-      <!--             <origin xyz="0 0 0.1293166" rpy="0 0 0"/> -->
-      <origin xyz="0 0 0.0793166" rpy="0 0 ${PI/2}"/>
-    </joint>
   </xacro:macro>
   <!-- Hand macros -->

File: models/hand.urdf.xacro (robot description, xacro)
@@ -29,4 +29,14 @@
   xmlns:xacro="http://www.ros.org/wiki/xacro">
   <include filename="$(find bard_urdf)/models/common.urdf.xacro"/>
+  <!-- Palm -->
+  <xacro:macro name="Palm" params="prefix">
+    <link name="${prefix}/PalmLink" />
+    <joint name="${prefix}/PalmJoint" type="fixed">
+      <parent link="${prefix}/LowerWristPalmLink"/>
+      <child link="${prefix}/PalmLink"/>
+      <!--             <origin xyz="0 0 0.1293166" rpy="0 0 0"/> -->
+      <origin xyz="0 0 0.0793166" rpy="0 0 ${PI/2}"/>
+    </joint>
+  </xacro:macro>
   <xacro:macro name="fingers" params="parent prefix number xyz rpy">
     <xacro:KnuckleTwo parent="${parent}" prefix="${prefix}" number="${number}" xyz="${xyz}" rpy="${rpy}" />
@@ -46,5 +56,123 @@
     </gazebo>
   </xacro:macro>
+  <xacro:macro name="LowerWristPalm" params="prefix">
+    <joint name="${prefix}/LowerWristPalmJoint" type="fixed">
+      <parent link="${prefix}/LowerWristYawLink"/>
+      <child link="${prefix}/LowerWristPalmLink"/>
+      <origin xyz="0 0 0" rpy="0 0 -${0.5 * PI}"/>
+      <provideFeedback value="true"/>
+    </joint>
+    <link name="${prefix}/LowerWristPalmLink" >
+      <inertial>
+        <origin xyz="0.00035500 -0.00499005 0.04864979" />
+        <mass value="0.63352875" />
+        <inertia  ixx="0.00102103" ixy="0.00000775"  ixz="-0.00001230"
+          iyy="0.00080944"  iyz="-0.00014417"
+          izz="0.00068788" />
+      </inertial>
+      <visual>
+        <material name="WAMGrey" />
+        <origin xyz="0 0 0" rpy="0 0 0" />
+        <geometry>
+          <mesh filename="${homeDirectory}/models/componentSTL/palm.DAE"/>
+        </geometry>
+      </visual>
+      <collision>
+        <origin xyz="0 0 0" rpy="0 0 0" />
+        <geometry>
+          <mesh filename="${homeDirectory}/models/componentSTL/palm.stl"/>
+        </geometry>
+      </collision>
+    </link>
+    <xacro:gazeboReferenceDAE name="${prefix}/LowerWristPalmLink"/>
+    <gazebo reference="${prefix}/LowerWristPalmJoint">
+      <provideFeedback value="true"/>
+    </gazebo>
+    <gazebo>
+      <controller:gazebo_ros_jointFeedback name="${prefix}_JointFTsensor" plugin="libgazebo_ros_jointFeedback.so">
+        <alwaysOn>true</alwaysOn>
+        <updateRate>100.0</updateRate>
+        <jointName>${prefix}/LowerWristPalmJoint</jointName>
+        <topicName>${prefix}/BHand/ForceTorqueSensor</topicName>
+        <bodyRelation>child</bodyRelation>
+        <frameName>${prefix}/LowerWristPalmLink</frameName>
+        <interface:position name="${prefix}_JointFTsensor_force_iface" />
+      </controller:gazebo_ros_jointFeedback>
+    </gazebo>
+    <gazebo reference="${prefix}/LowerWristPalmLink">
+      <sensor:contact name="${prefix}Palm_contact_sensor">
+        <geom>${prefix}/LowerWristPalmLink_geom</geom>
+        <updateRate>100.0</updateRate>
+        <controller:gazebo_ros_bumper name="${prefix}/LowerWristPalmLink/bumperController" plugin="libgazebo_ros_bumper.so">
+          <alwaysOn>true</alwaysOn>
+          <updateRate>100.0</updateRate>
+          <frameName>${prefix}/LowerWristPalmLink</frameName>
+          <bumperTopicName>${prefix}/BHand/Palm/bumper</bumperTopicName>
+          <interface:bumper name="DarmSim${prefix}ArmWAMLowerWristPalmLink_bumper_iface" />
+        </controller:gazebo_ros_bumper>
+      </sensor:contact>
+    </gazebo>
+  </xacro:macro>
+  <xacro:macro name="LowerWristPalmFT" params="prefix">
+    <joint name="${prefix}/LowerWristPalmJoint" type="fixed">
+      <parent link="${prefix}/LowerWristYawLink"/>
+      <child link="${prefix}/LowerWristPalmLink"/>
+      <origin xyz="0 0 0.0048" rpy="0 0 -${0.5 * PI}"/>
+      <provideFeedback value="true"/>
+    </joint>
+    <link name="${prefix}/LowerWristPalmLink" >
+      <inertial>
+        <origin xyz="0.00035500 -0.00499005 0.04864979" />
+        <mass value="0.63352875" />
+        <inertia  ixx="0.00102103" ixy="0.00000775"  ixz="-0.00001230"
+          iyy="0.00080944"  iyz="-0.00014417"
+          izz="0.00068788" />
+      </inertial>
+      <visual>
+        <material name="WAMGrey" />
+        <origin xyz="0 0 0" rpy="0 0 0" />
+        <geometry>
+          <mesh filename="${homeDirectory}/models/componentSTL/palm.DAE"/>
+        </geometry>
+      </visual>
+      <collision>
+        <origin xyz="0 0 0" rpy="0 0 0" />
+        <geometry>
+          <mesh filename="${homeDirectory}/models/componentSTL/palm.stl"/>
+        </geometry>
+      </collision>
+    </link>
+    <xacro:gazeboReferenceDAE name="${prefix}/LowerWristPalmLink"/>
+    <gazebo reference="${prefix}/LowerWristPalmJoint">
+      <provideFeedback value="true"/>
+    </gazebo>
+    <gazebo>
+      <controller:gazebo_ros_jointFeedback name="${prefix}_JointFTsensor" plugin="libgazebo_ros_jointFeedback.so">
+        <alwaysOn>true</alwaysOn>
+        <updateRate>100.0</updateRate>
+        <jointName>${prefix}/LowerWristPalmJoint</jointName>
+        <topicName>${prefix}/BHand/ForceTorqueSensor</topicName>
+        <bodyRelation>child</bodyRelation>
+        <frameName>${prefix}/LowerWristPalmLink</frameName>
+        <interface:position name="${prefix}_JointFTsensor_force_iface" />
+      </controller:gazebo_ros_jointFeedback>
+    </gazebo>
+    <gazebo reference="${prefix}/LowerWristPalmLink">
+      <sensor:contact name="${prefix}Palm_contact_sensor">
+        <geom>${prefix}/LowerWristPalmLink_geom</geom>
+        <updateRate>100.0</updateRate>
+        <controller:gazebo_ros_bumper name="${prefix}/LowerWristPalmLink/bumperController" plugin="libgazebo_ros_bumper.so">
+          <alwaysOn>true</alwaysOn>
+          <updateRate>100.0</updateRate>
+          <frameName>${prefix}/LowerWristPalmLink</frameName>
+          <bumperTopicName>${prefix}/BHand/Palm/bumper</bumperTopicName>
+          <interface:bumper name="DarmSim${prefix}ArmWAMLowerWristPalmLink_bumper_iface" />
+        </controller:gazebo_ros_bumper>
+      </sensor:contact>
+    </gazebo>
+  </xacro:macro>
   <xacro:macro name="barrett_hand" params="prefix">
+    <xacro:LowerWristPalm prefix="${prefix}"/>
+    <xacro:Palm prefix="${prefix}"/>
     <xacro:fingers prefix="${prefix}" parent="${prefix}/LowerWristPalmLink" number="Three" xyz="0 -0.05 0.0801966" rpy="-${0.5 * PI} -0.0429350996 -${0.5 * PI}"/>
     <xacro:KnuckleOne prefix="${prefix}" number="One" xyz=".02497 0 0.0587966" rpy="0 0 ${0.5 * PI}" axis="0 0 -1"/>
