Commit message: fixing wrist link

File: models/arm.urdf.xacro (robot description, xacro)
@@ -56,5 +56,5 @@
     <xacro:UpperWristYaw prefix="${prefix}"/>
     <xacro:UpperWristPitch prefix="${prefix}"/>
-    <xacro:LowerWrist prefix="${prefix}"/>
+    <!--xacro:LowerWrist prefix="${prefix}"/-->
   </xacro:macro>
   <!-- Define a macro to construct the arm with a Barrett BHand on the end of it -->

File: models/components.urdf.xacro (robot description, xacro)
@@ -282,5 +282,5 @@
           <color rgba="0.9 0.9 0.9 1.0"/>
         </material>
-        <origin xyz="0 0.02711 0" rpy="${PI} 0 0" />
+        <origin xyz="0 0.02711 0" rpy="${PI} ${0.5 * PI} 0" />
         <geometry>
           <mesh filename="${homeDirectory}/models/componentSTL/wamUpperWristYawLink.DAE"/>
@@ -288,5 +288,5 @@
       </visual>
       <collision>
-        <origin xyz="0 0.02711 0" rpy="${PI} 0 0" />
+        <origin xyz="0 0.02711 0" rpy="${PI} ${0.5 * PI} 0" />
         <geometry>
           <mesh filename="${homeDirectory}/models/componentSTL/wamUpperWristYawLink5.stl"/>
@@ -319,5 +319,5 @@
           <color rgba="0.9 0.9 0.9 1.0"/>
         </material>
-        <origin xyz="0 0 0" rpy="${0.5 * PI} 0 0" />
+        <origin xyz="0 0 0" rpy="${0.5 * PI} 0 ${-0.5 * PI}" />
         <geometry>
           <mesh filename="${homeDirectory}/models/componentSTL/wamUpperWristPitchLink6.dae"/>
@@ -325,5 +325,5 @@
       </visual>
       <collision>
-        <origin xyz="0 0 0" rpy="${0.5 * PI} 0 0" />
+        <origin xyz="0 0 0" rpy="${0.5 * PI} 0 ${-0.5 * PI}" />
         <geometry>
           <mesh filename="${homeDirectory}/models/componentSTL/wamUpperWristPitchLink6.stl"/>
@@ -372,3 +372,203 @@
     <xacro:control topicName="${prefix}/LowerWristYaw" name="DarmSim_${prefix}Arm_WAM_LowerWristYaw" linkName="${prefix}/LowerWristYawLink" jointName="${prefix}/LowerWristYawJoint" />
   </xacro:macro>
+  <!-- Palm without force-torque sensor -->
+  <xacro:macro name="LowerWrist" params="prefix">
+    <joint name="${prefix}/LowerWristYawJoint" type="revolute">
+      <parent link="${prefix}/UpperWristPitchLink"/>
+      <child link="${prefix}/LowerWristYawLink"/>
+      <origin xyz="0 0 0.065" rpy="0 0 0"/>
+      <axis xyz="0 0 1"/>
+      <limit effort="5" lower="-2.95" upper="2.95" velocity="0.20"/><!-- 2.95 is a limit taken in from 3 due to saftey and differences between arms. -->
+      <!-- <safety_controller k_position="100" k_velocity="3" soft_lower_limit="-100.0" soft_upper_limit="100.0" /> -->
+      <dynamics damping="1.0" friction="100.0"/>
+    </joint>
+    <link name="${prefix}/LowerWristYawLink" >
+      <inertial>
+        <origin xyz="-0.00000134 -0.00228167 -0.00000141" rpy="0 0 0" />
+        <mass value="0.08286134" />
+        <inertia  ixx="0.00010859" ixy="0.00000000"  ixz="-0.00000000"
+          iyy="0.00020683"  iyz="-0.0000000"
+          izz="0.00010851" />
+      </inertial>
+      <visual>
+        <material name="WAMGrey">
+          <color rgba="0.9 0.9 0.9 1.0"/>
+        </material>
+        <origin xyz="0 0 0" rpy="0 0 0" />
+        <geometry>
+          <mesh filename="${homeDirectory}/models/componentSTL/wamLowerWristLink7.dae"/>
+        </geometry>
+      </visual>
+      <collision>
+        <origin xyz="0 0 0" rpy="0 0 0" />
+        <geometry>
+          <mesh filename="${homeDirectory}/models/componentSTL/wamLowerWristLink7.stl"/>
+        </geometry>
+      </collision>
+    </link>
+    <xacro:gazeboReferenceDAE name="${prefix}/LowerWristYawLink"/>
+    <xacro:control topicName="${prefix}/LowerWristYaw" name="DarmSim_${prefix}Arm_WAM_LowerWristYaw" linkName="${prefix}/LowerWristYawLink" jointName="${prefix}/LowerWristYawJoint" />
+  </xacro:macro>
+  <!-- Palm with ForceTorque macros -->
+  <xacro:macro name="LowerWristFT" params="prefix">
+    <joint name="${prefix}/LowerWristYawJoint" type="revolute">
+      <parent link="${prefix}/UpperWristPitchLink"/>
+      <child link="${prefix}/LowerWristYawLink"/>
+      <origin xyz="0 0 0.06713340" rpy="0 0 0"/>
+      <axis xyz="0 0 1"/>
+      <limit effort="5" lower="-2.95" upper="2.95" velocity="0.20"/><!-- 2.95 is a limit taken in from 3 due to saftey and differences between arms. -->
+      <!-- <safety_controller k_position="100" k_velocity="3" soft_lower_limit="-100.0" soft_upper_limit="100.0" /> -->
+      <dynamics damping="1.0" friction="100.0"/>
+    </joint>
+    <link name="${prefix}/LowerWristYawLink" >
+      <inertial>
+        <origin xyz="-0.00000134 -0.00228167 -0.00000141" rpy="0 0 0" />
+        <mass value="0.17286134" />
+        <inertia  ixx="0.00010859" ixy="0.00000000"  ixz="-0.00000000"
+          iyy="0.00020683"  iyz="-0.0000000"
+          izz="0.00010851" />
+      </inertial>
+      <visual>
+        <material name="WAMGrey">
+          <color rgba="0.9 0.9 0.9 1.0"/>
+        </material>
+        <origin xyz="0 0 0" rpy="0 0 0" />
+        <geometry>
+          <mesh filename="${homeDirectory}/models/componentSTL/forceTorqueSensor.DAE"/>
+        </geometry>
+      </visual>
+      <collision>
+        <origin xyz="0 0 0" rpy="0 0 0" />
+        <geometry>
+          <mesh filename="${homeDirectory}/models/componentSTL/forceTorqueSensor.stl"/>
+        </geometry>
+      </collision>
+    </link>
+    <xacro:gazeboReferenceDAE name="${prefix}/LowerWristYawLink"/>
+    <xacro:control topicName="${prefix}/LowerWristYaw" name="DarmSim_${prefix}Arm_WAM_LowerWristYaw" linkName="${prefix}/LowerWristYawLink" jointName="${prefix}/LowerWristYawJoint" />
+  </xacro:macro>
+  <!-- Hand macros -->
+  <xacro:macro name="KnuckleOne" params="prefix number xyz rpy axis">
+    <joint name="${prefix}/BHand/Finger${number}/KnuckleOneJoint" type="revolute">
+      <parent link="${prefix}/LowerWristPalmLink"/>
+      <child link="${prefix}/BHand/Finger${number}/KnuckleOneLink"/>
+      <origin xyz="${xyz}" rpy="${rpy}"/>
+      <axis xyz="${axis}"/>
+      <limit effort="1" lower="0" upper="${PI}" velocity="0.20"/>
+      <dynamics damping="0.005" friction="100.0"/>
+    </joint>
+    <link name="${prefix}/BHand/Finger${number}/KnuckleOneLink">
+      <visual>
+        <material name="WAMGrey">
+          <color rgba="0.9 0.9 0.9 1.0"/>
+        </material>
+        <origin xyz="0 0 0" rpy="${0.5 * PI} 0 -${0.5 * PI}" />
+        <geometry>
+          <mesh filename="${homeDirectory}/models/componentSTL/firstFingerLink.DAE"/>
+        </geometry>
+      </visual>
+      <inertial>
+        <origin xyz="0.03201666 -0.00086502 0.00890075" />
+        <mass value="0.16252678" />
+        <inertia  ixx="0.00002567" ixy="-0.00000146"  ixz="0.00001128"
+          iyy="0.00008818"   iyz="-0.00000094"
+          izz="0.00007827" />
+      </inertial>
+      <collision>
+        <origin xyz="0 0 0" rpy="${0.5 * PI} 0 -${0.5 * PI}" />
+        <geometry>
+          <mesh filename="${homeDirectory}/models/componentSTL/firstFingerLink.stl"/>
+        </geometry>
+        <mu1 value="50000.0" />
+        <mu2 value="50000.0" />
+        <kp  value="1000000.0" />
+        <kd  value="1.0" />
+      </collision>
+    </link>
+    <xacro:gazeboReferenceDAE name="${prefix}/BHand/Finger${number}/KnuckleOneLink" />
+    <xacro:control topicName="${prefix}/BHand/Finger${number}/KnuckleOne" name="DarmSim_${prefix}Arm_BHand_Finger${number}KnuckleOne" linkName="${prefix}/BHand/Finger${number}/KnuckleOneLink" jointName="${prefix}/BHand/Finger${number}/KnuckleOneJoint" />
+  </xacro:macro>
+  <xacro:macro name="KnuckleTwo" params="parent prefix number xyz rpy">
+    <joint name="${prefix}/BHand/Finger${number}/KnuckleTwoJoint" type="revolute">
+      <parent link="${parent}"/>
+      <child link="${prefix}/BHand/Finger${number}/KnuckleTwoLink"/>
+      <origin xyz="${xyz}" rpy="${rpy}"/>
+      <axis xyz="0 0 -1"/>
+      <!-- 122 degrees - start orientation of 0.4 degrees-->
+      <limit effort="1" lower="0" upper="${2.12930169 - 0.00698131701}" velocity="1.50"/>
+      <dynamics damping="0.005" friction="100.0"/>
+    </joint>
+    <link name="${prefix}/BHand/Finger${number}/KnuckleTwoLink">
+      <visual>
+        <material name="WAMGrey">
+          <color rgba="0.9 0.9 0.9 1.0"/>
+        </material>
+        <origin xyz="0 0 0" rpy="${PI} ${0.5 * PI} 0" />
+        <geometry>
+          <mesh filename="${homeDirectory}/models/componentSTL/secondFingerLink.DAE"/>
+        </geometry>
+      </visual>
+      <inertial>
+        <origin xyz=".031720 .001070 -.000586" />
+        <mass value="0.057957" />
+        <inertia  ixx="0.00000461" ixy="0.00000003"  ixz="0.00000164"
+          iyy="0.00003590"  iyz="0.00000004"
+          izz="0.00003682" />
+      </inertial>
+      <collision>
+        <origin xyz="0 0 0" rpy="${PI} ${0.5 * PI} 0" />
+        <geometry>
+          <mesh filename="${homeDirectory}/models/componentSTL/secondFingerLink.stl"/>
+        </geometry>
+        <mu1 value="50000.0" />
+        <mu2 value="50000.0" />
+        <kp  value="1000000.0" />
+        <kd  value="1.0" />
+      </collision>
+    </link>
+    <xacro:gazeboReferenceDAE name="${prefix}/BHand/Finger${number}/KnuckleTwoLink"/>
+    <xacro:control topicName="${prefix}/BHand/Finger${number}/KnuckleTwo" name="DarmSim_${prefix}Arm_BHand_Finger${number}KnuckleTwo" linkName="${prefix}/BHand/Finger${number}/KnuckleTwoLink" jointName="${prefix}/BHand/Finger${number}/KnuckleTwoJoint" />
+  </xacro:macro>
+  <xacro:macro name="KnuckleThree" params="prefix number">
+    <joint name="${prefix}/BHand/Finger${number}/KnuckleThreeJoint" type="revolute">
+      <parent link="${prefix}/BHand/Finger${number}/KnuckleTwoLink"/>
+      <child link="${prefix}/BHand/Finger${number}/KnuckleThreeLink"/>
+      <!-- 42 degrees -->
+      <origin xyz="0.07 0 0" rpy="0 0 -0.733038286"/>
+      <axis xyz="0 0 -1"/>
+      <!-- measured max angle is 94.  so upper limit is 94 - start orientation (42 degrees)-->
+      <limit effort="1" lower="0" upper="${1.6406095 - 0.733038286}" velocity="1.50"/>
+      <dynamics damping="0.005" friction="100.0"/>
+    </joint>
+    <link name="${prefix}/BHand/Finger${number}/KnuckleThreeLink">
+      <visual>
+        <material name="WAMGrey">
+          <color rgba="0.9 0.9 0.9 1.0"/>
+        </material>
+        <origin xyz="0 0 0" rpy="0 ${0.5 * PI} 0" />
+        <geometry>
+          <mesh filename="${homeDirectory}/models/componentSTL/thirdFingerLink.DAE"/>
+        </geometry>
+      </visual>
+      <inertial>
+        <origin xyz="0.01970974 0.00182016 0.00020041" />
+        <mass value="0.03421781" />
+        <inertia  ixx="0.00000287" ixy="0.00000091"  ixz="-0.00000007"
+          iyy="0.00001329"  iyz="-0.00000002"
+          izz="0.00001214" />
+      </inertial>
+      <collision>
+        <origin xyz="0 0 0" rpy="0 ${0.5 * PI} 0" />
+        <geometry>
+          <mesh filename="${homeDirectory}/models/componentSTL/thirdFingerLink.stl"/>
+        </geometry>
+        <mu1 value="50000.0" />
+        <mu2 value="50000.0" />
+        <kp  value="1000000.0" />
+        <kd  value="1.0" />
+      </collision>
+    </link>
+    <xacro:gazeboReferenceDAE name="${prefix}/BHand/Finger${number}/KnuckleThreeLink"/>
+    <xacro:control topicName="${prefix}/BHand/Finger${number}/KnuckleThree" name="DarmSim_${prefix}Arm_BHand_Finger${number}KnuckleThree" linkName="${prefix}/BHand/Finger${number}/KnuckleThreeLink" jointName="${prefix}/BHand/Finger${number}/KnuckleThreeJoint" />
+  </xacro:macro>
 </robot>

Commit message: Removing big wall in base link, fixing damping-induced explosion when adding the last link

File: models/arm.urdf.xacro (robot description, xacro)
@@ -56,5 +56,5 @@
     <xacro:UpperWristYaw prefix="${prefix}"/>
     <xacro:UpperWristPitch prefix="${prefix}"/>
-    <!--xacro:LowerWrist prefix="${prefix}"/-->
+    <xacro:LowerWrist prefix="${prefix}"/>
   </xacro:macro>
   <!-- Define a macro to construct the arm with a Barrett BHand on the end of it -->

File: models/components.urdf.xacro (robot description, xacro)
@@ -339,51 +339,13 @@
       <parent link="${prefix}/UpperWristPitchLink"/>
       <child link="${prefix}/LowerWristYawLink"/>
-      <origin xyz="0 0 0.065" rpy="0 0 0"/>
+      <origin xyz="0 0 0.05" rpy="0 0 0"/>
       <axis xyz="0 0 1"/>
       <limit effort="5" lower="-2.95" upper="2.95" velocity="0.20"/><!-- 2.95 is a limit taken in from 3 due to saftey and differences between arms. -->
       <!-- <safety_controller k_position="100" k_velocity="3" soft_lower_limit="-100.0" soft_upper_limit="100.0" /> -->
-      <dynamics damping="1.0" friction="100.0"/>
+      <!--dynamics damping="1.0" friction="100.0"/-->
     </joint>
     <link name="${prefix}/LowerWristYawLink" >
       <inertial>
-        <origin xyz="-0.00000134 -0.00228167 -0.00000141" rpy="0 0 0" />
-        <mass value="0.08286134" />
-        <inertia  ixx="0.00010859" ixy="0.00000000"  ixz="-0.00000000"
-          iyy="0.00020683"  iyz="-0.0000000"
-          izz="0.00010851" />
-      </inertial>
-      <visual>
-        <material name="WAMGrey">
-          <color rgba="0.9 0.9 0.9 1.0"/>
-        </material>
-        <origin xyz="0 0 0" rpy="0 0 0" />
-        <geometry>
-          <mesh filename="${homeDirectory}/models/componentSTL/wamLowerWristLink7.dae"/>
-        </geometry>
-      </visual>
-      <collision>
-        <origin xyz="0 0 0" rpy="0 0 0" />
-        <geometry>
-          <mesh filename="${homeDirectory}/models/componentSTL/wamLowerWristLink7.stl"/>
-        </geometry>
-      </collision>
-    </link>
-    <xacro:gazeboReferenceDAE name="${prefix}/LowerWristYawLink"/>
-    <xacro:control topicName="${prefix}/LowerWristYaw" name="DarmSim_${prefix}Arm_WAM_LowerWristYaw" linkName="${prefix}/LowerWristYawLink" jointName="${prefix}/LowerWristYawJoint" />
-  </xacro:macro>
-  <!-- Palm without force-torque sensor -->
-  <xacro:macro name="LowerWrist" params="prefix">
-    <joint name="${prefix}/LowerWristYawJoint" type="revolute">
-      <parent link="${prefix}/UpperWristPitchLink"/>
-      <child link="${prefix}/LowerWristYawLink"/>
-      <origin xyz="0 0 0.065" rpy="0 0 0"/>
-      <axis xyz="0 0 1"/>
-      <limit effort="5" lower="-2.95" upper="2.95" velocity="0.20"/><!-- 2.95 is a limit taken in from 3 due to saftey and differences between arms. -->
-      <!-- <safety_controller k_position="100" k_velocity="3" soft_lower_limit="-100.0" soft_upper_limit="100.0" /> -->
-      <dynamics damping="1.0" friction="100.0"/>
-    </joint>
-    <link name="${prefix}/LowerWristYawLink" >
-      <inertial>
-        <origin xyz="-0.00000134 -0.00228167 -0.00000141" rpy="0 0 0" />
+        <origin xyz="0.0 0.0 0.0" rpy="0 0 0" />
         <mass value="0.08286134" />
         <inertia  ixx="0.00010859" ixy="0.00000000"  ixz="-0.00000000"

File: robots/wam_7dof_2x.urdf.xacro (robot description, xacro)
@@ -5,40 +5,12 @@
   <!-- Root link is in the world frame-->
   <link name="world"/>
-  <!-- Fix this robot to the world -->
-  <joint name="world_joint"  type="fixed">
-    <origin xyz="0 0 0" rpy="0 0 0" />
-    <parent link="world"/>
-    <child link="baseLink"/>
-  </joint>
-  <link name = "baseLink">
-    <inertial>
-      <origin xyz="-1 0 0" />
-      <mass value="100" />
-      <inertia
-        ixx="1" ixy="0"   ixz="0"
-                iyy="1"   iyz="0"
-                          izz="1" />
-    </inertial>
-    <visual>
-      <origin rpy="0 0 0 " xyz="-1 0 1"/>
-      <geometry>
-        <box size="2 5 2"/>
-      </geometry>
-    </visual>
-    <collision>
-      <origin rpy="0 0 0 " xyz="-1 0 1"/>
-      <geometry>
-        <box size="2 5 2"/>
-      </geometry>
-    </collision>
-  </link>
   <!--<gazebo reference="baseLink">
     <static>true</static>
      <turnGravityOff>true</turnGravityOff>
    </gazebo>-->
-  <xacro:wam_root prefix="wam_left" parentLink="baseLink" xyz="0.356 0.46 1" rpy="0 ${-0.5*PI} ${0.5*PI}"/>
+  <xacro:wam_root prefix="wam_left" parentLink="world" xyz="0.356 0.46 1" rpy="0 ${-0.5*PI} ${0.5*PI}"/>
   <xacro:wam_7dof prefix="wam_left" parentLink="wam_left/FixedLink" xyz="0 0 0" rpy="0 0 0" />
   <!--xacro:barrett_hand prefix="wam_left" /-->
-  <xacro:wam_root prefix="wam_right" parentLink="baseLink" xyz="0.356 -0.46 1" rpy="0 ${-0.5*PI} ${0.5*PI}"/>
+  <xacro:wam_root prefix="wam_right" parentLink="world" xyz="0.356 -0.46 1" rpy="0 ${-0.5*PI} ${0.5*PI}"/>
   <xacro:wam_7dof prefix="wam_right" parentLink="wam_right/FixedLink" xyz="0 0 0" rpy="0 0 0" />
   <!--xacro:barrett_hand prefix="wam_right" /-->
