Commit message: new and improved

File: models/arm.urdf.xacro (robot description, xacro)
@@ -24,7 +24,7 @@
 -->
 <robot xmlns:xacro="http://www.ros.org/wiki/xacro">
-  <include filename="$(find bard_urdf)/models/hand.urdf.xacro"/>
-  <include filename="$(find bard_urdf)/models/common.urdf.xacro"/>
-  <include filename="$(find bard_urdf)/models/components.urdf.xacro"/>
+  <include filename="$(find barrett_model)/models/hand.urdf.xacro"/>
+  <include filename="$(find barrett_model)/models/common.urdf.xacro"/>
+  <include filename="$(find barrett_model)/models/components.urdf.xacro"/>
   <!-- different types of arms -->
   <xacro:macro name="wam_4dof" params="prefix parentLink xyz rpy">
@@ -42,5 +42,6 @@
   <!-- upper arm only -->
   <xacro:macro name="wam_upper_arm" params="prefix parentLink xyz rpy">
-    <xacro:Shoulder prefix="${prefix}" parentLink="${parentLink}" xyz="${xyz}" rpy="${rpy}"/>
+    <xacro:Base prefix="${prefix}" parentLink="${parentLink}" xyz="${xyz}" rpy="${rpy}"/>
+    <xacro:Shoulder prefix="${prefix}"/>
     <xacro:UpperArmInShoulder prefix="${prefix}"/>
     <xacro:UpperArm prefix="${prefix}"/>

File: models/common.urdf.xacro (robot description, xacro)
@@ -31,6 +31,6 @@
   xmlns:xacro="http://ros.org/wiki/xacro">
   <!-- Directories -->
-  <xacro:property name="homeDirectory" value="package://bard_urdf" />
-  <xacro:property name="highResModelDirectory" value="${homeDirectory}/models/componentSTL/splitModels" />
+  <xacro:property name="models_path" value="package://barrett_model/models" />
+  <xacro:property name="highResModelDirectory" value="${models_path}/meshes/splitModels" />
   <!-- Constants -->
   <xacro:property name="PI" value="3.1415926535897931" />

File: models/components.urdf.xacro (robot description, xacro)
@@ -30,12 +30,53 @@
   xmlns:geom="http://playerstage.sourceforge.net/gazebo/xmlschema/#geom"
   xmlns:xacro="http://ros.org/wiki/xacro">
-  <include filename="$(find bard_urdf)/models/hand.urdf.xacro"/>
-  <include filename="$(find bard_urdf)/models/common.urdf.xacro"/>
+  <include filename="$(find barrett_model)/models/hand.urdf.xacro"/>
+  <include filename="$(find barrett_model)/models/common.urdf.xacro"/>
   <!-- Upper arm macros -->
-  <xacro:macro name="Shoulder" params="prefix parentLink xyz rpy">
+  <xacro:macro name="Base" params="prefix parentLink xyz rpy">
+    <joint name="${prefix}/FixedJoint" type="fixed">
+      <parent link="${parentLink}"/>
+      <child link="${prefix}/BaseLink"/>
+      <origin xyz="${xyz}" rpy="${rpy}"/>
+    </joint>
+    <!-- Create the $(arg robot_name) WAM -->
+    <link name = "${prefix}/BaseLink">
+      <inertial>
+        <origin xyz="0 0 0" />
+        <mass value="100" />
+        <inertia
+          ixx="1" ixy="0"   ixz="0"
+                  iyy="1"   iyz="0"
+                            izz="1" />
+      </inertial>
+      <visual>
+        <material name="WAMGrey">
+          <color rgba="0.9 0.9 0.9 0.0"/>
+        </material>
+        <!--  this orgin is not centered because the origin in our model is not at the same spot as the origin barret uses for inertia-->
+        <origin xyz="0 0.0 0" rpy="0 0 0"/>
+        <geometry>
+          <mesh filename="${models_path}/sw_meshes/base_link.STL"/>
+        </geometry>
+      </visual>
+      <collision>
+        <origin xyz="0 0.0 0" rpy="0 0 0" />
+        <geometry>
+          <mesh filename="${models_path}/sw_meshes/base_link.STL"/>
+        </geometry>
+      </collision>
+    </link>
+    <!-- Simulation stuff -->
+    <!--gazebo>
+      <controller:gazebo_ros_controller_manager name="gazebo_ros_controller_manager" plugin="libgazebo_ros_controller_manager.so">
+        <alwaysOn>true</alwaysOn>
+        <updateRate>1000.0</updateRate>
+      </controller:gazebo_ros_controller_manager>
+    </gazebo-->
+  </xacro:macro>
+  <xacro:macro name="Shoulder" params="prefix">
     <joint name="${prefix}/YawJoint" type="revolute">
-      <parent link="${parentLink}"/>
+      <parent link="${prefix}/BaseLink"/>
       <child link="${prefix}/ShoulderLink"/>
-      <origin xyz="${xyz}" rpy="${rpy}"/>
+      <origin xyz="0 0 0.346" rpy="0 0 0"/>
       <axis xyz="0 -1 0"/>
       <limit effort="30" lower="-2.6" upper="2.6" velocity="0.50"/>
@@ -58,5 +99,5 @@
         <origin xyz="0 .189 0" rpy="${PI} 0 0" />
         <geometry>
-          <mesh filename="${homeDirectory}/models/componentSTL/wamShoulderLink1.DAE"/>
+          <mesh filename="${models_path}/meshes/wamShoulderLink1.DAE"/>
         </geometry>
       </visual>
@@ -64,5 +105,5 @@
         <origin xyz="0 .189 0" rpy="${PI} 0 0" />
         <geometry>
-          <mesh filename="${homeDirectory}/models/componentSTL/wamShoulderLink1.stl"/>
+          <mesh filename="${models_path}/meshes/wamShoulderLink1.stl"/>
         </geometry>
       </collision>
@@ -88,5 +129,5 @@
         <origin xyz="0 0 0" rpy="${PI} 0 0" />
         <geometry>
-          <mesh filename="${homeDirectory}/models/componentSTL/wamUpperArmInShoulderLink.dae"/>
+          <mesh filename="${models_path}/meshes/wamUpperArmInShoulderLink.dae"/>
         </geometry>
       </visual>
@@ -101,5 +142,5 @@
         <origin xyz="0 0 0" rpy="${PI} 0 0" />
         <geometry>
-          <mesh filename="${homeDirectory}/models/componentSTL/wamUpperArmInShoulderLink2.stl"/>
+          <mesh filename="${models_path}/meshes/wamUpperArmInShoulderLink2.stl"/>
         </geometry>
       </collision>
@@ -132,5 +173,5 @@
         <origin xyz="0 0 0" rpy="0 0 0" />
         <geometry>
-          <mesh filename="${homeDirectory}/models/componentSTL/wamUpperArmLink3.dae"/>
+          <mesh filename="${models_path}/meshes/wamUpperArmLink3.dae"/>
         </geometry>
       </visual>
@@ -138,5 +179,5 @@
         <origin xyz="0 0 0" rpy="0 0 0" />
         <geometry>
-          <mesh filename="${homeDirectory}/models/componentSTL/wamUpperArmLink3.stl"/>
+          <mesh filename="${models_path}/meshes/wamUpperArmLink3.stl"/>
         </geometry>
       </collision>
@@ -171,5 +212,5 @@
         <origin xyz="0 0 0" rpy="-${PI} 0 0" />
         <geometry>
-          <mesh filename="${homeDirectory}/models/componentSTL/wamForeArmLink4.DAE"/>
+          <mesh filename="${models_path}/meshes/wamForeArmLink4.DAE"/>
         </geometry>
       </visual>
@@ -177,5 +218,5 @@
         <origin xyz="0 0 0" rpy="-${PI} 0 0" />
         <geometry>
-          <mesh filename="${homeDirectory}/models/componentSTL/wamForeArmLink4.stl"/>
+          <mesh filename="${models_path}/meshes/wamForeArmLink4.stl"/>
         </geometry>
       </collision>
@@ -208,5 +249,5 @@
         <origin xyz="0 0.02711 0" rpy="${PI} 0 0" />
         <geometry>
-          <mesh filename="${homeDirectory}/models/componentSTL/wamUpperWristYawLink.DAE"/>
+          <mesh filename="${models_path}/meshes/wamUpperWristYawLink.DAE"/>
         </geometry>
       </visual>
@@ -214,5 +255,5 @@
         <origin xyz="0 0.02711 0" rpy="${PI} 0 0" />
         <geometry>
-          <mesh filename="${homeDirectory}/models/componentSTL/wamUpperWristYawLink5.stl"/>
+          <mesh filename="${models_path}/meshes/wamUpperWristYawLink5.stl"/>
         </geometry>
       </collision>
@@ -247,5 +288,5 @@
         <origin xyz="0 0 0" rpy="-${PI} 0 0" />
         <geometry>
-          <mesh filename="${homeDirectory}/models/componentSTL/wamForeArmLink4.DAE"/>
+          <mesh filename="${models_path}/meshes/wamForeArmLink4.DAE"/>
         </geometry>
       </visual>
@@ -253,5 +294,5 @@
         <origin xyz="0 0 0" rpy="-${PI} 0 0" />
         <geometry>
-          <mesh filename="${homeDirectory}/models/componentSTL/wamForeArmLink4.stl"/>
+          <mesh filename="${models_path}/meshes/wamForeArmLink4.stl"/>
         </geometry>
       </collision>
@@ -284,5 +325,5 @@
         <origin xyz="0 0.02711 0" rpy="${PI} ${0.5 * PI} 0" />
         <geometry>
-          <mesh filename="${homeDirectory}/models/componentSTL/wamUpperWristYawLink.DAE"/>
+          <mesh filename="${models_path}/meshes/wamUpperWristYawLink.DAE"/>
         </geometry>
       </visual>
@@ -290,5 +331,5 @@
         <origin xyz="0 0.02711 0" rpy="${PI} ${0.5 * PI} 0" />
         <geometry>
-          <mesh filename="${homeDirectory}/models/componentSTL/wamUpperWristYawLink5.stl"/>
+          <mesh filename="${models_path}/meshes/wamUpperWristYawLink5.stl"/>
         </geometry>
       </collision>
@@ -321,5 +362,5 @@
         <origin xyz="0 0 0" rpy="${0.5 * PI} 0 ${-0.5 * PI}" />
         <geometry>
-          <mesh filename="${homeDirectory}/models/componentSTL/wamUpperWristPitchLink6.dae"/>
+          <mesh filename="${models_path}/meshes/wamUpperWristPitchLink6.dae"/>
         </geometry>
       </visual>
@@ -327,5 +368,5 @@
         <origin xyz="0 0 0" rpy="${0.5 * PI} 0 ${-0.5 * PI}" />
         <geometry>
-          <mesh filename="${homeDirectory}/models/componentSTL/wamUpperWristPitchLink6.stl"/>
+          <mesh filename="${models_path}/meshes/wamUpperWristPitchLink6.stl"/>
         </geometry>
       </collision>
@@ -359,5 +400,5 @@
         <origin xyz="0 0 0" rpy="0 0 0" />
         <geometry>
-          <mesh filename="${homeDirectory}/models/componentSTL/wamLowerWristLink7.dae"/>
+          <mesh filename="${models_path}/meshes/wamLowerWristLink7.dae"/>
         </geometry>
       </visual>
@@ -365,5 +406,5 @@
         <origin xyz="0 0 0" rpy="0 0 0" />
         <geometry>
-          <mesh filename="${homeDirectory}/models/componentSTL/wamLowerWristLink7.stl"/>
+          <mesh filename="${models_path}/meshes/wamLowerWristLink7.stl"/>
         </geometry>
       </collision>
@@ -397,5 +438,5 @@
         <origin xyz="0 0 0" rpy="0 0 0" />
         <geometry>
-          <mesh filename="${homeDirectory}/models/componentSTL/forceTorqueSensor.DAE"/>
+          <mesh filename="${models_path}/meshes/forceTorqueSensor.DAE"/>
         </geometry>
       </visual>
@@ -403,5 +444,5 @@
         <origin xyz="0 0 0" rpy="0 0 0" />
         <geometry>
-          <mesh filename="${homeDirectory}/models/componentSTL/forceTorqueSensor.stl"/>
+          <mesh filename="${models_path}/meshes/forceTorqueSensor.stl"/>
         </geometry>
       </collision>
@@ -427,5 +468,5 @@
         <origin xyz="0 0 0" rpy="${0.5 * PI} 0 -${0.5 * PI}" />
         <geometry>
-          <mesh filename="${homeDirectory}/models/componentSTL/firstFingerLink.DAE"/>
+          <mesh filename="${models_path}/meshes/firstFingerLink.DAE"/>
         </geometry>
       </visual>
@@ -440,5 +481,5 @@
         <origin xyz="0 0 0" rpy="${0.5 * PI} 0 -${0.5 * PI}" />
         <geometry>
-          <mesh filename="${homeDirectory}/models/componentSTL/firstFingerLink.stl"/>
+          <mesh filename="${models_path}/meshes/firstFingerLink.stl"/>
         </geometry>
         <mu1 value="50000.0" />
@@ -468,5 +509,5 @@
         <origin xyz="0 0 0" rpy="${PI} ${0.5 * PI} 0" />
         <geometry>
-          <mesh filename="${homeDirectory}/models/componentSTL/secondFingerLink.DAE"/>
+          <mesh filename="${models_path}/meshes/secondFingerLink.DAE"/>
         </geometry>
       </visual>
@@ -481,5 +522,5 @@
         <origin xyz="0 0 0" rpy="${PI} ${0.5 * PI} 0" />
         <geometry>
-          <mesh filename="${homeDirectory}/models/componentSTL/secondFingerLink.stl"/>
+          <mesh filename="${models_path}/meshes/secondFingerLink.stl"/>
         </geometry>
         <mu1 value="50000.0" />
@@ -510,5 +551,5 @@
         <origin xyz="0 0 0" rpy="0 ${0.5 * PI} 0" />
         <geometry>
-          <mesh filename="${homeDirectory}/models/componentSTL/thirdFingerLink.DAE"/>
+          <mesh filename="${models_path}/meshes/thirdFingerLink.DAE"/>
         </geometry>
       </visual>
@@ -523,5 +564,5 @@
         <origin xyz="0 0 0" rpy="0 ${0.5 * PI} 0" />
         <geometry>
-          <mesh filename="${homeDirectory}/models/componentSTL/thirdFingerLink.stl"/>
+          <mesh filename="${models_path}/meshes/thirdFingerLink.stl"/>
         </geometry>
         <mu1 value="50000.0" />

File: models/hand.urdf.xacro (robot description, xacro)
@@ -28,5 +28,5 @@
   xmlns:interface="http://playerstage.sourceforge.net/gazebo/xmlschema/#interface"
   xmlns:xacro="http://www.ros.org/wiki/xacro">
-  <include filename="$(find bard_urdf)/models/common.urdf.xacro"/>
+  <include filename="$(find barrett_model)/models/common.urdf.xacro"/>
   <!-- Palm -->
   <xacro:macro name="Palm" params="prefix">
@@ -77,5 +77,5 @@
         <origin xyz="0 0 0" rpy="0 0 0" />
         <geometry>
-          <mesh filename="${homeDirectory}/models/componentSTL/palm.DAE"/>
+          <mesh filename="${models_path}/meshes/palm.DAE"/>
         </geometry>
       </visual>
@@ -83,5 +83,5 @@
         <origin xyz="0 0 0" rpy="0 0 0" />
         <geometry>
-          <mesh filename="${homeDirectory}/models/componentSTL/palm.stl"/>
+          <mesh filename="${models_path}/meshes/palm.stl"/>
         </geometry>
       </collision>
@@ -137,5 +137,5 @@
         <origin xyz="0 0 0" rpy="0 0 0" />
         <geometry>
-          <mesh filename="${homeDirectory}/models/componentSTL/palm.DAE"/>
+          <mesh filename="${models_path}/meshes/palm.DAE"/>
         </geometry>
       </visual>
@@ -143,5 +143,5 @@
         <origin xyz="0 0 0" rpy="0 0 0" />
         <geometry>
-          <mesh filename="${homeDirectory}/models/componentSTL/palm.stl"/>
+          <mesh filename="${models_path}/meshes/palm.stl"/>
         </geometry>
       </collision>

File: models/unused.urdf.xacro (robot description, xacro)
@@ -14,11 +14,11 @@
         <origin xyz="0 0 0" rpy="0 0 0" />
         <geometry>
-          <mesh filename="${homeDirectory}/models/componentSTL/lowerPanUnit.DAE"/>
-        </geometry>
-      </visual>
-      <collision>
-        <origin xyz="0 0 0" rpy="0 0 0" />
-        <geometry>
-          <mesh filename="${homeDirectory}/models/componentSTL/lowerPanUnit.stl"/>
+          <mesh filename="${models_path}/meshes/lowerPanUnit.DAE"/>
+        </geometry>
+      </visual>
+      <collision>
+        <origin xyz="0 0 0" rpy="0 0 0" />
+        <geometry>
+          <mesh filename="${models_path}/meshes/lowerPanUnit.stl"/>
         </geometry>
       </collision>
@@ -50,11 +50,11 @@
         <origin xyz="0 0 0" rpy="0 0 0" />
         <geometry>
-          <mesh filename="${homeDirectory}/models/componentSTL/lowerTiltBeamsLink.DAE"/>
-        </geometry>
-      </visual>
-      <collision>
-        <origin xyz="0 0 0" rpy="0 0 0" />
-        <geometry>
-          <mesh filename="${homeDirectory}/models/componentSTL/lowerTiltBeamsLink.stl"/>
+          <mesh filename="${models_path}/meshes/lowerTiltBeamsLink.DAE"/>
+        </geometry>
+      </visual>
+      <collision>
+        <origin xyz="0 0 0" rpy="0 0 0" />
+        <geometry>
+          <mesh filename="${models_path}/meshes/lowerTiltBeamsLink.stl"/>
         </geometry>
       </collision>
@@ -79,5 +79,5 @@
         <origin xyz="0 0 0" rpy="0 0 0" />
         <geometry>
-          <mesh filename="${homeDirectory}/models/componentSTL/lowerTiltBeamsFrontLink.DAE"/>
+          <mesh filename="${models_path}/meshes/lowerTiltBeamsFrontLink.DAE"/>
         </geometry>
         <material name="base">
@@ -95,5 +95,5 @@
         <origin xyz="0 0 0" rpy="0 0 0" />
         <geometry>
-          <mesh filename="${homeDirectory}/models/componentSTL/lowerTiltBeamsFrontLink.stl"/>
+          <mesh filename="${models_path}/meshes/lowerTiltBeamsFrontLink.stl"/>
         </geometry>
       </collision>
@@ -116,5 +116,5 @@
         <origin xyz="0 0 0" rpy="0 0 0" />
         <geometry>
-          <mesh filename="${homeDirectory}/models/componentSTL/lowerTiltBeamsTopLink.DAE"/>
+          <mesh filename="${models_path}/meshes/lowerTiltBeamsTopLink.DAE"/>
         </geometry>
         <material name="base">
@@ -132,5 +132,5 @@
         <origin xyz="0 0 0" rpy="0 0 0" />
         <geometry>
-          <mesh filename="${homeDirectory}/models/componentSTL/lowerTiltBeamsTopLink.stl"/>
+          <mesh filename="${models_path}/meshes/lowerTiltBeamsTopLink.stl"/>
         </geometry>
       </collision>
@@ -171,5 +171,5 @@
         <origin xyz="0 0 0.0" rpy="0 0 0" />
         <geometry>
-          <mesh filename="${homeDirectory}/models/componentSTL/upperTiltUnitLink.DAE"/>
+          <mesh filename="${models_path}/meshes/upperTiltUnitLink.DAE"/>
         </geometry>
       </visual>
@@ -177,5 +177,5 @@
         <origin xyz="0 0 0.0" rpy="0 0 0" />
         <geometry>
-          <mesh filename="${homeDirectory}/models/componentSTL/upperTiltUnitLink.stl"/>
+          <mesh filename="${models_path}/meshes/upperTiltUnitLink.stl"/>
         </geometry>
       </collision>
@@ -205,11 +205,11 @@
         <origin xyz="0 0 0" rpy="0 0 0" />
         <geometry>
-          <mesh filename="${homeDirectory}/models/componentSTL/Re2_Head.DAE"/>
-        </geometry>
-      </visual>
-      <collision>
-        <origin xyz="0 0 0" rpy="0 0 0" />
-        <geometry>
-          <mesh filename="${homeDirectory}/models/componentSTL/skinMeshCollision.stl"/>
+          <mesh filename="${models_path}/meshes/Re2_Head.DAE"/>
+        </geometry>
+      </visual>
+      <collision>
+        <origin xyz="0 0 0" rpy="0 0 0" />
+        <geometry>
+          <mesh filename="${models_path}/meshes/skinMeshCollision.stl"/>
         </geometry>
       </collision>

File: models/wam_7dof.urdf.xacro (robot description, xacro)
@@ -2,5 +2,5 @@
   xmlns:xacro="http://www.ros.org/wiki/xacro">
   <!-- Includea all the WAM stuff -->
-  <include filename="$(find bard_urdf)/models/wam_top.urdf.xacro"/>
+  <include filename="$(find barrett_model)/models/wam_top.urdf.xacro"/>
   <!-- Root link is in the world frame-->
   <link name = "baseLink"/>

File: models/wam_top.urdf.xacro (robot description, xacro)
@@ -3,53 +3,12 @@
   xmlns:controller="http://playerstage.sourceforge.net/gazebo/xmlschema/#controller">
   <!-- Some macros used by the WAM urdf -->
-  <include filename="$(find bard_urdf)/models/common.urdf.xacro"/>
+  <include filename="$(find barrett_model)/models/common.urdf.xacro"/>
   <!-- Definition of a single WAM arm -->
-  <include filename="$(find bard_urdf)/models/arm.urdf.xacro"/>
+  <include filename="$(find barrett_model)/models/arm.urdf.xacro"/>
   <!-- Definition of all the different parts of a WAM arm -->
-  <include filename="$(find bard_urdf)/models/components.urdf.xacro"/>
+  <include filename="$(find barrett_model)/models/components.urdf.xacro"/>
   <!-- Materials -->
   <material name="WAMGrey">
     <color rgba="0.9 0.9 0.9 1.0"/>
   </material>
-  <xacro:macro name="wam_root" params="prefix parentLink xyz rpy">
-    <!-- Create the $(arg robot_name) WAM -->
-    <link name = "${prefix}/FixedLink">
-      <inertial>
-        <origin xyz="0 0 0" />
-        <mass value="100" />
-        <inertia
-          ixx="1" ixy="0"   ixz="0"
-                  iyy="1"   iyz="0"
-                            izz="1" />
-      </inertial>
-      <visual>
-        <material name="WAMGrey">
-          <color rgba="0.9 0.9 0.9 0.0"/>
-        </material>
-        <!--  this orgin is not centered because the origin in our model is not at the same spot as the origin barret uses for inertia-->
-        <origin xyz="0 0.346 0" rpy="${PI/2} 0 0"/>
-        <geometry>
-          <mesh filename="${homeDirectory}/models/componentSTL/wamBase.dae"/>
-        </geometry>
-      </visual>
-      <collision>
-        <origin xyz="0 0.346 0" rpy="${PI/2} 0 0" />
-        <geometry>
-          <mesh filename="${homeDirectory}/models/componentSTL/wamBase.stl"/>
-        </geometry>
-      </collision>
-    </link>
-    <joint name="${prefix}/FixedJoint" type="fixed">
-      <parent link="${parentLink}"/>
-      <child link="${prefix}/FixedLink"/>
-      <origin xyz="${xyz}" rpy="${rpy}"/>
-    </joint>
-    <!-- Simulation stuff -->
-    <!--gazebo>
-      <controller:gazebo_ros_controller_manager name="gazebo_ros_controller_manager" plugin="libgazebo_ros_controller_manager.so">
-        <alwaysOn>true</alwaysOn>
-        <updateRate>1000.0</updateRate>
-      </controller:gazebo_ros_controller_manager>
-    </gazebo-->
-  </xacro:macro>
 </robot>

File: robots/wam_4dof_wam.urdf.xacro (robot description, xacro)
@@ -2,5 +2,5 @@
   xmlns:xacro="http://www.ros.org/wiki/xacro">
   <!-- Includea all the WAM stuff -->
-  <include filename="$(find bard_urdf)/models/wam_top.urdf.xacro"/>
+  <include filename="$(find barrett_model)/models/wam_top.urdf.xacro"/>
   <!-- Root link is in the world frame-->
   <link name = "baseLink"/>

File: robots/wam_4dof_wam_left.urdf.xacro (robot description, xacro)
@@ -2,5 +2,5 @@
   xmlns:xacro="http://www.ros.org/wiki/xacro">
   <!-- Includea all the WAM stuff -->
-  <include filename="$(find bard_urdf)/models/wam_top.urdf.xacro"/>
+  <include filename="$(find barrett_model)/models/wam_top.urdf.xacro"/>
   <!-- Root link is in the world frame-->
   <link name = "baseLink"/>

File: robots/wam_4dof_wam_right.urdf.xacro (robot description, xacro)
@@ -2,5 +2,5 @@
   xmlns:xacro="http://www.ros.org/wiki/xacro">
   <!-- Includea all the WAM stuff -->
-  <include filename="$(find bard_urdf)/models/wam_top.urdf.xacro"/>
+  <include filename="$(find barrett_model)/models/wam_top.urdf.xacro"/>
   <!-- Root link is in the world frame-->
   <link name = "baseLink"/>

File: robots/wam_7dof_2x.urdf.xacro (robot description, xacro)
@@ -2,5 +2,5 @@
   xmlns:xacro="http://www.ros.org/wiki/xacro">
   <!-- Includea all the WAM stuff -->
-  <include filename="$(find bard_urdf)/models/wam_top.urdf.xacro"/>
+  <include filename="$(find barrett_model)/models/wam_top.urdf.xacro"/>
   <!-- Root link is in the world frame-->
   <link name="world"/>
@@ -23,5 +23,5 @@
       <origin rpy="0 0 0 " xyz="0 0 0"/>
       <geometry>
-        <mesh filename="${homeDirectory}/models/componentSTL/bench_lattice.dae"/>
+        <mesh filename="${models_path}/meshes/bench_lattice.dae"/>
       </geometry>
     </visual>
@@ -29,12 +29,12 @@
       <origin rpy="0 0 0 " xyz="0 0 0"/>
       <geometry>
-        <mesh filename="${homeDirectory}/models/componentSTL/bench_lattice.stl"/>
+        <mesh filename="${models_path}/meshes/bench_lattice.stl"/>
       </geometry>
     </collision>
   </link>
-  <!--<gazebo reference="baseLink">
+  <gazebo reference="baseLink">
     <static>true</static>
-     <turnGravityOff>true</turnGravityOff>
-   </gazebo>-->
+    <turnGravityOff>true</turnGravityOff>
+  </gazebo>
   <xacro:wam_root prefix="wam_left" parentLink="baseLink" xyz="0.356 0.46 1" rpy="0 ${-0.5*PI} ${0.5*PI}"/>
   <xacro:wam_7dof prefix="wam_left" parentLink="wam_left/FixedLink" xyz="0 0 0" rpy="0 0 0" />

File: robots/wam_7dof_wam.urdf.xacro (robot description, xacro)
@@ -2,5 +2,5 @@
   xmlns:xacro="http://www.ros.org/wiki/xacro">
   <!-- Includea all the WAM stuff -->
-  <include filename="$(find bard_urdf)/models/wam_top.urdf.xacro"/>
+  <include filename="$(find barrett_model)/models/wam_top.urdf.xacro"/>
   <!-- Root link is in the world frame-->
   <link name = "baseLink"/>
