Commit message: cleaning up...

File: models/arm.urdf.xacro (robot description, xacro)
@@ -24,45 +24,23 @@
 -->
 <robot xmlns:xacro="http://www.ros.org/wiki/xacro">
-  <include filename="$(find barrett_model)/models/hand.urdf.xacro"/>
   <include filename="$(find barrett_model)/models/common.urdf.xacro"/>
   <include filename="$(find barrett_model)/models/components.urdf.xacro"/>
-  <!-- different types of arms -->
-  <xacro:macro name="wam_4dof" params="prefix parentLink xyz rpy">
-    <xacro:wam_upper_arm prefix="${prefix}" parentLink="${parentLink}" xyz="${xyz}" rpy="${rpy}"/>
-    <xacro:hollow_forearm prefix="${prefix}"/>
-  </xacro:macro>
-  <xacro:macro name="wam_7dof" params="prefix parentLink xyz rpy">
-    <xacro:wam_upper_arm prefix="${prefix}" parentLink="${parentLink}" xyz="${xyz}" rpy="${rpy}"/>
-    <xacro:actuated_forearm prefix="${prefix}"/>
-  </xacro:macro>
-  <xacro:macro name="wam_7dof_ft" params="prefix parentLink xyz rpy">
-    <xacro:wam_upper_arm prefix="${prefix}" parentLink="${parentLink}" xyz="${xyz}" rpy="${rpy}"/>
-    <xacro:actuated_forearm_ft prefix="${prefix}"/>
+  <xacro:macro name="wam_7dof" params="prefix parent_link xyz rpy">
+    <xacro:wam prefix="${prefix}" parent_link="${parent_link}" xyz="${xyz}" rpy="${rpy}"/>
+    <xacro:wam_wrist prefix="${prefix}"/>
   </xacro:macro>
   <!-- upper arm only -->
-  <xacro:macro name="wam_upper_arm" params="prefix parentLink xyz rpy">
-    <xacro:Base prefix="${prefix}" parentLink="${parentLink}" xyz="${xyz}" rpy="${rpy}"/>
-    <xacro:Shoulder prefix="${prefix}"/>
-    <xacro:UpperArmInShoulder prefix="${prefix}"/>
-    <xacro:UpperArm prefix="${prefix}"/>
-  </xacro:macro>
-  <!-- forearm with no actuation "wrist" -->
-  <xacro:macro name="hollow_forearm" params="prefix">
-    <xacro:HollowForeArm prefix="${prefix}"/>
-    <xacro:HollowWrist prefix="${prefix}"/>
+  <xacro:macro name="wam" params="prefix parent_link xyz rpy">
+    <xacro:wam_base prefix="${prefix}" parent_link="${parent_link}" xyz="${xyz}" rpy="${rpy}"/>
+    <xacro:wam_shoulder_yaw prefix="${prefix}"/>
+    <xacro:wam_shoulder_pitch prefix="${prefix}"/>
+    <xacro:wam_upper_arm prefix="${prefix}"/>
   </xacro:macro>
   <!-- forearm with actuation "wrist" -->
-  <xacro:macro name="actuated_forearm" params="prefix">
-    <xacro:ForeArm prefix="${prefix}"/>
-    <xacro:UpperWristYaw prefix="${prefix}"/>
-    <xacro:UpperWristPitch prefix="${prefix}"/>
-    <xacro:LowerWrist prefix="${prefix}"/>
-  </xacro:macro>
-  <!-- Define a macro to construct the arm with a Barrett BHand on the end of it -->
-  <xacro:macro name="actuated_forearm_ft" params="prefix">
-    <xacro:ForeArm prefix="${prefix}"/>
-    <xacro:UpperWristYaw prefix="${prefix}"/>
-    <xacro:UpperWristPitch prefix="${prefix}"/>
-    <xacro:LowerWristFT prefix="${prefix}"/>
+  <xacro:macro name="wam_wrist" params="prefix">
+    <xacro:wam_forearm prefix="${prefix}"/>
+    <xacro:wam_wrist_yaw prefix="${prefix}"/>
+    <xacro:wam_wrist_pitch prefix="${prefix}"/>
+    <xacro:wam_palm prefix="${prefix}"/>
   </xacro:macro>
 </robot>

File: models/common.urdf.xacro (robot description, xacro)
@@ -23,11 +23,5 @@
  * of or in connection with the use or performance of this software.
 -->
-<robot xmlns:sensor="http://playerstage.sourceforge.net/gazebo/xmlschema/#sensor"
-  xmlns:controller="http://playerstage.sourceforge.net/gazebo/xmlschema/#controller"
-  xmlns:joint="http://playerstage.sourceforge.net/gazebo/xmlschema/#slider"
-  xmlns:interface="http://playerstage.sourceforge.net/gazebo/xmlschema/#interface"
-  xmlns:body="http://playerstage.sourceforge.net/gazebo/xmlschema/#body"
-  xmlns:geom="http://playerstage.sourceforge.net/gazebo/xmlschema/#geom"
-  xmlns:xacro="http://ros.org/wiki/xacro">
+<robot xmlns:xacro="http://ros.org/wiki/xacro">
   <!-- Directories -->
   <xacro:property name="models_path" value="package://barrett_model/models" />
@@ -36,18 +30,5 @@
   <xacro:property name="PI" value="3.1415926535897931" />
   <!-- Gazebo macros -->
-  <xacro:macro name="gazeboReference" params="name material">
-    <gazebo reference="${name}">
-      <material>
-        ${material}
-      </material>
-      <turnGravityOff>
-        false
-      </turnGravityOff>
-      <selfCollide>
-        true
-      </selfCollide>
-    </gazebo>
-  </xacro:macro>
-  <xacro:macro name="gazeboReferenceDAE" params="name">
+  <xacro:macro name="gazebo_reference" params="name">
     <gazebo reference="${name}">
       <turnGravityOff>
@@ -59,15 +40,3 @@
     </gazebo>
   </xacro:macro>
-  <!-- Controller macros -->
-  <xacro:macro name="control" params="name topicName linkName jointName">
-    <!--
-    <transmission type="pr2_mechanism_model/SimpleTransmission" name="${name}_trans">
-      <actuator name="${name}_motor" />
-      <joint name="${jointName}" />
-      <mechanicalReduction>1</mechanicalReduction>
-      <motorTorqueConstant>1</motorTorqueConstant>
-      <pulsesPerRevolution>90000</pulsesPerRevolution>
-    </transmission>
-    -->
-  </xacro:macro>
 </robot>

File: models/components.urdf.xacro (robot description, xacro)
@@ -23,22 +23,15 @@
  * of or in connection with the use or performance of this software.
 -->
-<robot xmlns:sensor="http://playerstage.sourceforge.net/gazebo/xmlschema/#sensor"
-  xmlns:controller="http://playerstage.sourceforge.net/gazebo/xmlschema/#controller"
-  xmlns:joint="http://playerstage.sourceforge.net/gazebo/xmlschema/#slider"
-  xmlns:interface="http://playerstage.sourceforge.net/gazebo/xmlschema/#interface"
-  xmlns:body="http://playerstage.sourceforge.net/gazebo/xmlschema/#body"
-  xmlns:geom="http://playerstage.sourceforge.net/gazebo/xmlschema/#geom"
-  xmlns:xacro="http://ros.org/wiki/xacro">
+<robot xmlns:xacro="http://ros.org/wiki/xacro">
   <include filename="$(find barrett_model)/models/hand.urdf.xacro"/>
   <include filename="$(find barrett_model)/models/common.urdf.xacro"/>
   <!-- Upper arm macros -->
-  <xacro:macro name="Base" params="prefix parentLink xyz rpy">
-    <joint name="${prefix}/FixedJoint" type="fixed">
-      <parent link="${parentLink}"/>
-      <child link="${prefix}/BaseLink"/>
+  <xacro:macro name="wam_base" params="prefix parent_link xyz rpy">
+    <joint name="${prefix}/wam_fixed_joint" type="fixed">
+      <parent link="${parent_link}"/>
+      <child link="${prefix}/base_link"/>
       <origin xyz="${xyz}" rpy="${rpy}"/>
     </joint>
-    <!-- Create the $(arg robot_name) WAM -->
-    <link name = "${prefix}/BaseLink">
+    <link name = "${prefix}/base_link">
       <inertial>
         <origin xyz="0 0 0" />
@@ -56,37 +49,30 @@
         <origin xyz="0 0.0 0" rpy="0 0 0"/>
         <geometry>
+          <mesh filename="${models_path}/sw_meshes/base_link_fine.STL"/>
+        </geometry>
+      </visual>
+      <collision>
+        <origin xyz="0 0.0 0" rpy="0 0 0" />
+        <geometry>
           <mesh filename="${models_path}/sw_meshes/base_link.STL"/>
         </geometry>
-      </visual>
-      <collision>
-        <origin xyz="0 0.0 0" rpy="0 0 0" />
-        <geometry>
-          <mesh filename="${models_path}/sw_meshes/base_link.STL"/>
-        </geometry>
-      </collision>
-    </link>
-    <!-- Simulation stuff -->
-    <!--gazebo>
-      <controller:gazebo_ros_controller_manager name="gazebo_ros_controller_manager" plugin="libgazebo_ros_controller_manager.so">
-        <alwaysOn>true</alwaysOn>
-        <updateRate>1000.0</updateRate>
-      </controller:gazebo_ros_controller_manager>
-    </gazebo-->
-  </xacro:macro>
-  <xacro:macro name="Shoulder" params="prefix">
-    <joint name="${prefix}/YawJoint" type="revolute">
-      <parent link="${prefix}/BaseLink"/>
-      <child link="${prefix}/ShoulderLink"/>
-      <origin xyz="0 0 0.346" rpy="0 0 0"/>
-      <axis xyz="0 -1 0"/>
+      </collision>
+    </link>
+  </xacro:macro>
+  <xacro:macro name="wam_shoulder_yaw" params="prefix">
+    <joint name="${prefix}/base_yaw_joint" type="revolute">
+      <parent link="${prefix}/base_link"/>
+      <child link="${prefix}/shoulder_yaw_link"/>
+      <origin xyz="0 0 0.160" rpy="0 0 0"/>
+      <axis xyz="0 0 1"/>
       <limit effort="30" lower="-2.6" upper="2.6" velocity="0.50"/>
-      <!-- <safety_controller k_position="10000000" k_velocity="10000000" soft_lower_limit="-100.0" soft_upper_limit="100.0" /> -->
-      <dynamics damping="1.0" friction="100.0"/>
-    </joint>
-    <link name="${prefix}/ShoulderLink" >
+      <dynamics damping="1.0" friction="100.0"/>
+    </joint>
+    <link name="${prefix}/shoulder_yaw_link" >
       <inertial>
         <origin xyz="-.00443422 0.1289039 -.00066489" />
         <mass value="10.7677" />
-        <inertia  ixx=".13488033" ixy="-.00213041"   ixz="-.00012485"
+        <inertia
+          ixx=".13488033"  ixy="-.00213041"   ixz="-.00012485"
           iyy=".11328369"  iyz=".00068555"
           izz=".09046330" />
@@ -96,38 +82,31 @@
           <color rgba="0.9 0.9 0.9 1.0"/>
         </material>
-        <!--  this orgin is not centered because the origin in our model is not at the same spot as the origin barret uses for inertia-->
-        <origin xyz="0 .189 0" rpy="${PI} 0 0" />
-        <geometry>
-          <mesh filename="${models_path}/meshes/wamShoulderLink1.DAE"/>
-        </geometry>
-      </visual>
-      <collision>
-        <origin xyz="0 .189 0" rpy="${PI} 0 0" />
-        <geometry>
-          <mesh filename="${models_path}/meshes/wamShoulderLink1.stl"/>
-        </geometry>
-      </collision>
-    </link>
-    <xacro:gazeboReferenceDAE name="${prefix}/ShoulderLink"/>
-    <xacro:control topicName="${prefix}/ShoulderYaw" name="DarmSim_${prefix}Arm_WAM_ShoulderYaw" linkName="${prefix}/ShoulderLink" jointName="${prefix}/YawJoint" />
-  </xacro:macro>
-  <xacro:macro name="UpperArmInShoulder" params="prefix">
-    <joint name="${prefix}/ShoulderPitchJoint" type="revolute">
-      <parent link="${prefix}/ShoulderLink"/>
-      <child link="${prefix}/UpperArmInShoulderLink"/>
-      <origin xyz="0 0 0" rpy="${0.5 * PI} 0 0"/>
-      <axis xyz="0 1 0"/>
+        <geometry>
+          <mesh filename="${models_path}/sw_meshes/shoulder_link_fine.STL"/>
+        </geometry>
+      </visual>
+      <collision>
+        <geometry>
+          <mesh filename="${models_path}/sw_meshes/shoulder_link.STL"/>
+        </geometry>
+      </collision>
+    </link>
+  </xacro:macro>
+  <xacro:macro name="wam_shoulder_pitch" params="prefix">
+    <joint name="${prefix}/shoulder_pitch_joint" type="revolute">
+      <parent link="${prefix}/shoulder_yaw_link"/>
+      <child link="${prefix}/shoulder_pitch_link"/>
+      <origin xyz="0 0 0.186" rpy="${-PI/2} 0 0"/>
+      <axis xyz="0 0 1"/>
       <limit effort="30" lower="-1.985" upper="1.985" velocity="0.5"/>
-      <!-- <safety_controller k_position="100" k_velocity="3" soft_lower_limit="-100.0" soft_upper_limit="100.0" /> -->
-      <dynamics damping="1.0" friction="100.0"/>
-    </joint>
-    <link name="${prefix}/UpperArmInShoulderLink" >
-      <visual>
-        <material name="WAMGrey">
-          <color rgba="0.9 0.9 0.9 1.0"/>
-        </material>
-        <origin xyz="0 0 0" rpy="${PI} 0 0" />
-        <geometry>
-          <mesh filename="${models_path}/meshes/wamUpperArmInShoulderLink.dae"/>
+      <dynamics damping="1.0" friction="100.0"/>
+    </joint>
+    <link name="${prefix}/shoulder_pitch_link" >
+      <visual>
+        <material name="WAMGrey">
+          <color rgba="0.9 0.9 0.9 1.0"/>
+        </material>
+        <geometry>
+          <mesh filename="${models_path}/sw_meshes/shoulder_pitch_link_fine.STL"/>
         </geometry>
       </visual>
@@ -135,34 +114,32 @@
         <origin xyz="-.00236981 .03105614 .01542114" />
         <mass value="3.87493756" />
-        <inertia  ixx=".02140958" ixy=".00027172"  ixz=".00002461"
+        <inertia
+          ixx=".02140958"  ixy=".00027172"  ixz=".00002461"
           iyy=".01377875"  iyz="-.00181920"
           izz=".01558906" />
       </inertial>
       <collision>
-        <origin xyz="0 0 0" rpy="${PI} 0 0" />
-        <geometry>
-          <mesh filename="${models_path}/meshes/wamUpperArmInShoulderLink2.stl"/>
-        </geometry>
-      </collision>
-    </link>
-    <xacro:gazeboReferenceDAE name="${prefix}/UpperArmInShoulderLink"/>
-    <xacro:control topicName="${prefix}/ShoulderPitch" name="DarmSim_${prefix}Arm_WAM_ShoulderPitch" linkName="${prefix}/UpperArmInShoulderLink" jointName="${prefix}/ShoulderPitchJoint" />
-  </xacro:macro>
-  <xacro:macro name="UpperArm" params="prefix">
-    <joint name="${prefix}/ShoulderYawJoint" type="revolute">
-      <parent link="${prefix}/UpperArmInShoulderLink"/>
-      <child link="${prefix}/UpperArmLink"/>
-      <origin xyz="0 0 0" rpy="-${0.5 * PI} 0 0"/>
-      <axis xyz="0 -1 0"/>
+        <geometry>
+          <mesh filename="${models_path}/sw_meshes/shoulder_pitch_link.STL"/>
+        </geometry>
+      </collision>
+    </link>
+  </xacro:macro>
+  <xacro:macro name="wam_upper_arm" params="prefix">
+    <joint name="${prefix}/shoulder_yaw_joint" type="revolute">
+      <parent link="${prefix}/shoulder_pitch_link"/>
+      <child link="${prefix}/upper_arm_link"/>
+      <origin xyz="0 0 0" rpy="${PI/2} 0 0"/>
+      <axis xyz="0 0 1"/>
       <limit effort="25" lower="-2.8" upper="2.8" velocity="0.5"/>
-      <!-- <safety_controller k_position="100" k_velocity="3" soft_lower_limit="-100.0" soft_upper_limit="100.0" /> -->
-      <dynamics damping="1.0" friction="100.0"/>
-    </joint>
-    <link name="${prefix}/UpperArmLink" >
+      <dynamics damping="1.0" friction="100.0"/>
+    </joint>
+    <link name="${prefix}/upper_arm_link" >
       <inertial>
         <origin xyz="-.03826 .20751 .00003" />
         <mass value="1.80228141" />
-        <inertia  ixx=".05911077" ixy="-.00249612"  ixz=".00000738"
-          iyy=".00324550"   iyz="-.00001767"
+        <inertia
+          ixx=".05911077"  ixy="-.00249612"  ixz=".00000738"
+          iyy=".00324550"  iyz="-.00001767"
           izz=".05927043" />
       </inertial>
@@ -173,35 +150,34 @@
         <origin xyz="0 0 0" rpy="0 0 0" />
         <geometry>
-          <mesh filename="${models_path}/meshes/wamUpperArmLink3.dae"/>
-        </geometry>
-      </visual>
-      <collision>
-        <origin xyz="0 0 0" rpy="0 0 0" />
-        <geometry>
-          <mesh filename="${models_path}/meshes/wamUpperArmLink3.stl"/>
-        </geometry>
-      </collision>
-    </link>
-    <xacro:gazeboReferenceDAE name="${prefix}/UpperArmLink" />
-    <xacro:control topicName="${prefix}/UpperArmYaw" name="DarmSim_${prefix}Arm_WAM_UpperArmYaw" linkName="${prefix}/UpperArmLink" jointName="${prefix}/ShoulderYawJoint" />
-  </xacro:macro>
-  <!-- Hollow forearm macros -->
-  <xacro:macro name="HollowForeArm" params="prefix">
-    <joint name="${prefix}/ElbowJoint" type="revolute">
-      <parent link="${prefix}/UpperArmLink"/>
-      <child link="${prefix}/ForeArmLink"/>
-      <origin xyz="0.045 -0.55 0" rpy="${0.5 * PI} 0 0"/>
-      <axis xyz="0 1 0"/>
-      <limit effort="15" lower="-0.9" upper="${PI}" velocity="0.50"/>
+          <mesh filename="${models_path}/sw_meshes/upper_arm_link_fine.STL"/>
+        </geometry>
+      </visual>
+      <collision>
+        <origin xyz="0 0 0" rpy="0 0 0" />
+        <geometry>
+          <mesh filename="${models_path}/sw_meshes/upper_arm_link.STL"/>
+        </geometry>
+      </collision>
+    </link>
+  </xacro:macro>
+  <!-- Forearm macros -->
+  <xacro:macro name="wam_forearm" params="prefix">
+    <joint name="${prefix}/elbow_pitch_joint" type="revolute">
+      <parent link="${prefix}/upper_arm_link"/>
+      <child link="${prefix}/forearm_link"/>
+      <origin xyz="0.045 0 0.55" rpy="${-PI/2} 0 0"/>
+      <axis xyz="0 0 1"/>
+      <limit effort="15" lower="-0.9" upper="${PI}" velocity="0.20"/>
       <!-- <safety_controller k_position="100" k_velocity="3" soft_lower_limit="-100.0" soft_upper_limit="100.0" /> -->
       <dynamics damping="1.0" friction="100.0"/>
     </joint>
-    <link name="${prefix}/ForeArmLink" >
+    <link name="${prefix}/forearm_link" >
       <inertial>
         <origin xyz="0 0 0" />
         <mass value="3.20016804" />
         <origin xyz="-0.04001488 -.00022942 .13271662" rpy="0 0 0" />
-        <inertia  ixx="0.01491672" ixy="0.00001741"   ixz="-0.00150604"
-          iyy="0.01482988"   iyz="-0.00002109"
+        <inertia
+          ixx="0.01491672"  ixy="0.00001741"   ixz="-0.00150604"
+          iyy="0.01482988"  iyz="-0.00002109"
           izz="0.00294463" />
       </inertial>
@@ -210,30 +186,41 @@
           <color rgba="0.9 0.9 0.9 1.0"/>
         </material>
-        <origin xyz="0 0 0" rpy="-${PI} 0 0" />
-        <geometry>
-          <mesh filename="${models_path}/meshes/wamForeArmLink4.DAE"/>
-        </geometry>
-      </visual>
-      <collision>
-        <origin xyz="0 0 0" rpy="-${PI} 0 0" />
-        <geometry>
-          <mesh filename="${models_path}/meshes/wamForeArmLink4.stl"/>
-        </geometry>
-      </collision>
-    </link>
-    <xacro:gazeboReferenceDAE name="${prefix}/ForeArmLink" />
-    <xacro:control topicName="${prefix}/ElbowPitch" name="DarmSim_${prefix}Arm_WAM_ElbowPitch" linkName="${prefix}/ForeArmLink" jointName="${prefix}/ElbowJoint" />
-  </xacro:macro>
-  <xacro:macro name="HollowWrist" params="prefix">
-    <joint name="${prefix}/UpperWristJoint" type="fixed">
-      <parent link="${prefix}/ForeArmLink"/>
-      <child link="${prefix}/LowerWristPalmLink"/>
-      <origin xyz="-0.045 0 .35" rpy="-${0.5 * PI} 0 ${0.5 * PI}"/>
-      <axis xyz="0 -1 0"/>
+        <geometry>
+          <mesh filename="${models_path}/sw_meshes/elbow_link_fine.STL"/>
+        </geometry>
+      </visual>
+      <collision>
+        <geometry>
+          <mesh filename="${models_path}/sw_meshes/elbow_link.STL"/>
+        </geometry>
+      </collision>
+      <visual>
+        <material name="WAMGrey">
+          <color rgba="0.9 0.9 0.9 1.0"/>
+        </material>
+        <origin xyz="-0.045 -0.0730 0" rpy="${PI/2} 0 0" />
+        <geometry>
+          <mesh filename="${models_path}/sw_meshes/forearm_link_fine.STL"/>
+        </geometry>
+      </visual>
+      <collision>
+        <origin xyz="-0.045 -0.0730 0" rpy="${PI/2} 0 0" />
+        <geometry>
+          <mesh filename="${models_path}/sw_meshes/forearm_link.STL"/>
+        </geometry>
+      </collision>
+    </link>
+  </xacro:macro>
+  <xacro:macro name="wam_wrist_yaw" params="prefix">
+    <joint name="${prefix}/wrist_yaw_joint" type="revolute">
+      <parent link="${prefix}/forearm_link"/>
+      <child link="${prefix}/wrist_yaw_link"/>
+      <origin xyz="-0.045 -0.3 0" rpy="${PI/2} 0 0"/>
+      <axis xyz="0 0 1"/>
       <limit effort="5" lower="-4.8" upper="1.3" velocity="0.20"/>
       <!-- <safety_controller k_position="100" k_velocity="3" soft_lower_limit="-100.0" soft_upper_limit="100.0" /> -->
       <dynamics damping="1.0" friction="100.0"/>
     </joint>
-    <link name="${prefix}/LowerWristPalmLink" >
+    <link name="${prefix}/wrist_yaw_link" >
       <inertial>
         <origin xyz="0.00008921 0.00511217 0.00435824" />
@@ -247,110 +234,33 @@
           <color rgba="0.9 0.9 0.9 1.0"/>
         </material>
-        <origin xyz="0 0.02711 0" rpy="${PI} 0 0" />
-        <geometry>
-          <mesh filename="${models_path}/meshes/wamUpperWristYawLink.DAE"/>
-        </geometry>
-      </visual>
-      <collision>
-        <origin xyz="0 0.02711 0" rpy="${PI} 0 0" />
-        <geometry>
-          <mesh filename="${models_path}/meshes/wamUpperWristYawLink5.stl"/>
-        </geometry>
-      </collision>
-    </link>
-    <xacro:gazeboReferenceDAE name="${prefix}/UpperWristYawLink" />
-    <xacro:control topicName="${prefix}/UpperWristYaw" name="DarmSim_${prefix}Arm_WAM_UpperWristYaw" linkName="${prefix}/UpperWristYawLink" jointName="${prefix}/UpperWristYawJoint" />
-  </xacro:macro>
-  <!-- Forearm macros -->
-  <xacro:macro name="ForeArm" params="prefix">
-    <joint name="${prefix}/ElbowJoint" type="revolute">
-      <parent link="${prefix}/UpperArmLink"/>
-      <child link="${prefix}/ForeArmLink"/>
-      <origin xyz="0.045 -0.55 0" rpy="${0.5 * PI} 0 0"/>
-      <axis xyz="0 1 0"/>
-      <limit effort="15" lower="-0.9" upper="${PI}" velocity="0.20"/>
-      <!-- <safety_controller k_position="100" k_velocity="3" soft_lower_limit="-100.0" soft_upper_limit="100.0" /> -->
-      <dynamics damping="1.0" friction="100.0"/>
-    </joint>
-    <link name="${prefix}/ForeArmLink" >
-      <inertial>
-        <origin xyz="0 0 0" />
-        <mass value="3.20016804" />
-        <origin xyz="-0.04001488 -.00022942 .13271662" rpy="0 0 0" />
-        <inertia  ixx="0.01491672" ixy="0.00001741"   ixz="-0.00150604"
-          iyy="0.01482988"   iyz="-0.00002109"
-          izz="0.00294463" />
-      </inertial>
-      <visual>
-        <material name="WAMGrey">
-          <color rgba="0.9 0.9 0.9 1.0"/>
-        </material>
-        <origin xyz="0 0 0" rpy="-${PI} 0 0" />
-        <geometry>
-          <mesh filename="${models_path}/meshes/wamForeArmLink4.DAE"/>
-        </geometry>
-      </visual>
-      <collision>
-        <origin xyz="0 0 0" rpy="-${PI} 0 0" />
-        <geometry>
-          <mesh filename="${models_path}/meshes/wamForeArmLink4.stl"/>
-        </geometry>
-      </collision>
-    </link>
-    <xacro:gazeboReferenceDAE name="${prefix}/ForeArmLink" />
-    <xacro:control topicName="${prefix}/ElbowPitch" name="DarmSim_${prefix}Arm_WAM_ElbowPitch" linkName="${prefix}/ForeArmLink" jointName="${prefix}/ElbowJoint" />
-  </xacro:macro>
-  <xacro:macro name="UpperWristYaw" params="prefix">
-    <joint name="${prefix}/UpperWristYawJoint" type="revolute">
-      <parent link="${prefix}/ForeArmLink"/>
-      <child link="${prefix}/UpperWristYawLink"/>
-      <origin xyz="-0.045 0 .3" rpy="-${0.5 * PI} 0 ${0.5 * PI}"/>
-      <axis xyz="0 -1 0"/>
-      <limit effort="5" lower="-4.8" upper="1.3" velocity="0.20"/>
-      <!-- <safety_controller k_position="100" k_velocity="3" soft_lower_limit="-100.0" soft_upper_limit="100.0" /> -->
-      <dynamics damping="1.0" friction="100.0"/>
-    </joint>
-    <link name="${prefix}/UpperWristYawLink" >
-      <inertial>
-        <origin xyz="0.00008921 0.00511217 0.00435824" />
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