Commit message: cleaning up...

File: models/hand.urdf.xacro (robot description, xacro)
@@ -1,187 +1,152 @@
-<!--
- * COPYRIGHT (C) 2010
- * RE2, INC.
- *
- * Author: RE2
- *
- * This file is a part of RobotModel, which was developed for the
- * DARPA ARM ROBOT Track C project.
- *
- * RobotModel is free software:
- * you can redistribute it and/or modify it under the terms of the GNU General
- * Public License as published by the Free Software Foundation, either version
- * 3 of the License, or (at your option) any later version.
- *
- * You should have received a copy of the GNU General Public License along
- * with this package.  If not, see <http://www.gnu.org/licenses/>.
- *
- * RE2, INC. disclaims all warranties with regard to this software, including
- * all implied warranties of merchantability and fitness, in no event shall
- * RE2, INC. be liable for any special, indirect or consequential damages or
- * any damages whatsoever resulting from loss of use, data or profits, whether
- * in an action of contract, negligence or other tortious action, arising out
- * of or in connection with the use or performance of this software.
--->
-<robot xmlns:sensor="http://playerstage.sourceforge.net/gazebo/xmlschema/#sensor"
-  xmlns:controller="http://playerstage.sourceforge.net/gazebo/xmlschema/#controller"
-  xmlns:geom="http://playerstage.sourceforge.net/gazebo/xmlschema/#geom"
-  xmlns:interface="http://playerstage.sourceforge.net/gazebo/xmlschema/#interface"
-  xmlns:xacro="http://www.ros.org/wiki/xacro">
+<robot xmlns:xacro="http://www.ros.org/wiki/xacro">
   <include filename="$(find barrett_model)/models/common.urdf.xacro"/>
-  <!-- Palm -->
-  <xacro:macro name="Palm" params="prefix">
-    <link name="${prefix}/PalmLink" />
-    <joint name="${prefix}/PalmJoint" type="fixed">
-      <parent link="${prefix}/LowerWristPalmLink"/>
-      <child link="${prefix}/PalmLink"/>
-      <!--             <origin xyz="0 0 0.1293166" rpy="0 0 0"/> -->
-      <origin xyz="0 0 0.0793166" rpy="0 0 ${PI/2}"/>
+  <!-- High-leveel hand macro -->
+  <xacro:macro name="bhand" params="parent_link prefix xyz rpy">
+    <xacro:bhand_palm parent_link="${parent_link}" prefix="${prefix}" xyz="${xyz}" rpy="${rpy}"/>
+    <xacro:bhand_finger_1 prefix="${prefix}"/>
+    <xacro:bhand_finger_2 prefix="${prefix}"/>
+    <xacro:bhand_finger_3 prefix="${prefix}"/>
+  </xacro:macro>
+  <!-- Fingers -->
+  <xacro:macro name="bhand_finger_1" params="prefix">
+    <xacro:bhand_finger_prox prefix="${prefix}/finger_1" parent_link="${prefix}/bhand_palm_link" xyz="0.025 0.0 0.0415" rpy="0 0 -${PI/2}" axis="0 0 1"/>
+    <xacro:bhand_finger_med prefix="${prefix}/finger_1" parent_link="${prefix}/finger_1/bhand_finger_prox_link" xyz="0.05 0.0 0.03390" rpy="${PI/2} 0 0"/>
+    <xacro:bhand_finger_dist prefix="${prefix}/finger_1"/>
+  </xacro:macro>
+  <xacro:macro name="bhand_finger_2" params="prefix">
+    <xacro:bhand_finger_prox prefix="${prefix}/finger_2" parent_link="${prefix}/bhand_palm_link" xyz="-0.025 0.0 0.0415" rpy="0 0 -${PI/2}" axis="0 0 -1"/>
+    <xacro:bhand_finger_med prefix="${prefix}/finger_2" parent_link="${prefix}/finger_2/bhand_finger_prox_link" xyz="0.05 0.0 0.03390" rpy="${PI/2} 0 0"/>
+    <xacro:bhand_finger_dist prefix="${prefix}/finger_2"/>
+  </xacro:macro>
+  <xacro:macro name="bhand_finger_3" params="prefix">
+    <xacro:bhand_finger_med prefix="${prefix}/finger_3" parent_link="${prefix}/bhand_palm_link" xyz="0 0.05 0.0754" rpy="${PI/2} 0 ${PI/2}"/>
+    <xacro:bhand_finger_dist prefix="${prefix}/finger_3"/>
+  </xacro:macro>
+  <!-- Components -->
+  <xacro:macro name="bhand_palm" params="prefix parent_link xyz rpy">
+    <joint name="${prefix}/bhand_base_joint" type="fixed">
+      <parent link="${parent_link}"/>
+      <child link="${prefix}/bhand_palm_link"/>
+      <origin xyz="${xyz}" rpy="${rpy}"/>
     </joint>
-  </xacro:macro>
-  <xacro:macro name="fingers" params="parent prefix number xyz rpy">
-    <xacro:KnuckleTwo parent="${parent}" prefix="${prefix}" number="${number}" xyz="${xyz}" rpy="${rpy}" />
-    <xacro:KnuckleThree prefix="${prefix}" number="${number}"/>
-    <gazebo reference="${prefix}/BHand/Finger${number}/KnuckleThreeLink">
-      <sensor:contact name="${prefix}Finger${number}_finger_contact_sensor">
-        <geom>${prefix}/BHand/Finger${number}/KnuckleThreeLink_geom</geom>
-        <updateRate>100.0</updateRate>
-        <controller:gazebo_ros_bumper name="${prefix}/BHand/Finger${number}/KnuckleThreeLink/bumperController" plugin="libgazebo_ros_bumper.so">
-          <alwaysOn>true</alwaysOn>
-          <updateRate>100.0</updateRate>
-          <frameName>${prefix}/BHand/Finger${number}/KnuckleThreeLink</frameName>
-          <bumperTopicName>${prefix}/BHand/Finger${number}/bumper</bumperTopicName>
-          <interface:bumper name="DarmSim${prefix}ArmBHandFinger${number}KnuckleThreeLink_bumper_iface" />
-        </controller:gazebo_ros_bumper>
-      </sensor:contact>
-    </gazebo>
-  </xacro:macro>
-  <xacro:macro name="LowerWristPalm" params="prefix">
-    <joint name="${prefix}/LowerWristPalmJoint" type="fixed">
-      <parent link="${prefix}/LowerWristYawLink"/>
-      <child link="${prefix}/LowerWristPalmLink"/>
-      <origin xyz="0 0 0" rpy="0 0 -${0.5 * PI}"/>
-      <provideFeedback value="true"/>
-    </joint>
-    <link name="${prefix}/LowerWristPalmLink" >
+    <link name="${prefix}/bhand_palm_link">
       <inertial>
-        <origin xyz="0.00035500 -0.00499005 0.04864979" />
-        <mass value="0.63352875" />
-        <inertia  ixx="0.00102103" ixy="0.00000775"  ixz="-0.00001230"
-          iyy="0.00080944"  iyz="-0.00014417"
-          izz="0.00068788" />
+        <origin xyz="5.1098e-005 -0.0050433 0.036671" />
+        <mass value="0.59573" />
+        <inertia
+          ixx="3.8374e-005" ixy="-5.604e-008"  ixz="-4.2034e-005"
+                           iyy="0.00022405"   iyz="1.3283e-007"
+                                              izz="0.00020045" />
       </inertial>
       <visual>
         <material name="WAMGrey">
-          <color rgba="0.9 0.9 0.9 1.0"/>
+          <color rgba="0.9 0.9 0.9 0.0"/>
         </material>
-        <origin xyz="0 0 0" rpy="0 0 0" />
         <geometry>
-          <mesh filename="${models_path}/meshes/palm.DAE"/>
+          <mesh filename="${models_path}/sw_meshes/bhand/bhand_palm_fine.STL"/>
         </geometry>
       </visual>
       <collision>
-        <origin xyz="0 0 0" rpy="0 0 0" />
         <geometry>
-          <mesh filename="${models_path}/meshes/palm.stl"/>
+          <mesh filename="${models_path}/sw_meshes/bhand/bhand_palm.STL"/>
         </geometry>
       </collision>
     </link>
-    <xacro:gazeboReferenceDAE name="${prefix}/LowerWristPalmLink"/>
-    <gazebo reference="${prefix}/LowerWristPalmJoint">
-      <provideFeedback value="true"/>
-    </gazebo>
-    <gazebo>
-      <controller:gazebo_ros_jointFeedback name="${prefix}_JointFTsensor" plugin="libgazebo_ros_jointFeedback.so">
-        <alwaysOn>true</alwaysOn>
-        <updateRate>100.0</updateRate>
-        <jointName>${prefix}/LowerWristPalmJoint</jointName>
-        <topicName>${prefix}/BHand/ForceTorqueSensor</topicName>
-        <bodyRelation>child</bodyRelation>
-        <frameName>${prefix}/LowerWristPalmLink</frameName>
-        <interface:position name="${prefix}_JointFTsensor_force_iface" />
-      </controller:gazebo_ros_jointFeedback>
-    </gazebo>
-    <gazebo reference="${prefix}/LowerWristPalmLink">
-      <sensor:contact name="${prefix}Palm_contact_sensor">
-        <geom>${prefix}/LowerWristPalmLink_geom</geom>
-        <updateRate>100.0</updateRate>
-        <controller:gazebo_ros_bumper name="${prefix}/LowerWristPalmLink/bumperController" plugin="libgazebo_ros_bumper.so">
-          <alwaysOn>true</alwaysOn>
-          <updateRate>100.0</updateRate>
-          <frameName>${prefix}/LowerWristPalmLink</frameName>
-          <bumperTopicName>${prefix}/BHand/Palm/bumper</bumperTopicName>
-          <interface:bumper name="DarmSim${prefix}ArmWAMLowerWristPalmLink_bumper_iface" />
-        </controller:gazebo_ros_bumper>
-      </sensor:contact>
-    </gazebo>
   </xacro:macro>
-  <xacro:macro name="LowerWristPalmFT" params="prefix">
-    <joint name="${prefix}/LowerWristPalmJoint" type="fixed">
-      <parent link="${prefix}/LowerWristYawLink"/>
-      <child link="${prefix}/LowerWristPalmLink"/>
-      <origin xyz="0 0 0.0048" rpy="0 0 -${0.5 * PI}"/>
-      <provideFeedback value="true"/>
+  <xacro:macro name="bhand_finger_prox" params="prefix parent_link xyz rpy axis">
+    <joint name="${prefix}/bhand_finger_prox_joint" type="revolute">
+      <parent link="${parent_link}"/>
+      <child link="${prefix}/bhand_finger_prox_link"/>
+      <origin xyz="${xyz}" rpy="${rpy}"/>
+      <axis xyz="${axis}"/>
+      <limit effort="5" lower="0" upper="${PI}" velocity="0.20"/>
     </joint>
-    <link name="${prefix}/LowerWristPalmLink" >
+    <link name="${prefix}/bhand_finger_prox_link">
       <inertial>
-        <origin xyz="0.00035500 -0.00499005 0.04864979" />
-        <mass value="0.63352875" />
-        <inertia  ixx="0.00102103" ixy="0.00000775"  ixz="-0.00001230"
-          iyy="0.00080944"  iyz="-0.00014417"
-          izz="0.00068788" />
+        <origin xyz="0.023133 0.00078642 0.00052792" />
+        <mass value="0.062139" />
+        <inertia
+          ixx="4.872e-006" ixy="1.7103e-006"  ixz="3.4041e-008"
+                           iyy="7.6588e-005"  iyz="2.3133e-008"
+                                              izz="7.7733e-005" />
       </inertial>
       <visual>
         <material name="WAMGrey">
-          <color rgba="0.9 0.9 0.9 1.0"/>
+          <color rgba="0.9 0.9 0.9 0.0"/>
         </material>
-        <origin xyz="0 0 0" rpy="0 0 0" />
         <geometry>
-          <mesh filename="${models_path}/meshes/palm.DAE"/>
+          <mesh filename="${models_path}/sw_meshes/bhand/bhand_finger_prox_link_fine.STL"/>
         </geometry>
       </visual>
       <collision>
-        <origin xyz="0 0 0" rpy="0 0 0" />
         <geometry>
-          <mesh filename="${models_path}/meshes/palm.stl"/>
+          <mesh filename="${models_path}/sw_meshes/bhand/bhand_finger_prox_link.STL"/>
         </geometry>
       </collision>
     </link>
-    <xacro:gazeboReferenceDAE name="${prefix}/LowerWristPalmLink"/>
-    <gazebo reference="${prefix}/LowerWristPalmJoint">
-      <provideFeedback value="true"/>
-    </gazebo>
-    <gazebo>
-      <controller:gazebo_ros_jointFeedback name="${prefix}_JointFTsensor" plugin="libgazebo_ros_jointFeedback.so">
-        <alwaysOn>true</alwaysOn>
-        <updateRate>100.0</updateRate>
-        <jointName>${prefix}/LowerWristPalmJoint</jointName>
-        <topicName>${prefix}/BHand/ForceTorqueSensor</topicName>
-        <bodyRelation>child</bodyRelation>
-        <frameName>${prefix}/LowerWristPalmLink</frameName>
-        <interface:position name="${prefix}_JointFTsensor_force_iface" />
-      </controller:gazebo_ros_jointFeedback>
-    </gazebo>
-    <gazebo reference="${prefix}/LowerWristPalmLink">
-      <sensor:contact name="${prefix}Palm_contact_sensor">
-        <geom>${prefix}/LowerWristPalmLink_geom</geom>
-        <updateRate>100.0</updateRate>
-        <controller:gazebo_ros_bumper name="${prefix}/LowerWristPalmLink/bumperController" plugin="libgazebo_ros_bumper.so">
-          <alwaysOn>true</alwaysOn>
-          <updateRate>100.0</updateRate>
-          <frameName>${prefix}/LowerWristPalmLink</frameName>
-          <bumperTopicName>${prefix}/BHand/Palm/bumper</bumperTopicName>
-          <interface:bumper name="DarmSim${prefix}ArmWAMLowerWristPalmLink_bumper_iface" />
-        </controller:gazebo_ros_bumper>
-      </sensor:contact>
-    </gazebo>
   </xacro:macro>
-  <xacro:macro name="barrett_hand" params="prefix">
-    <xacro:LowerWristPalm prefix="${prefix}"/>
-    <xacro:Palm prefix="${prefix}"/>
-    <xacro:fingers prefix="${prefix}" parent="${prefix}/LowerWristPalmLink" number="Three" xyz="0 -0.05 0.0801966" rpy="-${0.5 * PI} -0.0429350996 -${0.5 * PI}"/>
-    <xacro:KnuckleOne prefix="${prefix}" number="One" xyz=".02497 0 0.0587966" rpy="0 0 ${0.5 * PI}" axis="0 0 -1"/>
-    <xacro:fingers prefix="${prefix}" parent="${prefix}/BHand/FingerOne/KnuckleOneLink" number="One" xyz=".05 0 0.02140" rpy="-${0.5 * PI} -0.0429350996 0"/>
-    <xacro:KnuckleOne prefix="${prefix}" number="Two" xyz="-.02497 0 0.0587966" rpy="0 0 ${0.5 * PI}" axis ="0 0 1"/>
-    <xacro:fingers prefix="${prefix}" parent="${prefix}/BHand/FingerTwo/KnuckleOneLink" number="Two" xyz=".05 0 0.02140" rpy="-${0.5 * PI} -0.0429350996 0"/>
+  <xacro:macro name="bhand_finger_med" params="prefix parent_link xyz rpy">
+    <joint name="${prefix}/bhand_finger_med_joint" type="revolute">
+      <parent link="${parent_link}"/>
+      <child link="${prefix}/bhand_finger_med_link"/>
+      <origin xyz="${xyz}" rpy="${rpy}"/>
+      <axis xyz="0 0 1"/>
+      <limit effort="5" lower="0" upper="${140/180*PI}" velocity="0.20"/>
+    </joint>
+    <link name="${prefix}/bhand_finger_med_link">
+      <inertial>
+        <origin xyz="0.023133 0.00078642 0.00052792" />
+        <mass value="0.062139" />
+        <inertia
+          ixx="4.872e-006" ixy="1.7103e-006"  ixz="3.4041e-008"
+                           iyy="7.6588e-005"  iyz="2.3133e-008"
+                                              izz="7.7733e-005" />
+      </inertial>
+      <visual>
+        <material name="WAMGrey">
+          <color rgba="0.9 0.9 0.9 0.0"/>
+        </material>
+        <geometry>
+          <mesh filename="${models_path}/sw_meshes/bhand/bhand_finger_med_link_fine.STL"/>
+        </geometry>
+      </visual>
+      <collision>
+        <geometry>
+          <mesh filename="${models_path}/sw_meshes/bhand/bhand_finger_med_link.STL"/>
+        </geometry>
+      </collision>
+    </link>
+  </xacro:macro>
+  <xacro:macro name="bhand_finger_dist" params="prefix">
+    <joint name="${prefix}/bhand_finger_dist_joint" type="revolute">
+      <parent link="${prefix}/bhand_finger_med_link"/>
+      <child link="${prefix}/bhand_finger_dist_link"/>
+      <origin xyz="0.06994 0.003 0.0" rpy="0 0 0"/>
+      <axis xyz="0 0 1"/>
+      <limit effort="5" lower="0" upper="${48/180*PI}" velocity="0.20"/>
+    </joint>
+    <link name="${prefix}/bhand_finger_dist_link">
+      <inertial>
+        <origin xyz="0.022825 0.0010491 0.0004203" />
+        <mass value="0.041377" />
+        <inertia
+          ixx="3.1582e-006" ixy="1.4308e-006"  ixz="1.0106e-007"
+                           iyy="3.8376e-005"   iyz="0"
+                                              izz="3.7275e-005" />
+      </inertial>
+      <visual>
+        <material name="WAMGrey">
+          <color rgba="0.9 0.9 0.9 0.0"/>
+        </material>
+        <geometry>
+          <mesh filename="${models_path}/sw_meshes/bhand/bhand_finger_dist_link_fine.STL"/>
+        </geometry>
+      </visual>
+      <collision>
+        <geometry>
+          <mesh filename="${models_path}/sw_meshes/bhand/bhand_finger_dist_link.STL"/>
+        </geometry>
+      </collision>
+    </link>
   </xacro:macro>
 </robot>

File: models/wam_top.urdf.xacro (robot description, xacro)
@@ -8,4 +8,6 @@
   <!-- Definition of all the different parts of a WAM arm -->
   <include filename="$(find barrett_model)/models/components.urdf.xacro"/>
+  <!-- Definitions for the barrett hand -->
+  <include filename="$(find barrett_model)/models/hand.urdf.xacro"/>
   <!-- Materials -->
   <material name="WAMGrey">

Commit message: Updating inertial parameters from those observed in the lab. Adding stubby 4-dof WAM.

File: models/arm.urdf.xacro (robot description, xacro)
@@ -30,4 +30,8 @@
     <xacro:wam_wrist prefix="${prefix}"/>
   </xacro:macro>
+  <xacro:macro name="wam_4dof" params="prefix parent_link xyz rpy">
+    <xacro:wam prefix="${prefix}" parent_link="${parent_link}" xyz="${xyz}" rpy="${rpy}"/>
+    <xacro:wam_stump prefix="${prefix}"/>
+  </xacro:macro>
   <!-- upper arm only -->
   <xacro:macro name="wam" params="prefix parent_link xyz rpy">

File: models/components.urdf.xacro (robot description, xacro)
@@ -36,9 +36,9 @@
       <inertial>
         <origin xyz="0 0 0" />
-        <mass value="100" />
-        <inertia
-          ixx="1" ixy="0"   ixz="0"
-                  iyy="1"   iyz="0"
-                            izz="1" />
+        <mass value="1" />
+        <inertia
+          ixx="0.1" ixy="0"   ixz="0"
+                  iyy="0.1"   iyz="0"
+                            izz="0.1" />
       </inertial>
       <visual>
@@ -63,5 +63,5 @@
       <origin xyz="0 0 0.346" rpy="0 0 0"/>
       <axis xyz="0 0 1"/>
-      <limit effort="30" lower="-2.6" upper="2.6" velocity="0.50"/>
+      <limit effort="60" lower="-2.6" upper="2.6" velocity="0.50"/>
       <dynamics damping="1.0" friction="100.0"/>
     </joint>
@@ -69,5 +69,5 @@
       <inertial>
         <origin xyz="-.00443422 -.00066489 -0.1289039 " />
-        <mass value="10.7677" />
+        <mass value="0" />
         <inertia
           ixx=".13488033"  ixy="-0.00012485"   ixz="0.00213041"
@@ -96,5 +96,5 @@
       <origin xyz="0 0 0" rpy="${-PI/2} 0 0"/>
       <axis xyz="0 0 1"/>
-      <limit effort="30" lower="-1.985" upper="1.985" velocity="0.5"/>
+      <limit effort="60" lower="-1.985" upper="1.985" velocity="0.5"/>
       <dynamics damping="1.0" friction="100.0"/>
     </joint>
@@ -129,10 +129,10 @@
       <origin xyz="0 0 0" rpy="${PI/2} 0 0"/>
       <axis xyz="0 0 1"/>
-      <limit effort="25" lower="-2.8" upper="2.8" velocity="0.5"/>
+      <limit effort="45" lower="-2.8" upper="2.8" velocity="0.5"/>
       <dynamics damping="1.0" friction="100.0"/>
     </joint>
     <link name="${prefix}/upper_arm_link" >
       <inertial>
-        <origin xyz="-0.083258580000000 0.000033090000000 0.342492300000000" />
+        <origin xyz="0.00683258580000000 0.000033090000000 0.342492300000000" />
         <mass value="1.80228141" />
         <inertia
@@ -169,6 +169,6 @@
     <link name="${prefix}/forearm_link" >
       <inertial>
-        <mass value="2.40016804" />
-        <origin xyz="-0.04001488 -.13271662 -.00022942 " rpy="0 0 0" />
+        <mass value="1.50016804" />
+        <origin xyz="-0.04001488 -.08271662 -.00022942 " rpy="0 0 0" />
         <inertia
           ixx="0.01491672" ixy="0.001506040000000" ixz="0.000017410000000"
@@ -419,3 +419,37 @@
     <!--</link>-->
   <!--</xacro:macro>-->
+  <xacro:macro name="wam_stump" params="prefix">
+    <joint name="${prefix}/elbow_pitch_joint" type="revolute">
+      <parent link="${prefix}/upper_arm_link"/>
+      <child link="${prefix}/stump_link"/>
+      <origin xyz="0.045 0 0.55" rpy="${-PI/2} 0 0"/>
+      <axis xyz="0 0 1"/>
+      <limit effort="15" lower="-0.9" upper="${PI}" velocity="0.20"/>
+      <!-- <safety_controller k_position="100" k_velocity="3" soft_lower_limit="-100.0" soft_upper_limit="100.0" /> -->
+      <dynamics damping="1.0" friction="100.0"/>
+    </joint>
+    <link name="${prefix}/stump_link" >
+      <inertial>
+        <mass value="0.408" />
+        <origin xyz="-0.0195 -.02566 -.00022942 " rpy="0 0 0" />
+        <inertia
+          ixx="0.01491672" ixy="0.001506040000000" ixz="0.000017410000000"
+                           iyy="0.002944630000000" iyz="0.000021090000000"
+                                                   izz="0.014829880000000" />
+      </inertial>
+      <visual>
+        <material name="WAMGrey">
+          <color rgba="0.7 0.7 0.7 1.0"/>
+        </material>
+        <geometry>
+          <mesh filename="${models_path}/sw_meshes/elbow_link_fine.STL"/>
+        </geometry>
+      </visual>
+      <collision>
+        <geometry>
+          <mesh filename="${models_path}/sw_meshes/elbow_link.STL"/>
+        </geometry>
+      </collision>
+    </link>
+  </xacro:macro>
 </robot>

File: models/hand.urdf.xacro (robot description, xacro)
@@ -32,6 +32,6 @@
     <link name="${prefix}/bhand_palm_link">
       <inertial>
-        <origin xyz="5.1098e-005 -0.0050433 0.036671" />
-        <mass value="0.59573" />
+        <origin xyz="-5.1098e-005 0.0050433 0.036671"/>
+        <mass value="0.50573" />
         <inertia
           ixx="3.8374e-005" ixy="-5.604e-008"  ixz="-4.2034e-005"
@@ -65,5 +65,5 @@
       <inertial>
         <origin xyz="0.023133 0.00078642 0.00052792" />
-        <mass value="0.062139" />
+        <mass value="0.14109" />
         <inertia
           ixx="4.872e-006" ixy="1.7103e-006"  ixz="3.4041e-008"

File: robots/wam_4dof_wam.urdf.xacro (robot description, xacro)
@@ -4,7 +4,5 @@
   <include filename="$(find barrett_model)/models/wam_top.urdf.xacro"/>
   <!-- Root link is in the world frame-->
-  <link name = "baseLink"/>
-  <xacro:wam_root prefix="wam" parentLink="baseLink" xyz="0.0 0.5 1" rpy="0 ${-0.5*PI} ${0.5*PI}"/>
-  <xacro:wam_4dof prefix="wam" parentLink="wam/FixedLink" xyz="0 0 0" rpy="0 0 0" />
-  <!--xacro:barrett_hand prefix="wam_left" /-->
+  <link name = "world"/>
+  <xacro:wam_4dof prefix="wam" parent_link="world" xyz="0.02 0.46 1" rpy="0 0 0" />
 </robot>
