Commit message: adding additional frames for use as moveit end-effectors

File: models/arm.urdf.xacro (robot description, xacro)
@@ -29,4 +29,5 @@
     <xacro:wam prefix="${prefix}" parent_link="${parent_link}" xyz="${xyz}" rpy="${rpy}"/>
     <xacro:wam_wrist prefix="${prefix}"/>
+    <xacro:wam_wrist_palm_stump prefix="${prefix}"/>
   </xacro:macro>
   <xacro:macro name="wam_4dof" params="prefix parent_link xyz rpy">

File: models/components.urdf.xacro (robot description, xacro)
@@ -328,4 +328,20 @@
     </link>
   </xacro:macro>
+  <xacro:macro name="wam_wrist_palm_stump" params="prefix">
+    <joint name="${prefix}/wrist_palm_stump_joint" type="fixed">
+      <parent link="${prefix}/wrist_palm_link"/>
+      <child link="${prefix}/wrist_palm_stump_link"/>
+      <origin xyz="0 0 0.06" rpy="0 0 0"/>
+    </joint>
+    <link name="${prefix}/wrist_palm_stump_link" >
+      <inertial>
+        <mass value="0.000001" />
+        <inertia
+          ixx="0.0000001" ixy="0.0" ixz="0.0"
+          iyy="0.0000001" iyz="0.0"
+          izz="0.0000001" />
+      </inertial>
+    </link>
+  </xacro:macro>
   <!-- Hollow forearm macros -->
   <!--<xacro:macro name="wam_hollow_forearm" params="prefix">-->

File: models/hand.urdf.xacro (robot description, xacro)
@@ -61,4 +61,36 @@
       </collision>
     </link>
+    <joint name="${prefix}/bhand_palm_surface_joint" type="fixed">
+      <parent link="${prefix}/bhand_palm_link"/>
+      <child link="${prefix}/bhand_palm_surface_link"/>
+      <origin xyz="0 0 0.08" rpy="0 0 0"/>
+      <limit effort="5" lower="0" upper="${PI}" velocity="5.0"/>
+      <dynamics damping="1.5" friction="1"/>
+    </joint>
+    <link name="${prefix}/bhand_palm_surface_link">
+      <inertial>
+        <mass value="0.000001" />
+        <inertia
+          ixx="0.000001" ixy="0.0"  ixz="0.0"
+          iyy="0.000001" iyz="0.0"
+          izz="0.000001" />
+      </inertial>
+    </link>
+    <joint name="${prefix}/bhand_grasp_joint" type="fixed">
+      <parent link="${prefix}/bhand_palm_link"/>
+      <child link="${prefix}/bhand_grasp_link"/>
+      <origin xyz="0 0 0.12" rpy="0 0 0"/>
+      <limit effort="5" lower="0" upper="${PI}" velocity="5.0"/>
+      <dynamics damping="1.5" friction="1"/>
+    </joint>
+    <link name="${prefix}/bhand_grasp_link">
+      <inertial>
+        <mass value="0.000001" />
+        <inertia
+          ixx="0.000001" ixy="0.0"  ixz="0.0"
+          iyy="0.000001" iyz="0.0"
+          izz="0.000001" />
+      </inertial>
+    </link>
   </xacro:macro>
   <xacro:macro name="bhand_finger_prox" params="prefix parent_link xyz rpy axis">
