Commit message: updating wam ball

File: models/ball.urdf.xacro (robot description, xacro)
@@ -21,5 +21,5 @@
           <color rgba="0.9 0.9 0.9 0.0"/>
         </material>
-        <origin xyz="0 0 5" rpy="0 0 0"/>
+        <origin xyz="0 0 .005" rpy="0 0 0"/>
         <geometry>
           <cylinder radius="0.0415" length="0.01"/>
@@ -30,7 +30,7 @@
           <color rgba="0.9 0.9 0.9 0.0"/>
         </material>
-        <origin xyz="0 0 0.043" rpy="0 0 0"/>
+        <origin xyz="0 0 0.0425" rpy="0 0 0"/>
         <geometry>
-          <cylinder radius="0.0006" length="0.066"/>
+          <cylinder radius="0.006" length="0.065"/>
         </geometry>
       </visual>
@@ -44,4 +44,22 @@
         </geometry>
       </visual>
+      <collision>
+        <origin xyz="0 0 .005" rpy="0 0 0"/>
+        <geometry>
+          <cylinder radius="0.0415" length="0.01"/>
+        </geometry>
+      </collision>
+      <collision>
+        <origin xyz="0 0 0.0425" rpy="0 0 0"/>
+        <geometry>
+          <cylinder radius="0.006" length="0.065"/>
+        </geometry>
+      </collision>
+      <collision>
+        <origin xyz="0 0 0.1" rpy="0 0 0"/>
+        <geometry>
+          <sphere radius="0.0255"/>
+        </geometry>
+      </collision>
     </link>
   </xacro:macro>

File: models/wam_top.urdf.xacro (robot description, xacro)
@@ -10,4 +10,6 @@
   <!-- Definitions for the barrett hand -->
   <xacro:include filename="$(find barrett_model)/models/hand.urdf.xacro"/>
+  <!-- Definitions for the barrett ball -->
+  <xacro:include filename="$(find barrett_model)/models/ball.urdf.xacro"/>
   <!-- Materials -->
   <material name="WAMGrey">

Commit message: updating ball urdf to have a frame in the middle of the ball

File: models/ball.urdf.xacro (robot description, xacro)
@@ -63,4 +63,19 @@
       </collision>
     </link>
+    <joint name="${prefix}/bball_center_joint" type="fixed">
+      <parent link="${prefix}/bball_base_link"/>
+      <child link="${prefix}/bball_center_link"/>
+      <origin xyz="0 0 0.1" rpy="0 0 0"/>
+    </joint>
+    <link name="${prefix}/bball_center_link">
+      <inertial>
+        <origin xyz="0 0 0"/>
+        <mass value="0.00001" />
+        <inertia
+          ixx="0.0001" ixy="0"  ixz="0"
+                       iyy="0.0001"   iyz="0"
+                                      izz="0.0001" />
+      </inertial>
+    </link>
   </xacro:macro>
 </robot>
