Commit message: adding popeye bench lattice, will move soon

File: models/components.urdf.xacro (robot description, xacro)
@@ -32,32 +32,4 @@
   <include filename="$(find bard_urdf)/models/hand.urdf.xacro"/>
   <include filename="$(find bard_urdf)/models/common.urdf.xacro"/>
-  <xacro:macro name="base" params="xyz rpy parent">
-    <link name ="baseLink">
-      <inertial>
-        <origin xyz="0 0 0" rpy="0 0 0" />
-        <mass value="1.0" />
-        <inertia  ixx="1.0" ixy="0.0"  ixz="0.0"  iyy="100.0"  iyz="0.0"  izz="1.0" />
-      </inertial>
-      <visual>
-        <material name="WAMGrey" />
-        <origin xyz="0 0 0" rpy="${0.5 * PI} 0 0" />
-        <geometry>
-          <mesh filename="package://bard_urdf/models/componentSTL/Re2_Body.DAE"/>
-        </geometry>
-      </visual>
-      <collision>
-        <origin xyz="0 0 0" rpy="${0.5 * PI} 0 0" />
-        <geometry>
-          <mesh filename="package://bard_urdf/models/componentSTL/baseLinkTwoArms.stl"/>
-        </geometry>
-      </collision>
-    </link>
-    <xacro:gazeboReferenceDAE name="baseLink"/>
-    <joint name="baseJoint" type="fixed">
-      <parent link="${parent}"/>
-      <child link="baseLink"/>
-      <origin xyz="${xyz}" rpy="${rpy}"/>
-    </joint>
-  </xacro:macro>
   <xacro:macro name="Shoulder" params="prefix parentLink xyz rpy">
     <link name="${prefix}/ShoulderLink" >

File: models/root.urdf.xacro (robot description, xacro)
@@ -34,42 +34,45 @@
   </material>
   <link name = "world"/>
-  <xacro:base xyz="0 0 0.813372" rpy="0 0 0" parent="world"/>
-  <link name = "cylinderLink">
-    <inertial>
-      <origin xyz="0 0 0" rpy="0 0 0" />
-      <mass value="1.0" />
-      <inertia  ixx="1.0" ixy="0.0"  ixz="0.0"  iyy="100.0"  iyz="0.0"  izz="1.0" />
-    </inertial>
-    <visual>
-      <material name="WAMGrey" />
-      <origin xyz="0 0 0" rpy="0 0 0" />
-      <geometry>
-        <mesh filename="${homeDirectory}/models/componentSTL/armBase.DAE"/>
-      </geometry>
-    </visual>
-    <collision>
-      <origin xyz="0 0 0" rpy="0 0 0" />
-      <geometry>
-        <mesh filename="${homeDirectory}/models/componentSTL/armBase.stl"/>
-      </geometry>
-    </collision>
-  </link>
-  <xacro:gazeboReferenceDAE name="cylinderLink" />
+  <xacro:macro name="base" params="xyz rpy parent">
+    <link name ="baseLink">
+      <inertial>
+        <origin xyz="0 0 0" rpy="0 0 0" />
+        <mass value="1.0" />
+        <inertia  ixx="1.0" ixy="0.0"  ixz="0.0"  iyy="100.0"  iyz="0.0"  izz="1.0" />
+      </inertial>
+      <visual>
+        <material name="WAMGrey" />
+        <origin xyz="0 0 0" rpy="0 0 0" />
+        <geometry>
+          <!--box size="0.04 2.54 0.04"/-->
+          <mesh filename="package://bard_urdf/models/componentSTL/bench_lattice.dae"/>
+        </geometry>
+      </visual>
+      <collision>
+        <origin xyz="0 0 0" rpy="0 0 0" />
+        <geometry>
+          <mesh filename="package://bard_urdf/models/componentSTL/baseLinkTwoArms.stl"/>
+        </geometry>
+      </collision>
+    </link>
+    <xacro:gazeboReferenceDAE name="baseLink"/>
+    <joint name="baseJoint" type="fixed">
+      <parent link="${parent}"/>
+      <child link="baseLink"/>
+      <origin xyz="${xyz}" rpy="${rpy}"/>
+    </joint>
+  </xacro:macro>
+  <xacro:base xyz="0 0 0.68" rpy="0 0 0" parent="world"/>
   <link name = "LeftWAM/FixedLink" />
   <link name = "RightWAM/FixedLink" />
-  <joint name="cylinderJoint" type="fixed">
-    <parent link="baseLink"/>
-    <child link="cylinderLink"/>
-    <origin xyz="0 0 0" rpy="${0.5 * PI} 0 -${0.5 * PI}"/>
-  </joint>
   <joint name="rightFixedJoint" type="fixed">
     <parent link="baseLink"/>
     <child link="RightWAM/FixedLink"/>
-    <origin xyz="-0.350177361 -0.350177361 .37836125" rpy="0 ${-0.5*PI} ${0.25*PI}"/>
+    <origin xyz="0.346 -0.46 1" rpy="0 ${-0.5*PI} ${0.5*PI}"/>
   </joint>
   <joint name="leftFixedJoint" type="fixed">
     <parent link="baseLink"/>
     <child link="LeftWAM/FixedLink"/>
-    <origin xyz="0.350177361 -0.350177361 .37836125" rpy="0 ${-0.5*PI} ${0.75*PI}"/>
+    <origin xyz="0.356 0.46 1" rpy="0 ${-0.5*PI} ${0.5*PI}"/>
   </joint>
   <gazebo>

File: models/unused.urdf.xacro (robot description, xacro)
@@ -220,30 +220,2 @@
     </joint>
   </xacro:macro>
-  <xacro:macro name="base" params="xyz rpy parent">
-    <link name ="baseLink">
-      <inertial>
-        <origin xyz="0 0 0" rpy="0 0 0" />
-        <mass value="1.0" />
-        <inertia  ixx="1.0" ixy="0.0"  ixz="0.0"  iyy="100.0"  iyz="0.0"  izz="1.0" />
-      </inertial>
-      <visual>
-        <material name="WAMGrey" />
-        <origin xyz="0 0 0" rpy="${0.5 * PI} 0 0" />
-        <geometry>
-          <mesh filename="package://bard_urdf/models/componentSTL/Re2_Body.DAE"/>
-        </geometry>
-      </visual>
-      <collision>
-        <origin xyz="0 0 0" rpy="${0.5 * PI} 0 0" />
-        <geometry>
-          <mesh filename="package://bard_urdf/models/componentSTL/baseLinkTwoArms.stl"/>
-        </geometry>
-      </collision>
-    </link>
-    <xacro:gazeboReferenceDAE name="baseLink"/>
-    <joint name="baseJoint" type="fixed">
-      <parent link="${parent}"/>
-      <child link="baseLink"/>
-      <origin xyz="${xyz}" rpy="${rpy}"/>
-    </joint>
-  </xacro:macro>

Commit message: about to fix the wrist stuff

File: models/components.urdf.xacro (robot description, xacro)
@@ -244,47 +244,6 @@
     </joint>
   </xacro:macro>
-  <xacro:macro name="LowerWrist" params="prefix">
-    <link name="${prefix}/LowerWristLink" >
-      <inertial>
-        <origin xyz="0.00035500 -0.00499005 0.04864979" />
-        <mass value="0.63352875" />
-        <inertia  ixx="0.00102103" ixy="0.00000775"  ixz="-0.00001230"
-          iyy="0.00080944"  iyz="-0.00014417"
-          izz="0.00068788" />
-      </inertial>
-      <visual>
-        <material name="WAMGrey" />
-        <origin xyz="0 0 0" rpy="0 0 0" />
-        <geometry>
-          <mesh filename="${homeDirectory}/models/componentSTL/palm.DAE"/>
-        </geometry>
-      </visual>
-      <collision>
-        <origin xyz="0 0 0" rpy="0 0 0" />
-        <geometry>
-          <mesh filename="${homeDirectory}/models/componentSTL/palm.stl"/>
-        </geometry>
-      </collision>
-    </link>
-    <xacro:gazeboReferenceDAE name="${prefix}/LowerWristLink"/>
-    <joint name="${prefix}/LowerWristYawJoint" type="revolute">
-      <parent link="${prefix}/UpperWristPitchLink"/>
-      <child link="${prefix}/PalmLink"/>
-      <origin xyz="0 0 0.06713340" rpy="0 0 0"/>
-      <axis xyz="0 0 1"/>
-      <limit effort="5" lower="-2.95" upper="2.95" velocity="3.27"/><!-- 2.95 is a limit taken in from 3 due to saftey and differences between arms. -->
-      <!-- <safety_controller k_position="100" k_velocity="3" soft_lower_limit="-100.0" soft_upper_limit="100.0" /> -->
-      <dynamics damping="1.0" friction="100.0"/>
-    </joint>
-    <joint name="${prefix}/PalmJoint" type="fixed">
-      <parent link="${prefix}/ForceTorqueLink"/>
-      <child link="${prefix}/LowerWristFTPalmLink"/>
-      <origin xyz="0 0 0.0048" rpy="0 0 -${0.5 * PI}"/>
-      <provideFeedback value="true"/>
-    </joint>
-    <gazebo reference="${prefix}/PalmJoint">
-      <provideFeedback value="true"/>
-    </gazebo>
-  </xacro:macro>
+  <!-- Palm without force-torque sensor -->
+  <!-- ForceTorque macros -->
   <xacro:macro name="ForceTorque" params="prefix">
     <link name="${prefix}/ForceTorqueLink" >
@@ -380,4 +339,5 @@
     </gazebo>
   </xacro:macro>
+  <!-- Hand macros -->
   <xacro:macro name="KnuckleOne" params="prefix number xyz rpy axis">
     <link name="${prefix}/BHand/Finger${number}/KnuckleOneLink">

Commit message: working grav comp

File: models/components.urdf.xacro (robot description, xacro)
@@ -142,5 +142,5 @@
       <inertial>
         <origin xyz="0 0 0" />
-        <mass value="2.40016804" />
+        <mass value="3.40016804" />
         <origin xyz="-0.04001488 -.00022942 .13271662" rpy="0 0 0" />
         <inertia  ixx="0.01491672" ixy="0.00001741"   ixz="-0.00150604"
@@ -178,5 +178,5 @@
       <inertial>
         <origin xyz="0.00008921 0.00511217 0.00435824" />
-        <mass value="0.12376019" />
+        <mass value="1.12376019" />
         <inertia  ixx="0.00005029" ixy="0.00000020"  ixz="0.00007582"
           iyy="0.00007582"  iyz="-0.00000359"

Commit message: fixed joint effort limits, control switching could be made a bit less complex, joint traj controller is smooth, but could use more testing, experimentation with derivative gains needed

File: models/components.urdf.xacro (robot description, xacro)
@@ -39,5 +39,5 @@
       <origin xyz="${xyz}" rpy="${rpy}"/>
       <axis xyz="0 -1 0"/>
-      <limit effort="25" lower="-2.6" upper="2.6" velocity="3.27"/>
+      <limit effort="30" lower="-2.6" upper="2.6" velocity="3.27"/>
       <!-- <safety_controller k_position="10000000" k_velocity="10000000" soft_lower_limit="-100.0" soft_upper_limit="100.0" /> -->
       <dynamics damping="1.0" friction="100.0"/>
@@ -75,5 +75,5 @@
       <origin xyz="0 0 0" rpy="${0.5 * PI} 0 0"/>
       <axis xyz="0 1 0"/>
-      <limit effort="20" lower="-1.985" upper="1.985" velocity="3.27"/>
+      <limit effort="30" lower="-1.985" upper="1.985" velocity="3.27"/>
       <!-- <safety_controller k_position="100" k_velocity="3" soft_lower_limit="-100.0" soft_upper_limit="100.0" /> -->
       <dynamics damping="1.0" friction="100.0"/>
@@ -110,5 +110,5 @@
       <origin xyz="0 0 0" rpy="-${0.5 * PI} 0 0"/>
       <axis xyz="0 -1 0"/>
-      <limit effort="15" lower="-2.8" upper="2.8" velocity="3.27"/>
+      <limit effort="25" lower="-2.8" upper="2.8" velocity="3.27"/>
       <!-- <safety_controller k_position="100" k_velocity="3" soft_lower_limit="-100.0" soft_upper_limit="100.0" /> -->
       <dynamics damping="1.0" friction="100.0"/>

Commit message: smooth gains, happy IK

File: models/components.urdf.xacro (robot description, xacro)
@@ -39,5 +39,5 @@
       <origin xyz="${xyz}" rpy="${rpy}"/>
       <axis xyz="0 -1 0"/>
-      <limit effort="30" lower="-2.6" upper="2.6" velocity="3.27"/>
+      <limit effort="30" lower="-2.6" upper="2.6" velocity="0.50"/>
       <!-- <safety_controller k_position="10000000" k_velocity="10000000" soft_lower_limit="-100.0" soft_upper_limit="100.0" /> -->
       <dynamics damping="1.0" friction="100.0"/>
@@ -75,5 +75,5 @@
       <origin xyz="0 0 0" rpy="${0.5 * PI} 0 0"/>
       <axis xyz="0 1 0"/>
-      <limit effort="30" lower="-1.985" upper="1.985" velocity="3.27"/>
+      <limit effort="30" lower="-1.985" upper="1.985" velocity="0.5"/>
       <!-- <safety_controller k_position="100" k_velocity="3" soft_lower_limit="-100.0" soft_upper_limit="100.0" /> -->
       <dynamics damping="1.0" friction="100.0"/>
@@ -110,5 +110,5 @@
       <origin xyz="0 0 0" rpy="-${0.5 * PI} 0 0"/>
       <axis xyz="0 -1 0"/>
-      <limit effort="25" lower="-2.8" upper="2.8" velocity="3.27"/>
+      <limit effort="25" lower="-2.8" upper="2.8" velocity="0.5"/>
       <!-- <safety_controller k_position="100" k_velocity="3" soft_lower_limit="-100.0" soft_upper_limit="100.0" /> -->
       <dynamics damping="1.0" friction="100.0"/>
@@ -146,5 +146,5 @@
       <origin xyz="0.045 -0.55 0" rpy="${0.5 * PI} 0 0"/>
       <axis xyz="0 1 0"/>
-      <limit effort="15" lower="-0.9" upper="${PI}" velocity="3.27"/>
+      <limit effort="15" lower="-0.9" upper="${PI}" velocity="0.50"/>
       <!-- <safety_controller k_position="100" k_velocity="3" soft_lower_limit="-100.0" soft_upper_limit="100.0" /> -->
       <dynamics damping="1.0" friction="100.0"/>
@@ -182,5 +182,5 @@
       <origin xyz="-0.045 0 .35" rpy="-${0.5 * PI} 0 ${0.5 * PI}"/>
       <axis xyz="0 -1 0"/>
-      <limit effort="5" lower="-4.8" upper="1.3" velocity="3.27"/>
+      <limit effort="5" lower="-4.8" upper="1.3" velocity="0.20"/>
       <!-- <safety_controller k_position="100" k_velocity="3" soft_lower_limit="-100.0" soft_upper_limit="100.0" /> -->
       <dynamics damping="1.0" friction="100.0"/>
@@ -218,5 +218,5 @@
       <origin xyz="0.045 -0.55 0" rpy="${0.5 * PI} 0 0"/>
       <axis xyz="0 1 0"/>
-      <limit effort="15" lower="-0.9" upper="${PI}" velocity="3.27"/>
+      <limit effort="15" lower="-0.9" upper="${PI}" velocity="0.20"/>
       <!-- <safety_controller k_position="100" k_velocity="3" soft_lower_limit="-100.0" soft_upper_limit="100.0" /> -->
       <dynamics damping="1.0" friction="100.0"/>
@@ -254,5 +254,5 @@
       <origin xyz="-0.045 0 .3" rpy="-${0.5 * PI} 0 ${0.5 * PI}"/>
       <axis xyz="0 -1 0"/>
-      <limit effort="5" lower="-4.8" upper="1.3" velocity="3.27"/>
+      <limit effort="5" lower="-4.8" upper="1.3" velocity="0.20"/>
       <!-- <safety_controller k_position="100" k_velocity="3" soft_lower_limit="-100.0" soft_upper_limit="100.0" /> -->
       <dynamics damping="1.0" friction="100.0"/>
@@ -289,5 +289,5 @@
       <origin xyz="0 0 0" rpy="${0.5 * PI} ${PI} 0"/>
       <axis xyz="0 1 0"/>
-      <limit effort="5" lower="-1.45" upper="1.45" velocity="3.27"/><!-- 1.45 is a limit taken in from 1.5 due to saftey and differences between arms. -->
+      <limit effort="5" lower="-1.45" upper="1.45" velocity="0.20"/><!-- 1.45 is a limit taken in from 1.5 due to saftey and differences between arms. -->
       <!-- <safety_controller k_position="100" k_velocity="3" soft_lower_limit="-100.0" soft_upper_limit="100.0" /> -->
       <dynamics damping="1.0" friction="100.0"/>
@@ -325,5 +325,5 @@
       <origin xyz="0 0 0.060" rpy="0 0 0"/>
       <axis xyz="0 0 1"/>
-      <limit effort="5" lower="-2.95" upper="2.95" velocity="3.27"/><!-- 2.95 is a limit taken in from 3 due to saftey and differences between arms. -->
+      <limit effort="5" lower="-2.95" upper="2.95" velocity="0.20"/><!-- 2.95 is a limit taken in from 3 due to saftey and differences between arms. -->
       <!-- <safety_controller k_position="100" k_velocity="3" soft_lower_limit="-100.0" soft_upper_limit="100.0" /> -->
       <dynamics damping="1.0" friction="100.0"/>
@@ -361,5 +361,5 @@
       <origin xyz="0 0 0.06713340" rpy="0 0 0"/>
       <axis xyz="0 0 1"/>
-      <limit effort="5" lower="-2.95" upper="2.95" velocity="3.27"/><!-- 2.95 is a limit taken in from 3 due to saftey and differences between arms. -->
+      <limit effort="5" lower="-2.95" upper="2.95" velocity="0.20"/><!-- 2.95 is a limit taken in from 3 due to saftey and differences between arms. -->
       <!-- <safety_controller k_position="100" k_velocity="3" soft_lower_limit="-100.0" soft_upper_limit="100.0" /> -->
       <dynamics damping="1.0" friction="100.0"/>
@@ -397,5 +397,5 @@
       <origin xyz="${xyz}" rpy="${rpy}"/>
       <axis xyz="${axis}"/>
-      <limit effort="1" lower="0" upper="${PI}" velocity="3.27"/>
+      <limit effort="1" lower="0" upper="${PI}" velocity="0.20"/>
       <dynamics damping="0.005" friction="100.0"/>
     </joint>
@@ -436,5 +436,5 @@
       <axis xyz="0 0 -1"/>
       <!-- 122 degrees - start orientation of 0.4 degrees-->
-      <limit effort="1" lower="0" upper="${2.12930169 - 0.00698131701}" velocity="3.27"/>
+      <limit effort="1" lower="0" upper="${2.12930169 - 0.00698131701}" velocity="1.50"/>
       <dynamics damping="0.005" friction="100.0"/>
     </joint>
@@ -476,5 +476,5 @@
       <axis xyz="0 0 -1"/>
       <!-- measured max angle is 94.  so upper limit is 94 - start orientation (42 degrees)-->
-      <limit effort="1" lower="0" upper="${1.6406095 - 0.733038286}" velocity="3.27"/>
+      <limit effort="1" lower="0" upper="${1.6406095 - 0.733038286}" velocity="1.50"/>
       <dynamics damping="0.005" friction="100.0"/>
     </joint>

Commit message: Fixing two arm test, non-FT urdf wrist

File: models/components.urdf.xacro (robot description, xacro)
@@ -323,5 +323,5 @@
       <parent link="${prefix}/UpperWristPitchLink"/>
       <child link="${prefix}/LowerWristYawLink"/>
-      <origin xyz="0 0 0.060" rpy="0 0 0"/>
+      <origin xyz="0 0 0.065" rpy="0 0 0"/>
       <axis xyz="0 0 1"/>
       <limit effort="5" lower="-2.95" upper="2.95" velocity="0.20"/><!-- 2.95 is a limit taken in from 3 due to saftey and differences between arms. -->
@@ -341,5 +341,5 @@
         <origin xyz="0 0 0" rpy="0 0 0" />
         <geometry>
-          <mesh filename="${homeDirectory}/models/componentSTL/forceTorqueSensor.DAE"/>
+          <mesh filename="${homeDirectory}/models/componentSTL/wamLowerWristLink7.dae" scale="0.01 0.01 0.01"/>
         </geometry>
       </visual>
@@ -347,5 +347,5 @@
         <origin xyz="0 0 0" rpy="0 0 0" />
         <geometry>
-          <mesh filename="${homeDirectory}/models/componentSTL/forceTorqueSensor.stl"/>
+          <mesh filename="${homeDirectory}/models/componentSTL/wamLowerWristLink7.stl" scale="0.01 0.01 0.01"/>
         </geometry>
       </collision>
