Commit message: Fixing more stuff in urdf, making base link fixed to the world

File: models/components.urdf.xacro (robot description, xacro)
@@ -260,5 +260,4 @@
     <xacro:control topicName="${prefix}/ElbowPitch" name="DarmSim_${prefix}Arm_WAM_ElbowPitch" linkName="${prefix}/ForeArmLink" jointName="${prefix}/ElbowJoint" />
   </xacro:macro>
-  <!-- DEBUG HERE -->
   <xacro:macro name="UpperWristYaw" params="prefix">
     <joint name="${prefix}/UpperWristYawJoint" type="revolute">
@@ -320,5 +319,5 @@
           <color rgba="0.9 0.9 0.9 1.0"/>
         </material>
-        <origin xyz="0 0 0" rpy="${0.5 * PI} 0 ${0.5 * PI}" />
+        <origin xyz="0 0 0" rpy="${0.5 * PI} 0 0" />
         <geometry>
           <mesh filename="${homeDirectory}/models/componentSTL/wamUpperWristPitchLink6.dae"/>
@@ -326,5 +325,5 @@
       </visual>
       <collision>
-        <origin xyz="0 0 0" rpy="${0.5 * PI} 0 ${0.5 * PI}" />
+        <origin xyz="0 0 0" rpy="${0.5 * PI} 0 0" />
         <geometry>
           <mesh filename="${homeDirectory}/models/componentSTL/wamUpperWristPitchLink6.stl"/>
@@ -360,5 +359,5 @@
         <origin xyz="0 0 0" rpy="0 0 0" />
         <geometry>
-          <mesh filename="${homeDirectory}/models/componentSTL/wamLowerWristLink7.dae" scale="0.01 0.01 0.01"/>
+          <mesh filename="${homeDirectory}/models/componentSTL/wamLowerWristLink7.dae"/>
         </geometry>
       </visual>
@@ -366,5 +365,5 @@
         <origin xyz="0 0 0" rpy="0 0 0" />
         <geometry>
-          <mesh filename="${homeDirectory}/models/componentSTL/wamLowerWristLink7.stl" scale="0.01 0.01 0.01"/>
+          <mesh filename="${homeDirectory}/models/componentSTL/wamLowerWristLink7.stl"/>
         </geometry>
       </collision>
@@ -373,165 +372,3 @@
     <xacro:control topicName="${prefix}/LowerWristYaw" name="DarmSim_${prefix}Arm_WAM_LowerWristYaw" linkName="${prefix}/LowerWristYawLink" jointName="${prefix}/LowerWristYawJoint" />
   </xacro:macro>
-  <!-- Palm with ForceTorque macros -->
-  <xacro:macro name="LowerWristFT" params="prefix">
-    <joint name="${prefix}/LowerWristYawJoint" type="revolute">
-      <parent link="${prefix}/UpperWristPitchLink"/>
-      <child link="${prefix}/LowerWristYawLink"/>
-      <origin xyz="0 0 0.06713340" rpy="0 0 0"/>
-      <axis xyz="0 0 1"/>
-      <limit effort="5" lower="-2.95" upper="2.95" velocity="0.20"/><!-- 2.95 is a limit taken in from 3 due to saftey and differences between arms. -->
-      <!-- <safety_controller k_position="100" k_velocity="3" soft_lower_limit="-100.0" soft_upper_limit="100.0" /> -->
-      <dynamics damping="1.0" friction="100.0"/>
-    </joint>
-    <link name="${prefix}/LowerWristYawLink" >
-      <inertial>
-        <origin xyz="-0.00000134 -0.00228167 -0.00000141" rpy="0 0 0" />
-        <mass value="0.17286134" />
-        <inertia  ixx="0.00010859" ixy="0.00000000"  ixz="-0.00000000"
-          iyy="0.00020683"  iyz="-0.0000000"
-          izz="0.00010851" />
-      </inertial>
-      <visual>
-        <material name="WAMGrey">
-          <color rgba="0.9 0.9 0.9 1.0"/>
-        </material>
-        <origin xyz="0 0 0" rpy="0 0 0" />
-        <geometry>
-          <mesh filename="${homeDirectory}/models/componentSTL/forceTorqueSensor.DAE"/>
-        </geometry>
-      </visual>
-      <collision>
-        <origin xyz="0 0 0" rpy="0 0 0" />
-        <geometry>
-          <mesh filename="${homeDirectory}/models/componentSTL/forceTorqueSensor.stl"/>
-        </geometry>
-      </collision>
-    </link>
-    <xacro:gazeboReferenceDAE name="${prefix}/LowerWristYawLink"/>
-    <xacro:control topicName="${prefix}/LowerWristYaw" name="DarmSim_${prefix}Arm_WAM_LowerWristYaw" linkName="${prefix}/LowerWristYawLink" jointName="${prefix}/LowerWristYawJoint" />
-  </xacro:macro>
-  <!-- Hand macros -->
-  <xacro:macro name="KnuckleOne" params="prefix number xyz rpy axis">
-    <joint name="${prefix}/BHand/Finger${number}/KnuckleOneJoint" type="revolute">
-      <parent link="${prefix}/LowerWristPalmLink"/>
-      <child link="${prefix}/BHand/Finger${number}/KnuckleOneLink"/>
-      <origin xyz="${xyz}" rpy="${rpy}"/>
-      <axis xyz="${axis}"/>
-      <limit effort="1" lower="0" upper="${PI}" velocity="0.20"/>
-      <dynamics damping="0.005" friction="100.0"/>
-    </joint>
-    <link name="${prefix}/BHand/Finger${number}/KnuckleOneLink">
-      <visual>
-        <material name="WAMGrey">
-          <color rgba="0.9 0.9 0.9 1.0"/>
-        </material>
-        <origin xyz="0 0 0" rpy="${0.5 * PI} 0 -${0.5 * PI}" />
-        <geometry>
-          <mesh filename="${homeDirectory}/models/componentSTL/firstFingerLink.DAE"/>
-        </geometry>
-      </visual>
-      <inertial>
-        <origin xyz="0.03201666 -0.00086502 0.00890075" />
-        <mass value="0.16252678" />
-        <inertia  ixx="0.00002567" ixy="-0.00000146"  ixz="0.00001128"
-          iyy="0.00008818"   iyz="-0.00000094"
-          izz="0.00007827" />
-      </inertial>
-      <collision>
-        <origin xyz="0 0 0" rpy="${0.5 * PI} 0 -${0.5 * PI}" />
-        <geometry>
-          <mesh filename="${homeDirectory}/models/componentSTL/firstFingerLink.stl"/>
-        </geometry>
-        <mu1 value="50000.0" />
-        <mu2 value="50000.0" />
-        <kp  value="1000000.0" />
-        <kd  value="1.0" />
-      </collision>
-    </link>
-    <xacro:gazeboReferenceDAE name="${prefix}/BHand/Finger${number}/KnuckleOneLink" />
-    <xacro:control topicName="${prefix}/BHand/Finger${number}/KnuckleOne" name="DarmSim_${prefix}Arm_BHand_Finger${number}KnuckleOne" linkName="${prefix}/BHand/Finger${number}/KnuckleOneLink" jointName="${prefix}/BHand/Finger${number}/KnuckleOneJoint" />
-  </xacro:macro>
-  <xacro:macro name="KnuckleTwo" params="parent prefix number xyz rpy">
-    <joint name="${prefix}/BHand/Finger${number}/KnuckleTwoJoint" type="revolute">
-      <parent link="${parent}"/>
-      <child link="${prefix}/BHand/Finger${number}/KnuckleTwoLink"/>
-      <origin xyz="${xyz}" rpy="${rpy}"/>
-      <axis xyz="0 0 -1"/>
-      <!-- 122 degrees - start orientation of 0.4 degrees-->
-      <limit effort="1" lower="0" upper="${2.12930169 - 0.00698131701}" velocity="1.50"/>
-      <dynamics damping="0.005" friction="100.0"/>
-    </joint>
-    <link name="${prefix}/BHand/Finger${number}/KnuckleTwoLink">
-      <visual>
-        <material name="WAMGrey">
-          <color rgba="0.9 0.9 0.9 1.0"/>
-        </material>
-        <origin xyz="0 0 0" rpy="${PI} ${0.5 * PI} 0" />
-        <geometry>
-          <mesh filename="${homeDirectory}/models/componentSTL/secondFingerLink.DAE"/>
-        </geometry>
-      </visual>
-      <inertial>
-        <origin xyz=".031720 .001070 -.000586" />
-        <mass value="0.057957" />
-        <inertia  ixx="0.00000461" ixy="0.00000003"  ixz="0.00000164"
-          iyy="0.00003590"  iyz="0.00000004"
-          izz="0.00003682" />
-      </inertial>
-      <collision>
-        <origin xyz="0 0 0" rpy="${PI} ${0.5 * PI} 0" />
-        <geometry>
-          <mesh filename="${homeDirectory}/models/componentSTL/secondFingerLink.stl"/>
-        </geometry>
-        <mu1 value="50000.0" />
-        <mu2 value="50000.0" />
-        <kp  value="1000000.0" />
-        <kd  value="1.0" />
-      </collision>
-    </link>
-    <xacro:gazeboReferenceDAE name="${prefix}/BHand/Finger${number}/KnuckleTwoLink"/>
-    <xacro:control topicName="${prefix}/BHand/Finger${number}/KnuckleTwo" name="DarmSim_${prefix}Arm_BHand_Finger${number}KnuckleTwo" linkName="${prefix}/BHand/Finger${number}/KnuckleTwoLink" jointName="${prefix}/BHand/Finger${number}/KnuckleTwoJoint" />
-  </xacro:macro>
-  <xacro:macro name="KnuckleThree" params="prefix number">
-    <joint name="${prefix}/BHand/Finger${number}/KnuckleThreeJoint" type="revolute">
-      <parent link="${prefix}/BHand/Finger${number}/KnuckleTwoLink"/>
-      <child link="${prefix}/BHand/Finger${number}/KnuckleThreeLink"/>
-      <!-- 42 degrees -->
-      <origin xyz="0.07 0 0" rpy="0 0 -0.733038286"/>
-      <axis xyz="0 0 -1"/>
-      <!-- measured max angle is 94.  so upper limit is 94 - start orientation (42 degrees)-->
-      <limit effort="1" lower="0" upper="${1.6406095 - 0.733038286}" velocity="1.50"/>
-      <dynamics damping="0.005" friction="100.0"/>
-    </joint>
-    <link name="${prefix}/BHand/Finger${number}/KnuckleThreeLink">
-      <visual>
-        <material name="WAMGrey">
-          <color rgba="0.9 0.9 0.9 1.0"/>
-        </material>
-        <origin xyz="0 0 0" rpy="0 ${0.5 * PI} 0" />
-        <geometry>
-          <mesh filename="${homeDirectory}/models/componentSTL/thirdFingerLink.DAE"/>
-        </geometry>
-      </visual>
-      <inertial>
-        <origin xyz="0.01970974 0.00182016 0.00020041" />
-        <mass value="0.03421781" />
-        <inertia  ixx="0.00000287" ixy="0.00000091"  ixz="-0.00000007"
-          iyy="0.00001329"  iyz="-0.00000002"
-          izz="0.00001214" />
-      </inertial>
-      <collision>
-        <origin xyz="0 0 0" rpy="0 ${0.5 * PI} 0" />
-        <geometry>
-          <mesh filename="${homeDirectory}/models/componentSTL/thirdFingerLink.stl"/>
-        </geometry>
-        <mu1 value="50000.0" />
-        <mu2 value="50000.0" />
-        <kp  value="1000000.0" />
-        <kd  value="1.0" />
-      </collision>
-    </link>
-    <xacro:gazeboReferenceDAE name="${prefix}/BHand/Finger${number}/KnuckleThreeLink"/>
-    <xacro:control topicName="${prefix}/BHand/Finger${number}/KnuckleThree" name="DarmSim_${prefix}Arm_BHand_Finger${number}KnuckleThree" linkName="${prefix}/BHand/Finger${number}/KnuckleThreeLink" jointName="${prefix}/BHand/Finger${number}/KnuckleThreeJoint" />
-  </xacro:macro>
 </robot>

File: models/wam_top.urdf.xacro (robot description, xacro)
@@ -25,5 +25,5 @@
       <visual>
         <material name="WAMGrey">
-          <color rgba="0.9 0.9 0.9 1.0"/>
+          <color rgba="0.9 0.9 0.9 0.0"/>
         </material>
         <!--  this orgin is not centered because the origin in our model is not at the same spot as the origin barret uses for inertia-->

File: robots/wam_7dof_2x.urdf.xacro (robot description, xacro)
@@ -4,8 +4,15 @@
   <include filename="$(find bard_urdf)/models/wam_top.urdf.xacro"/>
   <!-- Root link is in the world frame-->
+  <link name="world"/>
+  <!-- Fix this robot to the world -->
+  <joint name="world_joint"  type="fixed">
+    <origin xyz="0 0 0" rpy="0 0 0" />
+    <parent link="world"/>
+    <child link="baseLink"/>
+  </joint>
   <link name = "baseLink">
     <inertial>
       <origin xyz="-1 0 0" />
-      <mass value="1000" />
+      <mass value="100" />
       <inertia
         ixx="1" ixy="0"   ixz="0"

Commit message: fixing base link coordinate frame

File: models/components.urdf.xacro (robot description, xacro)
@@ -46,6 +46,4 @@
           <color rgba="0.7 0.7 0.7 0.0"/>
         </material>
-        <!--  this orgin is not centered because the origin in our model is not at the same spot as the origin barret uses for inertia-->
-        <origin xyz="0 0.0 0" rpy="0 0 0"/>
         <geometry>
           <mesh filename="${models_path}/sw_meshes/base_link_fine.STL"/>
@@ -53,5 +51,4 @@
       </visual>
       <collision>
-        <origin xyz="0 0.0 0" rpy="0 0 0" />
         <geometry>
           <mesh filename="${models_path}/sw_meshes/base_link.STL"/>
@@ -64,5 +61,5 @@
       <parent link="${prefix}/base_link"/>
       <child link="${prefix}/shoulder_yaw_link"/>
-      <origin xyz="0 0 0.160" rpy="0 0 0"/>
+      <origin xyz="0 0 0.346" rpy="0 0 0"/>
       <axis xyz="0 0 1"/>
       <limit effort="30" lower="-2.6" upper="2.6" velocity="0.50"/>
@@ -97,5 +94,5 @@
       <parent link="${prefix}/shoulder_yaw_link"/>
       <child link="${prefix}/shoulder_pitch_link"/>
-      <origin xyz="0 0 0.186" rpy="${-PI/2} 0 0"/>
+      <origin xyz="0 0 0" rpy="${-PI/2} 0 0"/>
       <axis xyz="0 0 1"/>
       <limit effort="30" lower="-1.985" upper="1.985" velocity="0.5"/>
@@ -148,5 +145,4 @@
           <color rgba="0.7 0.7 0.7 1.0"/>
         </material>
-        <origin xyz="0 0 0" rpy="0 0 0" />
         <geometry>
           <mesh filename="${models_path}/sw_meshes/upper_arm_link_fine.STL"/>
@@ -154,5 +150,4 @@
       </visual>
       <collision>
-        <origin xyz="0 0 0" rpy="0 0 0" />
         <geometry>
           <mesh filename="${models_path}/sw_meshes/upper_arm_link.STL"/>

File: models/hand.urdf.xacro (robot description, xacro)
@@ -11,10 +11,10 @@
   <xacro:macro name="bhand_finger_1" params="prefix">
     <xacro:bhand_finger_prox prefix="${prefix}/finger_1" parent_link="${prefix}/bhand_palm_link" xyz="0.025 0.0 0.0415" rpy="0 0 -${PI/2}" axis="0 0 1"/>
-    <xacro:bhand_finger_med prefix="${prefix}/finger_1" parent_link="${prefix}/finger_1/bhand_finger_prox_link" xyz="0.05 0.0 0.03390" rpy="${PI/2} 0 0"/>
+    <xacro:bhand_finger_med prefix="${prefix}/finger_1" parent_link="${prefix}/finger_1/prox_link" xyz="0.05 0.0 0.03390" rpy="${PI/2} 0 0"/>
     <xacro:bhand_finger_dist prefix="${prefix}/finger_1"/>
   </xacro:macro>
   <xacro:macro name="bhand_finger_2" params="prefix">
     <xacro:bhand_finger_prox prefix="${prefix}/finger_2" parent_link="${prefix}/bhand_palm_link" xyz="-0.025 0.0 0.0415" rpy="0 0 -${PI/2}" axis="0 0 -1"/>
-    <xacro:bhand_finger_med prefix="${prefix}/finger_2" parent_link="${prefix}/finger_2/bhand_finger_prox_link" xyz="0.05 0.0 0.03390" rpy="${PI/2} 0 0"/>
+    <xacro:bhand_finger_med prefix="${prefix}/finger_2" parent_link="${prefix}/finger_2/prox_link" xyz="0.05 0.0 0.03390" rpy="${PI/2} 0 0"/>
     <xacro:bhand_finger_dist prefix="${prefix}/finger_2"/>
   </xacro:macro>
@@ -55,12 +55,12 @@
   </xacro:macro>
   <xacro:macro name="bhand_finger_prox" params="prefix parent_link xyz rpy axis">
-    <joint name="${prefix}/bhand_finger_prox_joint" type="revolute">
+    <joint name="${prefix}/prox_joint" type="revolute">
       <parent link="${parent_link}"/>
-      <child link="${prefix}/bhand_finger_prox_link"/>
+      <child link="${prefix}/prox_link"/>
       <origin xyz="${xyz}" rpy="${rpy}"/>
       <axis xyz="${axis}"/>
       <limit effort="5" lower="0" upper="${PI}" velocity="0.20"/>
     </joint>
-    <link name="${prefix}/bhand_finger_prox_link">
+    <link name="${prefix}/prox_link">
       <inertial>
         <origin xyz="0.023133 0.00078642 0.00052792" />
@@ -87,12 +87,12 @@
   </xacro:macro>
   <xacro:macro name="bhand_finger_med" params="prefix parent_link xyz rpy">
-    <joint name="${prefix}/bhand_finger_med_joint" type="revolute">
+    <joint name="${prefix}/med_joint" type="revolute">
       <parent link="${parent_link}"/>
-      <child link="${prefix}/bhand_finger_med_link"/>
+      <child link="${prefix}/med_link"/>
       <origin xyz="${xyz}" rpy="${rpy}"/>
       <axis xyz="0 0 1"/>
       <limit effort="5" lower="0" upper="${140/180*PI}" velocity="0.20"/>
     </joint>
-    <link name="${prefix}/bhand_finger_med_link">
+    <link name="${prefix}/med_link">
       <inertial>
         <origin xyz="0.023133 0.00078642 0.00052792" />
@@ -119,12 +119,12 @@
   </xacro:macro>
   <xacro:macro name="bhand_finger_dist" params="prefix">
-    <joint name="${prefix}/bhand_finger_dist_joint" type="revolute">
-      <parent link="${prefix}/bhand_finger_med_link"/>
-      <child link="${prefix}/bhand_finger_dist_link"/>
+    <joint name="${prefix}/dist_joint" type="revolute">
+      <parent link="${prefix}/med_link"/>
+      <child link="${prefix}/dist_link"/>
       <origin xyz="0.06994 0.003 0.0" rpy="0 0 0"/>
       <axis xyz="0 0 1"/>
       <limit effort="5" lower="0" upper="${48/180*PI}" velocity="0.20"/>
     </joint>
-    <link name="${prefix}/bhand_finger_dist_link">
+    <link name="${prefix}/dist_link">
       <inertial>
         <origin xyz="0.022825 0.0010491 0.0004203" />

Commit message: Fixing inertial properties

File: models/components.urdf.xacro (robot description, xacro)
@@ -68,10 +68,10 @@
     <link name="${prefix}/shoulder_yaw_link" >
       <inertial>
-        <origin xyz="-.00443422 0.1289039 -.00066489" />
+        <origin xyz="-.00443422 -.00066489 -0.1289039 " />
         <mass value="10.7677" />
         <inertia
-          ixx=".13488033"  ixy="-.00213041"   ixz="-.00012485"
-          iyy=".11328369"  iyz=".00068555"
-          izz=".09046330" />
+          ixx=".13488033"  ixy="-0.00012485"   ixz="0.00213041"
+                           iyy=".09046330"    iyz="-.00068555"
+                                              izz=".11328369" />
       </inertial>
       <visual>
@@ -109,10 +109,10 @@
       </visual>
       <inertial>
-        <origin xyz="-.00236981 .03105614 .01542114" />
+        <origin xyz="-.00236981 -.01542114 .03105614 " />
         <mass value="3.87493756" />
         <inertia
-          ixx=".02140958"  ixy=".00027172"  ixz=".00002461"
-          iyy=".01377875"  iyz="-.00181920"
-          izz=".01558906" />
+          ixx="0.02140958"  ixy="-0.00002461"  ixz="0.00027172"
+                            iyy="0.015589060"  iyz="0.0018192"
+                                               izz="0.01377875" />
       </inertial>
       <collision>
@@ -134,10 +134,10 @@
     <link name="${prefix}/upper_arm_link" >
       <inertial>
-        <origin xyz="-.03826 .20751 .00003" />
+        <origin xyz="-0.083258580000000 0.000033090000000 0.342492300000000" />
         <mass value="1.80228141" />
         <inertia
-          ixx=".05911077"  ixy="-.00249612"  ixz=".00000738"
-          iyy=".00324550"  iyz="-.00001767"
-          izz=".05927043" />
+          ixx=".05911077"  ixy="-0.00000738"  ixz="-0.00249612"
+                           iyy="0.05927043"   iyz="0.00001767"
+                                              izz="0.0032455" />
       </inertial>
       <visual>
@@ -169,11 +169,10 @@
     <link name="${prefix}/forearm_link" >
       <inertial>
-        <origin xyz="0 0 0" />
-        <mass value="3.20016804" />
-        <origin xyz="-0.04001488 -.00022942 .13271662" rpy="0 0 0" />
-        <inertia
-          ixx="0.01491672"  ixy="0.00001741"   ixz="-0.00150604"
-          iyy="0.01482988"  iyz="-0.00002109"
-          izz="0.00294463" />
+        <mass value="2.40016804" />
+        <origin xyz="-0.04001488 -.13271662 -.00022942 " rpy="0 0 0" />
+        <inertia
+          ixx="0.01491672" ixy="0.001506040000000" ixz="0.000017410000000"
+                           iyy="0.002944630000000" iyz="0.000021090000000"
+                                                   izz="0.014829880000000" />
       </inertial>
       <visual>
@@ -219,5 +218,5 @@
     <link name="${prefix}/wrist_yaw_link" >
       <inertial>
-        <origin xyz="0.00008921 0.00511217 0.00435824" />
+        <origin xyz="0.00008921 0.00435824 -0.00511217 " />
         <mass value="1.12376019" />
         <inertia  ixx="0.00005029" ixy="0.00000020"  ixz="0.00007582"
@@ -254,5 +253,5 @@
     <link name="${prefix}/wrist_pitch_link" >
       <inertial>
-        <origin xyz="-0.00012262 -0.01703194 0.02468336" rpy="0 0 0" />
+        <origin xyz="-0.00012262 -0.02468336 -0.01703194 " rpy="0 0 0" />
         <mass value="0.51797364" />
         <inertia

Commit message: updating inertial properties

File: models/components.urdf.xacro (robot description, xacro)
@@ -169,6 +169,6 @@
     <link name="${prefix}/forearm_link" >
       <inertial>
-        <mass value="1.50016804" />
-        <origin xyz="-0.04001488 -.08271662 -.00022942 " rpy="0 0 0" />
+        <mass value="1.00016804" />
+        <origin xyz="-0.04001488 -.12271662 -.00022942 " rpy="0 0 0" />
         <inertia
           ixx="0.01491672" ixy="0.001506040000000" ixz="0.000017410000000"

Commit message: Adding missing mass to link, this was angering gazebo

File: models/components.urdf.xacro (robot description, xacro)
@@ -69,5 +69,5 @@
       <inertial>
         <origin xyz="-.00443422 -.00066489 -0.1289039 " />
-        <mass value="0" />
+        <mass value="5.0" />
         <inertia
           ixx=".13488033"  ixy="-0.00012485"   ixz="0.00213041"
