Commit message: Removing old dynamics tags, replacing with new gazebo xacro

File: models/components.urdf.xacro (robot description, xacro)
@@ -26,4 +26,12 @@
   <include filename="$(find barrett_model)/models/hand.urdf.xacro"/>
   <include filename="$(find barrett_model)/models/common.urdf.xacro"/>
+  <xacro:macro name="gz_joint">
+      <physics>
+        <ode>
+          <cfm_damping>true</cfm_damping>
+          <cfm>0.0</cfm>
+        </ode>
+      </physics>
+  </xacro:macro>
   <!-- Upper arm macros -->
   <xacro:macro name="wam_base" params="prefix parent_link xyz rpy">
@@ -58,4 +66,7 @@
   </xacro:macro>
   <xacro:macro name="wam_shoulder_yaw" params="prefix">
+    <gazebo reference="${prefix}/base_yaw_joint">
+      <xacro:gz_joint/>
+    </gazebo>
     <joint name="${prefix}/base_yaw_joint" type="revolute">
       <parent link="${prefix}/base_link"/>
@@ -64,5 +75,5 @@
       <axis xyz="0 0 1"/>
       <limit effort="60" lower="-2.6" upper="2.6" velocity="0.50"/>
-      <dynamics damping="1.0" friction="100.0"/>
+      <!--<dynamics damping="1.0" friction="100.0"/>-->
     </joint>
     <link name="${prefix}/shoulder_yaw_link" >
@@ -91,4 +102,7 @@
   </xacro:macro>
   <xacro:macro name="wam_shoulder_pitch" params="prefix">
+    <gazebo reference="${prefix}/shoulder_pitch_joint">
+      <xacro:gz_joint/>
+    </gazebo>
     <joint name="${prefix}/shoulder_pitch_joint" type="revolute">
       <parent link="${prefix}/shoulder_yaw_link"/>
@@ -97,5 +111,5 @@
       <axis xyz="0 0 1"/>
       <limit effort="60" lower="-1.985" upper="1.985" velocity="0.5"/>
-      <dynamics damping="1.0" friction="100.0"/>
+      <!--<dynamics damping="1.0" friction="100.0"/>-->
     </joint>
     <link name="${prefix}/shoulder_pitch_link" >
@@ -124,4 +138,7 @@
   </xacro:macro>
   <xacro:macro name="wam_upper_arm" params="prefix">
+    <gazebo reference="${prefix}/shoulder_yaw_joint">
+      <xacro:gz_joint/>
+    </gazebo>
     <joint name="${prefix}/shoulder_yaw_joint" type="revolute">
       <parent link="${prefix}/shoulder_pitch_link"/>
@@ -130,5 +147,5 @@
       <axis xyz="0 0 1"/>
       <limit effort="45" lower="-2.8" upper="2.8" velocity="0.5"/>
-      <dynamics damping="1.0" friction="100.0"/>
+      <!--<dynamics damping="1.0" friction="100.0"/>-->
     </joint>
     <link name="${prefix}/upper_arm_link" >
@@ -158,4 +175,7 @@
   <!-- Forearm macros -->
   <xacro:macro name="wam_forearm" params="prefix">
+    <gazebo reference="${prefix}/elbow_pitch_joint">
+      <xacro:gz_joint/>
+    </gazebo>
     <joint name="${prefix}/elbow_pitch_joint" type="revolute">
       <parent link="${prefix}/upper_arm_link"/>
@@ -163,7 +183,7 @@
       <origin xyz="0.045 0 0.55" rpy="${-PI/2} 0 0"/>
       <axis xyz="0 0 1"/>
-      <limit effort="15" lower="-0.9" upper="${PI}" velocity="0.20"/>
+      <limit effort="20" lower="-0.9" upper="${PI}" velocity="0.20"/>
       <!-- <safety_controller k_position="100" k_velocity="3" soft_lower_limit="-100.0" soft_upper_limit="100.0" /> -->
-      <dynamics damping="1.0" friction="100.0"/>
+      <!--<dynamics damping="1.0" friction="100.0"/>-->
     </joint>
     <link name="${prefix}/forearm_link" >
@@ -207,4 +227,7 @@
   </xacro:macro>
   <xacro:macro name="wam_wrist_yaw" params="prefix">
+    <gazebo reference="${prefix}/wrist_yaw_joint">
+      <xacro:gz_joint/>
+    </gazebo>
     <joint name="${prefix}/wrist_yaw_joint" type="revolute">
       <parent link="${prefix}/forearm_link"/>
@@ -214,5 +237,5 @@
       <limit effort="5" lower="-4.8" upper="1.3" velocity="0.20"/>
       <!-- <safety_controller k_position="100" k_velocity="3" soft_lower_limit="-100.0" soft_upper_limit="100.0" /> -->
-      <dynamics damping="1.0" friction="100.0"/>
+      <!--<dynamics damping="1.0" friction="100.0"/>-->
     </joint>
     <link name="${prefix}/wrist_yaw_link" >
@@ -242,4 +265,7 @@
   </xacro:macro>
   <xacro:macro name="wam_wrist_pitch" params="prefix">
+    <gazebo reference="${prefix}/wrist_pitch_joint">
+      <xacro:gz_joint/>
+    </gazebo>
     <joint name="${prefix}/wrist_pitch_joint" type="revolute">
       <parent link="${prefix}/wrist_yaw_link"/>
@@ -249,5 +275,5 @@
       <limit effort="5" lower="-1.45" upper="1.45" velocity="0.20"/><!-- 1.45 is a limit taken in from 1.5 due to saftey and differences between arms. -->
       <!-- <safety_controller k_position="100" k_velocity="3" soft_lower_limit="-100.0" soft_upper_limit="100.0" /> -->
-      <dynamics damping="1.0" friction="100.0"/>
+      <!--<dynamics damping="1.0" friction="100.0"/>-->
     </joint>
     <link name="${prefix}/wrist_pitch_link" >
@@ -277,4 +303,7 @@
   <!-- Palm without force-torque sensor -->
   <xacro:macro name="wam_palm" params="prefix">
+    <gazebo reference="${prefix}/palm_yaw_joint">
+      <xacro:gz_joint/>
+    </gazebo>
     <joint name="${prefix}/palm_yaw_joint" type="revolute">
       <parent link="${prefix}/wrist_pitch_link"/>
@@ -284,5 +313,5 @@
       <limit effort="5" lower="-2.95" upper="2.95" velocity="0.20"/><!-- 2.95 is a limit taken in from 3 due to saftey and differences between arms. -->
       <!-- <safety_controller k_position="100" k_velocity="3" soft_lower_limit="-100.0" soft_upper_limit="100.0" /> -->
-      <!--dynamics damping="1.0" friction="100.0"/-->
+      <!--<dynamics damping="0.0" friction="100"/>-->
     </joint>
     <link name="${prefix}/wrist_palm_link" >
@@ -427,5 +456,5 @@
       <limit effort="15" lower="-0.9" upper="${PI}" velocity="0.20"/>
       <!-- <safety_controller k_position="100" k_velocity="3" soft_lower_limit="-100.0" soft_upper_limit="100.0" /> -->
-      <dynamics damping="1.0" friction="100.0"/>
+      <!--<dynamics damping="1.0" friction="100.0"/>-->
     </joint>
     <link name="${prefix}/stump_link" >

Commit message: updating wrist pitch limits

File: models/components.urdf.xacro (robot description, xacro)
@@ -273,5 +273,5 @@
       <origin xyz="0 0 0" rpy="${-PI/2} 0 0"/>
       <axis xyz="0 0 1"/>
-      <limit effort="5" lower="-1.45" upper="1.45" velocity="0.20"/><!-- 1.45 is a limit taken in from 1.5 due to saftey and differences between arms. -->
+      <limit effort="5" lower="-1.5707" upper="1.5707" velocity="0.20"/><!-- 1.45 is a limit taken in from 1.5 due to saftey and differences between arms. -->
       <!-- <safety_controller k_position="100" k_velocity="3" soft_lower_limit="-100.0" soft_upper_limit="100.0" /> -->
       <!--<dynamics damping="1.0" friction="100.0"/>-->

Commit message: Cleaning up robot urdfs

File: models/components.urdf.xacro (robot description, xacro)
@@ -75,5 +75,4 @@
       <axis xyz="0 0 1"/>
       <limit effort="60" lower="-2.6" upper="2.6" velocity="0.50"/>
-      <!--<dynamics damping="1.0" friction="100.0"/>-->
     </joint>
     <link name="${prefix}/shoulder_yaw_link" >
@@ -111,5 +110,4 @@
       <axis xyz="0 0 1"/>
       <limit effort="60" lower="-1.985" upper="1.985" velocity="0.5"/>
-      <!--<dynamics damping="1.0" friction="100.0"/>-->
     </joint>
     <link name="${prefix}/shoulder_pitch_link" >
@@ -147,5 +145,4 @@
       <axis xyz="0 0 1"/>
       <limit effort="45" lower="-2.8" upper="2.8" velocity="0.5"/>
-      <!--<dynamics damping="1.0" friction="100.0"/>-->
     </joint>
     <link name="${prefix}/upper_arm_link" >
@@ -184,6 +181,4 @@
       <axis xyz="0 0 1"/>
       <limit effort="20" lower="-0.9" upper="${PI}" velocity="0.20"/>
-      <!-- <safety_controller k_position="100" k_velocity="3" soft_lower_limit="-100.0" soft_upper_limit="100.0" /> -->
-      <!--<dynamics damping="1.0" friction="100.0"/>-->
     </joint>
     <link name="${prefix}/forearm_link" >
@@ -236,6 +231,4 @@
       <axis xyz="0 0 1"/>
       <limit effort="5" lower="-4.8" upper="1.3" velocity="0.20"/>
-      <!-- <safety_controller k_position="100" k_velocity="3" soft_lower_limit="-100.0" soft_upper_limit="100.0" /> -->
-      <!--<dynamics damping="1.0" friction="100.0"/>-->
     </joint>
     <link name="${prefix}/wrist_yaw_link" >
@@ -273,7 +266,5 @@
       <origin xyz="0 0 0" rpy="${-PI/2} 0 0"/>
       <axis xyz="0 0 1"/>
-      <limit effort="5" lower="-1.5707" upper="1.5707" velocity="0.20"/><!-- 1.45 is a limit taken in from 1.5 due to saftey and differences between arms. -->
-      <!-- <safety_controller k_position="100" k_velocity="3" soft_lower_limit="-100.0" soft_upper_limit="100.0" /> -->
-      <!--<dynamics damping="1.0" friction="100.0"/>-->
+      <limit effort="5" lower="-1.5707" upper="1.5707" velocity="0.20"/>
     </joint>
     <link name="${prefix}/wrist_pitch_link" >
@@ -312,6 +303,4 @@
       <axis xyz="0 0 1"/>
       <limit effort="5" lower="-2.95" upper="2.95" velocity="0.20"/><!-- 2.95 is a limit taken in from 3 due to saftey and differences between arms. -->
-      <!-- <safety_controller k_position="100" k_velocity="3" soft_lower_limit="-100.0" soft_upper_limit="100.0" /> -->
-      <!--<dynamics damping="0.0" friction="100"/>-->
     </joint>
     <link name="${prefix}/wrist_palm_link" >
@@ -455,6 +444,4 @@
       <axis xyz="0 0 1"/>
       <limit effort="15" lower="-0.9" upper="${PI}" velocity="0.20"/>
-      <!-- <safety_controller k_position="100" k_velocity="3" soft_lower_limit="-100.0" soft_upper_limit="100.0" /> -->
-      <!--<dynamics damping="1.0" friction="100.0"/>-->
     </joint>
     <link name="${prefix}/stump_link" >

File: robots/wam4_stump.urdf.xacro (robot description, xacro)
@@ -4,6 +4,8 @@
   <include filename="$(find barrett_model)/models/wam_top.urdf.xacro"/>
   <!-- Root link is in the world frame-->
-  <link name = "world"/>
-  <xacro:wam_7dof prefix="wam" parent_link="world" xyz="0.02 0.46 1" rpy="0 0 0" />
-  <!--xacro:barrett_hand prefix="wam_left" /-->
+  <link name="world"/>
+  <!-- 4-DOF Wam -->
+  <xacro:wam_4dof prefix="wam" parent_link="world" xyz="0.0 0.0 1" rpy="0 0 0" />
+  <!-- Hollow forearm (stump) -->
+  <xacro:wam_stump prefix="wam" />
 </robot>

File: robots/wam7.urdf.xacro (robot description, xacro)
@@ -4,5 +4,8 @@
   <include filename="$(find barrett_model)/models/wam_top.urdf.xacro"/>
   <!-- Root link is in the world frame-->
-  <link name = "world"/>
-  <xacro:wam_4dof prefix="wam" parent_link="world" xyz="0.02 0.46 1" rpy="0 0 0" />
+  <link name="world"/>
+  <!-- 7-DOF Wam -->
+  <xacro:wam_7dof prefix="wam" parent_link="world" xyz="0.0 0.0 1.0" rpy="0 0 0" />
+  <!-- BHand -->
+  <!--xacro:barrett_hand prefix="wam" /-->
 </robot>

Commit message: adding in damping that gazebo actually reads

File: models/components.urdf.xacro (robot description, xacro)
@@ -27,10 +27,13 @@
   <include filename="$(find barrett_model)/models/common.urdf.xacro"/>
   <xacro:macro name="gz_joint">
-      <physics>
-        <ode>
-          <cfm_damping>true</cfm_damping>
-          <cfm>0.0</cfm>
-        </ode>
-      </physics>
+    <!--<dynamics damping="0.5" friction="1"/>-->
+    <!--
+       -<physics>
+       -  <ode>
+       -    <cfm_damping>true</cfm_damping>
+       -    <cfm>10.0</cfm>
+       -  </ode>
+       -</physics>
+       -->
   </xacro:macro>
   <!-- Upper arm macros -->
@@ -66,7 +69,4 @@
   </xacro:macro>
   <xacro:macro name="wam_shoulder_yaw" params="prefix">
-    <gazebo reference="${prefix}/base_yaw_joint">
-      <xacro:gz_joint/>
-    </gazebo>
     <joint name="${prefix}/base_yaw_joint" type="revolute">
       <parent link="${prefix}/base_link"/>
@@ -75,5 +75,9 @@
       <axis xyz="0 0 1"/>
       <limit effort="60" lower="-2.6" upper="2.6" velocity="0.50"/>
-    </joint>
+      <dynamics damping="0.5" friction="1"/>
+    </joint>
+    <gazebo reference="${prefix}/base_yaw_joint">
+      <xacro:gz_joint/>
+    </gazebo>
     <link name="${prefix}/shoulder_yaw_link" >
       <inertial>
@@ -101,7 +105,4 @@
   </xacro:macro>
   <xacro:macro name="wam_shoulder_pitch" params="prefix">
-    <gazebo reference="${prefix}/shoulder_pitch_joint">
-      <xacro:gz_joint/>
-    </gazebo>
     <joint name="${prefix}/shoulder_pitch_joint" type="revolute">
       <parent link="${prefix}/shoulder_yaw_link"/>
@@ -110,5 +111,9 @@
       <axis xyz="0 0 1"/>
       <limit effort="60" lower="-1.985" upper="1.985" velocity="0.5"/>
-    </joint>
+      <dynamics damping="0.5" friction="1"/>
+    </joint>
+    <gazebo reference="${prefix}/shoulder_pitch_joint">
+      <xacro:gz_joint/>
+    </gazebo>
     <link name="${prefix}/shoulder_pitch_link" >
       <visual>
@@ -136,7 +141,4 @@
   </xacro:macro>
   <xacro:macro name="wam_upper_arm" params="prefix">
-    <gazebo reference="${prefix}/shoulder_yaw_joint">
-      <xacro:gz_joint/>
-    </gazebo>
     <joint name="${prefix}/shoulder_yaw_joint" type="revolute">
       <parent link="${prefix}/shoulder_pitch_link"/>
@@ -145,5 +147,9 @@
       <axis xyz="0 0 1"/>
       <limit effort="45" lower="-2.8" upper="2.8" velocity="0.5"/>
-    </joint>
+      <dynamics damping="0.5" friction="1"/>
+    </joint>
+    <gazebo reference="${prefix}/shoulder_yaw_joint">
+      <xacro:gz_joint/>
+    </gazebo>
     <link name="${prefix}/upper_arm_link" >
       <inertial>
@@ -172,7 +178,4 @@
   <!-- Forearm macros -->
   <xacro:macro name="wam_forearm" params="prefix">
-    <gazebo reference="${prefix}/elbow_pitch_joint">
-      <xacro:gz_joint/>
-    </gazebo>
     <joint name="${prefix}/elbow_pitch_joint" type="revolute">
       <parent link="${prefix}/upper_arm_link"/>
@@ -181,5 +184,9 @@
       <axis xyz="0 0 1"/>
       <limit effort="20" lower="-0.9" upper="${PI}" velocity="0.20"/>
-    </joint>
+      <dynamics damping="0.5" friction="1"/>
+    </joint>
+    <gazebo reference="${prefix}/elbow_pitch_joint">
+      <xacro:gz_joint/>
+    </gazebo>
     <link name="${prefix}/forearm_link" >
       <inertial>
@@ -222,7 +229,4 @@
   </xacro:macro>
   <xacro:macro name="wam_wrist_yaw" params="prefix">
-    <gazebo reference="${prefix}/wrist_yaw_joint">
-      <xacro:gz_joint/>
-    </gazebo>
     <joint name="${prefix}/wrist_yaw_joint" type="revolute">
       <parent link="${prefix}/forearm_link"/>
@@ -231,5 +235,9 @@
       <axis xyz="0 0 1"/>
       <limit effort="5" lower="-4.8" upper="1.3" velocity="0.20"/>
-    </joint>
+      <dynamics damping="0.5" friction="1"/>
+    </joint>
+    <gazebo reference="${prefix}/wrist_yaw_joint">
+      <xacro:gz_joint/>
+    </gazebo>
     <link name="${prefix}/wrist_yaw_link" >
       <inertial>
@@ -258,7 +266,4 @@
   </xacro:macro>
   <xacro:macro name="wam_wrist_pitch" params="prefix">
-    <gazebo reference="${prefix}/wrist_pitch_joint">
-      <xacro:gz_joint/>
-    </gazebo>
     <joint name="${prefix}/wrist_pitch_joint" type="revolute">
       <parent link="${prefix}/wrist_yaw_link"/>
@@ -267,5 +272,9 @@
       <axis xyz="0 0 1"/>
       <limit effort="5" lower="-1.5707" upper="1.5707" velocity="0.20"/>
-    </joint>
+      <dynamics damping="0.5" friction="1"/>
+    </joint>
+    <gazebo reference="${prefix}/wrist_pitch_joint">
+      <xacro:gz_joint/>
+    </gazebo>
     <link name="${prefix}/wrist_pitch_link" >
       <inertial>
@@ -294,7 +303,4 @@
   <!-- Palm without force-torque sensor -->
   <xacro:macro name="wam_palm" params="prefix">
-    <gazebo reference="${prefix}/palm_yaw_joint">
-      <xacro:gz_joint/>
-    </gazebo>
     <joint name="${prefix}/palm_yaw_joint" type="revolute">
       <parent link="${prefix}/wrist_pitch_link"/>
@@ -303,5 +309,9 @@
       <axis xyz="0 0 1"/>
       <limit effort="5" lower="-2.95" upper="2.95" velocity="0.20"/><!-- 2.95 is a limit taken in from 3 due to saftey and differences between arms. -->
-    </joint>
+      <dynamics damping="0.5" friction="1"/>
+    </joint>
+    <gazebo reference="${prefix}/palm_yaw_joint">
+      <xacro:gz_joint/>
+    </gazebo>
     <link name="${prefix}/wrist_palm_link" >
       <inertial>
@@ -444,4 +454,5 @@
       <axis xyz="0 0 1"/>
       <limit effort="15" lower="-0.9" upper="${PI}" velocity="0.20"/>
+      <dynamics damping="0.5" friction="1"/>
     </joint>
     <link name="${prefix}/stump_link" >

Commit message: Adding better damping characterization

File: models/components.urdf.xacro (robot description, xacro)
@@ -26,6 +26,9 @@
   <xacro:include filename="$(find barrett_model)/models/hand.urdf.xacro"/>
   <xacro:include filename="$(find barrett_model)/models/common.urdf.xacro"/>
+  <!-- Gazebo joint configuration -->
   <xacro:macro name="gz_joint">
-    <!--<dynamics damping="0.5" friction="1"/>-->
+    <provideFeedback>true</provideFeedback>
+    <cfmDamping>true</cfmDamping>
+    <!--<dynamics damping="5.5" friction="1"/>-->
     <!--
        -<physics>
@@ -75,5 +78,5 @@
       <axis xyz="0 0 1"/>
       <limit effort="60" lower="-2.6" upper="2.6" velocity="0.50"/>
-      <dynamics damping="0.5" friction="1"/>
+      <dynamics damping="5.5" friction="1"/>
     </joint>
     <gazebo reference="${prefix}/base_yaw_joint">
@@ -111,5 +114,5 @@
       <axis xyz="0 0 1"/>
       <limit effort="60" lower="-1.985" upper="1.985" velocity="0.5"/>
-      <dynamics damping="0.5" friction="1"/>
+      <dynamics damping="5.5" friction="1"/>
     </joint>
     <gazebo reference="${prefix}/shoulder_pitch_joint">
@@ -147,5 +150,5 @@
       <axis xyz="0 0 1"/>
       <limit effort="45" lower="-2.8" upper="2.8" velocity="0.5"/>
-      <dynamics damping="0.5" friction="1"/>
+      <dynamics damping="5.5" friction="1"/>
     </joint>
     <gazebo reference="${prefix}/shoulder_yaw_joint">
@@ -184,5 +187,5 @@
       <axis xyz="0 0 1"/>
       <limit effort="20" lower="-0.9" upper="${PI}" velocity="0.20"/>
-      <dynamics damping="0.5" friction="1"/>
+      <dynamics damping="5.5" friction="1"/>
     </joint>
     <gazebo reference="${prefix}/elbow_pitch_joint">
@@ -454,5 +457,5 @@
       <axis xyz="0 0 1"/>
       <limit effort="15" lower="-0.9" upper="${PI}" velocity="0.20"/>
-      <dynamics damping="0.5" friction="1"/>
+      <dynamics damping="5.5" friction="1"/>
     </joint>
     <link name="${prefix}/stump_link" >
