Commit message: fixing velocity limits which were messing up high-performance motions in gazebo

File: models/components.urdf.xacro (robot description, xacro)
@@ -63,6 +63,6 @@
       <origin xyz="0 0 0.346" rpy="0 0 0"/>
       <axis xyz="0 0 1"/>
-      <limit effort="60" lower="-2.6" upper="2.6" velocity="0.50"/>
-      <dynamics damping="5.5" friction="1"/>
+      <limit effort="60" lower="-2.6" upper="2.6" velocity="1.0"/>
+      <dynamics damping="1.1" friction="0"/>
     </joint>
     <gazebo reference="${prefix}/base_yaw_joint">
@@ -99,6 +99,6 @@
       <origin xyz="0 0 0" rpy="${-PI/2} 0 0"/>
       <axis xyz="0 0 1"/>
-      <limit effort="60" lower="-1.985" upper="1.985" velocity="0.5"/>
-      <dynamics damping="5.5" friction="1"/>
+      <limit effort="60" lower="-1.985" upper="1.985" velocity="1.0"/>
+      <dynamics damping="1.1" friction="0"/>
     </joint>
     <gazebo reference="${prefix}/shoulder_pitch_joint">
@@ -135,6 +135,6 @@
       <origin xyz="0 0 0" rpy="${PI/2} 0 0"/>
       <axis xyz="0 0 1"/>
-      <limit effort="45" lower="-2.8" upper="2.8" velocity="0.5"/>
-      <dynamics damping="5.5" friction="1"/>
+      <limit effort="45" lower="-2.8" upper="2.8" velocity="1.0"/>
+      <dynamics damping="1.1" friction="0"/>
     </joint>
     <gazebo reference="${prefix}/shoulder_yaw_joint">
@@ -172,6 +172,6 @@
       <origin xyz="0.045 0 0.55" rpy="${-PI/2} 0 0"/>
       <axis xyz="0 0 1"/>
-      <limit effort="20" lower="-0.9" upper="${PI}" velocity="0.20"/>
-      <dynamics damping="5.5" friction="1"/>
+      <limit effort="30" lower="-0.9" upper="${PI}" velocity="1.00"/>
+      <dynamics damping="1.1" friction="0"/>
     </joint>
     <gazebo reference="${prefix}/elbow_pitch_joint">
@@ -223,6 +223,6 @@
       <origin xyz="-0.045 -0.3 0" rpy="${PI/2} 0 0"/>
       <axis xyz="0 0 1"/>
-      <limit effort="5" lower="-4.8" upper="1.3" velocity="0.20"/>
-      <dynamics damping="0.5" friction="1"/>
+      <limit effort="5" lower="-4.8" upper="1.3" velocity="1.0"/>
+      <dynamics damping="1.1" friction="0"/>
     </joint>
     <gazebo reference="${prefix}/wrist_yaw_joint">
@@ -260,6 +260,6 @@
       <origin xyz="0 0 0" rpy="${-PI/2} 0 0"/>
       <axis xyz="0 0 1"/>
-      <limit effort="5" lower="-1.5707" upper="1.5707" velocity="0.20"/>
-      <dynamics damping="0.5" friction="1"/>
+      <limit effort="5" lower="-1.5707" upper="1.5707" velocity="1.00"/>
+      <dynamics damping="1.1" friction="0"/>
     </joint>
     <gazebo reference="${prefix}/wrist_pitch_joint">
@@ -297,6 +297,6 @@
       <origin xyz="0 0 0" rpy="${PI/2} 0 0"/>
       <axis xyz="0 0 1"/>
-      <limit effort="5" lower="-2.95" upper="2.95" velocity="0.20"/><!-- 2.95 is a limit taken in from 3 due to saftey and differences between arms. -->
-      <dynamics damping="0.5" friction="1"/>
+      <limit effort="5" lower="-2.95" upper="2.95" velocity="1.00"/><!-- 2.95 is a limit taken in from 3 due to saftey and differences between arms. -->
+      <dynamics damping="1.1" friction="0"/>
     </joint>
     <gazebo reference="${prefix}/palm_yaw_joint">
@@ -442,6 +442,6 @@
       <origin xyz="0.045 0 0.55" rpy="${-PI/2} 0 0"/>
       <axis xyz="0 0 1"/>
-      <limit effort="15" lower="-0.9" upper="${PI}" velocity="0.20"/>
-      <dynamics damping="5.5" friction="1"/>
+      <limit effort="15" lower="-0.9" upper="${PI}" velocity="1.00"/>
+      <dynamics damping="1.1" friction="0"/>
     </joint>
     <link name="${prefix}/stump_link" >

File: models/hand.urdf.xacro (robot description, xacro)
@@ -23,4 +23,9 @@
     <xacro:bhand_finger_dist prefix="${prefix}/finger_3"/>
   </xacro:macro>
+  <xacro:macro name="gz_hand_link">
+    <mu1>0.8</mu1>
+    <mu2>0.8</mu2>
+    <selfCollide>true</selfCollide>
+  </xacro:macro>
   <!-- Components -->
   <xacro:macro name="bhand_palm" params="prefix parent_link xyz rpy">
@@ -30,4 +35,7 @@
       <origin xyz="${xyz}" rpy="${rpy}"/>
     </joint>
+    <gazebo reference="${prefix}/bhand_palm_link">
+      <xacro:gz_hand_link/>
+    </gazebo>
     <link name="${prefix}/bhand_palm_link">
       <inertial>
@@ -60,9 +68,12 @@
       <origin xyz="${xyz}" rpy="${rpy}"/>
       <axis xyz="${axis}"/>
-      <limit effort="5" lower="0" upper="${PI}" velocity="0.20"/>
+      <limit effort="5" lower="0" upper="${PI}" velocity="2.0"/>
       <dynamics damping="1.5" friction="1"/>
     </joint>
     <gazebo reference="${prefix}/prox_joint">
       <xacro:gz_joint/>
+    </gazebo>
+    <gazebo reference="${prefix}/prox_link">
+      <xacro:gz_hand_link/>
     </gazebo>
     <link name="${prefix}/prox_link">
@@ -96,9 +107,12 @@
       <origin xyz="${xyz}" rpy="${rpy}"/>
       <axis xyz="0 0 1"/>
-      <limit effort="5" lower="0" upper="${140/180*PI}" velocity="0.20"/>
+      <limit effort="5" lower="0" upper="${140/180*PI}" velocity="2.00"/>
       <dynamics damping="1.5" friction="1"/>
     </joint>
     <gazebo reference="${prefix}/med_joint">
       <xacro:gz_joint/>
+    </gazebo>
+    <gazebo reference="${prefix}/med_link">
+      <xacro:gz_hand_link/>
     </gazebo>
     <link name="${prefix}/med_link">
@@ -132,9 +146,12 @@
       <origin xyz="0.06994 0.003 0.0" rpy="0 0 0"/>
       <axis xyz="0 0 1"/>
-      <limit effort="5" lower="0" upper="${48/180*PI}" velocity="0.20"/>
+      <limit effort="5" lower="0" upper="${48/180*PI}" velocity="2.00"/>
       <dynamics damping="1.5" friction="1"/>
     </joint>
     <gazebo reference="${prefix}/dist_joint">
       <xacro:gz_joint/>
+    </gazebo>
+    <gazebo reference="${prefix}/dist_link">
+      <xacro:gz_hand_link/>
     </gazebo>
     <link name="${prefix}/dist_link">

Commit message: Tweaking limits

File: models/components.urdf.xacro (robot description, xacro)
@@ -63,5 +63,5 @@
       <origin xyz="0 0 0.346" rpy="0 0 0"/>
       <axis xyz="0 0 1"/>
-      <limit effort="60" lower="-2.6" upper="2.6" velocity="1.0"/>
+      <limit effort="60" lower="-2.6" upper="2.6" velocity="2.0"/>
       <dynamics damping="1.1" friction="0"/>
     </joint>
@@ -99,5 +99,5 @@
       <origin xyz="0 0 0" rpy="${-PI/2} 0 0"/>
       <axis xyz="0 0 1"/>
-      <limit effort="60" lower="-1.985" upper="1.985" velocity="1.0"/>
+      <limit effort="60" lower="-1.985" upper="1.985" velocity="2.0"/>
       <dynamics damping="1.1" friction="0"/>
     </joint>
@@ -135,5 +135,5 @@
       <origin xyz="0 0 0" rpy="${PI/2} 0 0"/>
       <axis xyz="0 0 1"/>
-      <limit effort="45" lower="-2.8" upper="2.8" velocity="1.0"/>
+      <limit effort="45" lower="-2.8" upper="2.8" velocity="2.0"/>
       <dynamics damping="1.1" friction="0"/>
     </joint>
@@ -172,5 +172,5 @@
       <origin xyz="0.045 0 0.55" rpy="${-PI/2} 0 0"/>
       <axis xyz="0 0 1"/>
-      <limit effort="30" lower="-0.9" upper="${PI}" velocity="1.00"/>
+      <limit effort="30" lower="-0.9" upper="${PI}" velocity="2.00"/>
       <dynamics damping="1.1" friction="0"/>
     </joint>
@@ -223,5 +223,5 @@
       <origin xyz="-0.045 -0.3 0" rpy="${PI/2} 0 0"/>
       <axis xyz="0 0 1"/>
-      <limit effort="5" lower="-4.8" upper="1.3" velocity="1.0"/>
+      <limit effort="6" lower="-4.8" upper="1.3" velocity="2.0"/>
       <dynamics damping="1.1" friction="0"/>
     </joint>
@@ -260,5 +260,5 @@
       <origin xyz="0 0 0" rpy="${-PI/2} 0 0"/>
       <axis xyz="0 0 1"/>
-      <limit effort="5" lower="-1.5707" upper="1.5707" velocity="1.00"/>
+      <limit effort="6" lower="-1.5707" upper="1.5707" velocity="2.00"/>
       <dynamics damping="1.1" friction="0"/>
     </joint>
@@ -297,5 +297,5 @@
       <origin xyz="0 0 0" rpy="${PI/2} 0 0"/>
       <axis xyz="0 0 1"/>
-      <limit effort="5" lower="-2.95" upper="2.95" velocity="1.00"/><!-- 2.95 is a limit taken in from 3 due to saftey and differences between arms. -->
+      <limit effort="6" lower="-2.95" upper="2.95" velocity="2.00"/><!-- 2.95 is a limit taken in from 3 due to saftey and differences between arms. -->
       <dynamics damping="1.1" friction="0"/>
     </joint>
@@ -442,5 +442,5 @@
       <origin xyz="0.045 0 0.55" rpy="${-PI/2} 0 0"/>
       <axis xyz="0 0 1"/>
-      <limit effort="15" lower="-0.9" upper="${PI}" velocity="1.00"/>
+      <limit effort="15" lower="-0.9" upper="${PI}" velocity="2.0"/>
       <dynamics damping="1.1" friction="0"/>
     </joint>

File: models/hand.urdf.xacro (robot description, xacro)
@@ -68,5 +68,5 @@
       <origin xyz="${xyz}" rpy="${rpy}"/>
       <axis xyz="${axis}"/>
-      <limit effort="5" lower="0" upper="${PI}" velocity="2.0"/>
+      <limit effort="5" lower="0" upper="${PI}" velocity="5.0"/>
       <dynamics damping="1.5" friction="1"/>
     </joint>
@@ -107,5 +107,5 @@
       <origin xyz="${xyz}" rpy="${rpy}"/>
       <axis xyz="0 0 1"/>
-      <limit effort="5" lower="0" upper="${140/180*PI}" velocity="2.00"/>
+      <limit effort="5" lower="0" upper="${140/180*PI}" velocity="5.00"/>
       <dynamics damping="1.5" friction="1"/>
     </joint>
@@ -146,5 +146,5 @@
       <origin xyz="0.06994 0.003 0.0" rpy="0 0 0"/>
       <axis xyz="0 0 1"/>
-      <limit effort="5" lower="0" upper="${48/180*PI}" velocity="2.00"/>
+      <limit effort="5" lower="0" upper="${48/180*PI}" velocity="5.00"/>
       <dynamics damping="1.5" friction="1"/>
     </joint>

Commit message: adding realistic velocity limits, damping

File: models/components.urdf.xacro (robot description, xacro)
@@ -64,5 +64,5 @@
       <axis xyz="0 0 1"/>
       <limit effort="60" lower="-2.6" upper="2.6" velocity="2.0"/>
-      <dynamics damping="1.1" friction="0"/>
+      <dynamics damping="2.0" friction="0"/>
     </joint>
     <gazebo reference="${prefix}/base_yaw_joint">
@@ -100,5 +100,5 @@
       <axis xyz="0 0 1"/>
       <limit effort="60" lower="-1.985" upper="1.985" velocity="2.0"/>
-      <dynamics damping="1.1" friction="0"/>
+      <dynamics damping="2.0" friction="0"/>
     </joint>
     <gazebo reference="${prefix}/shoulder_pitch_joint">
@@ -136,5 +136,5 @@
       <axis xyz="0 0 1"/>
       <limit effort="45" lower="-2.8" upper="2.8" velocity="2.0"/>
-      <dynamics damping="1.1" friction="0"/>
+      <dynamics damping="2.0" friction="0"/>
     </joint>
     <gazebo reference="${prefix}/shoulder_yaw_joint">
@@ -173,5 +173,5 @@
       <axis xyz="0 0 1"/>
       <limit effort="30" lower="-0.9" upper="${PI}" velocity="2.00"/>
-      <dynamics damping="1.1" friction="0"/>
+      <dynamics damping="1.5" friction="0"/>
     </joint>
     <gazebo reference="${prefix}/elbow_pitch_joint">

Commit message: adding simplified collision geometry

File: models/components.urdf.xacro (robot description, xacro)
@@ -47,10 +47,10 @@
         </material>
         <geometry>
-          <mesh filename="${models_path}/sw_meshes/base_link_fine.STL"/>
-        </geometry>
-      </visual>
-      <collision>
-        <geometry>
-          <mesh filename="${models_path}/sw_meshes/base_link.STL"/>
+          <mesh filename="${models_path}/sw_meshes/base_link_fine.stl"/>
+        </geometry>
+      </visual>
+      <collision>
+        <geometry>
+          <mesh filename="${models_path}/sw_meshes/base_link_convex.stl"/>
         </geometry>
       </collision>
@@ -83,10 +83,10 @@
         </material>
         <geometry>
-          <mesh filename="${models_path}/sw_meshes/shoulder_link_fine.STL"/>
-        </geometry>
-      </visual>
-      <collision>
-        <geometry>
-          <mesh filename="${models_path}/sw_meshes/shoulder_link.STL"/>
+          <mesh filename="${models_path}/sw_meshes/shoulder_link_fine.stl"/>
+        </geometry>
+      </visual>
+      <collision>
+        <geometry>
+          <mesh filename="${models_path}/sw_meshes/shoulder_link_convex_decomposition.dae"/>
         </geometry>
       </collision>
@@ -111,5 +111,5 @@
         </material>
         <geometry>
-          <mesh filename="${models_path}/sw_meshes/shoulder_pitch_link_fine.STL"/>
+          <mesh filename="${models_path}/sw_meshes/shoulder_pitch_link_fine.stl"/>
         </geometry>
       </visual>
@@ -124,5 +124,5 @@
       <collision>
         <geometry>
-          <mesh filename="${models_path}/sw_meshes/shoulder_pitch_link.STL"/>
+          <mesh filename="${models_path}/sw_meshes/shoulder_pitch_link_convex.stl"/>
         </geometry>
       </collision>
@@ -155,10 +155,10 @@
         </material>
         <geometry>
-          <mesh filename="${models_path}/sw_meshes/upper_arm_link_fine.STL"/>
-        </geometry>
-      </visual>
-      <collision>
-        <geometry>
-          <mesh filename="${models_path}/sw_meshes/upper_arm_link.STL"/>
+          <mesh filename="${models_path}/sw_meshes/upper_arm_link_fine.stl"/>
+        </geometry>
+      </visual>
+      <collision>
+        <geometry>
+          <mesh filename="${models_path}/sw_meshes/upper_arm_link_convex_decomposition.dae"/>
         </geometry>
       </collision>
@@ -192,10 +192,10 @@
         </material>
         <geometry>
-          <mesh filename="${models_path}/sw_meshes/elbow_link_fine.STL"/>
-        </geometry>
-      </visual>
-      <collision>
-        <geometry>
-          <mesh filename="${models_path}/sw_meshes/elbow_link.STL"/>
+          <mesh filename="${models_path}/sw_meshes/elbow_link_fine.stl"/>
+        </geometry>
+      </visual>
+      <collision>
+        <geometry>
+          <mesh filename="${models_path}/sw_meshes/elbow_link_convex.stl"/>
         </geometry>
       </collision>
@@ -206,5 +206,5 @@
         <origin xyz="-0.045 -0.0730 0" rpy="${PI/2} 0 0" />
         <geometry>
-          <mesh filename="${models_path}/sw_meshes/forearm_link_fine.STL"/>
+          <mesh filename="${models_path}/sw_meshes/forearm_link_fine.stl"/>
         </geometry>
       </visual>
@@ -212,5 +212,5 @@
         <origin xyz="-0.045 -0.0730 0" rpy="${PI/2} 0 0" />
         <geometry>
-          <mesh filename="${models_path}/sw_meshes/forearm_link.STL"/>
+          <mesh filename="${models_path}/sw_meshes/forearm_link_convex_decomposition.dae"/>
         </geometry>
       </collision>
@@ -243,5 +243,5 @@
         <origin xyz="0 0 0" rpy="0 0 0" />
         <geometry>
-          <mesh filename="${models_path}/sw_meshes/wrist_yaw_link_fine.STL"/>
+          <mesh filename="${models_path}/sw_meshes/wrist_yaw_link_fine.stl"/>
         </geometry>
       </visual>
@@ -249,5 +249,5 @@
         <origin xyz="0 0 0" rpy="0 0 0" />
         <geometry>
-          <mesh filename="${models_path}/sw_meshes/wrist_yaw_link.STL"/>
+          <mesh filename="${models_path}/sw_meshes/wrist_yaw_link_convex_decomposition.dae"/>
         </geometry>
       </collision>
@@ -280,10 +280,10 @@
         </material>
         <geometry>
-          <mesh filename="${models_path}/sw_meshes/wrist_pitch_link_fine.STL"/>
-        </geometry>
-      </visual>
-      <collision>
-        <geometry>
-          <mesh filename="${models_path}/sw_meshes/wrist_pitch_link.STL"/>
+          <mesh filename="${models_path}/sw_meshes/wrist_pitch_link_fine.stl"/>
+        </geometry>
+      </visual>
+      <collision>
+        <geometry>
+          <mesh filename="${models_path}/sw_meshes/wrist_pitch_link_convex_decomposition.dae"/>
         </geometry>
       </collision>
@@ -317,5 +317,5 @@
         <origin xyz="0 0 0" rpy="0 0 0" />
         <geometry>
-          <mesh filename="${models_path}/sw_meshes/wrist_palm_link_fine.STL"/>
+          <mesh filename="${models_path}/sw_meshes/wrist_palm_link_fine.stl"/>
         </geometry>
       </visual>
@@ -323,5 +323,5 @@
         <origin xyz="0 0 0" rpy="0 0 0" />
         <geometry>
-          <mesh filename="${models_path}/sw_meshes/wrist_palm_link.STL"/>
+          <mesh filename="${models_path}/sw_meshes/wrist_palm_link.stl"/>
         </geometry>
       </collision>
@@ -459,10 +459,10 @@
         </material>
         <geometry>
-          <mesh filename="${models_path}/sw_meshes/elbow_link_fine.STL"/>
-        </geometry>
-      </visual>
-      <collision>
-        <geometry>
-          <mesh filename="${models_path}/sw_meshes/elbow_link.STL"/>
+          <mesh filename="${models_path}/sw_meshes/elbow_link_fine.stl"/>
+        </geometry>
+      </visual>
+      <collision>
+        <geometry>
+          <mesh filename="${models_path}/sw_meshes/elbow_link.stl"/>
         </geometry>
       </collision>

File: models/hand.urdf.xacro (robot description, xacro)
@@ -52,10 +52,10 @@
         </material>
         <geometry>
-          <mesh filename="${models_path}/sw_meshes/bhand/bhand_palm_fine.STL"/>
+          <mesh filename="${models_path}/sw_meshes/bhand/bhand_palm_fine.stl"/>
         </geometry>
       </visual>
       <collision>
         <geometry>
-          <mesh filename="${models_path}/sw_meshes/bhand/bhand_palm.STL"/>
+          <mesh filename="${models_path}/sw_meshes/bhand/bhand_palm_link_convex_decomposition.dae"/>
         </geometry>
       </collision>
@@ -91,10 +91,10 @@
         </material>
         <geometry>
-          <mesh filename="${models_path}/sw_meshes/bhand/bhand_finger_prox_link_fine.STL"/>
+          <mesh filename="${models_path}/sw_meshes/bhand/bhand_finger_prox_link_fine.stl"/>
         </geometry>
       </visual>
       <collision>
         <geometry>
-          <mesh filename="${models_path}/sw_meshes/bhand/bhand_finger_prox_link.STL"/>
+          <mesh filename="${models_path}/sw_meshes/bhand/bhand_finger_prox_link_convex_decomposition.dae"/>
         </geometry>
       </collision>
@@ -130,10 +130,10 @@
         </material>
         <geometry>
-          <mesh filename="${models_path}/sw_meshes/bhand/bhand_finger_med_link_fine.STL"/>
+          <mesh filename="${models_path}/sw_meshes/bhand/bhand_finger_med_link_fine.stl"/>
         </geometry>
       </visual>
       <collision>
         <geometry>
-          <mesh filename="${models_path}/sw_meshes/bhand/bhand_finger_med_link.STL"/>
+          <mesh filename="${models_path}/sw_meshes/bhand/bhand_finger_med_link_convex.stl"/>
         </geometry>
       </collision>
@@ -169,10 +169,10 @@
         </material>
         <geometry>
-          <mesh filename="${models_path}/sw_meshes/bhand/bhand_finger_dist_link_fine.STL"/>
+          <mesh filename="${models_path}/sw_meshes/bhand/bhand_finger_dist_link_fine.stl"/>
         </geometry>
       </visual>
       <collision>
         <geometry>
-          <mesh filename="${models_path}/sw_meshes/bhand/bhand_finger_dist_link.STL"/>
+          <mesh filename="${models_path}/sw_meshes/bhand/bhand_finger_dist_link_convex.stl"/>
         </geometry>
       </collision>

Commit message: decreasing damping

File: models/components.urdf.xacro (robot description, xacro)
@@ -224,5 +224,5 @@
       <axis xyz="0 0 1"/>
       <limit effort="6" lower="-4.8" upper="1.3" velocity="2.0"/>
-      <dynamics damping="1.1" friction="0"/>
+      <dynamics damping="0.5" friction="0"/>
     </joint>
     <gazebo reference="${prefix}/wrist_yaw_joint">
@@ -261,5 +261,5 @@
       <axis xyz="0 0 1"/>
       <limit effort="6" lower="-1.5707" upper="1.5707" velocity="2.00"/>
-      <dynamics damping="1.1" friction="0"/>
+      <dynamics damping="0.5" friction="0"/>
     </joint>
     <gazebo reference="${prefix}/wrist_pitch_joint">
@@ -298,5 +298,5 @@
       <axis xyz="0 0 1"/>
       <limit effort="6" lower="-2.95" upper="2.95" velocity="2.00"/><!-- 2.95 is a limit taken in from 3 due to saftey and differences between arms. -->
-      <dynamics damping="1.1" friction="0"/>
+      <dynamics damping="0.5" friction="0"/>
     </joint>
     <gazebo reference="${prefix}/palm_yaw_joint">

Commit message: fixing palm link, forearm, and upper arm inertia (palm link was in the wrong place)

File: models/components.urdf.xacro (robot description, xacro)
@@ -143,6 +143,6 @@
     <link name="${prefix}/upper_arm_link" >
       <inertial>
-        <origin xyz="0.00683258580000000 0.000033090000000 0.342492300000000" />
-        <mass value="1.80228141" />
+        <origin xyz="0.00683258580000000 0.000033090000000 0.392492300000000" />
+        <mass value="2.20228141" />
         <inertia
           ixx=".05911077"  ixy="-0.00000738"  ixz="-0.00249612"
@@ -180,6 +180,6 @@
     <link name="${prefix}/forearm_link" >
       <inertial>
-        <mass value="1.00016804" />
-        <origin xyz="-0.04001488 -.12271662 -.00022942 " rpy="0 0 0" />
+        <mass value="0.50016804" />
+        <origin xyz="-0.04001488 -.14271662 -.00022942 " rpy="0 0 0" />
         <inertia
           ixx="0.01491672" ixy="0.001506040000000" ixz="0.000017410000000"
@@ -232,5 +232,5 @@
       <inertial>
         <origin xyz="0.00008921 0.00435824 -0.00511217 " />
-        <mass value="1.12376019" />
+        <mass value="1.05376019" />
         <inertia  ixx="0.00005029" ixy="0.00000020"  ixz="0.00007582"
           iyy="0.00007582"  iyz="-0.00000359"
@@ -305,5 +305,5 @@
     <link name="${prefix}/wrist_palm_link" >
       <inertial>
-        <origin xyz="0.0 0.0 0.0" rpy="0 0 0" />
+        <origin xyz="0.0 0.0 0.055" rpy="0 0 0" />
         <mass value="0.08286134" />
         <inertia  ixx="0.00010859" ixy="0.00000000"  ixz="-0.00000000"

Commit message: more realistic damping

File: models/components.urdf.xacro (robot description, xacro)
@@ -64,5 +64,5 @@
       <axis xyz="0 0 1"/>
       <limit effort="60" lower="-2.6" upper="2.6" velocity="2.0"/>
-      <dynamics damping="2.0" friction="0"/>
+      <dynamics damping="0.5" friction="0"/>
     </joint>
     <gazebo reference="${prefix}/base_yaw_joint">
@@ -100,5 +100,5 @@
       <axis xyz="0 0 1"/>
       <limit effort="60" lower="-1.985" upper="1.985" velocity="2.0"/>
-      <dynamics damping="2.0" friction="0"/>
+      <dynamics damping="0.5" friction="0"/>
     </joint>
     <gazebo reference="${prefix}/shoulder_pitch_joint">
@@ -136,5 +136,5 @@
       <axis xyz="0 0 1"/>
       <limit effort="45" lower="-2.8" upper="2.8" velocity="2.0"/>
-      <dynamics damping="2.0" friction="0"/>
+      <dynamics damping="0.5" friction="0"/>
     </joint>
     <gazebo reference="${prefix}/shoulder_yaw_joint">
@@ -173,5 +173,5 @@
       <axis xyz="0 0 1"/>
       <limit effort="30" lower="-0.9" upper="${PI}" velocity="2.00"/>
-      <dynamics damping="1.5" friction="0"/>
+      <dynamics damping="0.5" friction="0"/>
     </joint>
     <gazebo reference="${prefix}/elbow_pitch_joint">
@@ -298,5 +298,5 @@
       <axis xyz="0 0 1"/>
       <limit effort="6" lower="-2.95" upper="2.95" velocity="2.00"/><!-- 2.95 is a limit taken in from 3 due to saftey and differences between arms. -->
-      <dynamics damping="0.5" friction="0"/>
+      <dynamics damping="0.2" friction="0"/>
     </joint>
     <gazebo reference="${prefix}/palm_yaw_joint">
@@ -443,5 +443,5 @@
       <axis xyz="0 0 1"/>
       <limit effort="15" lower="-0.9" upper="${PI}" velocity="2.0"/>
-      <dynamics damping="1.1" friction="0"/>
+      <dynamics damping="0.5" friction="0"/>
     </joint>
     <link name="${prefix}/stump_link" >
