Commit message: fixing joint limits

File: models/components.urdf.xacro (robot description, xacro)
@@ -223,5 +223,5 @@
       <origin xyz="-0.045 -0.3 0" rpy="${PI/2} 0 0"/>
       <axis xyz="0 0 1"/>
-      <limit effort="6" lower="-4.8" upper="1.3" velocity="2.0"/>
+      <limit effort="6" lower="-4.55" upper="1.25" velocity="2.0"/>
       <dynamics damping="0.5" friction="0"/>
     </joint>

Commit message: increasing damping for simulation stability

File: models/components.urdf.xacro (robot description, xacro)
@@ -64,5 +64,5 @@
       <axis xyz="0 0 1"/>
       <limit effort="60" lower="-2.6" upper="2.6" velocity="2.0"/>
-      <dynamics damping="0.5" friction="0"/>
+      <dynamics damping="15.0" friction="0"/>
     </joint>
     <gazebo reference="${prefix}/base_yaw_joint">
@@ -100,5 +100,5 @@
       <axis xyz="0 0 1"/>
       <limit effort="60" lower="-1.985" upper="1.985" velocity="2.0"/>
-      <dynamics damping="0.5" friction="0"/>
+      <dynamics damping="15.0" friction="0"/>
     </joint>
     <gazebo reference="${prefix}/shoulder_pitch_joint">
@@ -136,5 +136,5 @@
       <axis xyz="0 0 1"/>
       <limit effort="45" lower="-2.8" upper="2.8" velocity="2.0"/>
-      <dynamics damping="0.5" friction="0"/>
+      <dynamics damping="15.0" friction="0"/>
     </joint>
     <gazebo reference="${prefix}/shoulder_yaw_joint">
@@ -173,5 +173,5 @@
       <axis xyz="0 0 1"/>
       <limit effort="30" lower="-0.9" upper="${PI}" velocity="2.00"/>
-      <dynamics damping="0.5" friction="0"/>
+      <dynamics damping="15.0" friction="0"/>
     </joint>
     <gazebo reference="${prefix}/elbow_pitch_joint">
@@ -224,5 +224,5 @@
       <axis xyz="0 0 1"/>
       <limit effort="6" lower="-4.55" upper="1.25" velocity="2.0"/>
-      <dynamics damping="0.5" friction="0"/>
+      <dynamics damping="15.0" friction="0"/>
     </joint>
     <gazebo reference="${prefix}/wrist_yaw_joint">
@@ -261,5 +261,5 @@
       <axis xyz="0 0 1"/>
       <limit effort="6" lower="-1.5707" upper="1.5707" velocity="2.00"/>
-      <dynamics damping="0.5" friction="0"/>
+      <dynamics damping="15.0" friction="0"/>
     </joint>
     <gazebo reference="${prefix}/wrist_pitch_joint">
@@ -298,5 +298,5 @@
       <axis xyz="0 0 1"/>
       <limit effort="6" lower="-2.95" upper="2.95" velocity="2.00"/><!-- 2.95 is a limit taken in from 3 due to saftey and differences between arms. -->
-      <dynamics damping="0.2" friction="0"/>
+      <dynamics damping="15.0" friction="0"/>
     </joint>
     <gazebo reference="${prefix}/palm_yaw_joint">
@@ -337,5 +337,5 @@
       <!--<limit effort="15" lower="-0.9" upper="${PI}" velocity="0.50"/>-->
       <!--[> <safety_controller k_position="100" k_velocity="3" soft_lower_limit="-100.0" soft_upper_limit="100.0" /> <]-->
-      <!--<dynamics damping="1.0" friction="100.0"/>-->
+      <!--<dynamics damping="15.0" friction="100.0"/>-->
     <!--</joint>-->
     <!--<link name="${prefix}/forearm_link" >-->
@@ -373,5 +373,5 @@
       <!--<limit effort="5" lower="-4.8" upper="1.3" velocity="0.20"/>-->
       <!--[> <safety_controller k_position="100" k_velocity="3" soft_lower_limit="-100.0" soft_upper_limit="100.0" /> <]-->
-      <!--<dynamics damping="1.0" friction="100.0"/>-->
+      <!--<dynamics damping="15.0" friction="100.0"/>-->
     <!--</joint>-->
     <!--<link name="${prefix}/LowerWristPalmLink" >-->
@@ -409,5 +409,5 @@
       <!--<limit effort="5" lower="-2.95" upper="2.95" velocity="0.20"/>[> 2.95 is a limit taken in from 3 due to saftey and differences between arms. <]-->
       <!--[> <safety_controller k_position="100" k_velocity="3" soft_lower_limit="-100.0" soft_upper_limit="100.0" /> <]-->
-      <!--<dynamics damping="1.0" friction="100.0"/>-->
+      <!--<dynamics damping="15.0" friction="100.0"/>-->
     <!--</joint>-->
     <!--<link name="${prefix}/LowerWristYawLink" >-->
@@ -443,5 +443,5 @@
       <axis xyz="0 0 1"/>
       <limit effort="15" lower="-0.9" upper="${PI}" velocity="2.0"/>
-      <dynamics damping="0.5" friction="0"/>
+      <dynamics damping="15.0" friction="0"/>
     </joint>
     <link name="${prefix}/stump_link" >

Commit message: decreasing damping for wam joints to increase performance

File: models/components.urdf.xacro (robot description, xacro)
@@ -64,5 +64,5 @@
       <axis xyz="0 0 1"/>
       <limit effort="60" lower="-2.6" upper="2.6" velocity="2.0"/>
-      <dynamics damping="15.0" friction="0"/>
+      <dynamics damping="5.0" friction="0"/>
     </joint>
     <gazebo reference="${prefix}/base_yaw_joint">
@@ -100,5 +100,5 @@
       <axis xyz="0 0 1"/>
       <limit effort="60" lower="-1.985" upper="1.985" velocity="2.0"/>
-      <dynamics damping="15.0" friction="0"/>
+      <dynamics damping="5.0" friction="0"/>
     </joint>
     <gazebo reference="${prefix}/shoulder_pitch_joint">
@@ -136,5 +136,5 @@
       <axis xyz="0 0 1"/>
       <limit effort="45" lower="-2.8" upper="2.8" velocity="2.0"/>
-      <dynamics damping="15.0" friction="0"/>
+      <dynamics damping="5.0" friction="0"/>
     </joint>
     <gazebo reference="${prefix}/shoulder_yaw_joint">
@@ -173,5 +173,5 @@
       <axis xyz="0 0 1"/>
       <limit effort="30" lower="-0.9" upper="${PI}" velocity="2.00"/>
-      <dynamics damping="15.0" friction="0"/>
+      <dynamics damping="5.0" friction="0"/>
     </joint>
     <gazebo reference="${prefix}/elbow_pitch_joint">
@@ -224,5 +224,5 @@
       <axis xyz="0 0 1"/>
       <limit effort="6" lower="-4.55" upper="1.25" velocity="2.0"/>
-      <dynamics damping="15.0" friction="0"/>
+      <dynamics damping="2.0" friction="0"/>
     </joint>
     <gazebo reference="${prefix}/wrist_yaw_joint">
@@ -261,5 +261,5 @@
       <axis xyz="0 0 1"/>
       <limit effort="6" lower="-1.5707" upper="1.5707" velocity="2.00"/>
-      <dynamics damping="15.0" friction="0"/>
+      <dynamics damping="2.0" friction="0"/>
     </joint>
     <gazebo reference="${prefix}/wrist_pitch_joint">
@@ -298,5 +298,5 @@
       <axis xyz="0 0 1"/>
       <limit effort="6" lower="-2.95" upper="2.95" velocity="2.00"/><!-- 2.95 is a limit taken in from 3 due to saftey and differences between arms. -->
-      <dynamics damping="15.0" friction="0"/>
+      <dynamics damping="2.0" friction="0"/>
     </joint>
     <gazebo reference="${prefix}/palm_yaw_joint">
@@ -337,5 +337,5 @@
       <!--<limit effort="15" lower="-0.9" upper="${PI}" velocity="0.50"/>-->
       <!--[> <safety_controller k_position="100" k_velocity="3" soft_lower_limit="-100.0" soft_upper_limit="100.0" /> <]-->
-      <!--<dynamics damping="15.0" friction="100.0"/>-->
+      <!--<dynamics damping="5.0" friction="100.0"/>-->
     <!--</joint>-->
     <!--<link name="${prefix}/forearm_link" >-->
@@ -373,5 +373,5 @@
       <!--<limit effort="5" lower="-4.8" upper="1.3" velocity="0.20"/>-->
       <!--[> <safety_controller k_position="100" k_velocity="3" soft_lower_limit="-100.0" soft_upper_limit="100.0" /> <]-->
-      <!--<dynamics damping="15.0" friction="100.0"/>-->
+      <!--<dynamics damping="5.0" friction="100.0"/>-->
     <!--</joint>-->
     <!--<link name="${prefix}/LowerWristPalmLink" >-->
@@ -409,5 +409,5 @@
       <!--<limit effort="5" lower="-2.95" upper="2.95" velocity="0.20"/>[> 2.95 is a limit taken in from 3 due to saftey and differences between arms. <]-->
       <!--[> <safety_controller k_position="100" k_velocity="3" soft_lower_limit="-100.0" soft_upper_limit="100.0" /> <]-->
-      <!--<dynamics damping="15.0" friction="100.0"/>-->
+      <!--<dynamics damping="5.0" friction="100.0"/>-->
     <!--</joint>-->
     <!--<link name="${prefix}/LowerWristYawLink" >-->
@@ -443,5 +443,5 @@
       <axis xyz="0 0 1"/>
       <limit effort="15" lower="-0.9" upper="${PI}" velocity="2.0"/>
-      <dynamics damping="15.0" friction="0"/>
+      <dynamics damping="5.0" friction="0"/>
     </joint>
     <link name="${prefix}/stump_link" >

Commit message: decreasing joint damping for simulation

File: models/components.urdf.xacro (robot description, xacro)
@@ -64,5 +64,5 @@
       <axis xyz="0 0 1"/>
       <limit effort="60" lower="-2.6" upper="2.6" velocity="2.0"/>
-      <dynamics damping="5.0" friction="0"/>
+      <dynamics damping="1.5" friction="0"/>
     </joint>
     <gazebo reference="${prefix}/base_yaw_joint">
@@ -100,5 +100,5 @@
       <axis xyz="0 0 1"/>
       <limit effort="60" lower="-1.985" upper="1.985" velocity="2.0"/>
-      <dynamics damping="5.0" friction="0"/>
+      <dynamics damping="1.5" friction="0"/>
     </joint>
     <gazebo reference="${prefix}/shoulder_pitch_joint">
@@ -136,5 +136,5 @@
       <axis xyz="0 0 1"/>
       <limit effort="45" lower="-2.8" upper="2.8" velocity="2.0"/>
-      <dynamics damping="5.0" friction="0"/>
+      <dynamics damping="1.5" friction="0"/>
     </joint>
     <gazebo reference="${prefix}/shoulder_yaw_joint">
@@ -173,5 +173,5 @@
       <axis xyz="0 0 1"/>
       <limit effort="30" lower="-0.9" upper="${PI}" velocity="2.00"/>
-      <dynamics damping="5.0" friction="0"/>
+      <dynamics damping="1.5" friction="0"/>
     </joint>
     <gazebo reference="${prefix}/elbow_pitch_joint">
@@ -224,5 +224,5 @@
       <axis xyz="0 0 1"/>
       <limit effort="6" lower="-4.55" upper="1.25" velocity="2.0"/>
-      <dynamics damping="2.0" friction="0"/>
+      <dynamics damping="1.5" friction="0"/>
     </joint>
     <gazebo reference="${prefix}/wrist_yaw_joint">
@@ -261,5 +261,5 @@
       <axis xyz="0 0 1"/>
       <limit effort="6" lower="-1.5707" upper="1.5707" velocity="2.00"/>
-      <dynamics damping="2.0" friction="0"/>
+      <dynamics damping="1.5" friction="0"/>
     </joint>
     <gazebo reference="${prefix}/wrist_pitch_joint">
@@ -298,5 +298,5 @@
       <axis xyz="0 0 1"/>
       <limit effort="6" lower="-2.95" upper="2.95" velocity="2.00"/><!-- 2.95 is a limit taken in from 3 due to saftey and differences between arms. -->
-      <dynamics damping="2.0" friction="0"/>
+      <dynamics damping="1.5" friction="0"/>
     </joint>
     <gazebo reference="${prefix}/palm_yaw_joint">
@@ -337,5 +337,5 @@
       <!--<limit effort="15" lower="-0.9" upper="${PI}" velocity="0.50"/>-->
       <!--[> <safety_controller k_position="100" k_velocity="3" soft_lower_limit="-100.0" soft_upper_limit="100.0" /> <]-->
-      <!--<dynamics damping="5.0" friction="100.0"/>-->
+      <!--<dynamics damping="1.5" friction="100.0"/>-->
     <!--</joint>-->
     <!--<link name="${prefix}/forearm_link" >-->
@@ -373,5 +373,5 @@
       <!--<limit effort="5" lower="-4.8" upper="1.3" velocity="0.20"/>-->
       <!--[> <safety_controller k_position="100" k_velocity="3" soft_lower_limit="-100.0" soft_upper_limit="100.0" /> <]-->
-      <!--<dynamics damping="5.0" friction="100.0"/>-->
+      <!--<dynamics damping="1.5" friction="100.0"/>-->
     <!--</joint>-->
     <!--<link name="${prefix}/LowerWristPalmLink" >-->
@@ -409,5 +409,5 @@
       <!--<limit effort="5" lower="-2.95" upper="2.95" velocity="0.20"/>[> 2.95 is a limit taken in from 3 due to saftey and differences between arms. <]-->
       <!--[> <safety_controller k_position="100" k_velocity="3" soft_lower_limit="-100.0" soft_upper_limit="100.0" /> <]-->
-      <!--<dynamics damping="5.0" friction="100.0"/>-->
+      <!--<dynamics damping="1.5" friction="100.0"/>-->
     <!--</joint>-->
     <!--<link name="${prefix}/LowerWristYawLink" >-->
@@ -443,5 +443,5 @@
       <axis xyz="0 0 1"/>
       <limit effort="15" lower="-0.9" upper="${PI}" velocity="2.0"/>
-      <dynamics damping="5.0" friction="0"/>
+      <dynamics damping="1.5" friction="0"/>
     </joint>
     <link name="${prefix}/stump_link" >

Commit message: increasing max effort for wrist joints

File: models/components.urdf.xacro (robot description, xacro)
@@ -223,5 +223,5 @@
       <origin xyz="-0.045 -0.3 0" rpy="${PI/2} 0 0"/>
       <axis xyz="0 0 1"/>
-      <limit effort="6" lower="-4.55" upper="1.25" velocity="2.0"/>
+      <limit effort="10" lower="-4.55" upper="1.25" velocity="2.0"/>
       <dynamics damping="1.5" friction="0"/>
     </joint>
@@ -260,5 +260,5 @@
       <origin xyz="0 0 0" rpy="${-PI/2} 0 0"/>
       <axis xyz="0 0 1"/>
-      <limit effort="6" lower="-1.5707" upper="1.5707" velocity="2.00"/>
+      <limit effort="10" lower="-1.5707" upper="1.5707" velocity="2.00"/>
       <dynamics damping="1.5" friction="0"/>
     </joint>
@@ -297,5 +297,5 @@
       <origin xyz="0 0 0" rpy="${PI/2} 0 0"/>
       <axis xyz="0 0 1"/>
-      <limit effort="6" lower="-2.95" upper="2.95" velocity="2.00"/><!-- 2.95 is a limit taken in from 3 due to saftey and differences between arms. -->
+      <limit effort="10" lower="-2.95" upper="2.95" velocity="2.00"/><!-- 2.95 is a limit taken in from 3 due to saftey and differences between arms. -->
       <dynamics damping="1.5" friction="0"/>
     </joint>

Commit message: updating palm limits

File: models/components.urdf.xacro (robot description, xacro)
@@ -297,5 +297,5 @@
       <origin xyz="0 0 0" rpy="${PI/2} 0 0"/>
       <axis xyz="0 0 1"/>
-      <limit effort="10" lower="-2.95" upper="2.95" velocity="2.00"/><!-- 2.95 is a limit taken in from 3 due to saftey and differences between arms. -->
+      <limit effort="10" lower="-3.0" upper="3.0" velocity="2.00"/><!-- 2.95 is a limit taken in from 3 due to saftey and differences between arms. -->
       <dynamics damping="1.5" friction="0"/>
     </joint>

Commit message: adding non-zero friction

File: models/components.urdf.xacro (robot description, xacro)
@@ -64,5 +64,5 @@
       <axis xyz="0 0 1"/>
       <limit effort="60" lower="-2.6" upper="2.6" velocity="2.0"/>
-      <dynamics damping="1.5" friction="0"/>
+      <dynamics damping="1.5" friction="2.0"/>
     </joint>
     <gazebo reference="${prefix}/base_yaw_joint">
@@ -100,5 +100,5 @@
       <axis xyz="0 0 1"/>
       <limit effort="60" lower="-1.985" upper="1.985" velocity="2.0"/>
-      <dynamics damping="1.5" friction="0"/>
+      <dynamics damping="1.5" friction="2.0"/>
     </joint>
     <gazebo reference="${prefix}/shoulder_pitch_joint">
@@ -136,5 +136,5 @@
       <axis xyz="0 0 1"/>
       <limit effort="45" lower="-2.8" upper="2.8" velocity="2.0"/>
-      <dynamics damping="1.5" friction="0"/>
+      <dynamics damping="1.5" friction="1.0"/>
     </joint>
     <gazebo reference="${prefix}/shoulder_yaw_joint">
@@ -173,5 +173,5 @@
       <axis xyz="0 0 1"/>
       <limit effort="30" lower="-0.9" upper="${PI}" velocity="2.00"/>
-      <dynamics damping="1.5" friction="0"/>
+      <dynamics damping="1.5" friction="1.1"/>
     </joint>
     <gazebo reference="${prefix}/elbow_pitch_joint">
@@ -224,5 +224,5 @@
       <axis xyz="0 0 1"/>
       <limit effort="6" lower="-4.55" upper="1.25" velocity="2.0"/>
-      <dynamics damping="1.5" friction="0"/>
+      <dynamics damping="1.5" friction="0.05"/>
     </joint>
     <gazebo reference="${prefix}/wrist_yaw_joint">
@@ -261,5 +261,5 @@
       <axis xyz="0 0 1"/>
       <limit effort="6" lower="-1.5707" upper="1.5707" velocity="2.00"/>
-      <dynamics damping="1.5" friction="0"/>
+      <dynamics damping="1.5" friction="0.4"/>
     </joint>
     <gazebo reference="${prefix}/wrist_pitch_joint">
@@ -298,5 +298,5 @@
       <axis xyz="0 0 1"/>
       <limit effort="6" lower="-2.95" upper="2.95" velocity="2.00"/><!-- 2.95 is a limit taken in from 3 due to saftey and differences between arms. -->
-      <dynamics damping="1.5" friction="0"/>
+      <dynamics damping="1.5" friction="0.03"/>
     </joint>
     <gazebo reference="${prefix}/palm_yaw_joint">

Commit message: decreasing damping for gazebo 2.2.3

File: models/components.urdf.xacro (robot description, xacro)
@@ -64,5 +64,5 @@
       <axis xyz="0 0 1"/>
       <limit effort="60" lower="-2.6" upper="2.6" velocity="2.0"/>
-      <dynamics damping="1.5" friction="0"/>
+      <dynamics damping="0.5" friction="0"/>
     </joint>
     <gazebo reference="${prefix}/base_yaw_joint">
@@ -100,5 +100,5 @@
       <axis xyz="0 0 1"/>
       <limit effort="60" lower="-1.985" upper="1.985" velocity="2.0"/>
-      <dynamics damping="1.5" friction="0"/>
+      <dynamics damping="0.5" friction="0"/>
     </joint>
     <gazebo reference="${prefix}/shoulder_pitch_joint">
@@ -136,5 +136,5 @@
       <axis xyz="0 0 1"/>
       <limit effort="45" lower="-2.8" upper="2.8" velocity="2.0"/>
-      <dynamics damping="1.5" friction="0"/>
+      <dynamics damping="0.5" friction="0"/>
     </joint>
     <gazebo reference="${prefix}/shoulder_yaw_joint">
@@ -173,5 +173,5 @@
       <axis xyz="0 0 1"/>
       <limit effort="30" lower="-0.9" upper="${PI}" velocity="2.00"/>
-      <dynamics damping="1.5" friction="0"/>
+      <dynamics damping="0.5" friction="0"/>
     </joint>
     <gazebo reference="${prefix}/elbow_pitch_joint">
@@ -224,5 +224,5 @@
       <axis xyz="0 0 1"/>
       <limit effort="10" lower="-4.55" upper="1.25" velocity="2.0"/>
-      <dynamics damping="1.5" friction="0"/>
+      <dynamics damping="0.5" friction="0"/>
     </joint>
     <gazebo reference="${prefix}/wrist_yaw_joint">
@@ -261,5 +261,5 @@
       <axis xyz="0 0 1"/>
       <limit effort="10" lower="-1.5707" upper="1.5707" velocity="2.00"/>
-      <dynamics damping="1.5" friction="0"/>
+      <dynamics damping="0.5" friction="0"/>
     </joint>
     <gazebo reference="${prefix}/wrist_pitch_joint">
@@ -298,5 +298,5 @@
       <axis xyz="0 0 1"/>
       <limit effort="10" lower="-3.0" upper="3.0" velocity="2.00"/><!-- 2.95 is a limit taken in from 3 due to saftey and differences between arms. -->
-      <dynamics damping="1.5" friction="0"/>
+      <dynamics damping="0.5" friction="0"/>
     </joint>
     <gazebo reference="${prefix}/palm_yaw_joint">
@@ -353,5 +353,5 @@
       <!--<limit effort="15" lower="-0.9" upper="${PI}" velocity="0.50"/>-->
       <!--[> <safety_controller k_position="100" k_velocity="3" soft_lower_limit="-100.0" soft_upper_limit="100.0" /> <]-->
-      <!--<dynamics damping="1.5" friction="100.0"/>-->
+      <!--<dynamics damping="0.5" friction="100.0"/>-->
     <!--</joint>-->
     <!--<link name="${prefix}/forearm_link" >-->
@@ -389,5 +389,5 @@
       <!--<limit effort="5" lower="-4.8" upper="1.3" velocity="0.20"/>-->
       <!--[> <safety_controller k_position="100" k_velocity="3" soft_lower_limit="-100.0" soft_upper_limit="100.0" /> <]-->
-      <!--<dynamics damping="1.5" friction="100.0"/>-->
+      <!--<dynamics damping="0.5" friction="100.0"/>-->
     <!--</joint>-->
     <!--<link name="${prefix}/LowerWristPalmLink" >-->
@@ -425,5 +425,5 @@
       <!--<limit effort="5" lower="-2.95" upper="2.95" velocity="0.20"/>[> 2.95 is a limit taken in from 3 due to saftey and differences between arms. <]-->
       <!--[> <safety_controller k_position="100" k_velocity="3" soft_lower_limit="-100.0" soft_upper_limit="100.0" /> <]-->
-      <!--<dynamics damping="1.5" friction="100.0"/>-->
+      <!--<dynamics damping="0.5" friction="100.0"/>-->
     <!--</joint>-->
     <!--<link name="${prefix}/LowerWristYawLink" >-->
@@ -459,5 +459,5 @@
       <axis xyz="0 0 1"/>
       <limit effort="15" lower="-0.9" upper="${PI}" velocity="2.0"/>
-      <dynamics damping="1.5" friction="0"/>
+      <dynamics damping="0.5" friction="0"/>
     </joint>
     <link name="${prefix}/stump_link" >

Commit message: increasing simulated damping on last joint

File: models/components.urdf.xacro (robot description, xacro)
@@ -299,5 +299,5 @@
       <axis xyz="0 0 1"/>
       <limit effort="10" lower="-3.0" upper="3.0" velocity="2.00"/><!-- 2.95 is a limit taken in from 3 due to saftey and differences between arms. -->
-      <dynamics damping="${0.1*b}" friction="0"/>
+      <dynamics damping="${0.3*b}" friction="0"/>
     </joint>
     <gazebo reference="${prefix}/palm_yaw_joint">

Commit message: fixing color

File: models/components.urdf.xacro (robot description, xacro)
@@ -47,7 +47,7 @@
       </inertial>
       <visual>
-        <!--<material name="WAMGrey">-->
-          <!--<color rgba="0.7 0.7 0.7 0.0"/>-->
-        <!--</material>-->
+        <material name="WAMGrey">
+          <color rgba="0.7 0.7 0.7 0.0"/>
+        </material>
         <geometry>
           <mesh filename="${models_path}/sw_meshes/base_link_fine.stl"/>
@@ -86,7 +86,7 @@
       </inertial>
       <visual>
-        <!--<material name="WAMGrey">-->
-          <!--<color rgba="0.7 0.7 0.7 1.0"/>-->
-        <!--</material>-->
+        <material name="WAMGrey">
+          <color rgba="0.7 0.7 0.7 1.0"/>
+        </material>
         <geometry>
           <mesh filename="${models_path}/sw_meshes/shoulder_link_fine.stl"/>
@@ -117,7 +117,7 @@
     <link name="${prefix}/shoulder_pitch_link" >
       <visual>
-        <!--<material name="WAMGrey">-->
-          <!--<color rgba="0.7 0.7 0.7 1.0"/>-->
-        <!--</material>-->
+        <material name="WAMGrey">
+          <color rgba="0.7 0.7 0.7 1.0"/>
+        </material>
         <geometry>
           <mesh filename="${models_path}/sw_meshes/shoulder_pitch_link_fine.stl"/>
@@ -164,7 +164,7 @@
       </inertial>
       <visual>
-        <!--<material name="WAMGrey">-->
-          <!--<color rgba="0.7 0.7 0.7 1.0"/>-->
-        <!--</material>-->
+        <material name="WAMGrey">
+          <color rgba="0.7 0.7 0.7 1.0"/>
+        </material>
         <geometry>
           <mesh filename="${models_path}/sw_meshes/upper_arm_link_fine.stl"/>
@@ -204,7 +204,7 @@
       </inertial>
       <visual>
-        <!--<material name="WAMGrey">-->
-          <!--<color rgba="0.7 0.7 0.7 1.0"/>-->
-        <!--</material>-->
+        <material name="WAMGrey">
+          <color rgba="0.7 0.7 0.7 1.0"/>
+        </material>
         <geometry>
           <mesh filename="${models_path}/sw_meshes/elbow_link_fine.stl"/>
@@ -217,7 +217,7 @@
       </collision>
       <visual>
-        <!--<material name="WAMGrey2">-->
-          <!--<color rgba="0.1 0.1 0.1 1.0"/>-->
-        <!--</material>-->
+        <material name="WAMGrey2">
+          <color rgba="0.1 0.1 0.1 1.0"/>
+        </material>
         <origin xyz="-0.045 -0.0730 0" rpy="${PI/2} 0 0" />
         <geometry>
@@ -298,7 +298,7 @@
       </inertial>
       <visual>
-        <!--<material name="WAMGrey">-->
-          <!--<color rgba="0.7 0.7 0.7 1.0"/>-->
-        <!--</material>-->
+        <material name="WAMGrey">
+          <color rgba="0.7 0.7 0.7 1.0"/>
+        </material>
         <geometry>
           <mesh filename="${models_path}/sw_meshes/wrist_pitch_link_fine.stl"/>
@@ -337,7 +337,7 @@
       </inertial>
       <visual>
-        <!--<material name="WAMGrey">-->
-          <!--<color rgba="0.7 0.7 0.7 1.0"/>-->
-        <!--</material>-->
+        <material name="WAMGrey">
+          <color rgba="0.7 0.7 0.7 1.0"/>
+        </material>
         <origin xyz="0 0 0" rpy="0 0 0" />
         <geometry>
@@ -496,7 +496,7 @@
       </inertial>
       <visual>
-        <!--<material name="WAMGrey">-->
-          <!--<color rgba="0.7 0.7 0.7 1.0"/>-->
-        <!--</material>-->
+        <material name="WAMGrey">
+          <color rgba="0.7 0.7 0.7 1.0"/>
+        </material>
         <geometry>
           <mesh filename="${models_path}/sw_meshes/elbow_link_fine.stl"/>
