Commit message: adding wrist link color

File: models/components.urdf.xacro (robot description, xacro)
@@ -257,7 +257,7 @@
       </inertial>
       <visual>
-        <!--<material name="WAMGrey">-->
-          <!--<color rgba="0.7 0.7 0.7 1.0"/>-->
-        <!--</material>-->
+        <material name="WAMGrey">
+          <color rgba="0.7 0.7 0.7 1.0"/>
+        </material>
         <origin xyz="0 0 0" rpy="0 0 0" />
         <geometry>
