Commit message: adding base back in

File: models/common.urdf.xacro (robot description, xacro)
@@ -35,8 +35,4 @@
   <!-- Constants -->
   <xacro:property name="PI" value="3.1415926535897931" />
-  <!-- Materials -->
-  <material name="WAMGrey">
-    <color rgba="0.9 0.9 0.9 1.0"/>
-  </material>
   <!-- Gazebo macros -->
   <xacro:macro name="gazeboReference" params="name material">

File: models/components.urdf.xacro (robot description, xacro)
@@ -32,4 +32,32 @@
   <include filename="$(find bard_urdf)/models/hand.urdf.xacro"/>
   <include filename="$(find bard_urdf)/models/common.urdf.xacro"/>
+  <xacro:macro name="base" params="xyz rpy parent">
+    <link name ="baseLink">
+      <inertial>
+        <origin xyz="0 0 0" rpy="0 0 0" />
+        <mass value="1.0" />
+        <inertia  ixx="1.0" ixy="0.0"  ixz="0.0"  iyy="100.0"  iyz="0.0"  izz="1.0" />
+      </inertial>
+      <visual>
+        <material name="WAMGrey" />
+        <origin xyz="0 0 0" rpy="${0.5 * PI} 0 0" />
+        <geometry>
+          <mesh filename="package://bard_urdf/models/componentSTL/Re2_Body.DAE"/>
+        </geometry>
+      </visual>
+      <collision>
+        <origin xyz="0 0 0" rpy="${0.5 * PI} 0 0" />
+        <geometry>
+          <mesh filename="package://bard_urdf/models/componentSTL/baseLinkTwoArms.stl"/>
+        </geometry>
+      </collision>
+    </link>
+    <xacro:gazeboReferenceDAE name="baseLink"/>
+    <joint name="baseJoint" type="fixed">
+      <parent link="${parent}"/>
+      <child link="baseLink"/>
+      <origin xyz="${xyz}" rpy="${rpy}"/>
+    </joint>
+  </xacro:macro>
   <xacro:macro name="Shoulder" params="prefix parentLink xyz rpy">
     <link name="${prefix}/ShoulderLink" >

File: models/root.urdf.xacro (robot description, xacro)
@@ -29,4 +29,8 @@
   <include filename="$(find bard_urdf)/models/arm.urdf.xacro"/>
   <include filename="$(find bard_urdf)/models/components.urdf.xacro"/>
+  <!-- Materials -->
+  <material name="WAMGrey">
+    <color rgba="0.9 0.9 0.9 1.0"/>
+  </material>
   <link name = "world"/>
   <xacro:base xyz="0 0 0.813372" rpy="0 0 0" parent="world"/>
@@ -75,6 +79,6 @@
     </controller:gazebo_ros_controller_manager>
   </gazebo>
-  <xacro:darpa_arm prefix="RightWAM" parentLink="baseLink" xyz="-0.350177361 -0.350177361 .37836125" rpy="-${0.5 * PI} -${0.5 * PI} ${0.25*PI}" />
-  <xacro:darpa_arm prefix="LeftWAM" parentLink="baseLink" xyz="0.350177361 -0.350177361 .37836125" rpy="-${0.5 * PI} -${0.5 * PI} ${0.75*PI}" />
-  <xacro:darpa_head_assembly parent="baseLink" xyz="0 -.1292225 .52971" rpy="${0.5 * PI} 0 0"/>
+  <!-- Construct the actual arms -->
+  <xacro:darpa_arm prefix="RightWAM" parentLink="RightWAM/FixedLink" xyz="0 0 0 " rpy="0 0 0" />
+  <xacro:darpa_arm prefix="LeftWAM" parentLink="LeftWAM/FixedLink" xyz="0 0 0" rpy="0 0 0" />
 </robot>

Commit message: Updates, getting things running in gazebo

File: models/common.urdf.xacro (robot description, xacro)
@@ -42,5 +42,5 @@
       </material>
       <turnGravityOff>
-        true
+        false
       </turnGravityOff>
       <selfCollide>
@@ -52,5 +52,5 @@
     <gazebo reference="${name}">
       <turnGravityOff>
-        true
+        false
       </turnGravityOff>
       <selfCollide>
@@ -61,4 +61,5 @@
   <!-- Controller macros -->
   <xacro:macro name="control" params="name topicName linkName jointName">
+    <!--
     <transmission type="pr2_mechanism_model/SimpleTransmission" name="${name}_trans">
       <actuator name="${name}_motor" />
@@ -68,4 +69,5 @@
       <pulsesPerRevolution>90000</pulsesPerRevolution>
     </transmission>
+    -->
   </xacro:macro>
 </robot>

File: models/components.urdf.xacro (robot description, xacro)
@@ -52,5 +52,7 @@
       </inertial>
       <visual>
-        <material name="WAMGrey" />
+        <material name="WAMGrey">
+          <color rgba="0.9 0.9 0.9 1.0"/>
+        </material>
         <!--  this orgin is not centered because the origin in our model is not at the same spot as the origin barret uses for inertia-->
         <origin xyz="0 .189 0" rpy="${PI} 0 0" />
@@ -81,8 +83,10 @@
     <link name="${prefix}/UpperArmInShoulderLink" >
       <visual>
-        <material name="WAMGrey" />
+        <material name="WAMGrey">
+          <color rgba="0.9 0.9 0.9 1.0"/>
+        </material>
         <origin xyz="0 0 0" rpy="${PI} 0 0" />
         <geometry>
-          <mesh filename="${homeDirectory}/models/componentSTL/wamUpperArmInShoulderLink.DAE"/>
+          <mesh filename="${homeDirectory}/models/componentSTL/wamUpperArmInShoulderLink.dae"/>
         </geometry>
       </visual>
@@ -123,8 +127,10 @@
       </inertial>
       <visual>
-        <material name="WAMGrey" />
+        <material name="WAMGrey">
+          <color rgba="0.9 0.9 0.9 1.0"/>
+        </material>
         <origin xyz="0 0 0" rpy="0 0 0" />
         <geometry>
-          <mesh filename="${homeDirectory}/models/componentSTL/wamUpperArmLink3.DAE"/>
+          <mesh filename="${homeDirectory}/models/componentSTL/wamUpperArmLink3.dae"/>
         </geometry>
       </visual>
@@ -160,5 +166,7 @@
       </inertial>
       <visual>
-        <material name="WAMGrey" />
+        <material name="WAMGrey">
+          <color rgba="0.9 0.9 0.9 1.0"/>
+        </material>
         <origin xyz="0 0 0" rpy="-${PI} 0 0" />
         <geometry>
@@ -195,5 +203,7 @@
       </inertial>
       <visual>
-        <material name="WAMGrey" />
+        <material name="WAMGrey">
+          <color rgba="0.9 0.9 0.9 1.0"/>
+        </material>
         <origin xyz="0 0.02711 0" rpy="${PI} 0 0" />
         <geometry>
@@ -232,5 +242,7 @@
       </inertial>
       <visual>
-        <material name="WAMGrey" />
+        <material name="WAMGrey">
+          <color rgba="0.9 0.9 0.9 1.0"/>
+        </material>
         <origin xyz="0 0 0" rpy="-${PI} 0 0" />
         <geometry>
@@ -248,4 +260,5 @@
     <xacro:control topicName="${prefix}/ElbowPitch" name="DarmSim_${prefix}Arm_WAM_ElbowPitch" linkName="${prefix}/ForeArmLink" jointName="${prefix}/ElbowJoint" />
   </xacro:macro>
+  <!-- DEBUG HERE -->
   <xacro:macro name="UpperWristYaw" params="prefix">
     <joint name="${prefix}/UpperWristYawJoint" type="revolute">
@@ -267,5 +280,7 @@
       </inertial>
       <visual>
-        <material name="WAMGrey" />
+        <material name="WAMGrey">
+          <color rgba="0.9 0.9 0.9 1.0"/>
+        </material>
         <origin xyz="0 0.02711 0" rpy="${PI} 0 0" />
         <geometry>
@@ -302,8 +317,10 @@
       </inertial>
       <visual>
-        <material name="WAMGrey" />
+        <material name="WAMGrey">
+          <color rgba="0.9 0.9 0.9 1.0"/>
+        </material>
         <origin xyz="0 0 0" rpy="${0.5 * PI} 0 ${0.5 * PI}" />
         <geometry>
-          <mesh filename="${homeDirectory}/models/componentSTL/wamUpperWristPitchLink6.DAE"/>
+          <mesh filename="${homeDirectory}/models/componentSTL/wamUpperWristPitchLink6.dae"/>
         </geometry>
       </visual>
@@ -338,5 +355,7 @@
       </inertial>
       <visual>
-        <material name="WAMGrey" />
+        <material name="WAMGrey">
+          <color rgba="0.9 0.9 0.9 1.0"/>
+        </material>
         <origin xyz="0 0 0" rpy="0 0 0" />
         <geometry>
@@ -374,5 +393,7 @@
       </inertial>
       <visual>
-        <material name="WAMGrey" />
+        <material name="WAMGrey">
+          <color rgba="0.9 0.9 0.9 1.0"/>
+        </material>
         <origin xyz="0 0 0" rpy="0 0 0" />
         <geometry>
@@ -402,5 +423,7 @@
     <link name="${prefix}/BHand/Finger${number}/KnuckleOneLink">
       <visual>
-        <material name="WAMGrey" />
+        <material name="WAMGrey">
+          <color rgba="0.9 0.9 0.9 1.0"/>
+        </material>
         <origin xyz="0 0 0" rpy="${0.5 * PI} 0 -${0.5 * PI}" />
         <geometry>
@@ -441,5 +464,7 @@
     <link name="${prefix}/BHand/Finger${number}/KnuckleTwoLink">
       <visual>
-        <material name="WAMGrey" />
+        <material name="WAMGrey">
+          <color rgba="0.9 0.9 0.9 1.0"/>
+        </material>
         <origin xyz="0 0 0" rpy="${PI} ${0.5 * PI} 0" />
         <geometry>
@@ -481,5 +506,7 @@
     <link name="${prefix}/BHand/Finger${number}/KnuckleThreeLink">
       <visual>
-        <material name="WAMGrey" />
+        <material name="WAMGrey">
+          <color rgba="0.9 0.9 0.9 1.0"/>
+        </material>
         <origin xyz="0 0 0" rpy="0 ${0.5 * PI} 0" />
         <geometry>

File: models/hand.urdf.xacro (robot description, xacro)
@@ -72,5 +72,7 @@
       </inertial>
       <visual>
-        <material name="WAMGrey" />
+        <material name="WAMGrey">
+          <color rgba="0.9 0.9 0.9 1.0"/>
+        </material>
         <origin xyz="0 0 0" rpy="0 0 0" />
         <geometry>
@@ -130,5 +132,7 @@
       </inertial>
       <visual>
-        <material name="WAMGrey" />
+        <material name="WAMGrey">
+          <color rgba="0.9 0.9 0.9 1.0"/>
+        </material>
         <origin xyz="0 0 0" rpy="0 0 0" />
         <geometry>

File: models/unused.urdf.xacro (robot description, xacro)
@@ -9,5 +9,7 @@
       </inertial>
       <visual>
-        <material name="WAMGrey" />
+        <material name="WAMGrey">
+          <color rgba="0.9 0.9 0.9 1.0"/>
+        </material>
         <origin xyz="0 0 0" rpy="0 0 0" />
         <geometry>
@@ -43,5 +45,7 @@
       </inertial>
       <visual>
-        <material name="WAMGrey" />
+        <material name="WAMGrey">
+          <color rgba="0.9 0.9 0.9 1.0"/>
+        </material>
         <origin xyz="0 0 0" rpy="0 0 0" />
         <geometry>
@@ -70,5 +74,7 @@
     <link name="DarmSim/lowerTiltBeamsFrontLink">
       <visual>
-        <material name="WAMGrey" />
+        <material name="WAMGrey">
+          <color rgba="0.9 0.9 0.9 1.0"/>
+        </material>
         <origin xyz="0 0 0" rpy="0 0 0" />
         <geometry>

File: models/wam_top.urdf.xacro (robot description, xacro)
@@ -15,6 +15,16 @@
     <!-- Create the $(arg robot_name) WAM -->
     <link name = "${prefix}/FixedLink">
+      <inertial>
+        <origin xyz="0 0 0" />
+        <mass value="100" />
+        <inertia
+          ixx="1" ixy="0"   ixz="0"
+                  iyy="1"   iyz="0"
+                            izz="1" />
+      </inertial>
       <visual>
-        <material name="WAMGrey" />
+        <material name="WAMGrey">
+          <color rgba="0.9 0.9 0.9 1.0"/>
+        </material>
         <!--  this orgin is not centered because the origin in our model is not at the same spot as the origin barret uses for inertia-->
         <origin xyz="0 0.346 0" rpy="${PI/2} 0 0"/>
@@ -24,5 +34,5 @@
       </visual>
       <collision>
-        <origin xyz="0 .189 0" rpy="0 0 0" />
+        <origin xyz="0 0.346 0" rpy="${PI/2} 0 0" />
         <geometry>
           <mesh filename="${homeDirectory}/models/componentSTL/wamBase.stl"/>
@@ -36,10 +46,10 @@
     </joint>
     <!-- Simulation stuff -->
-    <gazebo>
+    <!--gazebo>
       <controller:gazebo_ros_controller_manager name="gazebo_ros_controller_manager" plugin="libgazebo_ros_controller_manager.so">
         <alwaysOn>true</alwaysOn>
         <updateRate>1000.0</updateRate>
       </controller:gazebo_ros_controller_manager>
-    </gazebo>
+    </gazebo-->
   </xacro:macro>
 </robot>

File: robots/wam_7dof_2x.urdf.xacro (robot description, xacro)
@@ -4,5 +4,30 @@
   <include filename="$(find bard_urdf)/models/wam_top.urdf.xacro"/>
   <!-- Root link is in the world frame-->
-  <link name = "baseLink"/>
+  <link name = "baseLink">
+    <inertial>
+      <origin xyz="-1 0 0" />
+      <mass value="1000" />
+      <inertia
+        ixx="1" ixy="0"   ixz="0"
+                iyy="1"   iyz="0"
+                          izz="1" />
+    </inertial>
+    <visual>
+      <origin rpy="0 0 0 " xyz="-1 0 1"/>
+      <geometry>
+        <box size="2 5 2"/>
+      </geometry>
+    </visual>
+    <collision>
+      <origin rpy="0 0 0 " xyz="-1 0 1"/>
+      <geometry>
+        <box size="2 5 2"/>
+      </geometry>
+    </collision>
+  </link>
+  <!--<gazebo reference="baseLink">
+    <static>true</static>
+     <turnGravityOff>true</turnGravityOff>
+   </gazebo>-->
   <xacro:wam_root prefix="wam_left" parentLink="baseLink" xyz="0.356 0.46 1" rpy="0 ${-0.5*PI} ${0.5*PI}"/>
   <xacro:wam_7dof prefix="wam_left" parentLink="wam_left/FixedLink" xyz="0 0 0" rpy="0 0 0" />

Commit message: moving gz tags to common and adding them to the hand

File: models/common.urdf.xacro (robot description, xacro)
@@ -40,3 +40,10 @@
     </gazebo>
   </xacro:macro>
+  <!-- Gazebo joint configuration -->
+  <xacro:macro name="gz_joint">
+    <provideFeedback>true</provideFeedback>
+    <implicitSpringDamper>true</implicitSpringDamper>
+    <!--<cfmDamping>true</cfmDamping>-->
+    <!--<dynamics damping="5.5" friction="1"/>-->
+  </xacro:macro>
 </robot>

File: models/components.urdf.xacro (robot description, xacro)
@@ -26,11 +26,4 @@
   <xacro:include filename="$(find barrett_model)/models/hand.urdf.xacro"/>
   <xacro:include filename="$(find barrett_model)/models/common.urdf.xacro"/>
-  <!-- Gazebo joint configuration -->
-  <xacro:macro name="gz_joint">
-    <provideFeedback>true</provideFeedback>
-    <implicitSpringDamper>true</implicitSpringDamper>
-    <!--<cfmDamping>true</cfmDamping>-->
-    <!--<dynamics damping="5.5" friction="1"/>-->
-  </xacro:macro>
   <!-- Upper arm macros -->
   <xacro:macro name="wam_base" params="prefix parent_link xyz rpy">

File: models/hand.urdf.xacro (robot description, xacro)
@@ -61,5 +61,9 @@
       <axis xyz="${axis}"/>
       <limit effort="5" lower="0" upper="${PI}" velocity="0.20"/>
+      <dynamics damping="0.5" friction="1"/>
     </joint>
+    <gazebo reference="${prefix}/prox_joint">
+      <xacro:gz_joint/>
+    </gazebo>
     <link name="${prefix}/prox_link">
       <inertial>
@@ -93,5 +97,9 @@
       <axis xyz="0 0 1"/>
       <limit effort="5" lower="0" upper="${140/180*PI}" velocity="0.20"/>
+      <dynamics damping="0.5" friction="1"/>
     </joint>
+    <gazebo reference="${prefix}/med_joint">
+      <xacro:gz_joint/>
+    </gazebo>
     <link name="${prefix}/med_link">
       <inertial>
@@ -125,5 +133,9 @@
       <axis xyz="0 0 1"/>
       <limit effort="5" lower="0" upper="${48/180*PI}" velocity="0.20"/>
+      <dynamics damping="0.5" friction="1"/>
     </joint>
+    <gazebo reference="${prefix}/dist_joint">
+      <xacro:gz_joint/>
+    </gazebo>
     <link name="${prefix}/dist_link">
       <inertial>

Commit message: updating damping to have a global scale factor

File: models/common.urdf.xacro (robot description, xacro)
@@ -44,4 +44,6 @@
     <provideFeedback>true</provideFeedback>
     <implicitSpringDamper>true</implicitSpringDamper>
+    <!--<kp>0.0</kp>[> CFM <]-->
+    <!--<kd>0.0</kd>[> ERP <]-->
     <!--<cfmDamping>true</cfmDamping>-->
     <!--<dynamics damping="5.5" friction="1"/>-->

File: models/components.urdf.xacro (robot description, xacro)
@@ -26,4 +26,5 @@
   <xacro:include filename="$(find barrett_model)/models/hand.urdf.xacro"/>
   <xacro:include filename="$(find barrett_model)/models/common.urdf.xacro"/>
+  <xacro:property name="b" value="0.5"/>
   <!-- Upper arm macros -->
   <xacro:macro name="wam_base" params="prefix parent_link xyz rpy">
@@ -64,5 +65,5 @@
       <axis xyz="0 0 1"/>
       <limit effort="60" lower="-2.6" upper="2.6" velocity="2.0"/>
-      <dynamics damping="0.5" friction="0"/>
+      <dynamics damping="${1.8*b}" friction="0"/>
     </joint>
     <gazebo reference="${prefix}/base_yaw_joint">
@@ -100,5 +101,5 @@
       <axis xyz="0 0 1"/>
       <limit effort="60" lower="-1.985" upper="1.985" velocity="2.0"/>
-      <dynamics damping="0.5" friction="0"/>
+      <dynamics damping="${0.5*b}" friction="0"/>
     </joint>
     <gazebo reference="${prefix}/shoulder_pitch_joint">
@@ -136,5 +137,5 @@
       <axis xyz="0 0 1"/>
       <limit effort="45" lower="-2.8" upper="2.8" velocity="2.0"/>
-      <dynamics damping="0.5" friction="0"/>
+      <dynamics damping="${1.5*b}" friction="0"/>
     </joint>
     <gazebo reference="${prefix}/shoulder_yaw_joint">
@@ -173,5 +174,5 @@
       <axis xyz="0 0 1"/>
       <limit effort="30" lower="-0.9" upper="${PI}" velocity="2.00"/>
-      <dynamics damping="0.5" friction="0"/>
+      <dynamics damping="${0.8*b}" friction="0"/>
     </joint>
     <gazebo reference="${prefix}/elbow_pitch_joint">
@@ -224,5 +225,5 @@
       <axis xyz="0 0 1"/>
       <limit effort="10" lower="-4.55" upper="1.25" velocity="2.0"/>
-      <dynamics damping="0.5" friction="0"/>
+      <dynamics damping="${0.5*b}" friction="0"/>
     </joint>
     <gazebo reference="${prefix}/wrist_yaw_joint">
@@ -261,5 +262,5 @@
       <axis xyz="0 0 1"/>
       <limit effort="10" lower="-1.5707" upper="1.5707" velocity="2.00"/>
-      <dynamics damping="0.5" friction="0"/>
+      <dynamics damping="${0.1*b}" friction="0"/>
     </joint>
     <gazebo reference="${prefix}/wrist_pitch_joint">
@@ -298,5 +299,5 @@
       <axis xyz="0 0 1"/>
       <limit effort="10" lower="-3.0" upper="3.0" velocity="2.00"/><!-- 2.95 is a limit taken in from 3 due to saftey and differences between arms. -->
-      <dynamics damping="0.5" friction="0"/>
+      <dynamics damping="${0.1*b}" friction="0"/>
     </joint>
     <gazebo reference="${prefix}/palm_yaw_joint">
@@ -353,5 +354,5 @@
       <!--<limit effort="15" lower="-0.9" upper="${PI}" velocity="0.50"/>-->
       <!--[> <safety_controller k_position="100" k_velocity="3" soft_lower_limit="-100.0" soft_upper_limit="100.0" /> <]-->
-      <!--<dynamics damping="0.5" friction="100.0"/>-->
+      <!--<dynamics damping="0.1" friction="100.0"/>-->
     <!--</joint>-->
     <!--<link name="${prefix}/forearm_link" >-->
@@ -389,5 +390,5 @@
       <!--<limit effort="5" lower="-4.8" upper="1.3" velocity="0.20"/>-->
       <!--[> <safety_controller k_position="100" k_velocity="3" soft_lower_limit="-100.0" soft_upper_limit="100.0" /> <]-->
-      <!--<dynamics damping="0.5" friction="100.0"/>-->
+      <!--<dynamics damping="0.1" friction="100.0"/>-->
     <!--</joint>-->
     <!--<link name="${prefix}/LowerWristPalmLink" >-->
@@ -425,5 +426,5 @@
       <!--<limit effort="5" lower="-2.95" upper="2.95" velocity="0.20"/>[> 2.95 is a limit taken in from 3 due to saftey and differences between arms. <]-->
       <!--[> <safety_controller k_position="100" k_velocity="3" soft_lower_limit="-100.0" soft_upper_limit="100.0" /> <]-->
-      <!--<dynamics damping="0.5" friction="100.0"/>-->
+      <!--<dynamics damping="0.1" friction="100.0"/>-->
     <!--</joint>-->
     <!--<link name="${prefix}/LowerWristYawLink" >-->
@@ -459,5 +460,5 @@
       <axis xyz="0 0 1"/>
       <limit effort="15" lower="-0.9" upper="${PI}" velocity="2.0"/>
-      <dynamics damping="0.5" friction="0"/>
+      <dynamics damping="${0.1*b}" friction="0"/>
     </joint>
     <link name="${prefix}/stump_link" >

File: models/hand.urdf.xacro (robot description, xacro)
@@ -1,4 +1,5 @@
 <robot xmlns:xacro="http://www.ros.org/wiki/xacro">
   <xacro:include filename="$(find barrett_model)/models/common.urdf.xacro"/>
+  <xacro:property name="b" value="1.1"/>
   <!-- High-leveel hand macro -->
   <xacro:macro name="bhand" params="parent_link prefix xyz rpy">
@@ -68,5 +69,5 @@
       <origin xyz="0 0 0.08" rpy="0 0 0"/>
       <limit effort="5" lower="0" upper="${PI}" velocity="5.0"/>
-      <dynamics damping="0.1" friction="0"/>
+      <dynamics damping="${0.1*b}" friction="0"/>
     </joint>
     <link name="${prefix}/bhand_palm_surface_link">
@@ -84,5 +85,5 @@
       <origin xyz="0 0 0.12" rpy="0 0 0"/>
       <limit effort="5" lower="0" upper="${PI}" velocity="5.0"/>
-      <dynamics damping="0.1" friction="0"/>
+      <dynamics damping="${0.1*b}" friction="0"/>
     </joint>
     <link name="${prefix}/bhand_grasp_link">
@@ -103,5 +104,5 @@
       <axis xyz="${axis}"/>
       <limit effort="5" lower="0" upper="${PI}" velocity="5.0"/>
-      <dynamics damping="0.1" friction="0"/>
+      <dynamics damping="${0.1*b}" friction="0"/>
     </joint>
     <gazebo reference="${prefix}/prox_joint">
@@ -142,5 +143,5 @@
       <axis xyz="0 0 1"/>
       <limit effort="5" lower="0" upper="${140/180*PI}" velocity="5.00"/>
-      <dynamics damping="0.1" friction="0"/>
+      <dynamics damping="${0.1*b}" friction="0"/>
     </joint>
     <gazebo reference="${prefix}/med_joint">
@@ -181,5 +182,5 @@
       <axis xyz="0 0 1"/>
       <limit effort="5" lower="0" upper="${48/180*PI}" velocity="5.00"/>
-      <dynamics damping="0.1" friction="0"/>
+      <dynamics damping="${0.1*b}" friction="0"/>
     </joint>
     <gazebo reference="${prefix}/dist_joint">

Commit message: making hand finger links more compliant

File: models/common.urdf.xacro (robot description, xacro)
@@ -49,3 +49,8 @@
     <!--<dynamics damping="5.5" friction="1"/>-->
   </xacro:macro>
+  <!-- Gazebo "soft" link which has compliant surface stiffness -->
+  <xacro:macro name="gz_soft_link">
+    <kp>10000</kp>
+    <kd>0.01</kd>
+  </xacro:macro>
 </robot>

File: models/hand.urdf.xacro (robot description, xacro)
@@ -1,5 +1,5 @@
 <robot xmlns:xacro="http://www.ros.org/wiki/xacro">
   <xacro:include filename="$(find barrett_model)/models/common.urdf.xacro"/>
-  <xacro:property name="b" value="6.0"/>
+  <xacro:property name="b" value="0.1"/>
   <!-- High-leveel hand macro -->
   <xacro:macro name="bhand" params="parent_link prefix xyz rpy">
@@ -28,6 +28,6 @@
   </xacro:macro>
   <xacro:macro name="gz_hand_link" params="collide">
-    <mu1>1.8</mu1>
-    <mu2>1.8</mu2>
+    <mu1>2.8</mu1>
+    <mu2>2.8</mu2>
     <xacro:if value="${collide}">
       <selfCollide>true</selfCollide>
@@ -72,5 +72,4 @@
       <origin xyz="0 0 0.08" rpy="0 0 0"/>
       <limit effort="5" lower="0" upper="${PI}" velocity="5.0"/>
-      <dynamics damping="${0.1*b}" friction="0"/>
     </joint>
     <link name="${prefix}/bhand_palm_surface_link">
@@ -88,5 +87,4 @@
       <origin xyz="0 0 0.12" rpy="0 0 0"/>
       <limit effort="5" lower="0" upper="${PI}" velocity="5.0"/>
-      <dynamics damping="${0.1*b}" friction="0"/>
     </joint>
     <link name="${prefix}/bhand_grasp_link">
@@ -110,5 +108,5 @@
     </joint>
     <gazebo reference="${prefix}/prox_joint">
-      <xacro:gz_joint/>
+      <provideFeedback>true</provideFeedback>
     </gazebo>
     <gazebo reference="${prefix}/prox_link">
@@ -149,8 +147,9 @@
     </joint>
     <gazebo reference="${prefix}/med_joint">
-      <xacro:gz_joint/>
+      <provideFeedback>true</provideFeedback>
     </gazebo>
     <gazebo reference="${prefix}/med_link">
       <xacro:gz_hand_link collide="false"/>
+      <xacro:gz_soft_link/>
     </gazebo>
     <link name="${prefix}/med_link">
@@ -188,8 +187,9 @@
     </joint>
     <gazebo reference="${prefix}/dist_joint">
-      <xacro:gz_joint/>
+      <provideFeedback>true</provideFeedback>
     </gazebo>
     <gazebo reference="${prefix}/dist_link">
       <xacro:gz_hand_link collide="true"/>
+      <xacro:gz_soft_link/>
     </gazebo>
     <link name="${prefix}/dist_link">
