Commit message: making hand primitive model configurable

File: models/common.urdf.xacro (robot description, xacro)
@@ -51,6 +51,6 @@
   <!-- Gazebo "soft" link which has compliant surface stiffness -->
   <xacro:macro name="gz_soft_link">
-    <kp>10000</kp>
-    <kd>0.01</kd>
+    <kp>5000</kp>
+    <kd>0.02</kd>
   </xacro:macro>
 </robot>

File: models/hand.urdf.xacro (robot description, xacro)
@@ -1,10 +1,9 @@
 <robot xmlns:xacro="http://www.ros.org/wiki/xacro">
   <xacro:include filename="$(find barrett_model)/models/common.urdf.xacro"/>
-  <xacro:property name="primitive" value="true"/>
   <!-- link properties -->
   <xacro:macro name="gz_hand_link" params="soft collide">
     <mu1>2.8</mu1>
     <mu2>2.8</mu2>
-    <maxContacts>2</maxContacts>
+    <maxContacts>1</maxContacts>
     <xacro:if value="${collide}">
       <selfCollide>false</selfCollide>
@@ -26,9 +25,9 @@
   </xacro:macro>
   <!-- High-level hand macro -->
-  <xacro:macro name="bhand" params="parent_link prefix xyz rpy">
-    <xacro:bhand_palm parent_link="${parent_link}" prefix="${prefix}" xyz="${xyz}" rpy="${rpy}"/>
-    <xacro:bhand_finger_1 prefix="${prefix}"/>
-    <xacro:bhand_finger_2 prefix="${prefix}"/>
-    <xacro:bhand_finger_3 prefix="${prefix}"/>
+  <xacro:macro name="bhand" params="parent_link prefix xyz rpy primitive">
+    <xacro:bhand_palm parent_link="${parent_link}" prefix="${prefix}" xyz="${xyz}" rpy="${rpy}" primitive="${primitive}/>
+    <xacro:bhand_finger_1 prefix="${prefix}" primitive="${primitive}/>
+    <xacro:bhand_finger_2 prefix="${prefix}" primitive="${primitive}/>
+    <xacro:bhand_finger_3 prefix="${prefix}" primitive="${primitive}/>
     <!-- don't use the gazebo gripper plugin, just slows down the sim -->
     <xacro:if value="false">
@@ -55,23 +54,23 @@
   </xacro:macro>
   <!-- Fingers -->
-  <xacro:macro name="bhand_finger_1" params="prefix">
-    <xacro:bhand_finger_prox prefix="${prefix}/finger_1" parent_link="${prefix}/bhand_palm_link" xyz="-0.025 0.0 0.0415" rpy="0 0 -${PI/2}" axis="0 0 -1"/>
-    <xacro:bhand_finger_med prefix="${prefix}/finger_1" parent_link="${prefix}/finger_1/prox_link" xyz="0.05 0.0 0.03390" rpy="${PI/2} 0 0"/>
-    <xacro:bhand_finger_dist prefix="${prefix}/finger_1"/>
+  <xacro:macro name="bhand_finger_1" params="prefix primitive">
+    <xacro:bhand_finger_prox prefix="${prefix}/finger_1" primitive="${primitive} parent_link="${prefix}/bhand_palm_link" xyz="-0.025 0.0 0.0415" rpy="0 0 -${PI/2}" axis="0 0 -1"/>
+    <xacro:bhand_finger_med prefix="${prefix}/finger_1" primitive="${primitive} parent_link="${prefix}/finger_1/prox_link" xyz="0.05 0.0 0.03390" rpy="${PI/2} 0 0"/>
+    <xacro:bhand_finger_dist prefix="${prefix}/finger_1" primitive="${primitive}/>
     <xacro:bhand_finger_tip prefix="${prefix}/finger_1"/>
   </xacro:macro>
-  <xacro:macro name="bhand_finger_2" params="prefix">
-    <xacro:bhand_finger_prox prefix="${prefix}/finger_2" parent_link="${prefix}/bhand_palm_link" xyz="0.025 0.0 0.0415" rpy="0 0 -${PI/2}" axis="0 0 1"/>
-    <xacro:bhand_finger_med prefix="${prefix}/finger_2" parent_link="${prefix}/finger_2/prox_link" xyz="0.05 0.0 0.03390" rpy="${PI/2} 0 0"/>
-    <xacro:bhand_finger_dist prefix="${prefix}/finger_2"/>
+  <xacro:macro name="bhand_finger_2" params="prefix primitive">
+    <xacro:bhand_finger_prox prefix="${prefix}/finger_2" primitive="${primitive} parent_link="${prefix}/bhand_palm_link" xyz="0.025 0.0 0.0415" rpy="0 0 -${PI/2}" axis="0 0 1"/>
+    <xacro:bhand_finger_med prefix="${prefix}/finger_2" primitive="${primitive} parent_link="${prefix}/finger_2/prox_link" xyz="0.05 0.0 0.03390" rpy="${PI/2} 0 0"/>
+    <xacro:bhand_finger_dist prefix="${prefix}/finger_2" primitive="${primitive}/>
     <xacro:bhand_finger_tip prefix="${prefix}/finger_2"/>
   </xacro:macro>
-  <xacro:macro name="bhand_finger_3" params="prefix">
-    <xacro:bhand_finger_med prefix="${prefix}/finger_3" parent_link="${prefix}/bhand_palm_link" xyz="0 0.05 0.0754" rpy="${PI/2} 0 ${PI/2}"/>
-    <xacro:bhand_finger_dist prefix="${prefix}/finger_3"/>
+  <xacro:macro name="bhand_finger_3" params="prefix primitive">
+    <xacro:bhand_finger_med prefix="${prefix}/finger_3" primitive="${primitive} parent_link="${prefix}/bhand_palm_link" xyz="0 0.05 0.0754" rpy="${PI/2} 0 ${PI/2}"/>
+    <xacro:bhand_finger_dist prefix="${prefix}/finger_3" primitive="${primitive}/>
     <xacro:bhand_finger_tip prefix="${prefix}/finger_3"/>
   </xacro:macro>
   <!-- Components -->
-  <xacro:macro name="bhand_palm" params="prefix parent_link xyz rpy">
+  <xacro:macro name="bhand_palm" params="prefix parent_link xyz rpy primitive">
     <joint name="${prefix}/bhand_base_joint" type="fixed">
       <parent link="${parent_link}"/>
@@ -121,5 +120,5 @@
       <child link="${prefix}/bhand_palm_surface_link"/>
       <origin xyz="0 0 0.08" rpy="0 0 0"/>
-      <limit effort="5" lower="0" upper="${PI}" velocity="5.0"/>
+      <limit effort="30" lower="0" upper="${PI}" velocity="5.0"/>
     </joint>
     <link name="${prefix}/bhand_palm_surface_link">
@@ -136,5 +135,5 @@
       <child link="${prefix}/bhand_grasp_link"/>
       <origin xyz="0 0 0.12" rpy="0 0 0"/>
-      <limit effort="5" lower="0" upper="${PI}" velocity="5.0"/>
+      <limit effort="30" lower="0" upper="${PI}" velocity="5.0"/>
     </joint>
     <link name="${prefix}/bhand_grasp_link">
@@ -148,5 +147,5 @@
     </link>
   </xacro:macro>
-  <xacro:macro name="bhand_finger_prox" params="prefix parent_link xyz rpy axis">
+  <xacro:macro name="bhand_finger_prox" params="prefix parent_link xyz rpy axis primitive">
     <joint name="${prefix}/prox_joint" type="revolute">
       <parent link="${parent_link}"/>
@@ -196,5 +195,5 @@
     </link>
   </xacro:macro>
-  <xacro:macro name="bhand_finger_med" params="prefix parent_link xyz rpy">
+  <xacro:macro name="bhand_finger_med" params="prefix parent_link xyz rpy primitive">
     <joint name="${prefix}/med_joint" type="revolute">
       <parent link="${parent_link}"/>
@@ -202,5 +201,5 @@
       <origin xyz="${xyz}" rpy="${rpy}"/>
       <axis xyz="0 0 1"/>
-      <limit effort="3" lower="0" upper="${140/180*PI}" velocity="10.00"/>
+      <limit effort="30" lower="0" upper="${140/180*PI}" velocity="10.00"/>
       <dynamics damping="0.15" friction="${f}"/>
     </joint>
@@ -244,5 +243,5 @@
     </link>
   </xacro:macro>
-  <xacro:macro name="bhand_finger_dist" params="prefix">
+  <xacro:macro name="bhand_finger_dist" params="prefix primitive">
     <joint name="${prefix}/dist_joint" type="revolute">
       <parent link="${prefix}/med_link"/>
@@ -250,5 +249,5 @@
       <origin xyz="0.06994 0.003 0.0" rpy="0 0 ${PI/4}"/>
       <axis xyz="0 0 1"/>
-      <limit effort="10" lower="0" upper="${48/180*PI}" velocity="10.00"/>
+      <limit effort="30" lower="0" upper="${48/180*PI}" velocity="10.00"/>
       <dynamics damping="0.15" friction="${f}"/>
     </joint>

File: robots/wam7_bhand.urdf.xacro (robot description, xacro)
@@ -8,4 +8,4 @@
   <xacro:wam_7dof prefix="wam" parent_link="world" xyz="0.0 0.0 1.0" rpy="0 0 0" />
   <!-- BHand -->
-  <xacro:bhand prefix="wam/bhand" parent_link="wam/wrist_palm_link" xyz="0 0 0.06" rpy="0 0 0"/>
+  <xacro:bhand prefix="wam/bhand" parent_link="wam/wrist_palm_link" xyz="0 0 0.06" rpy="0 0 0" primitive="true"/>
 </robot>

File: robots/wam_7dof_wam_bhand.urdf.xacro (robot description, xacro)
@@ -6,4 +6,4 @@
   <link name = "world"/>
   <xacro:wam_7dof prefix="wam" parent_link="world" xyz="0.02 0.46 1" rpy="0 0 0" />
-  <xacro:bhand prefix="wam/bhand" parent_link="wam/wrist_palm_link" xyz="0 0 0.06" rpy="0 0 ${PI}"/>
+  <xacro:bhand prefix="wam/bhand" parent_link="wam/wrist_palm_link" xyz="0 0 0.06" rpy="0 0 ${PI}" primitive="true"/>
 </robot>

Commit message: making wam shiny

File: models/common.urdf.xacro (robot description, xacro)
@@ -54,3 +54,13 @@
     <kd>0.02</kd>
   </xacro:macro>
+  <xacro:macro name="gz_shiny">
+    <visual name='visual_shiny'>
+      <material>
+        <ambient>0.7 0.7 0.7 1</ambient>
+        <diffuse>0.9 0.9 0.9 1</diffuse>
+        <specular>0.5 0.5 0.5 0.3</specular>
+        <emissive>0 0 0 0</emissive>
+      </material>
+    </visual>
+  </xacro:macro>
 </robot>

File: models/components.urdf.xacro (robot description, xacro)
@@ -34,4 +34,7 @@
       <origin xyz="${xyz}" rpy="${rpy}"/>
     </joint>
+    <gazebo reference="${prefix}/base_link">
+      <xacro:gz_shiny/>
+    </gazebo>
     <link name = "${prefix}/base_link">
       <inertial>
@@ -44,7 +47,7 @@
       </inertial>
       <visual>
-        <material name="WAMGrey">
-          <color rgba="0.7 0.7 0.7 0.0"/>
-        </material>
+        <!--<material name="WAMGrey">-->
+          <!--<color rgba="0.7 0.7 0.7 0.0"/>-->
+        <!--</material>-->
         <geometry>
           <mesh filename="${models_path}/sw_meshes/base_link_fine.stl"/>
@@ -70,4 +73,7 @@
       <xacro:gz_joint/>
     </gazebo>
+    <gazebo reference="${prefix}/shoulder_yaw_link">
+      <xacro:gz_shiny/>
+    </gazebo>
     <link name="${prefix}/shoulder_yaw_link" >
       <inertial>
@@ -80,7 +86,7 @@
       </inertial>
       <visual>
-        <material name="WAMGrey">
-          <color rgba="0.7 0.7 0.7 1.0"/>
-        </material>
+        <!--<material name="WAMGrey">-->
+          <!--<color rgba="0.7 0.7 0.7 1.0"/>-->
+        <!--</material>-->
         <geometry>
           <mesh filename="${models_path}/sw_meshes/shoulder_link_fine.stl"/>
@@ -106,9 +112,12 @@
       <xacro:gz_joint/>
     </gazebo>
+    <gazebo reference="${prefix}/shoulder_pitch_link">
+      <xacro:gz_shiny/>
+    </gazebo>
     <link name="${prefix}/shoulder_pitch_link" >
       <visual>
-        <material name="WAMGrey">
-          <color rgba="0.7 0.7 0.7 1.0"/>
-        </material>
+        <!--<material name="WAMGrey">-->
+          <!--<color rgba="0.7 0.7 0.7 1.0"/>-->
+        <!--</material>-->
         <geometry>
           <mesh filename="${models_path}/sw_meshes/shoulder_pitch_link_fine.stl"/>
@@ -142,4 +151,7 @@
       <xacro:gz_joint/>
     </gazebo>
+    <gazebo reference="${prefix}/upper_arm_link">
+      <xacro:gz_shiny/>
+    </gazebo>
     <link name="${prefix}/upper_arm_link" >
       <inertial>
@@ -152,7 +164,7 @@
       </inertial>
       <visual>
-        <material name="WAMGrey">
-          <color rgba="0.7 0.7 0.7 1.0"/>
-        </material>
+        <!--<material name="WAMGrey">-->
+          <!--<color rgba="0.7 0.7 0.7 1.0"/>-->
+        <!--</material>-->
         <geometry>
           <mesh filename="${models_path}/sw_meshes/upper_arm_link_fine.stl"/>
@@ -179,4 +191,7 @@
       <xacro:gz_joint/>
     </gazebo>
+    <gazebo reference="${prefix}/forearm_link">
+      <xacro:gz_shiny/>
+    </gazebo>
     <link name="${prefix}/forearm_link" >
       <inertial>
@@ -189,7 +204,7 @@
       </inertial>
       <visual>
-        <material name="WAMGrey">
-          <color rgba="0.7 0.7 0.7 1.0"/>
-        </material>
+        <!--<material name="WAMGrey">-->
+          <!--<color rgba="0.7 0.7 0.7 1.0"/>-->
+        <!--</material>-->
         <geometry>
           <mesh filename="${models_path}/sw_meshes/elbow_link_fine.stl"/>
@@ -202,7 +217,7 @@
       </collision>
       <visual>
-        <material name="WAMGrey">
-          <color rgba="0.7 0.7 0.7 1.0"/>
-        </material>
+        <!--<material name="WAMGrey2">-->
+          <!--<color rgba="0.1 0.1 0.1 1.0"/>-->
+        <!--</material>-->
         <origin xyz="-0.045 -0.0730 0" rpy="${PI/2} 0 0" />
         <geometry>
@@ -230,4 +245,7 @@
       <xacro:gz_joint/>
     </gazebo>
+    <gazebo reference="${prefix}/wrist_yaw_link">
+      <xacro:gz_shiny/>
+    </gazebo>
     <link name="${prefix}/wrist_yaw_link" >
       <inertial>
@@ -239,7 +257,7 @@
       </inertial>
       <visual>
-        <material name="WAMGrey">
-          <color rgba="0.7 0.7 0.7 1.0"/>
-        </material>
+        <!--<material name="WAMGrey">-->
+          <!--<color rgba="0.7 0.7 0.7 1.0"/>-->
+        <!--</material>-->
         <origin xyz="0 0 0" rpy="0 0 0" />
         <geometry>
@@ -267,4 +285,7 @@
       <xacro:gz_joint/>
     </gazebo>
+    <gazebo reference="${prefix}/wrist_pitch_link">
+      <xacro:gz_shiny/>
+    </gazebo>
     <link name="${prefix}/wrist_pitch_link" >
       <inertial>
@@ -277,7 +298,7 @@
       </inertial>
       <visual>
-        <material name="WAMGrey">
-          <color rgba="0.7 0.7 0.7 1.0"/>
-        </material>
+        <!--<material name="WAMGrey">-->
+          <!--<color rgba="0.7 0.7 0.7 1.0"/>-->
+        <!--</material>-->
         <geometry>
           <mesh filename="${models_path}/sw_meshes/wrist_pitch_link_fine.stl"/>
@@ -304,4 +325,7 @@
       <xacro:gz_joint/>
     </gazebo>
+    <gazebo reference="${prefix}/wrist_palm_link">
+      <xacro:gz_shiny/>
+    </gazebo>
     <link name="${prefix}/wrist_palm_link" >
       <inertial>
@@ -313,7 +337,7 @@
       </inertial>
       <visual>
-        <material name="WAMGrey">
-          <color rgba="0.7 0.7 0.7 1.0"/>
-        </material>
+        <!--<material name="WAMGrey">-->
+          <!--<color rgba="0.7 0.7 0.7 1.0"/>-->
+        <!--</material>-->
         <origin xyz="0 0 0" rpy="0 0 0" />
         <geometry>
@@ -472,7 +496,7 @@
       </inertial>
       <visual>
-        <material name="WAMGrey">
-          <color rgba="0.7 0.7 0.7 1.0"/>
-        </material>
+        <!--<material name="WAMGrey">-->
+          <!--<color rgba="0.7 0.7 0.7 1.0"/>-->
+        <!--</material>-->
         <geometry>
           <mesh filename="${models_path}/sw_meshes/elbow_link_fine.stl"/>

Commit message: improving vistualization in gazebo and improving simulation stability

File: models/common.urdf.xacro (robot description, xacro)
@@ -56,10 +56,30 @@
   <xacro:macro name="gz_shiny">
     <visual name='visual_shiny'>
-      <material>
-        <ambient>0.7 0.7 0.7 1</ambient>
-        <diffuse>0.9 0.9 0.9 1</diffuse>
-        <specular>0.5 0.5 0.5 0.3</specular>
-        <emissive>0 0 0 0</emissive>
-      </material>
+      <xacro:if value="true">
+        <material>
+          <script>
+            <uri>file://$(find barrett_model)/materials/barrett.material</uri>
+            <name>Wam/Aluminum</name>
+          </script>
+        </material>
+      </xacro:if>
+      <xacro:if value="false">
+        <material>
+          <ambient>0.7 0.7 0.7 1</ambient>
+          <diffuse>0.9 0.9 0.9 1</diffuse>
+          <specular>0.5 0.5 0.5 0.3</specular>
+          <emissive>0 0 0 0</emissive>
+        </material>
+      </xacro:if>
+    </visual>
+  </xacro:macro>
+  <xacro:macro name="gz_shiny_blue">
+    <visual name='visual_shiny'>
+        <material>
+          <script>
+            <uri>file://$(find barrett_model)/materials/barrett.material</uri>
+            <name>BHand/BlueAluminum</name>
+          </script>
+        </material>
     </visual>
   </xacro:macro>

File: models/components.urdf.xacro (robot description, xacro)
@@ -47,7 +47,7 @@
       </inertial>
       <visual>
-        <material name="WAMGrey">
-          <color rgba="0.7 0.7 0.7 0.0"/>
-        </material>
+        <!--<material name="WAMGrey">-->
+          <!--<color rgba="0.7 0.7 0.7 0.0"/>-->
+        <!--</material>-->
         <geometry>
           <mesh filename="${models_path}/sw_meshes/base_link_fine.stl"/>
@@ -86,7 +86,7 @@
       </inertial>
       <visual>
-        <material name="WAMGrey">
-          <color rgba="0.7 0.7 0.7 1.0"/>
-        </material>
+        <!--<material name="WAMGrey">-->
+          <!--<color rgba="0.7 0.7 0.7 1.0"/>-->
+        <!--</material>-->
         <geometry>
           <mesh filename="${models_path}/sw_meshes/shoulder_link_fine.stl"/>
@@ -117,7 +117,7 @@
     <link name="${prefix}/shoulder_pitch_link" >
       <visual>
-        <material name="WAMGrey">
-          <color rgba="0.7 0.7 0.7 1.0"/>
-        </material>
+        <!--<material name="WAMGrey">-->
+          <!--<color rgba="0.7 0.7 0.7 1.0"/>-->
+        <!--</material>-->
         <geometry>
           <mesh filename="${models_path}/sw_meshes/shoulder_pitch_link_fine.stl"/>
@@ -164,7 +164,7 @@
       </inertial>
       <visual>
-        <material name="WAMGrey">
-          <color rgba="0.7 0.7 0.7 1.0"/>
-        </material>
+        <!--<material name="WAMGrey">-->
+          <!--<color rgba="0.7 0.7 0.7 1.0"/>-->
+        <!--</material>-->
         <geometry>
           <mesh filename="${models_path}/sw_meshes/upper_arm_link_fine.stl"/>
@@ -204,7 +204,7 @@
       </inertial>
       <visual>
-        <material name="WAMGrey">
-          <color rgba="0.7 0.7 0.7 1.0"/>
-        </material>
+        <!--<material name="WAMGrey">-->
+          <!--<color rgba="0.7 0.7 0.7 1.0"/>-->
+        <!--</material>-->
         <geometry>
           <mesh filename="${models_path}/sw_meshes/elbow_link_fine.stl"/>
@@ -217,7 +217,7 @@
       </collision>
       <visual>
-        <material name="WAMGrey2">
-          <color rgba="0.1 0.1 0.1 1.0"/>
-        </material>
+        <!--<material name="WAMGrey2">-->
+          <!--<color rgba="0.1 0.1 0.1 1.0"/>-->
+        <!--</material>-->
         <origin xyz="-0.045 -0.0730 0" rpy="${PI/2} 0 0" />
         <geometry>
@@ -257,7 +257,7 @@
       </inertial>
       <visual>
-        <material name="WAMGrey">
-          <color rgba="0.7 0.7 0.7 1.0"/>
-        </material>
+        <!--<material name="WAMGrey">-->
+          <!--<color rgba="0.7 0.7 0.7 1.0"/>-->
+        <!--</material>-->
         <origin xyz="0 0 0" rpy="0 0 0" />
         <geometry>
@@ -298,7 +298,7 @@
       </inertial>
       <visual>
-        <material name="WAMGrey">
-          <color rgba="0.7 0.7 0.7 1.0"/>
-        </material>
+        <!--<material name="WAMGrey">-->
+          <!--<color rgba="0.7 0.7 0.7 1.0"/>-->
+        <!--</material>-->
         <geometry>
           <mesh filename="${models_path}/sw_meshes/wrist_pitch_link_fine.stl"/>
@@ -337,7 +337,7 @@
       </inertial>
       <visual>
-        <material name="WAMGrey">
-          <color rgba="0.7 0.7 0.7 1.0"/>
-        </material>
+        <!--<material name="WAMGrey">-->
+          <!--<color rgba="0.7 0.7 0.7 1.0"/>-->
+        <!--</material>-->
         <origin xyz="0 0 0" rpy="0 0 0" />
         <geometry>
@@ -496,7 +496,7 @@
       </inertial>
       <visual>
-        <material name="WAMGrey">
-          <color rgba="0.7 0.7 0.7 1.0"/>
-        </material>
+        <!--<material name="WAMGrey">-->
+          <!--<color rgba="0.7 0.7 0.7 1.0"/>-->
+        <!--</material>-->
         <geometry>
           <mesh filename="${models_path}/sw_meshes/elbow_link_fine.stl"/>

File: models/hand.urdf.xacro (robot description, xacro)
@@ -3,6 +3,6 @@
   <!-- link properties -->
   <xacro:macro name="gz_hand_link" params="soft collide">
-    <mu1>2.8</mu1>
-    <mu2>2.8</mu2>
+    <mu1>0.95</mu1>
+    <mu2>0.95</mu2>
     <maxContacts>1</maxContacts>
     <xacro:if value="${collide}">
@@ -80,4 +80,5 @@
     <gazebo reference="${prefix}/bhand_palm_link">
       <xacro:gz_hand_link collide="false" soft="false"/>
+      <xacro:gz_shiny_blue/>
     </gazebo>
     <link name="${prefix}/bhand_palm_link">
@@ -91,7 +92,7 @@
       </inertial>
       <visual>
-        <material name="WAMGrey">
-          <color rgba="0.9 0.9 0.9 0.0"/>
-        </material>
+        <!--<material name="WAMGrey">-->
+          <!--<color rgba="0.9 0.9 0.9 0.0"/>-->
+        <!--</material>-->
         <geometry>
           <mesh filename="${models_path}/sw_meshes/bhand/bhand_palm_fine.stl"/>
@@ -168,4 +169,5 @@
     <gazebo reference="${prefix}/prox_link">
       <xacro:gz_hand_link collide="false" soft="false"/>
+      <xacro:gz_shiny_blue/>
     </gazebo>
     <link name="${prefix}/prox_link">
@@ -216,4 +218,5 @@
     <gazebo reference="${prefix}/med_link">
       <xacro:gz_hand_link collide="false" soft="true"/>
+      <xacro:gz_shiny/>
     </gazebo>
     <link name="${prefix}/med_link">
@@ -264,4 +267,5 @@
     <gazebo reference="${prefix}/dist_link">
       <xacro:gz_hand_link collide="true" soft="true"/>
+      <xacro:gz_shiny/>
     </gazebo>
     <link name="${prefix}/dist_link">
