Commit message: increasing bhand damping in simulation

File: models/hand.urdf.xacro (robot description, xacro)
@@ -61,5 +61,5 @@
       <axis xyz="${axis}"/>
       <limit effort="5" lower="0" upper="${PI}" velocity="0.20"/>
-      <dynamics damping="0.5" friction="1"/>
+      <dynamics damping="1.5" friction="1"/>
     </joint>
     <gazebo reference="${prefix}/prox_joint">
@@ -97,5 +97,5 @@
       <axis xyz="0 0 1"/>
       <limit effort="5" lower="0" upper="${140/180*PI}" velocity="0.20"/>
-      <dynamics damping="0.5" friction="1"/>
+      <dynamics damping="1.5" friction="1"/>
     </joint>
     <gazebo reference="${prefix}/med_joint">
@@ -133,5 +133,5 @@
       <axis xyz="0 0 1"/>
       <limit effort="5" lower="0" upper="${48/180*PI}" velocity="0.20"/>
-      <dynamics damping="0.5" friction="1"/>
+      <dynamics damping="1.5" friction="1"/>
     </joint>
     <gazebo reference="${prefix}/dist_joint">

Commit message: reducing friction and disabling collision for some links

File: models/hand.urdf.xacro (robot description, xacro)
@@ -23,8 +23,10 @@
     <xacro:bhand_finger_dist prefix="${prefix}/finger_3"/>
   </xacro:macro>
-  <xacro:macro name="gz_hand_link">
+  <xacro:macro name="gz_hand_link" params="collide">
     <mu1>0.8</mu1>
     <mu2>0.8</mu2>
-    <selfCollide>true</selfCollide>
+    <xacro:if value="${collide}">
+      <selfCollide>true</selfCollide>
+    </xacro:if>
   </xacro:macro>
   <!-- Components -->
@@ -36,5 +38,5 @@
     </joint>
     <gazebo reference="${prefix}/bhand_palm_link">
-      <xacro:gz_hand_link/>
+      <xacro:gz_hand_link collide="false"/>
     </gazebo>
     <link name="${prefix}/bhand_palm_link">
@@ -66,5 +68,5 @@
       <origin xyz="0 0 0.08" rpy="0 0 0"/>
       <limit effort="5" lower="0" upper="${PI}" velocity="5.0"/>
-      <dynamics damping="1.5" friction="1"/>
+      <dynamics damping="0.1" friction="0"/>
     </joint>
     <link name="${prefix}/bhand_palm_surface_link">
@@ -82,5 +84,5 @@
       <origin xyz="0 0 0.12" rpy="0 0 0"/>
       <limit effort="5" lower="0" upper="${PI}" velocity="5.0"/>
-      <dynamics damping="1.5" friction="1"/>
+      <dynamics damping="0.1" friction="0"/>
     </joint>
     <link name="${prefix}/bhand_grasp_link">
@@ -101,5 +103,5 @@
       <axis xyz="${axis}"/>
       <limit effort="5" lower="0" upper="${PI}" velocity="5.0"/>
-      <dynamics damping="1.5" friction="1"/>
+      <dynamics damping="0.1" friction="0"/>
     </joint>
     <gazebo reference="${prefix}/prox_joint">
@@ -107,5 +109,5 @@
     </gazebo>
     <gazebo reference="${prefix}/prox_link">
-      <xacro:gz_hand_link/>
+      <xacro:gz_hand_link collide="false"/>
     </gazebo>
     <link name="${prefix}/prox_link">
@@ -140,5 +142,5 @@
       <axis xyz="0 0 1"/>
       <limit effort="5" lower="0" upper="${140/180*PI}" velocity="5.00"/>
-      <dynamics damping="1.5" friction="1"/>
+      <dynamics damping="0.1" friction="0"/>
     </joint>
     <gazebo reference="${prefix}/med_joint">
@@ -146,5 +148,5 @@
     </gazebo>
     <gazebo reference="${prefix}/med_link">
-      <xacro:gz_hand_link/>
+      <xacro:gz_hand_link collide="false"/>
     </gazebo>
     <link name="${prefix}/med_link">
@@ -179,5 +181,5 @@
       <axis xyz="0 0 1"/>
       <limit effort="5" lower="0" upper="${48/180*PI}" velocity="5.00"/>
-      <dynamics damping="1.5" friction="1"/>
+      <dynamics damping="0.1" friction="0"/>
     </joint>
     <gazebo reference="${prefix}/dist_joint">
@@ -185,5 +187,5 @@
     </gazebo>
     <gazebo reference="${prefix}/dist_link">
-      <xacro:gz_hand_link/>
+      <xacro:gz_hand_link collide="true"/>
     </gazebo>
     <link name="${prefix}/dist_link">

Commit message: adding tf frame for fingertips, fixing naming of the first two fingers

File: models/hand.urdf.xacro (robot description, xacro)
@@ -11,16 +11,19 @@
   <!-- Fingers -->
   <xacro:macro name="bhand_finger_1" params="prefix">
-    <xacro:bhand_finger_prox prefix="${prefix}/finger_1" parent_link="${prefix}/bhand_palm_link" xyz="0.025 0.0 0.0415" rpy="0 0 -${PI/2}" axis="0 0 1"/>
+    <xacro:bhand_finger_prox prefix="${prefix}/finger_1" parent_link="${prefix}/bhand_palm_link" xyz="-0.025 0.0 0.0415" rpy="0 0 -${PI/2}" axis="0 0 -1"/>
     <xacro:bhand_finger_med prefix="${prefix}/finger_1" parent_link="${prefix}/finger_1/prox_link" xyz="0.05 0.0 0.03390" rpy="${PI/2} 0 0"/>
     <xacro:bhand_finger_dist prefix="${prefix}/finger_1"/>
+    <xacro:bhand_finger_tip prefix="${prefix}/finger_1"/>
   </xacro:macro>
   <xacro:macro name="bhand_finger_2" params="prefix">
-    <xacro:bhand_finger_prox prefix="${prefix}/finger_2" parent_link="${prefix}/bhand_palm_link" xyz="-0.025 0.0 0.0415" rpy="0 0 -${PI/2}" axis="0 0 -1"/>
+    <xacro:bhand_finger_prox prefix="${prefix}/finger_2" parent_link="${prefix}/bhand_palm_link" xyz="0.025 0.0 0.0415" rpy="0 0 -${PI/2}" axis="0 0 1"/>
     <xacro:bhand_finger_med prefix="${prefix}/finger_2" parent_link="${prefix}/finger_2/prox_link" xyz="0.05 0.0 0.03390" rpy="${PI/2} 0 0"/>
     <xacro:bhand_finger_dist prefix="${prefix}/finger_2"/>
+    <xacro:bhand_finger_tip prefix="${prefix}/finger_2"/>
   </xacro:macro>
   <xacro:macro name="bhand_finger_3" params="prefix">
     <xacro:bhand_finger_med prefix="${prefix}/finger_3" parent_link="${prefix}/bhand_palm_link" xyz="0 0.05 0.0754" rpy="${PI/2} 0 ${PI/2}"/>
     <xacro:bhand_finger_dist prefix="${prefix}/finger_3"/>
+    <xacro:bhand_finger_tip prefix="${prefix}/finger_3"/>
   </xacro:macro>
   <xacro:macro name="gz_hand_link" params="collide">
@@ -179,5 +182,5 @@
       <parent link="${prefix}/med_link"/>
       <child link="${prefix}/dist_link"/>
-      <origin xyz="0.06994 0.003 0.0" rpy="0 0 0"/>
+      <origin xyz="0.06994 0.003 0.0" rpy="0 0 ${PI/4}"/>
       <axis xyz="0 0 1"/>
       <limit effort="5" lower="0" upper="${48/180*PI}" velocity="5.00"/>
@@ -192,5 +195,5 @@
     <link name="${prefix}/dist_link">
       <inertial>
-        <origin xyz="0.022825 0.0010491 0.0004203" />
+        <origin xyz="0.022825 0.0010491 0.0004203" rpy="0 0 ${-PI/4}"/>
         <mass value="0.041377" />
         <inertia
@@ -200,4 +203,5 @@
       </inertial>
       <visual>
+        <origin rpy="0 0 ${-PI/4}"/>
         <material name="WAMGrey">
           <color rgba="0.9 0.9 0.9 0.0"/>
@@ -208,4 +212,5 @@
       </visual>
       <collision>
+        <origin rpy="0 0 ${-PI/4}"/>
         <geometry>
           <mesh filename="${models_path}/sw_meshes/bhand/bhand_finger_dist_link_convex.stl"/>
@@ -214,3 +219,19 @@
     </link>
   </xacro:macro>
+  <xacro:macro name="bhand_finger_tip" params="prefix">
+    <joint name="${prefix}/tip_joint" type="fixed">
+      <parent link="${prefix}/dist_link"/>
+      <child link="${prefix}/tip_link"/>
+      <origin xyz="0.05 0.0 0.0" rpy="0 0 0"/>
+    </joint>
+    <link name="${prefix}/tip_link">
+      <inertial>
+        <mass value="1E-6" />
+        <inertia
+          ixx="1E-6" ixy="0"    ixz="0"
+                     iyy="1E-6" iyz="0"
+                                izz="1E-6" />
+      </inertial>
+    </link>
+  </xacro:macro>
 </robot>

Commit message: bhand: inertial properties for 3d-printed fingertips

File: models/hand.urdf.xacro (robot description, xacro)
@@ -47,5 +47,5 @@
       <inertial>
         <origin xyz="-5.1098e-005 0.0050433 0.036671"/>
-        <mass value="0.50573" />
+        <mass value="0.40573" />
         <inertia
           ixx="3.8374e-005" ixy="-5.604e-008"  ixz="-4.2034e-005"

Commit message: fixing orientation of bhand inertia

File: models/hand.urdf.xacro (robot description, xacro)
@@ -195,5 +195,5 @@
     <link name="${prefix}/dist_link">
       <inertial>
-        <origin xyz="0.022825 0.0010491 0.0004203" rpy="0 0 ${-PI/4}"/>
+        <origin xyz="0.022825 0.0010491 0.0004203" rpy="0 0 0"/>
         <mass value="0.041377" />
         <inertia

Commit message: adding vertex normals to all collision meshes

File: models/hand.urdf.xacro (robot description, xacro)
@@ -173,5 +173,5 @@
       <collision>
         <geometry>
-          <mesh filename="${models_path}/sw_meshes/bhand/bhand_finger_med_link_convex.stl"/>
+          <mesh filename="${models_path}/sw_meshes/bhand/bhand_finger_med_link_convex.dae"/>
         </geometry>
       </collision>
@@ -214,5 +214,5 @@
         <origin rpy="0 0 ${-PI/4}"/>
         <geometry>
-          <mesh filename="${models_path}/sw_meshes/bhand/bhand_finger_dist_link_convex.stl"/>
+          <mesh filename="${models_path}/sw_meshes/bhand/bhand_finger_dist_link_convex.dae"/>
         </geometry>
       </collision>

Commit message: increasing damping

File: models/hand.urdf.xacro (robot description, xacro)
@@ -1,5 +1,5 @@
 <robot xmlns:xacro="http://www.ros.org/wiki/xacro">
   <xacro:include filename="$(find barrett_model)/models/common.urdf.xacro"/>
-  <xacro:property name="b" value="1.1"/>
+  <xacro:property name="b" value="6.0"/>
   <!-- High-leveel hand macro -->
   <xacro:macro name="bhand" params="parent_link prefix xyz rpy">

Commit message: increasing bhand damping

File: models/hand.urdf.xacro (robot description, xacro)
@@ -1,5 +1,5 @@
 <robot xmlns:xacro="http://www.ros.org/wiki/xacro">
   <xacro:include filename="$(find barrett_model)/models/common.urdf.xacro"/>
-  <xacro:property name="b" value="0.1"/>
+  <xacro:property name="b" value="0.3"/>
   <!-- High-leveel hand macro -->
   <xacro:macro name="bhand" params="parent_link prefix xyz rpy">

Commit message: updating hand collision model to use primitive composition

File: models/hand.urdf.xacro (robot description, xacro)
@@ -2,5 +2,6 @@
   <xacro:include filename="$(find barrett_model)/models/common.urdf.xacro"/>
   <xacro:property name="b" value="0.3"/>
-  <!-- High-leveel hand macro -->
+  <xacro:property name="primitive" value="true"/>
+  <!-- High-level hand macro -->
   <xacro:macro name="bhand" params="parent_link prefix xyz rpy">
     <xacro:bhand_palm parent_link="${parent_link}" prefix="${prefix}" xyz="${xyz}" rpy="${rpy}"/>
@@ -8,4 +9,25 @@
     <xacro:bhand_finger_2 prefix="${prefix}"/>
     <xacro:bhand_finger_3 prefix="${prefix}"/>
+    <xacro:if value="false">
+      <gazebo>
+        <gripper name="bhand">
+          <grasp_check>
+              <attach_steps>10</attach_steps>
+              <detach_steps>20</detach_steps>
+              <min_contact_count>2</min_contact_count>
+          </grasp_check>
+          <palm_link>${prefix}/bhand_palm_link</palm_link>
+          <gripper_link>${prefix}/finger_1/med_link</gripper_link>
+          <gripper_link>${prefix}/finger_2/med_link</gripper_link>
+          <gripper_link>${prefix}/finger_3/med_link</gripper_link>
+          <gripper_link>${prefix}/finger_1/dist_link</gripper_link>
+          <gripper_link>${prefix}/finger_2/dist_link</gripper_link>
+          <gripper_link>${prefix}/finger_3/dist_link</gripper_link>
+          <!--<gripper_link>${prefix}/finger_1/tip_link</gripper_link>-->
+          <!--<gripper_link>${prefix}/finger_2/tip_link</gripper_link>-->
+          <!--<gripper_link>${prefix}/finger_3/tip_link</gripper_link>-->
+        </gripper>
+      </gazebo>
+    </xacro:if>
   </xacro:macro>
   <!-- Fingers -->
@@ -28,8 +50,11 @@
   </xacro:macro>
   <xacro:macro name="gz_hand_link" params="collide">
+    <kp>1</kp>
+    <kd>0.01</kd>
     <mu1>2.8</mu1>
     <mu2>2.8</mu2>
+    <maxContacts>2</maxContacts>
     <xacro:if value="${collide}">
-      <selfCollide>true</selfCollide>
+      <selfCollide>false</selfCollide>
     </xacro:if>
   </xacro:macro>
@@ -61,9 +86,21 @@
         </geometry>
       </visual>
-      <collision>
-        <geometry>
-          <mesh filename="${models_path}/sw_meshes/bhand/bhand_palm_link_convex_decomposition.dae"/>
-        </geometry>
-      </collision>
+      <xacro:if value="${primitive}">
+        <!-- wrist -->
+        <collision><origin xyz="0 0 0.02029"/><geometry><cylinder radius="0.045" length="0.042"/></geometry></collision>
+        <!-- spine -->
+        <collision><origin xyz="0 0.01105 0.05768"/><geometry><box size="0.024 0.108 0.033"/></geometry></collision>
+        <!-- palm -->
+        <collision><origin xyz="0 0 0.07243"/><geometry><box size="0.076 0.046 0.012"/></geometry></collision>
+        <!-- F1 knuckle -->
+        <collision><origin xyz="0 0.05 0.07527" rpy="0 1.5707 0"/><geometry><cylinder radius="0.015" length="0.024"/></geometry></collision>
+      </xacro:if>
+      <xacro:unless value="${primitive}">
+        <collision>
+          <geometry>
+            <mesh filename="${models_path}/sw_meshes/bhand/bhand_palm_link_convex_decomposition.dae"/>
+          </geometry>
+        </collision>
+      </xacro:unless>
     </link>
     <joint name="${prefix}/bhand_palm_surface_joint" type="fixed">
@@ -75,5 +112,5 @@
     <link name="${prefix}/bhand_palm_surface_link">
       <inertial>
-        <mass value="0.000001" />
+        <mass value="0.00001" />
         <inertia
           ixx="0.000001" ixy="0.0"  ixz="0.0"
@@ -90,5 +127,5 @@
     <link name="${prefix}/bhand_grasp_link">
       <inertial>
-        <mass value="0.000001" />
+        <mass value="0.00001" />
         <inertia
           ixx="0.000001" ixy="0.0"  ixz="0.0"
@@ -130,9 +167,17 @@
         </geometry>
       </visual>
-      <collision>
-        <geometry>
-          <mesh filename="${models_path}/sw_meshes/bhand/bhand_finger_prox_link_convex_decomposition.dae"/>
-        </geometry>
-      </collision>
+      <xacro:if value="${primitive}">
+        <!-- base -->
+        <collision><origin xyz="0.03217 0.0 0.01674"/><geometry><box size="0.066 0.024 0.033"/></geometry></collision>
+        <!-- F2/F3 knuckle -->
+        <collision><origin xyz="0.05 0.0 0.034" rpy="1.5707 0 0"/><geometry><cylinder radius="0.015" length="0.024"/></geometry></collision>
+      </xacro:if>
+      <xacro:unless value="${primitive}">
+        <collision>
+          <geometry>
+            <mesh filename="${models_path}/sw_meshes/bhand/bhand_finger_prox_link_convex_decomposition.dae"/>
+          </geometry>
+        </collision>
+      </xacro:unless>
     </link>
   </xacro:macro>
@@ -170,9 +215,17 @@
         </geometry>
       </visual>
-      <collision>
-        <geometry>
-          <mesh filename="${models_path}/sw_meshes/bhand/bhand_finger_med_link_convex.dae"/>
-        </geometry>
-      </collision>
+      <xacro:if value="${primitive}">
+        <!-- spine -->
+        <collision><origin xyz="0.03493 0.003 -0.0007"/><geometry><box size="0.07 0.019 0.006"/></geometry></collision>
+        <!-- protrusion -->
+        <collision><origin xyz="0.03894 0.00376 -0.0007"/><geometry><box size="0.031 0.023 0.019"/></geometry></collision>
+      </xacro:if>
+      <xacro:unless value="${primitive}">
+        <collision>
+          <geometry>
+            <mesh filename="${models_path}/sw_meshes/bhand/bhand_finger_med_link_convex.dae"/>
+          </geometry>
+        </collision>
+      </xacro:unless>
     </link>
   </xacro:macro>
@@ -188,4 +241,6 @@
     <gazebo reference="${prefix}/dist_joint">
       <provideFeedback>true</provideFeedback>
+      <!--<kp>10</kp>-->
+      <!--<kd>0.01</kd>-->
     </gazebo>
     <gazebo reference="${prefix}/dist_link">
@@ -211,10 +266,22 @@
         </geometry>
       </visual>
-      <collision>
-        <origin rpy="0 0 ${-PI/4}"/>
-        <geometry>
-          <mesh filename="${models_path}/sw_meshes/bhand/bhand_finger_dist_link_convex.dae"/>
-        </geometry>
-      </collision>
+      <xacro:if value="${primitive}">
+        <!-- base -->
+        <collision><origin xyz="0 0 -0.0007"/><geometry><cylinder length="0.023" radius="0.0095"/></geometry></collision>
+        <!-- tip -->
+        <collision><origin xyz="0.05047 -0.00236 -0.0007"/><geometry><cylinder length="0.023" radius="0.0065"/></geometry></collision>
+        <!-- outer -->
+        <collision><origin xyz="0.02896 -0.00853 -0.0007" rpy="0 0 0"/><geometry><box size="0.059 0.002 0.023"/></geometry></collision>
+        <!-- inner -->
+        <collision><origin xyz="0.02538 0.00124 -0.0007" rpy="0 0 ${-6.0/180.0*PI}"/><geometry><box size="0.052 0.011 0.023"/></geometry></collision>
+      </xacro:if>
+      <xacro:unless value="${primitive}">
+        <collision>
+          <origin rpy="0 0 ${-PI/4}"/>
+          <geometry>
+            <mesh filename="${models_path}/sw_meshes/bhand/bhand_finger_dist_link_convex.dae"/>
+          </geometry>
+        </collision>
+      </xacro:unless>
     </link>
   </xacro:macro>

Commit message: more stable hand parameters

File: models/hand.urdf.xacro (robot description, xacro)
@@ -1,6 +1,28 @@
 <robot xmlns:xacro="http://www.ros.org/wiki/xacro">
   <xacro:include filename="$(find barrett_model)/models/common.urdf.xacro"/>
-  <xacro:property name="b" value="0.3"/>
   <xacro:property name="primitive" value="true"/>
+  <!-- link properties -->
+  <xacro:macro name="gz_hand_link" params="soft collide">
+    <mu1>2.8</mu1>
+    <mu2>2.8</mu2>
+    <maxContacts>2</maxContacts>
+    <xacro:if value="${collide}">
+      <selfCollide>false</selfCollide>
+    </xacro:if>
+    <xacro:if value="${soft}">
+      <xacro:gz_soft_link/>
+    </xacro:if>
+  </xacro:macro>
+  <!-- joint properties -->
+  <xacro:property name="b" value="0.5"/>
+  <xacro:property name="f" value="0"/>
+  <xacro:macro name="gz_hand_joint" params="feedback">
+    <provideFeedback>${feedback}</provideFeedback>
+    <!--<cfmDamping>true</cfmDamping>-->
+    <!--<kp>0.001</kp>-->
+    <!--<kd>0.01</kd>-->
+    <!--<stopCfm>0.5</stopCfm>-->
+    <!--<stopErp>0.5</stopErp>-->
+  </xacro:macro>
   <!-- High-level hand macro -->
   <xacro:macro name="bhand" params="parent_link prefix xyz rpy">
@@ -9,4 +31,5 @@
     <xacro:bhand_finger_2 prefix="${prefix}"/>
     <xacro:bhand_finger_3 prefix="${prefix}"/>
+    <!-- don't use the gazebo gripper plugin, just slows down the sim -->
     <xacro:if value="false">
       <gazebo>
@@ -49,14 +72,4 @@
     <xacro:bhand_finger_tip prefix="${prefix}/finger_3"/>
   </xacro:macro>
-  <xacro:macro name="gz_hand_link" params="collide">
-    <kp>1</kp>
-    <kd>0.01</kd>
-    <mu1>2.8</mu1>
-    <mu2>2.8</mu2>
-    <maxContacts>2</maxContacts>
-    <xacro:if value="${collide}">
-      <selfCollide>false</selfCollide>
-    </xacro:if>
-  </xacro:macro>
   <!-- Components -->
   <xacro:macro name="bhand_palm" params="prefix parent_link xyz rpy">
@@ -67,5 +80,5 @@
     </joint>
     <gazebo reference="${prefix}/bhand_palm_link">
-      <xacro:gz_hand_link collide="false"/>
+      <xacro:gz_hand_link collide="false" soft="false"/>
     </gazebo>
     <link name="${prefix}/bhand_palm_link">
@@ -141,12 +154,13 @@
       <origin xyz="${xyz}" rpy="${rpy}"/>
       <axis xyz="${axis}"/>
-      <limit effort="5" lower="0" upper="${PI}" velocity="5.0"/>
-      <dynamics damping="${0.1*b}" friction="0"/>
+      <limit effort="5" lower="0" upper="${PI}" velocity="10.0"/>
+      <dynamics damping="0.15" friction="${f}"/>
     </joint>
     <gazebo reference="${prefix}/prox_joint">
-      <provideFeedback>true</provideFeedback>
+      <xacro:gz_hand_joint feedback="true"/>
+      <cfmDamping>true</cfmDamping>
     </gazebo>
     <gazebo reference="${prefix}/prox_link">
-      <xacro:gz_hand_link collide="false"/>
+      <xacro:gz_hand_link collide="false" soft="false"/>
     </gazebo>
     <link name="${prefix}/prox_link">
@@ -188,13 +202,13 @@
       <origin xyz="${xyz}" rpy="${rpy}"/>
       <axis xyz="0 0 1"/>
-      <limit effort="5" lower="0" upper="${140/180*PI}" velocity="5.00"/>
-      <dynamics damping="${0.1*b}" friction="0"/>
+      <limit effort="5" lower="0" upper="${140/180*PI}" velocity="10.00"/>
+      <dynamics damping="0.15" friction="${f}"/>
     </joint>
     <gazebo reference="${prefix}/med_joint">
-      <provideFeedback>true</provideFeedback>
+      <xacro:gz_hand_joint feedback="true"/>
+      <cfmDamping>true</cfmDamping>
     </gazebo>
     <gazebo reference="${prefix}/med_link">
-      <xacro:gz_hand_link collide="false"/>
-      <xacro:gz_soft_link/>
+      <xacro:gz_hand_link collide="false" soft="true"/>
     </gazebo>
     <link name="${prefix}/med_link">
@@ -236,15 +250,13 @@
       <origin xyz="0.06994 0.003 0.0" rpy="0 0 ${PI/4}"/>
       <axis xyz="0 0 1"/>
-      <limit effort="5" lower="0" upper="${48/180*PI}" velocity="5.00"/>
-      <dynamics damping="${0.1*b}" friction="0"/>
+      <limit effort="5" lower="0" upper="${48/180*PI}" velocity="10.00"/>
+      <dynamics damping="0.15" friction="${f}"/>
     </joint>
     <gazebo reference="${prefix}/dist_joint">
-      <provideFeedback>true</provideFeedback>
-      <!--<kp>10</kp>-->
-      <!--<kd>0.01</kd>-->
+      <xacro:gz_hand_joint feedback="true"/>
+      <cfmDamping>true</cfmDamping>
     </gazebo>
     <gazebo reference="${prefix}/dist_link">
-      <xacro:gz_hand_link collide="true"/>
-      <xacro:gz_soft_link/>
+      <xacro:gz_hand_link collide="true" soft="true"/>
     </gazebo>
     <link name="${prefix}/dist_link">

Commit message: limiting bhand finger torque

File: models/hand.urdf.xacro (robot description, xacro)
@@ -202,5 +202,5 @@
       <origin xyz="${xyz}" rpy="${rpy}"/>
       <axis xyz="0 0 1"/>
-      <limit effort="5" lower="0" upper="${140/180*PI}" velocity="10.00"/>
+      <limit effort="3" lower="0" upper="${140/180*PI}" velocity="10.00"/>
       <dynamics damping="0.15" friction="${f}"/>
     </joint>
@@ -250,5 +250,5 @@
       <origin xyz="0.06994 0.003 0.0" rpy="0 0 ${PI/4}"/>
       <axis xyz="0 0 1"/>
-      <limit effort="5" lower="0" upper="${48/180*PI}" velocity="10.00"/>
+      <limit effort="3" lower="0" upper="${48/180*PI}" velocity="10.00"/>
       <dynamics damping="0.15" friction="${f}"/>
     </joint>

Commit message: increasing max hand effort

File: models/hand.urdf.xacro (robot description, xacro)
@@ -250,5 +250,5 @@
       <origin xyz="0.06994 0.003 0.0" rpy="0 0 ${PI/4}"/>
       <axis xyz="0 0 1"/>
-      <limit effort="3" lower="0" upper="${48/180*PI}" velocity="10.00"/>
+      <limit effort="10" lower="0" upper="${48/180*PI}" velocity="10.00"/>
       <dynamics damping="0.15" friction="${f}"/>
     </joint>

Commit message: https://github.com/ros-planning/moveit_core/issues/158

File: models/hand.urdf.xacro (robot description, xacro)
@@ -138,4 +138,10 @@
     </joint>
     <link name="${prefix}/bhand_grasp_link">
+      <collision><!-- https://github.com/ros-planning/moveit_core/issues/158 -->
+        <origin xyz="0 0 -0.13" rpy="0 0 0"/>
+        <geometry>
+          <sphere size="0.001 0.001 0.001"/>
+        </geometry>
+      </collision>
       <inertial>
         <mass value="0.00001" />

Commit message: https://github.com/ros-planning/moveit_core/issues/158

File: models/hand.urdf.xacro (robot description, xacro)
@@ -138,4 +138,10 @@
     </joint>
     <link name="${prefix}/bhand_grasp_link">
+      <collision><!-- https://github.com/ros-planning/moveit_core/issues/158 -->
+        <origin xyz="0 0 -0.13" rpy="0 0 0"/>
+        <geometry>
+          <sphere radius="0.001"/>
+        </geometry>
+      </collision>
       <inertial>
         <mass value="0.00001" />
