Commit message: adjusting hand sim paramters

File: models/hand.urdf.xacro (robot description, xacro)
@@ -2,8 +2,8 @@
   <xacro:include filename="$(find barrett_model)/models/common.urdf.xacro"/>
   <!-- link properties -->
-  <xacro:macro name="gz_hand_link" params="soft collide">
-    <mu1>1.0</mu1>
-    <mu2>1.0</mu2>
-    <maxContacts>1</maxContacts>
+  <xacro:macro name="gz_hand_link" params="soft collide contacts">
+    <mu1>0.5</mu1>
+    <mu2>0.5</mu2>
+    <maxContacts>${contacts}</maxContacts>
     <xacro:if value="${collide}">
       <selfCollide>false</selfCollide>
@@ -11,4 +11,6 @@
     <xacro:if value="${soft}">
       <xacro:gz_soft_link/>
+      <!--<kp>3000</kp>-->
+      <kd>0.1</kd>
     </xacro:if>
   </xacro:macro>
@@ -19,4 +21,6 @@
     <provideFeedback>${feedback}</provideFeedback>
     <!--<cfmDamping>true</cfmDamping>-->
+    <!--<kp>100</kp>-->
+    <!--<kd>0.01</kd>-->
     <!--<kp>0.001</kp>-->
     <!--<kd>0.01</kd>-->
@@ -79,5 +83,5 @@
     </joint>
     <gazebo reference="${prefix}/bhand_palm_link">
-      <xacro:gz_hand_link collide="false" soft="false"/>
+      <xacro:gz_hand_link collide="false" soft="false" contacts="3"/>
       <xacro:gz_shiny_blue/>
     </gazebo>
@@ -161,5 +165,5 @@
       <axis xyz="${axis}"/>
       <limit effort="5" lower="0" upper="${PI}" velocity="10.0"/>
-      <dynamics damping="0.15" friction="${f}"/>
+      <dynamics damping="0.35" friction="${f}"/>
     </joint>
     <gazebo reference="${prefix}/prox_joint">
@@ -168,5 +172,5 @@
     </gazebo>
     <gazebo reference="${prefix}/prox_link">
-      <xacro:gz_hand_link collide="false" soft="false"/>
+      <xacro:gz_hand_link collide="false" soft="false" contacts="1"/>
       <xacro:gz_shiny_blue/>
     </gazebo>
@@ -210,5 +214,5 @@
       <axis xyz="0 0 1"/>
       <limit effort="30" lower="0" upper="${140/180*PI}" velocity="10.00"/>
-      <dynamics damping="0.15" friction="${f}"/>
+      <dynamics damping="0.35" friction="${f}"/>
     </joint>
     <gazebo reference="${prefix}/med_joint">
@@ -217,5 +221,5 @@
     </gazebo>
     <gazebo reference="${prefix}/med_link">
-      <xacro:gz_hand_link collide="false" soft="true"/>
+      <xacro:gz_hand_link collide="false" soft="true" contacts="1"/>
       <xacro:gz_shiny/>
     </gazebo>
@@ -259,5 +263,5 @@
       <axis xyz="0 0 1"/>
       <limit effort="30" lower="0" upper="${48/180*PI}" velocity="10.00"/>
-      <dynamics damping="0.15" friction="${f}"/>
+      <dynamics damping="0.35" friction="${f}"/>
     </joint>
     <gazebo reference="${prefix}/dist_joint">
@@ -266,5 +270,5 @@
     </gazebo>
     <gazebo reference="${prefix}/dist_link">
-      <xacro:gz_hand_link collide="true" soft="true"/>
+      <xacro:gz_hand_link collide="true" soft="true" contacts="1"/>
       <xacro:gz_shiny/>
     </gazebo>
