Commit message: add in bench lattice to urdf

File: robots/wam_7dof_2x.urdf.xacro (robot description, xacro)
@@ -5,12 +5,40 @@
   <!-- Root link is in the world frame-->
   <link name="world"/>
+  <!-- Fix this robot to the world -->
+  <joint name="world_joint"  type="fixed">
+    <origin xyz="0 0 0" rpy="0 0 0" />
+    <parent link="world"/>
+    <child link="baseLink"/>
+  </joint>
+  <link name = "baseLink">
+    <inertial>
+      <origin xyz="0 0 0" />
+      <mass value="100" />
+      <inertia
+        ixx="1" ixy="0"   ixz="0"
+                iyy="1"   iyz="0"
+                          izz="1" />
+    </inertial>
+    <visual>
+      <origin rpy="0 0 0 " xyz="0 0 0"/>
+      <geometry>
+        <mesh filename="${homeDirectory}/models/componentSTL/bench_lattice.dae"/>
+      </geometry>
+    </visual>
+    <collision>
+      <origin rpy="0 0 0 " xyz="0 0 0"/>
+      <geometry>
+        <mesh filename="${homeDirectory}/models/componentSTL/bench_lattice.stl"/>
+      </geometry>
+    </collision>
+  </link>
   <!--<gazebo reference="baseLink">
     <static>true</static>
      <turnGravityOff>true</turnGravityOff>
    </gazebo>-->
-  <xacro:wam_root prefix="wam_left" parentLink="world" xyz="0.356 0.46 1" rpy="0 ${-0.5*PI} ${0.5*PI}"/>
+  <xacro:wam_root prefix="wam_left" parentLink="baseLink" xyz="0.356 0.46 1" rpy="0 ${-0.5*PI} ${0.5*PI}"/>
   <xacro:wam_7dof prefix="wam_left" parentLink="wam_left/FixedLink" xyz="0 0 0" rpy="0 0 0" />
   <!--xacro:barrett_hand prefix="wam_left" /-->
-  <xacro:wam_root prefix="wam_right" parentLink="world" xyz="0.356 -0.46 1" rpy="0 ${-0.5*PI} ${0.5*PI}"/>
+  <xacro:wam_root prefix="wam_right" parentLink="baseLink" xyz="0.356 -0.46 1" rpy="0 ${-0.5*PI} ${0.5*PI}"/>
   <xacro:wam_7dof prefix="wam_right" parentLink="wam_right/FixedLink" xyz="0 0 0" rpy="0 0 0" />
   <!--xacro:barrett_hand prefix="wam_right" /-->

Commit message: fixing top-level xacro files

File: robots/wam_7dof_2x.urdf.xacro (robot description, xacro)
@@ -37,9 +37,9 @@
     <turnGravityOff>true</turnGravityOff>
   </gazebo>
-  <xacro:wam_root prefix="wam_left" parentLink="baseLink" xyz="0.356 0.46 1" rpy="0 ${-0.5*PI} ${0.5*PI}"/>
-  <xacro:wam_7dof prefix="wam_left" parentLink="wam_left/FixedLink" xyz="0 0 0" rpy="0 0 0" />
+  <xacro:wam_root prefix="wam_left" parent_link="baseLink" xyz="0.356 0.46 1" rpy="0 ${-0.5*PI} ${0.5*PI}"/>
+  <xacro:wam_7dof prefix="wam_left" parent_link="wam_left/FixedLink" xyz="0 0 0" rpy="0 0 0" />
   <!--xacro:barrett_hand prefix="wam_left" /-->
-  <xacro:wam_root prefix="wam_right" parentLink="baseLink" xyz="0.356 -0.46 1" rpy="0 ${-0.5*PI} ${0.5*PI}"/>
-  <xacro:wam_7dof prefix="wam_right" parentLink="wam_right/FixedLink" xyz="0 0 0" rpy="0 0 0" />
+  <xacro:wam_root prefix="wam_right" parent_link="baseLink" xyz="0.356 -0.46 1" rpy="0 ${-0.5*PI} ${0.5*PI}"/>
+  <xacro:wam_7dof prefix="wam_right" parent_link="wam_right/FixedLink" xyz="0 0 0" rpy="0 0 0" />
   <!--xacro:barrett_hand prefix="wam_right" /-->
 </robot>

File: robots/wam_7dof_wam.urdf.xacro (robot description, xacro)
@@ -4,7 +4,6 @@
   <include filename="$(find barrett_model)/models/wam_top.urdf.xacro"/>
   <!-- Root link is in the world frame-->
-  <link name = "baseLink"/>
-  <xacro:wam_root prefix="wam" parentLink="baseLink" xyz="0.0 0.5 1" rpy="0 ${-0.5*PI} ${0.5*PI}"/>
-  <xacro:wam_7dof prefix="wam" parentLink="wam/FixedLink" xyz="0 0 0" rpy="0 0 0" />
+  <link name = "world"/>
+  <xacro:wam_7dof prefix="wam" parent_link="world" xyz="0.02 0.46 1" rpy="0 0 0" />
   <!--xacro:barrett_hand prefix="wam_left" /-->
 </robot>
